File: Hardware/BUFFER.sch (KiCad schematic (older format))
At the start: 3 parts, among them U18 NC7SZ125P5X, U19 NC7SZ125P5X, U20 NC7SZ125P5X

Commit message: branch to make PR for review
I should have made a separate branch for the development and then merged
it, but its too late now.
Parts:
- renumbered U18 to U17, U19 to U18, U20 to U19
Changed lines of the file:
@@
 $EndDescr
 $Comp
-L NC7SZ125P5X U20
+L NC7SZ125P5X U19
 U 1 1 59290140
 P 2450 2850
-F 0 "U20" H 2450 3550 60  0000 C CNN
+F 0 "U19" H 2450 3550 60  0000 C CNN
 F 1 "NC7SZ125P5X" H 2400 2350 60  0000 C CNN
 F 2 "" H 2400 2850 60  0001 C CNN
@@
 PPM_OUT
 $Comp
-L NC7SZ125P5X U19
+L NC7SZ125P5X U18
 U 1 1 5929020C
 P 2400 4300
-F 0 "U19" H 2400 5000 60  0000 C CNN
+F 0 "U18" H 2400 5000 60  0000 C CNN
 F 1 "NC7SZ125P5X" H 2350 3800 60  0000 C CNN
 F 2 "" H 2350 4300 60  0001 C CNN
@@
 VCC
 $Comp
-L NC7SZ125P5X U18
+L NC7SZ125P5X U17
 U 1 1 59290291
 P 2300 5650
-F 0 "U18" H 2300 6350 60  0000 C CNN
+F 0 "U17" H 2300 6350 60  0000 C CNN
 F 1 "NC7SZ125P5X" H 2250 5150 60  0000 C CNN
 F 2 "" H 2250 5650 60  0001 C CNN
