File: Hardware/BUFFER.sch (KiCad schematic (older format))
At the start: 3 parts, among them U17 NC7SZ125P5X, U18 NC7SZ125P5X, U19 NC7SZ125P5X

Commit message: Fixed some BOM stuff
fixed BOM for non RLC components
Parts:
- removed U18: NC7SZ125P5X, symbol NC7SZ125P5X
- added R57, R58: 0, symbol R
- U42: renamed from U17; Digikey # NC7SZ125P5XCT-ND -> (none); part_num (none) -> CHIP-002
- U43: renamed from U19; Digikey # NC7SZ125P5XCT-ND -> (none); part_num (none) -> CHIP-002
Connections:
- net labels removed: CK_IN, CK_OUT
- wire segments 7 -> 17
Changed lines of the file:
@@
 $EndDescr
 $Comp
-L NC7SZ125P5X U19
+L NC7SZ125P5X U43
 U 1 1 59290140
 P 2450 2850
-F 0 "U19" H 2450 3550 60  0000 C CNN
+F 0 "U43" H 2450 3550 60  0000 C CNN
 F 1 "NC7SZ125P5X" H 2400 2350 60  0000 C CNN
 F 2 "" H 2400 2850 60  0001 C CNN
 F 3 "" H 2400 2850 60  0001 C CNN
-F 4 "NC7SZ125P5XCT-ND" H 2550 3650 60  0001 C CNN "Digikey #"
+F 4 "CHIP-002" H 2450 2850 60  0001 C CNN "part_num"
 	1    2450 2850
 	1    0    0    -1
@@
 Wire Wire Line
 	2000 3050 2450 3050
-Text HLabel 2000 2550 0    60   Input ~ 0
+Text HLabel 1750 2550 0    60   Input ~ 0
 PPM_IN
-Text HLabel 2950 2650 2    60   Input ~ 0
+Text HLabel 3150 2650 2    60   Input ~ 0
 PPM_OUT
-$Comp
-L NC7SZ125P5X U18
-U 1 1 5929020C
-P 2400 4300
-F 0 "U18" H 2400 5000 60  0000 C CNN
-F 1 "NC7SZ125P5X" H 2350 3800 60  0000 C CNN
-F 2 "" H 2350 4300 60  0001 C CNN
-F 3 "" H 2350 4300 60  0001 C CNN
-F 4 "NC7SZ125P5XCT-ND" H 2500 5100 60  0001 C CNN "Digikey #"
-	1    2400 4300
-	1    0    0    -1
-$EndComp
-Wire Wire Line
-	1950 4200 1950 4500
-Wire Wire Line
-	1950 4500 2400 4500
-Text HLabel 1950 4000 0    60   Input ~ 0
-CK_IN
-Text HLabel 2900 4100 2    60   Input ~ 0
-CK_OUT
 Text HLabel 1550 1900 0    60   Input ~ 0
 VCC
@@
 Text Label 2550 3050 0    60   ~ 0
 VCC
-Text Label 2500 4500 0    60   ~ 0
-VCC
 $Comp
-L NC7SZ125P5X U17
+L NC7SZ125P5X U42
 U 1 1 59290291
 P 2300 5650
-F 0 "U17" H 2300 6350 60  0000 C CNN
+F 0 "U42" H 2300 6350 60  0000 C CNN
 F 1 "NC7SZ125P5X" H 2250 5150 60  0000 C CNN
 F 2 "" H 2250 5650 60  0001 C CNN
-F 3 "" H 2250 5650 60  0001 C CNN
-F 4 "NC7SZ125P5XCT-ND" H 2400 6450 60  0001 C CNN "Digikey #"
+F 3 "CHIP-002" H 2250 5650 60  0001 C CNN
+F 4 "CHIP-002" H 2300 5650 60  0001 C CNN "part_num"
 	1    2300 5650
 	1    0    0    -1
@@
 Wire Wire Line
 	1850 5850 2300 5850
-Text HLabel 1850 5350 0    60   Input ~ 0
+Text HLabel 1600 5350 0    60   Input ~ 0
 RX_IN
-Text HLabel 2800 5450 2    60   Input ~ 0
+Text HLabel 3050 5450 2    60   Input ~ 0
 RX_OUT
 Text Label 2400 5850 0    60   ~ 0
 VCC
+Wire Wire Line
+	1750 2550 2000 2550
+Wire Wire Line
+	3150 2650 2950 2650
+$Comp
+L R R58
+U 1 1 5931D2C2
+P 2450 2300
+F 0 "R58" V 2530 2300 50  0000 C CNN
+F 1 "0" V 2450 2300 50  0000 C CNN
+F 2 "" V 2380 2300 50  0001 C CNN
+F 3 "" H 2450 2300 50  0001 C CNN
+	1    2450 2300
+	0    1    1    0
+$EndComp
+Wire Wire Line
+	2300 2300 1900 2300
+Wire Wire Line
+	1900 2300 1900 2550
+Connection ~ 1900 2550
+Wire Wire Line
+	2600 2300 3050 2300
+Wire Wire Line
+	3050 2300 3050 2650
+Connection ~ 3050 2650
+Wire Wire Line
+	3050 5450 2800 5450
+Wire Wire Line
+	1850 5350 1600 5350
+Wire Wire Line
+	1750 5350 1750 5050
+Wire Wire Line
+	1750 5050 2150 5050
+Connection ~ 1750 5350
+$Comp
+L R R57
+U 1 1 5931D3E3
+P 2300 5050
+F 0 "R57" V 2380 5050 50  0000 C CNN
+F 1 "0" V 2300 5050 50  0000 C CNN
+F 2 "" V 2230 5050 50  0001 C CNN
+F 3 "" H 2300 5050 50  0001 C CNN
+	1    2300 5050
+	0    1    1    0
+$EndComp
+Wire Wire Line
+	2450 5050 2900 5050
+Wire Wire Line
+	2900 5050 2900 5450
+Connection ~ 2900 5450
 $EndSCHEMATC

Commit message: Finished RLC bom stuff
Parts:
- R57, R58: part_num (none) -> RESS-001
- renumbered U42 to U17, U43 to U18
Changed lines of the file:
@@
 $EndDescr
 $Comp
-L NC7SZ125P5X U43
+L NC7SZ125P5X U18
 U 1 1 59290140
 P 2450 2850
-F 0 "U43" H 2450 3550 60  0000 C CNN
+F 0 "U18" H 2450 3550 60  0000 C CNN
 F 1 "NC7SZ125P5X" H 2400 2350 60  0000 C CNN
 F 2 "" H 2400 2850 60  0001 C CNN
@@
 VCC
 $Comp
-L NC7SZ125P5X U42
+L NC7SZ125P5X U17
 U 1 1 59290291
 P 2300 5650
-F 0 "U42" H 2300 6350 60  0000 C CNN
+F 0 "U17" H 2300 6350 60  0000 C CNN
 F 1 "NC7SZ125P5X" H 2250 5150 60  0000 C CNN
 F 2 "" H 2250 5650 60  0001 C CNN
@@
 F 2 "" V 2380 2300 50  0001 C CNN
 F 3 "" H 2450 2300 50  0001 C CNN
+F 4 "RESS-001" V 2450 2300 60  0001 C CNN "part_num"
 	1    2450 2300
 	0    1    1    0
@@
 F 2 "" V 2230 5050 50  0001 C CNN
 F 3 "" H 2300 5050 50  0001 C CNN
+F 4 "RESS-001" V 2300 5050 60  0001 C CNN "part_num"
 	1    2300 5050
 	0    1    1    0

Commit message: Added ressistor footprint
Parts:
- R57, R58: footprint (none) -> Resistors_SMD:R_0603_HandSoldering
Connections:
- wire segments 17 -> 20
Other:
- moved on the sheet: R57
Changed lines of the file:
@@
 Text HLabel 3150 2650 2    60   Input ~ 0
 PPM_OUT
-Text HLabel 1550 1900 0    60   Input ~ 0
+Text HLabel 3700 3350 3    60   Input ~ 0
 VCC
-Wire Wire Line
-	1550 1900 1900 1900
-Text Label 1900 1900 2    60   ~ 0
-VCC
-Text Label 2550 3050 0    60   ~ 0
+Text Label 3550 3150 2    60   ~ 0
 VCC
 $Comp
 L NC7SZ125P5X U17
 U 1 1 59290291
-P 2300 5650
-F 0 "U17" H 2300 6350 60  0000 C CNN
-F 1 "NC7SZ125P5X" H 2250 5150 60  0000 C CNN
-F 2 "" H 2250 5650 60  0001 C CNN
-F 3 "CHIP-002" H 2250 5650 60  0001 C CNN
-F 4 "CHIP-002" H 2300 5650 60  0001 C CNN "part_num"
-	1    2300 5650
+P 5100 2850
+F 0 "U17" H 5100 3550 60  0000 C CNN
+F 1 "NC7SZ125P5X" H 5050 2350 60  0000 C CNN
+F 2 "" H 5050 2850 60  0001 C CNN
+F 3 "CHIP-002" H 5050 2850 60  0001 C CNN
+F 4 "CHIP-002" H 5100 2850 60  0001 C CNN "part_num"
+	1    5100 2850
 	1    0    0    -1
 $EndComp
 Wire Wire Line
-	1850 5550 1850 5850
+	4650 2750 4650 3050
 Wire Wire Line
-	1850 5850 2300 5850
-Text HLabel 1600 5350 0    60   Input ~ 0
+	4650 3050 5100 3050
+Text HLabel 4400 2550 0    60   Input ~ 0
 RX_IN
-Text HLabel 3050 5450 2    60   Input ~ 0
+Text HLabel 5850 2650 2    60   Input ~ 0
 RX_OUT
-Text Label 2400 5850 0    60   ~ 0
-VCC
 Wire Wire Line
 	1750 2550 2000 2550
@@
 F 0 "R58" V 2530 2300 50  0000 C CNN
 F 1 "0" V 2450 2300 50  0000 C CNN
-F 2 "" V 2380 2300 50  0001 C CNN
+F 2 "Resistors_SMD:R_0603_HandSoldering" V 2380 2300 50  0001 C CNN
 F 3 "" H 2450 2300 50  0001 C CNN
 F 4 "RESS-001" V 2450 2300 60  0001 C CNN "part_num"
@@
 Connection ~ 3050 2650
 Wire Wire Line
-	3050 5450 2800 5450
+	5850 2650 5600 2650
 Wire Wire Line
-	1850 5350 1600 5350
+	4650 2550 4400 2550
 Wire Wire Line
-	1750 5350 1750 5050
+	4550 2550 4550 2250
 Wire Wire Line
-	1750 5050 2150 5050
-Connection ~ 1750 5350
+	4550 2250 4950 2250
+Connection ~ 4550 2550
 $Comp
 L R R57
 U 1 1 5931D3E3
-P 2300 5050
-F 0 "R57" V 2380 5050 50  0000 C CNN
-F 1 "0" V 2300 5050 50  0000 C CNN
-F 2 "" V 2230 5050 50  0001 C CNN
-F 3 "" H 2300 5050 50  0001 C CNN
-F 4 "RESS-001" V 2300 5050 60  0001 C CNN "part_num"
-	1    2300 5050
+P 5100 2250
+F 0 "R57" V 5180 2250 50  0000 C CNN
+F 1 "0" V 5100 2250 50  0000 C CNN
+F 2 "Resistors_SMD:R_0603_HandSoldering" V 5030 2250 50  0001 C CNN
+F 3 "" H 5100 2250 50  0001 C CNN
+F 4 "RESS-001" V 5100 2250 60  0001 C CNN "part_num"
+	1    5100 2250
 	0    1    1    0
 $EndComp
 Wire Wire Line
-	2450 5050 2900 5050
+	5250 2250 5700 2250
 Wire Wire Line
-	2900 5050 2900 5450
-Connection ~ 2900 5450
+	5700 2250 5700 2650
+Connection ~ 5700 2650
+Wire Wire Line
+	2550 3050 2550 3150
+Wire Wire Line
+	2550 3150 5200 3150
+Wire Wire Line
+	5200 3150 5200 3050
+Wire Wire Line
+	3700 3350 3700 3150
+Connection ~ 3700 3150
 $EndSCHEMATC

Commit message: PCB?!
Added initial PCB file with ratsnest. footprint library still needs to
be setup.
Parts:
- U17, U18: footprint (none) -> TO_SOT_Packages_SMD:SOT-353_SC-70-5_Handsoldering
- renumbered R58 to R82, R57 to R83
Changed lines of the file:
@@
 Comment4 ""
 $EndDescr
-$Comp
-L NC7SZ125P5X U18
-U 1 1 59290140
-P 2450 2850
-F 0 "U18" H 2450 3550 60  0000 C CNN
-F 1 "NC7SZ125P5X" H 2400 2350 60  0000 C CNN
-F 2 "" H 2400 2850 60  0001 C CNN
-F 3 "" H 2400 2850 60  0001 C CNN
-F 4 "CHIP-002" H 2450 2850 60  0001 C CNN "part_num"
-	1    2450 2850
-	1    0    0    -1
-$EndComp
 Wire Wire Line
 	2000 2750 2000 3050
@@
 Text Label 3550 3150 2    60   ~ 0
 VCC
-$Comp
-L NC7SZ125P5X U17
-U 1 1 59290291
-P 5100 2850
-F 0 "U17" H 5100 3550 60  0000 C CNN
-F 1 "NC7SZ125P5X" H 5050 2350 60  0000 C CNN
-F 2 "" H 5050 2850 60  0001 C CNN
-F 3 "CHIP-002" H 5050 2850 60  0001 C CNN
-F 4 "CHIP-002" H 5100 2850 60  0001 C CNN "part_num"
-	1    5100 2850
-	1    0    0    -1
-$EndComp
 Wire Wire Line
 	4650 2750 4650 3050
@@
 	3150 2650 2950 2650
 $Comp
-L R R58
+L R R82
 U 1 1 5931D2C2
 P 2450 2300
-F 0 "R58" V 2530 2300 50  0000 C CNN
+F 0 "R82" V 2530 2300 50  0000 C CNN
 F 1 "0" V 2450 2300 50  0000 C CNN
 F 2 "Resistors_SMD:R_0603_HandSoldering" V 2380 2300 50  0001 C CNN
@@
 Connection ~ 4550 2550
 $Comp
-L R R57
+L R R83
 U 1 1 5931D3E3
 P 5100 2250
-F 0 "R57" V 5180 2250 50  0000 C CNN
+F 0 "R83" V 5180 2250 50  0000 C CNN
 F 1 "0" V 5100 2250 50  0000 C CNN
 F 2 "Resistors_SMD:R_0603_HandSoldering" V 5030 2250 50  0001 C CNN
@@
 	3700 3350 3700 3150
 Connection ~ 3700 3150
+$Comp
+L NC7SZ125P5X U17
+U 1 1 595FABF1
+P 2450 2850
+F 0 "U17" H 2450 3550 60  0000 C CNN
+F 1 "NC7SZ125P5X" H 2400 2350 60  0000 C CNN
+F 2 "TO_SOT_Packages_SMD:SOT-353_SC-70-5_Handsoldering" H 2400 2850 60  0001 C CNN
+F 3 "" H 2400 2850 60  0001 C CNN
+F 4 "CHIP-002" H 2550 3650 60  0000 C CNN "part_num"
+	1    2450 2850
+	1    0    0    -1
+$EndComp
+$Comp
+L NC7SZ125P5X U18
+U 1 1 595FAC26
+P 5100 2850
+F 0 "U18" H 5100 3550 60  0000 C CNN
+F 1 "NC7SZ125P5X" H 5050 2350 60  0000 C CNN
+F 2 "TO_SOT_Packages_SMD:SOT-353_SC-70-5_Handsoldering" H 5050 2850 60  0001 C CNN
+F 3 "" H 5050 2850 60  0001 C CNN
+F 4 "CHIP-002" H 5200 3650 60  0000 C CNN "part_num"
+	1    5100 2850
+	1    0    0    -1
+$EndComp
 $EndSCHEMATC

Commit message: Fixed serge suggestions
Parts:
- removed R82, R83: 0, Resistors_SMD:R_0603_HandSoldering, symbol R
- added SH1, SH2: SHORT, symbol SHORT
Changed lines of the file:
@@
 $Descr A4 11693 8268
 encoding utf-8
-Sheet 18 20
+Sheet 18 21
 Title ""
 Date ""
@@
 	1750 2550 2000 2550
 Wire Wire Line
-	3150 2650 2950 2650
-$Comp
-L R R82
-U 1 1 5931D2C2
-P 2450 2300
-F 0 "R82" V 2530 2300 50  0000 C CNN
-F 1 "0" V 2450 2300 50  0000 C CNN
-F 2 "Resistors_SMD:R_0603_HandSoldering" V 2380 2300 50  0001 C CNN
-F 3 "" H 2450 2300 50  0001 C CNN
-F 4 "RESS-001" V 2450 2300 60  0001 C CNN "part_num"
-	1    2450 2300
-	0    1    1    0
-$EndComp
+	2950 2650 3150 2650
 Wire Wire Line
 	2300 2300 1900 2300
@@
 Connection ~ 1900 2550
 Wire Wire Line
-	2600 2300 3050 2300
+	2650 2300 3050 2300
 Wire Wire Line
 	3050 2300 3050 2650
 Connection ~ 3050 2650
 Wire Wire Line
-	5850 2650 5600 2650
+	5600 2650 5850 2650
 Wire Wire Line
-	4650 2550 4400 2550
+	4400 2550 4650 2550
 Wire Wire Line
 	4550 2550 4550 2250
 Wire Wire Line
-	4550 2250 4950 2250
+	4550 2250 4900 2250
 Connection ~ 4550 2550
-$Comp
-L R R83
-U 1 1 5931D3E3
-P 5100 2250
-F 0 "R83" V 5180 2250 50  0000 C CNN
-F 1 "0" V 5100 2250 50  0000 C CNN
-F 2 "Resistors_SMD:R_0603_HandSoldering" V 5030 2250 50  0001 C CNN
-F 3 "" H 5100 2250 50  0001 C CNN
-F 4 "RESS-001" V 5100 2250 60  0001 C CNN "part_num"
-	1    5100 2250
-	0    1    1    0
-$EndComp
 Wire Wire Line
 	5250 2250 5700 2250
@@
 	1    0    0    -1
 $EndComp
+$Comp
+L SHORT SH1
+U 1 1 59675A90
+P 2450 2300
+F 0 "SH1" H 2450 2450 60  0000 C CNN
+F 1 "SHORT" H 2450 2200 60  0000 C CNN
+F 2 "" H 2450 2300 60  0001 C CNN
+F 3 "" H 2450 2300 60  0001 C CNN
+	1    2450 2300
+	1    0    0    -1
+$EndComp
+$Comp
+L SHORT SH2
+U 1 1 59675ABF
+P 5050 2250
+F 0 "SH2" H 5050 2400 60  0000 C CNN
+F 1 "SHORT" H 5050 2150 60  0000 C CNN
+F 2 "" H 5050 2250 60  0001 C CNN
+F 3 "" H 5050 2250 60  0001 C CNN
+	1    5050 2250
+	1    0    0    -1
+$EndComp

Commit message: commit before my computer restarts
Parts:
- SH1, SH2: footprint (none) -> WARG:solder_bridge
Changed lines of the file:
@@
 Text HLabel 1750 2550 0    60   Input ~ 0
 PPM_IN
-Text HLabel 3150 2650 2    60   Input ~ 0
+Text HLabel 3150 2650 2    60   Output ~ 0
 PPM_OUT
 Text HLabel 3700 3350 3    60   Input ~ 0
@@
 Text HLabel 4400 2550 0    60   Input ~ 0
 RX_IN
-Text HLabel 5850 2650 2    60   Input ~ 0
+Text HLabel 5850 2650 2    60   Output ~ 0
 RX_OUT
 Wire Wire Line
@@
 $Comp
 L SHORT SH1
-U 1 1 59675A90
-P 2450 2300
-F 0 "SH1" H 2450 2450 60  0000 C CNN
-F 1 "SHORT" H 2450 2200 60  0000 C CNN
-F 2 "" H 2450 2300 60  0001 C CNN
-F 3 "" H 2450 2300 60  0001 C CNN
-	1    2450 2300
+U 1 1 596CF8A7
+P 2500 2300
+F 0 "SH1" H 2500 2450 60  0000 C CNN
+F 1 "SHORT" H 2500 2200 60  0000 C CNN
+F 2 "WARG:solder_bridge" H 2400 2350 60  0001 C CNN
+F 3 "" H 2500 2300 60  0001 C CNN
+	1    2500 2300
 	1    0    0    -1
 $EndComp
 $Comp
 L SHORT SH2
-U 1 1 59675ABF
-P 5050 2250
-F 0 "SH2" H 5050 2400 60  0000 C CNN
-F 1 "SHORT" H 5050 2150 60  0000 C CNN
-F 2 "" H 5050 2250 60  0001 C CNN
-F 3 "" H 5050 2250 60  0001 C CNN
-	1    5050 2250
+U 1 1 596CF8D2
+P 5100 2250
+F 0 "SH2" H 5100 2400 60  0000 C CNN
+F 1 "SHORT" H 5100 2150 60  0000 C CNN
+F 2 "WARG:solder_bridge" H 5000 2300 60  0001 C CNN
+F 3 "" H 5100 2250 60  0001 C CNN
+	1    5100 2250
 	1    0    0    -1
 $EndComp

Commit message: placed headers in roughly correct spot
Connections:
- net labels added: GND
- wire segments 20 -> 24
Changed lines of the file:
@@
 	1    0    0    -1
 $EndComp
+$Comp
+L GND #PWR?
+U 1 1 592EC337
+P 4500 2950
+F 0 "#PWR?" H 4500 2700 50  0001 C CNN
+F 1 "GND" H 4500 2800 50  0000 C CNN
+F 2 "" H 4500 2950 50  0001 C CNN
+F 3 "" H 4500 2950 50  0001 C CNN
+	1    4500 2950
+	1    0    0    -1
+$EndComp
+Wire Wire Line
+	4500 2950 4500 2900
+Wire Wire Line
+	4500 2900 4650 2900
+Connection ~ 4650 2900
+Connection ~ 4650 3000
+$Comp
+L GND #PWR?
+U 1 1 592EC3EA
+P 1800 3000
+F 0 "#PWR?" H 1800 2750 50  0001 C CNN
+F 1 "GND" H 1800 2850 50  0000 C CNN
+F 2 "" H 1800 3000 50  0001 C CNN
+F 3 "" H 1800 3000 50  0001 C CNN
+	1    1800 3000
+	1    0    0    -1
+$EndComp
+Wire Wire Line
+	1800 3000 1800 2900
+Wire Wire Line
+	1800 2900 2000 2900
+Connection ~ 2000 2900
 $EndSCHEMATC
