File: Hardware/PWM.sch (KiCad schematic (older format))
At the start: 7 parts, among them P1 PWM, U1 NLAS4599

Commit message: first rough draft without headers
Changed lines of the file:
@@
 $Descr A4 11693 8268
 encoding utf-8
-Sheet 6 18
+Sheet 5 19
 Title "PWM Switching Circuit"
 Date "2017-05-13"
@@
 AR Path="/591E6415/591EA4FC/5917D576" Ref="P11"  Part="1"
 AR Path="/591E6415/591EA50E/5917D576" Ref="P12"  Part="1"
-F 0 "P4" H 6350 2600 50  0001 C CNN
+F 0 "P3" H 6350 2600 50  0001 C CNN
 F 1 "PWM" V 6450 2400 50  0000 C CNN
 F 2 "" H 6350 2400 50  0000 C CNN
@@
 AR Path="/591E6415/591EA4FC/5917D57C" Ref="U11"  Part="1"
 AR Path="/591E6415/591EA50E/5917D57C" Ref="U12"  Part="1"
-F 0 "U4" H 4500 3250 60  0000 C CNN
+F 0 "U3" H 4500 3250 60  0000 C CNN
 F 1 "NLAS4599" H 4550 2500 60  0000 C CNN
 F 2 "" H 4300 2350 60  0001 C CNN
@@
 	4900 2500 6150 2500
 $Comp
-L GND #PWR01
+L GND #PWR03
 U 1 1 5917D836
 P 5100 2700
-AR Path="/591E6415/591EA448/5917D836" Ref="#PWR01"  Part="1"
-AR Path="/591E6415/591EA45A/5917D836" Ref="#PWR03"  Part="1"
-AR Path="/591E6415/591EA46C/5917D836" Ref="#PWR05"  Part="1"
-AR Path="/591E6415/591EA47E/5917D836" Ref="#PWR07"  Part="1"
-AR Path="/591E6415/591EA490/5917D836" Ref="#PWR09"  Part="1"
-AR Path="/591E6415/591EA4A2/5917D836" Ref="#PWR011"  Part="1"
-AR Path="/591E6415/591EA4B4/5917D836" Ref="#PWR013"  Part="1"
-AR Path="/591E6415/591EA4C6/5917D836" Ref="#PWR015"  Part="1"
-AR Path="/591E6415/591EA4D8/5917D836" Ref="#PWR017"  Part="1"
-AR Path="/591E6415/591EA4EA/5917D836" Ref="#PWR019"  Part="1"
-AR Path="/591E6415/591EA4FC/5917D836" Ref="#PWR021"  Part="1"
-AR Path="/591E6415/591EA50E/5917D836" Ref="#PWR023"  Part="1"
+AR Path="/591E6415/591EA448/5917D836" Ref="#PWR03"  Part="1"
+AR Path="/591E6415/591EA45A/5917D836" Ref="#PWR05"  Part="1"
+AR Path="/591E6415/591EA46C/5917D836" Ref="#PWR07"  Part="1"
+AR Path="/591E6415/591EA47E/5917D836" Ref="#PWR09"  Part="1"
+AR Path="/591E6415/591EA490/5917D836" Ref="#PWR011"  Part="1"
+AR Path="/591E6415/591EA4A2/5917D836" Ref="#PWR013"  Part="1"
+AR Path="/591E6415/591EA4B4/5917D836" Ref="#PWR015"  Part="1"
+AR Path="/591E6415/591EA4C6/5917D836" Ref="#PWR017"  Part="1"
+AR Path="/591E6415/591EA4D8/5917D836" Ref="#PWR019"  Part="1"
+AR Path="/591E6415/591EA4EA/5917D836" Ref="#PWR021"  Part="1"
+AR Path="/591E6415/591EA4FC/5917D836" Ref="#PWR023"  Part="1"
+AR Path="/591E6415/591EA50E/5917D836" Ref="#PWR025"  Part="1"
 F 0 "#PWR07" H 5100 2450 50  0001 C CNN
 F 1 "GND" H 5100 2550 50  0000 C CNN
@@
 AR Path="/591E6415/591EA4FC/591EF19A" Ref="D11"  Part="1"
 AR Path="/591E6415/591EA50E/591EF19A" Ref="D12"  Part="1"
-F 0 "D4" H 3550 3100 50  0000 C CNN
+F 0 "D3" H 3550 3100 50  0000 C CNN
 F 1 "LED" H 3550 2900 50  0000 C CNN
 F 2 "" H 3550 3000 50  0000 C CNN
@@
 AR Path="/591E6415/591EA4FC/591EF2D3" Ref="R32"  Part="1"
 AR Path="/591E6415/591EA50E/591EF2D3" Ref="R35"  Part="1"
-F 0 "R11" V 3630 2650 50  0000 C CNN
+F 0 "R8" V 3630 2650 50  0000 C CNN
 F 1 "250" V 3550 2650 50  0000 C CNN
 F 2 "" V 3480 2650 50  0000 C CNN
@@
 Connection ~ 3550 2450
 $Comp
-L GND #PWR02
+L GND #PWR04
 U 1 1 591EF3D9
 P 3350 3250
-AR Path="/591E6415/591EA448/591EF3D9" Ref="#PWR02"  Part="1"
-AR Path="/591E6415/591EA45A/591EF3D9" Ref="#PWR04"  Part="1"
-AR Path="/591E6415/591EA46C/591EF3D9" Ref="#PWR06"  Part="1"
-AR Path="/591E6415/591EA47E/591EF3D9" Ref="#PWR08"  Part="1"
-AR Path="/591E6415/591EA490/591EF3D9" Ref="#PWR010"  Part="1"
-AR Path="/591E6415/591EA4A2/591EF3D9" Ref="#PWR012"  Part="1"
-AR Path="/591E6415/591EA4B4/591EF3D9" Ref="#PWR014"  Part="1"
-AR Path="/591E6415/591EA4C6/591EF3D9" Ref="#PWR016"  Part="1"
-AR Path="/591E6415/591EA4D8/591EF3D9" Ref="#PWR018"  Part="1"
-AR Path="/591E6415/591EA4EA/591EF3D9" Ref="#PWR020"  Part="1"
-AR Path="/591E6415/591EA4FC/591EF3D9" Ref="#PWR022"  Part="1"
-AR Path="/591E6415/591EA50E/591EF3D9" Ref="#PWR024"  Part="1"
+AR Path="/591E6415/591EA448/591EF3D9" Ref="#PWR04"  Part="1"
+AR Path="/591E6415/591EA45A/591EF3D9" Ref="#PWR06"  Part="1"
+AR Path="/591E6415/591EA46C/591EF3D9" Ref="#PWR08"  Part="1"
+AR Path="/591E6415/591EA47E/591EF3D9" Ref="#PWR010"  Part="1"
+AR Path="/591E6415/591EA490/591EF3D9" Ref="#PWR012"  Part="1"
+AR Path="/591E6415/591EA4A2/591EF3D9" Ref="#PWR014"  Part="1"
+AR Path="/591E6415/591EA4B4/591EF3D9" Ref="#PWR016"  Part="1"
+AR Path="/591E6415/591EA4C6/591EF3D9" Ref="#PWR018"  Part="1"
+AR Path="/591E6415/591EA4D8/591EF3D9" Ref="#PWR020"  Part="1"
+AR Path="/591E6415/591EA4EA/591EF3D9" Ref="#PWR022"  Part="1"
+AR Path="/591E6415/591EA4FC/591EF3D9" Ref="#PWR024"  Part="1"
+AR Path="/591E6415/591EA50E/591EF3D9" Ref="#PWR026"  Part="1"
 F 0 "#PWR08" H 3350 3000 50  0001 C CNN
 F 1 "GND" H 3350 3100 50  0000 C CNN
@@
 AR Path="/591E6415/591EA4FC/591F0A89" Ref="R31"  Part="1"
 AR Path="/591E6415/591EA50E/591F0A89" Ref="R34"  Part="1"
-F 0 "R10" V 3230 2650 50  0000 C CNN
+F 0 "R7" V 3230 2650 50  0000 C CNN
 F 1 "10K" V 3150 2650 50  0000 C CNN
 F 2 "" V 3080 2650 50  0000 C CNN
@@
 AR Path="/591E6415/591EA4FC/591F0BAE" Ref="R33"  Part="1"
 AR Path="/591E6415/591EA50E/591F0BAE" Ref="R36"  Part="1"
-F 0 "R12" V 3880 2450 50  0000 C CNN
+F 0 "R9" V 3880 2450 50  0000 C CNN
 F 1 "0" V 3800 2450 50  0000 C CNN
 F 2 "" V 3730 2450 50  0000 C CNN
@@
 AR Path="/591E6415/591EA4FC/591F0CEF" Ref="TP11"  Part="1"
 AR Path="/591E6415/591EA50E/591F0CEF" Ref="TP12"  Part="1"
-F 0 "TP4" H 4000 2900 50  0000 C BNN
+F 0 "TP3" H 4000 2900 50  0000 C BNN
 F 1 "TEST" H 4000 2850 50  0000 C CNN
 F 2 "" H 4000 2600 50  0000 C CNN

Commit message: branch to make PR for review
I should have made a separate branch for the development and then merged
it, but its too late now.
Parts:
- renumbered R1 to R5, R2 to R6, R3 to R7
Changed lines of the file:
@@
 $Descr A4 11693 8268
 encoding utf-8
-Sheet 5 19
+Sheet 14 19
 Title "PWM Switching Circuit"
 Date "2017-05-13"
@@
 AR Path="/591E6415/591EA4FC/5917D576" Ref="P11"  Part="1"
 AR Path="/591E6415/591EA50E/5917D576" Ref="P12"  Part="1"
-F 0 "P3" H 6350 2600 50  0001 C CNN
+F 0 "P12" H 6350 2600 50  0001 C CNN
 F 1 "PWM" V 6450 2400 50  0000 C CNN
 F 2 "" H 6350 2400 50  0000 C CNN
@@
 AR Path="/591E6415/591EA4FC/5917D57C" Ref="U11"  Part="1"
 AR Path="/591E6415/591EA50E/5917D57C" Ref="U12"  Part="1"
-F 0 "U3" H 4500 3250 60  0000 C CNN
+F 0 "U12" H 4500 3250 60  0000 C CNN
 F 1 "NLAS4599" H 4550 2500 60  0000 C CNN
 F 2 "" H 4300 2350 60  0001 C CNN
@@
 	4900 2500 6150 2500
 $Comp
-L GND #PWR03
+L GND #PWR4
 U 1 1 5917D836
 P 5100 2700
-AR Path="/591E6415/591EA448/5917D836" Ref="#PWR03"  Part="1"
-AR Path="/591E6415/591EA45A/5917D836" Ref="#PWR05"  Part="1"
-AR Path="/591E6415/591EA46C/5917D836" Ref="#PWR07"  Part="1"
-AR Path="/591E6415/591EA47E/5917D836" Ref="#PWR09"  Part="1"
-AR Path="/591E6415/591EA490/5917D836" Ref="#PWR011"  Part="1"
-AR Path="/591E6415/591EA4A2/5917D836" Ref="#PWR013"  Part="1"
-AR Path="/591E6415/591EA4B4/5917D836" Ref="#PWR015"  Part="1"
-AR Path="/591E6415/591EA4C6/5917D836" Ref="#PWR017"  Part="1"
-AR Path="/591E6415/591EA4D8/5917D836" Ref="#PWR019"  Part="1"
-AR Path="/591E6415/591EA4EA/5917D836" Ref="#PWR021"  Part="1"
-AR Path="/591E6415/591EA4FC/5917D836" Ref="#PWR023"  Part="1"
-AR Path="/591E6415/591EA50E/5917D836" Ref="#PWR025"  Part="1"
-F 0 "#PWR07" H 5100 2450 50  0001 C CNN
+AR Path="/591E6415/591EA448/5917D836" Ref="#PWR4"  Part="1"
+AR Path="/591E6415/591EA45A/5917D836" Ref="#PWR6"  Part="1"
+AR Path="/591E6415/591EA46C/5917D836" Ref="#PWR8"  Part="1"
+AR Path="/591E6415/591EA47E/5917D836" Ref="#PWR10"  Part="1"
+AR Path="/591E6415/591EA490/5917D836" Ref="#PWR12"  Part="1"
+AR Path="/591E6415/591EA4A2/5917D836" Ref="#PWR14"  Part="1"
+AR Path="/591E6415/591EA4B4/5917D836" Ref="#PWR16"  Part="1"
+AR Path="/591E6415/591EA4C6/5917D836" Ref="#PWR18"  Part="1"
+AR Path="/591E6415/591EA4D8/5917D836" Ref="#PWR20"  Part="1"
+AR Path="/591E6415/591EA4EA/5917D836" Ref="#PWR22"  Part="1"
+AR Path="/591E6415/591EA4FC/5917D836" Ref="#PWR24"  Part="1"
+AR Path="/591E6415/591EA50E/5917D836" Ref="#PWR26"  Part="1"
+F 0 "#PWR26" H 5100 2450 50  0001 C CNN
 F 1 "GND" H 5100 2550 50  0000 C CNN
 F 2 "" H 5100 2700 50  0000 C CNN
@@
 AR Path="/591E6415/591EA4FC/591EF19A" Ref="D11"  Part="1"
 AR Path="/591E6415/591EA50E/591EF19A" Ref="D12"  Part="1"
-F 0 "D3" H 3550 3100 50  0000 C CNN
+F 0 "D12" H 3550 3100 50  0000 C CNN
 F 1 "LED" H 3550 2900 50  0000 C CNN
 F 2 "" H 3550 3000 50  0000 C CNN
@@
 $EndComp
 $Comp
-L R R2
+L R R6
 U 1 1 591EF2D3
 P 3550 2650
-AR Path="/591E6415/591EA448/591EF2D3" Ref="R2"  Part="1"
-AR Path="/591E6415/591EA45A/591EF2D3" Ref="R5"  Part="1"
-AR Path="/591E6415/591EA46C/591EF2D3" Ref="R8"  Part="1"
-AR Path="/591E6415/591EA47E/591EF2D3" Ref="R11"  Part="1"
-AR Path="/591E6415/591EA490/591EF2D3" Ref="R14"  Part="1"
-AR Path="/591E6415/591EA4A2/591EF2D3" Ref="R17"  Part="1"
-AR Path="/591E6415/591EA4B4/591EF2D3" Ref="R20"  Part="1"
-AR Path="/591E6415/591EA4C6/591EF2D3" Ref="R23"  Part="1"
-AR Path="/591E6415/591EA4D8/591EF2D3" Ref="R26"  Part="1"
-AR Path="/591E6415/591EA4EA/591EF2D3" Ref="R29"  Part="1"
-AR Path="/591E6415/591EA4FC/591EF2D3" Ref="R32"  Part="1"
-AR Path="/591E6415/591EA50E/591EF2D3" Ref="R35"  Part="1"
-F 0 "R8" V 3630 2650 50  0000 C CNN
+AR Path="/591E6415/591EA448/591EF2D3" Ref="R6"  Part="1"
+AR Path="/591E6415/591EA45A/591EF2D3" Ref="R9"  Part="1"
+AR Path="/591E6415/591EA46C/591EF2D3" Ref="R12"  Part="1"
+AR Path="/591E6415/591EA47E/591EF2D3" Ref="R15"  Part="1"
+AR Path="/591E6415/591EA490/591EF2D3" Ref="R18"  Part="1"
+AR Path="/591E6415/591EA4A2/591EF2D3" Ref="R21"  Part="1"
+AR Path="/591E6415/591EA4B4/591EF2D3" Ref="R24"  Part="1"
+AR Path="/591E6415/591EA4C6/591EF2D3" Ref="R27"  Part="1"
+AR Path="/591E6415/591EA4D8/591EF2D3" Ref="R30"  Part="1"
+AR Path="/591E6415/591EA4EA/591EF2D3" Ref="R33"  Part="1"
+AR Path="/591E6415/591EA4FC/591EF2D3" Ref="R36"  Part="1"
+AR Path="/591E6415/591EA50E/591EF2D3" Ref="R39"  Part="1"
+F 0 "R39" V 3630 2650 50  0000 C CNN
 F 1 "250" V 3550 2650 50  0000 C CNN
 F 2 "" V 3480 2650 50  0000 C CNN
@@
 Connection ~ 3550 2450
 $Comp
-L GND #PWR04
+L GND #PWR3
 U 1 1 591EF3D9
 P 3350 3250
-AR Path="/591E6415/591EA448/591EF3D9" Ref="#PWR04"  Part="1"
-AR Path="/591E6415/591EA45A/591EF3D9" Ref="#PWR06"  Part="1"
-AR Path="/591E6415/591EA46C/591EF3D9" Ref="#PWR08"  Part="1"
-AR Path="/591E6415/591EA47E/591EF3D9" Ref="#PWR010"  Part="1"
-AR Path="/591E6415/591EA490/591EF3D9" Ref="#PWR012"  Part="1"
-AR Path="/591E6415/591EA4A2/591EF3D9" Ref="#PWR014"  Part="1"
-AR Path="/591E6415/591EA4B4/591EF3D9" Ref="#PWR016"  Part="1"
-AR Path="/591E6415/591EA4C6/591EF3D9" Ref="#PWR018"  Part="1"
-AR Path="/591E6415/591EA4D8/591EF3D9" Ref="#PWR020"  Part="1"
-AR Path="/591E6415/591EA4EA/591EF3D9" Ref="#PWR022"  Part="1"
-AR Path="/591E6415/591EA4FC/591EF3D9" Ref="#PWR024"  Part="1"
-AR Path="/591E6415/591EA50E/591EF3D9" Ref="#PWR026"  Part="1"
-F 0 "#PWR08" H 3350 3000 50  0001 C CNN
+AR Path="/591E6415/591EA448/591EF3D9" Ref="#PWR3"  Part="1"
+AR Path="/591E6415/591EA45A/591EF3D9" Ref="#PWR5"  Part="1"
+AR Path="/591E6415/591EA46C/591EF3D9" Ref="#PWR7"  Part="1"
+AR Path="/591E6415/591EA47E/591EF3D9" Ref="#PWR9"  Part="1"
+AR Path="/591E6415/591EA490/591EF3D9" Ref="#PWR11"  Part="1"
+AR Path="/591E6415/591EA4A2/591EF3D9" Ref="#PWR13"  Part="1"
+AR Path="/591E6415/591EA4B4/591EF3D9" Ref="#PWR15"  Part="1"
+AR Path="/591E6415/591EA4C6/591EF3D9" Ref="#PWR17"  Part="1"
+AR Path="/591E6415/591EA4D8/591EF3D9" Ref="#PWR19"  Part="1"
+AR Path="/591E6415/591EA4EA/591EF3D9" Ref="#PWR21"  Part="1"
+AR Path="/591E6415/591EA4FC/591EF3D9" Ref="#PWR23"  Part="1"
+AR Path="/591E6415/591EA50E/591EF3D9" Ref="#PWR25"  Part="1"
+F 0 "#PWR25" H 3350 3000 50  0001 C CNN
 F 1 "GND" H 3350 3100 50  0000 C CNN
 F 2 "" H 3350 3250 50  0000 C CNN
@@
 	3550 3200 3550 3150
 $Comp
-L R R1
+L R R5
 U 1 1 591F0A89
 P 3150 2650
-AR Path="/591E6415/591EA448/591F0A89" Ref="R1"  Part="1"
-AR Path="/591E6415/591EA45A/591F0A89" Ref="R4"  Part="1"
-AR Path="/591E6415/591EA46C/591F0A89" Ref="R7"  Part="1"
-AR Path="/591E6415/591EA47E/591F0A89" Ref="R10"  Part="1"
-AR Path="/591E6415/591EA490/591F0A89" Ref="R13"  Part="1"
-AR Path="/591E6415/591EA4A2/591F0A89" Ref="R16"  Part="1"
-AR Path="/591E6415/591EA4B4/591F0A89" Ref="R19"  Part="1"
-AR Path="/591E6415/591EA4C6/591F0A89" Ref="R22"  Part="1"
-AR Path="/591E6415/591EA4D8/591F0A89" Ref="R25"  Part="1"
-AR Path="/591E6415/591EA4EA/591F0A89" Ref="R28"  Part="1"
-AR Path="/591E6415/591EA4FC/591F0A89" Ref="R31"  Part="1"
-AR Path="/591E6415/591EA50E/591F0A89" Ref="R34"  Part="1"
-F 0 "R7" V 3230 2650 50  0000 C CNN
+AR Path="/591E6415/591EA448/591F0A89" Ref="R5"  Part="1"
+AR Path="/591E6415/591EA45A/591F0A89" Ref="R8"  Part="1"
+AR Path="/591E6415/591EA46C/591F0A89" Ref="R11"  Part="1"
+AR Path="/591E6415/591EA47E/591F0A89" Ref="R14"  Part="1"
+AR Path="/591E6415/591EA490/591F0A89" Ref="R17"  Part="1"
+AR Path="/591E6415/591EA4A2/591F0A89" Ref="R20"  Part="1"
+AR Path="/591E6415/591EA4B4/591F0A89" Ref="R23"  Part="1"
+AR Path="/591E6415/591EA4C6/591F0A89" Ref="R26"  Part="1"
+AR Path="/591E6415/591EA4D8/591F0A89" Ref="R29"  Part="1"
+AR Path="/591E6415/591EA4EA/591F0A89" Ref="R32"  Part="1"
+AR Path="/591E6415/591EA4FC/591F0A89" Ref="R35"  Part="1"
+AR Path="/591E6415/591EA50E/591F0A89" Ref="R38"  Part="1"
+F 0 "R38" V 3230 2650 50  0000 C CNN
 F 1 "10K" V 3150 2650 50  0000 C CNN
 F 2 "" V 3080 2650 50  0000 C CNN
@@
 Connection ~ 3150 2450
 $Comp
-L R R3
+L R R7
 U 1 1 591F0BAE
 P 3800 2450
-AR Path="/591E6415/591EA448/591F0BAE" Ref="R3"  Part="1"
-AR Path="/591E6415/591EA45A/591F0BAE" Ref="R6"  Part="1"
-AR Path="/591E6415/591EA46C/591F0BAE" Ref="R9"  Part="1"
-AR Path="/591E6415/591EA47E/591F0BAE" Ref="R12"  Part="1"
-AR Path="/591E6415/591EA490/591F0BAE" Ref="R15"  Part="1"
-AR Path="/591E6415/591EA4A2/591F0BAE" Ref="R18"  Part="1"
-AR Path="/591E6415/591EA4B4/591F0BAE" Ref="R21"  Part="1"
-AR Path="/591E6415/591EA4C6/591F0BAE" Ref="R24"  Part="1"
-AR Path="/591E6415/591EA4D8/591F0BAE" Ref="R27"  Part="1"
-AR Path="/591E6415/591EA4EA/591F0BAE" Ref="R30"  Part="1"
-AR Path="/591E6415/591EA4FC/591F0BAE" Ref="R33"  Part="1"
-AR Path="/591E6415/591EA50E/591F0BAE" Ref="R36"  Part="1"
-F 0 "R9" V 3880 2450 50  0000 C CNN
+AR Path="/591E6415/591EA448/591F0BAE" Ref="R7"  Part="1"
+AR Path="/591E6415/591EA45A/591F0BAE" Ref="R10"  Part="1"
+AR Path="/591E6415/591EA46C/591F0BAE" Ref="R13"  Part="1"
+AR Path="/591E6415/591EA47E/591F0BAE" Ref="R16"  Part="1"
+AR Path="/591E6415/591EA490/591F0BAE" Ref="R19"  Part="1"
+AR Path="/591E6415/591EA4A2/591F0BAE" Ref="R22"  Part="1"
+AR Path="/591E6415/591EA4B4/591F0BAE" Ref="R25"  Part="1"
+AR Path="/591E6415/591EA4C6/591F0BAE" Ref="R28"  Part="1"
+AR Path="/591E6415/591EA4D8/591F0BAE" Ref="R31"  Part="1"
+AR Path="/591E6415/591EA4EA/591F0BAE" Ref="R34"  Part="1"
+AR Path="/591E6415/591EA4FC/591F0BAE" Ref="R37"  Part="1"
+AR Path="/591E6415/591EA50E/591F0BAE" Ref="R40"  Part="1"
+F 0 "R40" V 3880 2450 50  0000 C CNN
 F 1 "0" V 3800 2450 50  0000 C CNN
 F 2 "" V 3730 2450 50  0000 C CNN
@@
 AR Path="/591E6415/591EA4FC/591F0CEF" Ref="TP11"  Part="1"
 AR Path="/591E6415/591EA50E/591F0CEF" Ref="TP12"  Part="1"
-F 0 "TP3" H 4000 2900 50  0000 C BNN
+F 0 "TP12" H 4000 2900 50  0000 C BNN
 F 1 "TEST" H 4000 2850 50  0000 C CNN
 F 2 "" H 4000 2600 50  0000 C CNN

Commit message: Added a lot of debug
Parts:
- added TP? (x2): TEST, symbol TEST
- added U? (x2): SHORT, symbol SHORT
- R6: value 250 -> 100
Connections:
- wire segments 21 -> 25
Other:
- moved on the sheet: R11
Changed lines of the file:
@@
 $Descr A4 11693 8268
 encoding utf-8
-Sheet 14 19
+Sheet 5 19
 Title "PWM Switching Circuit"
 Date "2017-05-13"
@@
 AR Path="/591E6415/591EA4FC/5917D576" Ref="P11"  Part="1"
 AR Path="/591E6415/591EA50E/5917D576" Ref="P12"  Part="1"
-F 0 "P12" H 6350 2600 50  0001 C CNN
+F 0 "P3" H 6350 2600 50  0001 C CNN
 F 1 "PWM" V 6450 2400 50  0000 C CNN
 F 2 "" H 6350 2400 50  0000 C CNN
@@
 AR Path="/591E6415/591EA4FC/5917D57C" Ref="U11"  Part="1"
 AR Path="/591E6415/591EA50E/5917D57C" Ref="U12"  Part="1"
-F 0 "U12" H 4500 3250 60  0000 C CNN
+F 0 "U3" H 4500 3250 60  0000 C CNN
 F 1 "NLAS4599" H 4550 2500 60  0000 C CNN
 F 2 "" H 4300 2350 60  0001 C CNN
@@
 AR Path="/591E6415/591EA4FC/5917D836" Ref="#PWR24"  Part="1"
 AR Path="/591E6415/591EA50E/5917D836" Ref="#PWR26"  Part="1"
-F 0 "#PWR26" H 5100 2450 50  0001 C CNN
+F 0 "#PWR8" H 5100 2450 50  0001 C CNN
 F 1 "GND" H 5100 2550 50  0000 C CNN
 F 2 "" H 5100 2700 50  0000 C CNN
@@
 OC
 Wire Wire Line
-	2750 2150 4100 2150
-Wire Wire Line
-	2750 2250 4100 2250
+	2750 2150 2950 2150
+Wire Wire Line
+	2750 2250 3200 2250
 Wire Wire Line
 	2750 2450 3650 2450
@@
 AR Path="/591E6415/591EA4FC/591EF19A" Ref="D11"  Part="1"
 AR Path="/591E6415/591EA50E/591EF19A" Ref="D12"  Part="1"
-F 0 "D12" H 3550 3100 50  0000 C CNN
+F 0 "D3" H 3550 3100 50  0000 C CNN
 F 1 "LED" H 3550 2900 50  0000 C CNN
 F 2 "" H 3550 3000 50  0000 C CNN
@@
 AR Path="/591E6415/591EA4FC/591EF2D3" Ref="R36"  Part="1"
 AR Path="/591E6415/591EA50E/591EF2D3" Ref="R39"  Part="1"
-F 0 "R39" V 3630 2650 50  0000 C CNN
-F 1 "250" V 3550 2650 50  0000 C CNN
+F 0 "R12" V 3630 2650 50  0000 C CNN
+F 1 "100" V 3550 2650 50  0000 C CNN
 F 2 "" V 3480 2650 50  0000 C CNN
 F 3 "" H 3550 2650 50  0000 C CNN
@@
 AR Path="/591E6415/591EA4FC/591EF3D9" Ref="#PWR23"  Part="1"
 AR Path="/591E6415/591EA50E/591EF3D9" Ref="#PWR25"  Part="1"
-F 0 "#PWR25" H 3350 3000 50  0001 C CNN
+F 0 "#PWR7" H 3350 3000 50  0001 C CNN
 F 1 "GND" H 3350 3100 50  0000 C CNN
 F 2 "" H 3350 3250 50  0000 C CNN
@@
 L R R5
 U 1 1 591F0A89
-P 3150 2650
+P 3150 2800
 AR Path="/591E6415/591EA448/591F0A89" Ref="R5"  Part="1"
 AR Path="/591E6415/591EA45A/591F0A89" Ref="R8"  Part="1"
@@
 AR Path="/591E6415/591EA4FC/591F0A89" Ref="R35"  Part="1"
 AR Path="/591E6415/591EA50E/591F0A89" Ref="R38"  Part="1"
-F 0 "R38" V 3230 2650 50  0000 C CNN
-F 1 "10K" V 3150 2650 50  0000 C CNN
-F 2 "" V 3080 2650 50  0000 C CNN
-F 3 "" H 3150 2650 50  0000 C CNN
-	1    3150 2650
+F 0 "R11" V 3230 2800 50  0000 C CNN
+F 1 "10K" V 3150 2800 50  0000 C CNN
+F 2 "" V 3080 2800 50  0000 C CNN
+F 3 "" H 3150 2800 50  0000 C CNN
+	1    3150 2800
 	1    0    0    -1
 $EndComp
@@
 	3150 3200 3550 3200
 Wire Wire Line
-	3150 2800 3150 3200
-Wire Wire Line
-	3150 2500 3150 2450
+	3150 2950 3150 3200
+Wire Wire Line
+	3150 2650 3150 2450
 Connection ~ 3150 2450
 $Comp
@@
 AR Path="/591E6415/591EA4FC/591F0BAE" Ref="R37"  Part="1"
 AR Path="/591E6415/591EA50E/591F0BAE" Ref="R40"  Part="1"
-F 0 "R40" V 3880 2450 50  0000 C CNN
+F 0 "R13" V 3880 2450 50  0000 C CNN
 F 1 "0" V 3800 2450 50  0000 C CNN
 F 2 "" V 3730 2450 50  0000 C CNN
@@
 AR Path="/591E6415/591EA4FC/591F0CEF" Ref="TP11"  Part="1"
 AR Path="/591E6415/591EA50E/591F0CEF" Ref="TP12"  Part="1"
-F 0 "TP12" H 4000 2900 50  0000 C BNN
+F 0 "TP3" H 4000 2900 50  0000 C BNN
 F 1 "TEST" H 4000 2850 50  0000 C CNN
 F 2 "" H 4000 2600 50  0000 C CNN
@@
 Wire Wire Line
 	5100 2400 4900 2400
+$Comp
+L TEST TP?
+U 1 1 592CAEE3
+P 3900 2050
+AR Path="/591E6415/591EA448/592CAEE3" Ref="TP?"  Part="1"
+AR Path="/591E6415/591EA46C/592CAEE3" Ref="TP?"  Part="1"
+F 0 "TP?" H 3900 2350 50  0000 C BNN
+F 1 "TEST" H 3900 2300 50  0000 C CNN
+F 2 "" H 3900 2050 50  0000 C CNN
+F 3 "" H 3900 2050 50  0000 C CNN
+	1    3900 2050
+	1    0    0    -1
+$EndComp
+$Comp
+L TEST TP?
+U 1 1 592CAF2C
+P 3700 2050
+AR Path="/591E6415/591EA448/592CAF2C" Ref="TP?"  Part="1"
+AR Path="/591E6415/591EA46C/592CAF2C" Ref="TP?"  Part="1"
+F 0 "TP?" H 3700 2350 50  0000 C BNN
+F 1 "TEST" H 3700 2300 50  0000 C CNN
+F 2 "" H 3700 2050 50  0000 C CNN
+F 3 "" H 3700 2050 50  0000 C CNN
+	1    3700 2050
+	1    0    0    -1
+$EndComp
+$Comp
+L SHORT U?
+U 1 1 592EB0C1
+P 3100 2150
+F 0 "U?" H 3100 2300 60  0000 C CNN
+F 1 "SHORT" H 3100 2050 60  0000 C CNN
+F 2 "" H 3100 2150 60  0001 C CNN
+F 3 "" H 3100 2150 60  0001 C CNN
+	1    3100 2150
+	1    0    0    -1
+$EndComp
+$Comp
+L SHORT U?
+U 1 1 592EB103
+P 3350 2250
+F 0 "U?" H 3350 2400 60  0000 C CNN
+F 1 "SHORT" H 3350 2150 60  0000 C CNN
+F 2 "" H 3350 2250 60  0001 C CNN
+F 3 "" H 3350 2250 60  0001 C CNN
+	1    3350 2250
+	1    0    0    -1
+$EndComp
+Wire Wire Line
+	3300 2150 4100 2150
+Wire Wire Line
+	4100 2250 3550 2250
+Wire Wire Line
+	3700 2050 3700 2150
+Connection ~ 3700 2150
+Wire Wire Line
+	3900 2050 3900 2250
+Connection ~ 3900 2250
 $EndSCHEMATC
