File: Hardware/PWM.sch (KiCad schematic (older format))
At the start: 11 parts, among them P1 PWM, U1 NLAS4599

Commit message: Fixed some BOM stuff
fixed BOM for non RLC components
Parts:
- removed U? (x2): SHORT, symbol SHORT
- added SH? (x2): SHORT, symbol SHORT
- D7: renamed from D1; part_num (none) -> DIOD-002
- J7: renamed from P1; part_num (none) -> CONN-007
- U15: renamed from U1; part_num (none) -> CHIP-004
- gave numbers to parts that had none: 2
- renumbered R5 to R19, R6 to R20, R7 to R21, TP1 to TP17

Commit message: Finished RLC bom stuff
Parts:
- R7: renamed from R19; part_num (none) -> RESS-005
- R8: renamed from R20; part_num (none) -> RESS-006
- R9: renamed from R21; part_num (none) -> RESS-001
- gave numbers to parts that had none: 2
- renumbered D7 to D3, J7 to J3, TP15 to TP3, TP16 to TP4, TP17 to TP5, U15 to U1

Commit message: Added ressistor footprint
Parts:
- R7, R8, R9: footprint (none) -> Resistors_SMD:R_0603_HandSoldering
Changed lines of the file:
@@
 $Descr A4 11693 8268
 encoding utf-8
-Sheet 3 20
+Sheet 11 20
 Title "PWM Switching Circuit"
 Date "2017-05-13"
@@
 AR Path="/591E6415/591EA4FC/5917D576" Ref="J13"  Part="1"
 AR Path="/591E6415/591EA50E/5917D576" Ref="J14"  Part="1"
-F 0 "J14" H 6350 2600 50  0001 C CNN
+F 0 "J11" H 6350 2600 50  0001 C CNN
 F 1 "PWM" V 6450 2400 50  0000 C CNN
 F 2 "" H 6350 2400 50  0000 C CNN
@@
 AR Path="/591E6415/591EA4FC/5917D57C" Ref="U11"  Part="1"
 AR Path="/591E6415/591EA50E/5917D57C" Ref="U12"  Part="1"
-F 0 "U12" H 4500 3250 60  0000 C CNN
+F 0 "U9" H 4500 3250 60  0000 C CNN
 F 1 "NLAS4599" H 4550 2500 60  0000 C CNN
 F 2 "" H 4300 2350 60  0001 C CNN
@@
 AR Path="/591E6415/591EA4FC/591EF19A" Ref="D13"  Part="1"
 AR Path="/591E6415/591EA50E/591EF19A" Ref="D14"  Part="1"
-F 0 "D14" H 3550 3100 50  0000 C CNN
+F 0 "D11" H 3550 3100 50  0000 C CNN
 F 1 "LED" H 3550 2900 50  0000 C CNN
 F 2 "" H 3550 3000 50  0000 C CNN
@@
 AR Path="/591E6415/591EA4FC/591EF2D3" Ref="R38"  Part="1"
 AR Path="/591E6415/591EA50E/591EF2D3" Ref="R41"  Part="1"
-F 0 "R41" V 3630 2650 50  0000 C CNN
+F 0 "R32" V 3630 2650 50  0000 C CNN
 F 1 "100" V 3550 2650 50  0000 C CNN
-F 2 "" V 3480 2650 50  0000 C CNN
+F 2 "Resistors_SMD:R_0603_HandSoldering" V 3480 2650 50  0001 C CNN
 F 3 "" H 3550 2650 50  0000 C CNN
 F 4 "RESS-006" V 3550 2650 60  0001 C CNN "part_num"
@@
 AR Path="/591E6415/591EA4FC/591F0A89" Ref="R37"  Part="1"
 AR Path="/591E6415/591EA50E/591F0A89" Ref="R40"  Part="1"
-F 0 "R40" V 3230 2800 50  0000 C CNN
+F 0 "R31" V 3230 2800 50  0000 C CNN
 F 1 "10K" V 3150 2800 50  0000 C CNN
-F 2 "" V 3080 2800 50  0000 C CNN
+F 2 "Resistors_SMD:R_0603_HandSoldering" V 3080 2800 50  0001 C CNN
 F 3 "" H 3150 2800 50  0000 C CNN
 F 4 "RESS-005" V 3150 2800 60  0001 C CNN "part_num"
@@
 AR Path="/591E6415/591EA4FC/591F0BAE" Ref="R39"  Part="1"
 AR Path="/591E6415/591EA50E/591F0BAE" Ref="R42"  Part="1"
-F 0 "R42" V 3880 2450 50  0000 C CNN
+F 0 "R33" V 3880 2450 50  0000 C CNN
 F 1 "0" V 3800 2450 50  0000 C CNN
-F 2 "" V 3730 2450 50  0000 C CNN
+F 2 "Resistors_SMD:R_0603_HandSoldering" V 3730 2450 50  0001 C CNN
 F 3 "" H 3800 2450 50  0000 C CNN
 F 4 "RESS-001" V 3800 2450 60  0001 C CNN "part_num"
@@
 AR Path="/591E6415/591EA4FC/591F0CEF" Ref="TP35"  Part="1"
 AR Path="/591E6415/591EA50E/591F0CEF" Ref="TP38"  Part="1"
-F 0 "TP38" H 4000 2900 50  0000 C BNN
+F 0 "TP29" H 4000 2900 50  0000 C BNN
 F 1 "TEST" H 4000 2850 50  0000 C CNN
 F 2 "" H 4000 2600 50  0000 C CNN
@@
 AR Path="/591E6415/591EA4FC/592CAEE3" Ref="TP34"  Part="1"
 AR Path="/591E6415/591EA50E/592CAEE3" Ref="TP37"  Part="1"
-F 0 "TP37" H 3900 2350 50  0000 C BNN
+F 0 "TP28" H 3900 2350 50  0000 C BNN
 F 1 "TEST" H 3900 2300 50  0000 C CNN
 F 2 "" H 3900 2050 50  0000 C CNN
@@
 AR Path="/591E6415/591EA4FC/592CAF2C" Ref="TP33"  Part="1"
 AR Path="/591E6415/591EA50E/592CAF2C" Ref="TP36"  Part="1"
-F 0 "TP36" H 3700 2350 50  0000 C BNN
+F 0 "TP27" H 3700 2350 50  0000 C BNN
 F 1 "TEST" H 3700 2300 50  0000 C CNN
 F 2 "" H 3700 2050 50  0000 C CNN
@@
 AR Path="/591E6415/591EA4FC/594E7E73" Ref="#PWR027"  Part="1"
 AR Path="/591E6415/591EA50E/594E7E73" Ref="#PWR029"  Part="1"
-F 0 "#PWR029" H 5100 2450 50  0001 C CNN
+F 0 "#PWR023" H 5100 2450 50  0001 C CNN
 F 1 "GND" H 5100 2550 50  0000 C CNN
 F 2 "" H 5100 2700 50  0001 C CNN
@@
 AR Path="/591E6415/591EA4FC/594EDAD2" Ref="#PWR028"  Part="1"
 AR Path="/591E6415/591EA50E/594EDAD2" Ref="#PWR030"  Part="1"
-F 0 "#PWR030" H 3350 3000 50  0001 C CNN
+F 0 "#PWR024" H 3350 3000 50  0001 C CNN
 F 1 "GND" H 3350 3100 50  0000 C CNN
 F 2 "" H 3350 3250 50  0001 C CNN
@@
 AR Path="/591E6415/591EA4FC/5957A292" Ref="SH21"  Part="1"
 AR Path="/591E6415/591EA50E/5957A292" Ref="SH23"  Part="1"
-F 0 "SH23" H 3100 2300 60  0000 C CNN
+F 0 "SH17" H 3100 2300 60  0000 C CNN
 F 1 "SHORT" H 3100 2050 60  0000 C CNN
 F 2 "" H 3100 2150 60  0001 C CNN
@@
 AR Path="/591E6415/591EA4FC/5957A2B7" Ref="SH22"  Part="1"
 AR Path="/591E6415/591EA50E/5957A2B7" Ref="SH24"  Part="1"
-F 0 "SH24" H 3350 2400 60  0000 C CNN
+F 0 "SH18" H 3350 2400 60  0000 C CNN
 F 1 "SHORT" H 3350 2150 60  0000 C CNN
 F 2 "" H 3350 2250 60  0001 C CNN

Commit message: PCB?!
Added initial PCB file with ratsnest. footprint library still needs to
be setup.
Parts:
- removed SH1, SH2: SHORT, symbol SHORT
- added R7, R9: 0, Resistors_SMD:R_0603_HandSoldering, symbol R
- D3: footprint (none) -> LEDs:LED_0603
- J3: footprint (none) -> Pin_Headers:Pin_Header_Straight_1x03_Pitch2.54mm
- TP3, TP4, TP5: footprint (none) -> Measurement_Points:Measurement_Point_Round-SMD-Pad_Big
- U1: footprint (none) -> TO_SOT_Packages_SMD:SOT-363_SC-70-6_Handsoldering
- renumbered R8 to R10, R9 to R11, R7 to R8

Commit message: Fixed serge suggestions
Parts:
- removed R11, R7, R9: 0, Resistors_SMD:R_0603_HandSoldering, symbol R
Connections:
- wire segments 25 -> 22
Changed lines of the file:
@@
 $Descr A4 11693 8268
 encoding utf-8
-Sheet 12 20
+Sheet 3 21
 Title "PWM Switching Circuit"
 Date "2017-05-13"
@@
 OC
 Wire Wire Line
-	2750 2150 3000 2150
-Wire Wire Line
-	2750 2250 3200 2250
-Wire Wire Line
-	2750 2450 3650 2450
+	2750 2150 4100 2150
+Wire Wire Line
+	2750 2250 4100 2250
+Wire Wire Line
+	2750 2450 4100 2450
 Wire Wire Line
 	4900 2200 4900 2300
@@
 	3150 2650 3150 2450
 Connection ~ 3150 2450
-$Comp
-L R R11
-U 1 1 591F0BAE
-P 3800 2450
-AR Path="/591E6415/591EA448/591F0BAE" Ref="R11"  Part="1"
-AR Path="/591E6415/591EA45A/591F0BAE" Ref="R16"  Part="1"
-AR Path="/591E6415/591EA46C/591F0BAE" Ref="R21"  Part="1"
-AR Path="/591E6415/591EA47E/591F0BAE" Ref="R26"  Part="1"
-AR Path="/591E6415/591EA490/591F0BAE" Ref="R31"  Part="1"
-AR Path="/591E6415/591EA4A2/591F0BAE" Ref="R36"  Part="1"
-AR Path="/591E6415/591EA4B4/591F0BAE" Ref="R41"  Part="1"
-AR Path="/591E6415/591EA4C6/591F0BAE" Ref="R46"  Part="1"
-AR Path="/591E6415/591EA4D8/591F0BAE" Ref="R51"  Part="1"
-AR Path="/591E6415/591EA4EA/591F0BAE" Ref="R56"  Part="1"
-AR Path="/591E6415/591EA4FC/591F0BAE" Ref="R61"  Part="1"
-AR Path="/591E6415/591EA50E/591F0BAE" Ref="R66"  Part="1"
-F 0 "R66" V 3880 2450 50  0000 C CNN
-F 1 "0" V 3800 2450 50  0000 C CNN
-F 2 "Resistors_SMD:R_0603_HandSoldering" V 3730 2450 50  0001 C CNN
-F 3 "" H 3800 2450 50  0000 C CNN
-F 4 "RESS-001" V 3800 2450 60  0001 C CNN "part_num"
-	1    3800 2450
-	0    1    1    0
-$EndComp
-Wire Wire Line
-	3950 2450 4100 2450
 Connection ~ 4000 2450
 $Comp
@@
 $EndComp
 Wire Wire Line
-	3300 2150 4100 2150
-Wire Wire Line
-	3500 2250 4100 2250
-Wire Wire Line
 	3700 2050 3700 2150
 Connection ~ 3700 2150
@@
 Connection ~ 3900 2250
 $Comp
-L GND #PWR7
+L GND #PWR04
 U 1 1 594E7E73
 P 5100 2700
-AR Path="/591E6415/591EA448/594E7E73" Ref="#PWR7"  Part="1"
-AR Path="/591E6415/591EA45A/594E7E73" Ref="#PWR9"  Part="1"
-AR Path="/591E6415/591EA46C/594E7E73" Ref="#PWR11"  Part="1"
-AR Path="/591E6415/591EA47E/594E7E73" Ref="#PWR13"  Part="1"
-AR Path="/591E6415/591EA490/594E7E73" Ref="#PWR15"  Part="1"
-AR Path="/591E6415/591EA4A2/594E7E73" Ref="#PWR17"  Part="1"
-AR Path="/591E6415/591EA4B4/594E7E73" Ref="#PWR19"  Part="1"
-AR Path="/591E6415/591EA4C6/594E7E73" Ref="#PWR21"  Part="1"
-AR Path="/591E6415/591EA4D8/594E7E73" Ref="#PWR23"  Part="1"
-AR Path="/591E6415/591EA4EA/594E7E73" Ref="#PWR25"  Part="1"
-AR Path="/591E6415/591EA4FC/594E7E73" Ref="#PWR27"  Part="1"
-AR Path="/591E6415/591EA50E/594E7E73" Ref="#PWR29"  Part="1"
-F 0 "#PWR29" H 5100 2450 50  0001 C CNN
+AR Path="/591E6415/591EA448/594E7E73" Ref="#PWR04"  Part="1"
+AR Path="/591E6415/591EA45A/594E7E73" Ref="#PWR06"  Part="1"
+AR Path="/591E6415/591EA46C/594E7E73" Ref="#PWR08"  Part="1"
+AR Path="/591E6415/591EA47E/594E7E73" Ref="#PWR010"  Part="1"
+AR Path="/591E6415/591EA490/594E7E73" Ref="#PWR012"  Part="1"
+AR Path="/591E6415/591EA4A2/594E7E73" Ref="#PWR014"  Part="1"
+AR Path="/591E6415/591EA4B4/594E7E73" Ref="#PWR016"  Part="1"
+AR Path="/591E6415/591EA4C6/594E7E73" Ref="#PWR018"  Part="1"
+AR Path="/591E6415/591EA4D8/594E7E73" Ref="#PWR020"  Part="1"
+AR Path="/591E6415/591EA4EA/594E7E73" Ref="#PWR022"  Part="1"
+AR Path="/591E6415/591EA4FC/594E7E73" Ref="#PWR024"  Part="1"
+AR Path="/591E6415/591EA50E/594E7E73" Ref="#PWR026"  Part="1"
+F 0 "#PWR026" H 5100 2450 50  0001 C CNN
 F 1 "GND" H 5100 2550 50  0000 C CNN
 F 2 "" H 5100 2700 50  0001 C CNN
@@
 $EndComp
 $Comp
-L GND #PWR6
+L GND #PWR05
 U 1 1 594EDAD2
 P 3350 3250
-AR Path="/591E6415/591EA448/594EDAD2" Ref="#PWR6"  Part="1"
-AR Path="/591E6415/591EA45A/594EDAD2" Ref="#PWR8"  Part="1"
-AR Path="/591E6415/591EA46C/594EDAD2" Ref="#PWR10"  Part="1"
-AR Path="/591E6415/591EA47E/594EDAD2" Ref="#PWR12"  Part="1"
-AR Path="/591E6415/591EA490/594EDAD2" Ref="#PWR14"  Part="1"
-AR Path="/591E6415/591EA4A2/594EDAD2" Ref="#PWR16"  Part="1"
-AR Path="/591E6415/591EA4B4/594EDAD2" Ref="#PWR18"  Part="1"
-AR Path="/591E6415/591EA4C6/594EDAD2" Ref="#PWR20"  Part="1"
-AR Path="/591E6415/591EA4D8/594EDAD2" Ref="#PWR22"  Part="1"
-AR Path="/591E6415/591EA4EA/594EDAD2" Ref="#PWR24"  Part="1"
-AR Path="/591E6415/591EA4FC/594EDAD2" Ref="#PWR26"  Part="1"
-AR Path="/591E6415/591EA50E/594EDAD2" Ref="#PWR28"  Part="1"
-F 0 "#PWR28" H 3350 3000 50  0001 C CNN
+AR Path="/591E6415/591EA448/594EDAD2" Ref="#PWR05"  Part="1"
+AR Path="/591E6415/591EA45A/594EDAD2" Ref="#PWR07"  Part="1"
+AR Path="/591E6415/591EA46C/594EDAD2" Ref="#PWR09"  Part="1"
+AR Path="/591E6415/591EA47E/594EDAD2" Ref="#PWR011"  Part="1"
+AR Path="/591E6415/591EA490/594EDAD2" Ref="#PWR013"  Part="1"
+AR Path="/591E6415/591EA4A2/594EDAD2" Ref="#PWR015"  Part="1"
+AR Path="/591E6415/591EA4B4/594EDAD2" Ref="#PWR017"  Part="1"
+AR Path="/591E6415/591EA4C6/594EDAD2" Ref="#PWR019"  Part="1"
+AR Path="/591E6415/591EA4D8/594EDAD2" Ref="#PWR021"  Part="1"
+AR Path="/591E6415/591EA4EA/594EDAD2" Ref="#PWR023"  Part="1"
+AR Path="/591E6415/591EA4FC/594EDAD2" Ref="#PWR025"  Part="1"
+AR Path="/591E6415/591EA50E/594EDAD2" Ref="#PWR027"  Part="1"
+F 0 "#PWR027" H 3350 3000 50  0001 C CNN
 F 1 "GND" H 3350 3100 50  0000 C CNN
 F 2 "" H 3350 3250 50  0001 C CNN
@@
 	3350 3250 3350 3200
 $Comp
-L R R9
-U 1 1 595EF0C9
-P 3350 2250
-AR Path="/591E6415/591EA448/595EF0C9" Ref="R9"  Part="1"
-AR Path="/591E6415/591EA45A/595EF0C9" Ref="R14"  Part="1"
-AR Path="/591E6415/591EA46C/595EF0C9" Ref="R19"  Part="1"
-AR Path="/591E6415/591EA47E/595EF0C9" Ref="R24"  Part="1"
-AR Path="/591E6415/591EA490/595EF0C9" Ref="R29"  Part="1"
-AR Path="/591E6415/591EA4A2/595EF0C9" Ref="R34"  Part="1"
-AR Path="/591E6415/591EA4B4/595EF0C9" Ref="R39"  Part="1"
-AR Path="/591E6415/591EA4C6/595EF0C9" Ref="R44"  Part="1"
-AR Path="/591E6415/591EA4D8/595EF0C9" Ref="R49"  Part="1"
-AR Path="/591E6415/591EA4EA/595EF0C9" Ref="R54"  Part="1"
-AR Path="/591E6415/591EA4FC/595EF0C9" Ref="R59"  Part="1"
-AR Path="/591E6415/591EA50E/595EF0C9" Ref="R64"  Part="1"
-F 0 "R64" V 3430 2250 50  0000 C CNN
-F 1 "0" V 3350 2250 50  0000 C CNN
-F 2 "Resistors_SMD:R_0603_HandSoldering" V 3280 2250 50  0001 C CNN
-F 3 "" H 3350 2250 50  0000 C CNN
-F 4 "RESS-001" V 3350 2250 60  0001 C CNN "part_num"
-	1    3350 2250
-	0    1    1    0
-$EndComp
-$Comp
-L R R7
-U 1 1 595EF0F1
-P 3150 2150
-AR Path="/591E6415/591EA448/595EF0F1" Ref="R7"  Part="1"
-AR Path="/591E6415/591EA45A/595EF0F1" Ref="R12"  Part="1"
-AR Path="/591E6415/591EA46C/595EF0F1" Ref="R17"  Part="1"
-AR Path="/591E6415/591EA47E/595EF0F1" Ref="R22"  Part="1"
-AR Path="/591E6415/591EA490/595EF0F1" Ref="R27"  Part="1"
-AR Path="/591E6415/591EA4A2/595EF0F1" Ref="R32"  Part="1"
-AR Path="/591E6415/591EA4B4/595EF0F1" Ref="R37"  Part="1"
-AR Path="/591E6415/591EA4C6/595EF0F1" Ref="R42"  Part="1"
-AR Path="/591E6415/591EA4D8/595EF0F1" Ref="R47"  Part="1"
-AR Path="/591E6415/591EA4EA/595EF0F1" Ref="R52"  Part="1"
-AR Path="/591E6415/591EA4FC/595EF0F1" Ref="R57"  Part="1"
-AR Path="/591E6415/591EA50E/595EF0F1" Ref="R62"  Part="1"
-F 0 "R62" V 3230 2150 50  0000 C CNN
-F 1 "0" V 3150 2150 50  0000 C CNN
-F 2 "Resistors_SMD:R_0603_HandSoldering" V 3080 2150 50  0001 C CNN
-F 3 "" H 3150 2150 50  0000 C CNN
-F 4 "RESS-001" V 3150 2150 60  0001 C CNN "part_num"
-	1    3150 2150
-	0    1    1    0
-$EndComp
-$Comp
 L NLAS4599 U1

Commit message: commit before my computer restarts
Parts:
- removed D3: LED, LEDs:LED_0603, symbol LED
- removed R10: 100, Resistors_SMD:R_0603_HandSoldering, symbol R
- renumbered J3 to J2, R8 to R1
Connections:
- wire segments 22 -> 17
Changed lines of the file:
@@
 $EndDescr
 $Comp
-L CONN_01X03 J3
+L CONN_01X03 J2
 U 1 1 5917D576
 P 6350 2400
-AR Path="/591E6415/591EA448/5917D576" Ref="J3"  Part="1"
-AR Path="/591E6415/591EA45A/5917D576" Ref="J4"  Part="1"
-AR Path="/591E6415/591EA46C/5917D576" Ref="J5"  Part="1"
-AR Path="/591E6415/591EA47E/5917D576" Ref="J6"  Part="1"
-AR Path="/591E6415/591EA490/5917D576" Ref="J7"  Part="1"
-AR Path="/591E6415/591EA4A2/5917D576" Ref="J8"  Part="1"
-AR Path="/591E6415/591EA4B4/5917D576" Ref="J9"  Part="1"
-AR Path="/591E6415/591EA4C6/5917D576" Ref="J10"  Part="1"
-AR Path="/591E6415/591EA4D8/5917D576" Ref="J11"  Part="1"
-AR Path="/591E6415/591EA4EA/5917D576" Ref="J12"  Part="1"
-AR Path="/591E6415/591EA4FC/5917D576" Ref="J13"  Part="1"
-AR Path="/591E6415/591EA50E/5917D576" Ref="J14"  Part="1"
-F 0 "J14" H 6350 2600 50  0001 C CNN
+AR Path="/591E6415/591EA448/5917D576" Ref="J2"  Part="1"
+AR Path="/591E6415/591EA45A/5917D576" Ref="J3"  Part="1"
+AR Path="/591E6415/591EA46C/5917D576" Ref="J4"  Part="1"
+AR Path="/591E6415/591EA47E/5917D576" Ref="J5"  Part="1"
+AR Path="/591E6415/591EA490/5917D576" Ref="J6"  Part="1"
+AR Path="/591E6415/591EA4A2/5917D576" Ref="J7"  Part="1"
+AR Path="/591E6415/591EA4B4/5917D576" Ref="J8"  Part="1"
+AR Path="/591E6415/591EA4C6/5917D576" Ref="J9"  Part="1"
+AR Path="/591E6415/591EA4D8/5917D576" Ref="J10"  Part="1"
+AR Path="/591E6415/591EA4EA/5917D576" Ref="J11"  Part="1"
+AR Path="/591E6415/591EA4FC/5917D576" Ref="J12"  Part="1"
+AR Path="/591E6415/591EA50E/5917D576" Ref="J13"  Part="1"
+F 0 "J4" H 6350 2600 50  0001 C CNN
 F 1 "PWM" V 6450 2400 50  0000 C CNN
 F 2 "Pin_Headers:Pin_Header_Straight_1x03_Pitch2.54mm" H 6350 2400 50  0001 C CNN
@@
 	4900 2300 6150 2300
 $Comp
-L LED D3
-U 1 1 591EF19A
-P 3550 3000
-AR Path="/591E6415/591EA448/591EF19A" Ref="D3"  Part="1"
-AR Path="/591E6415/591EA45A/591EF19A" Ref="D4"  Part="1"
-AR Path="/591E6415/591EA46C/591EF19A" Ref="D5"  Part="1"
-AR Path="/591E6415/591EA47E/591EF19A" Ref="D6"  Part="1"
-AR Path="/591E6415/591EA490/591EF19A" Ref="D7"  Part="1"
-AR Path="/591E6415/591EA4A2/591EF19A" Ref="D8"  Part="1"
-AR Path="/591E6415/591EA4B4/591EF19A" Ref="D9"  Part="1"
-AR Path="/591E6415/591EA4C6/591EF19A" Ref="D10"  Part="1"
-AR Path="/591E6415/591EA4D8/591EF19A" Ref="D11"  Part="1"
-AR Path="/591E6415/591EA4EA/591EF19A" Ref="D12"  Part="1"
-AR Path="/591E6415/591EA4FC/591EF19A" Ref="D13"  Part="1"
-AR Path="/591E6415/591EA50E/591EF19A" Ref="D14"  Part="1"
-F 0 "D14" H 3550 3100 50  0000 C CNN
-F 1 "LED" H 3550 2900 50  0000 C CNN
-F 2 "LEDs:LED_0603" H 3550 3000 50  0001 C CNN
-F 3 "" H 3550 3000 50  0000 C CNN
-F 4 "DIOD-002" H 3550 3000 60  0001 C CNN "part_num"
-	1    3550 3000
-	0    -1   -1   0
-$EndComp
-$Comp
-L R R10
-U 1 1 591EF2D3
-P 3550 2650
-AR Path="/591E6415/591EA448/591EF2D3" Ref="R10"  Part="1"
-AR Path="/591E6415/591EA45A/591EF2D3" Ref="R15"  Part="1"
-AR Path="/591E6415/591EA46C/591EF2D3" Ref="R20"  Part="1"
-AR Path="/591E6415/591EA47E/591EF2D3" Ref="R25"  Part="1"
-AR Path="/591E6415/591EA490/591EF2D3" Ref="R30"  Part="1"
-AR Path="/591E6415/591EA4A2/591EF2D3" Ref="R35"  Part="1"
-AR Path="/591E6415/591EA4B4/591EF2D3" Ref="R40"  Part="1"
-AR Path="/591E6415/591EA4C6/591EF2D3" Ref="R45"  Part="1"
-AR Path="/591E6415/591EA4D8/591EF2D3" Ref="R50"  Part="1"
-AR Path="/591E6415/591EA4EA/591EF2D3" Ref="R55"  Part="1"
-AR Path="/591E6415/591EA4FC/591EF2D3" Ref="R60"  Part="1"
-AR Path="/591E6415/591EA50E/591EF2D3" Ref="R65"  Part="1"
-F 0 "R65" V 3630 2650 50  0000 C CNN
-F 1 "100" V 3550 2650 50  0000 C CNN
-F 2 "Resistors_SMD:R_0603_HandSoldering" V 3480 2650 50  0001 C CNN
-F 3 "" H 3550 2650 50  0000 C CNN
-F 4 "RESS-006" V 3550 2650 60  0001 C CNN "part_num"
-	1    3550 2650
-	1    0    0    -1
-$EndComp
-Wire Wire Line
-	3550 2800 3550 2850
-Wire Wire Line
-	3550 2450 3550 2500
-Connection ~ 3550 2450
-Wire Wire Line
-	3550 3200 3550 3150
-$Comp
-L R R8
+L R R1
 U 1 1 591F0A89
 P 3150 2800
-AR Path="/591E6415/591EA448/591F0A89" Ref="R8"  Part="1"
-AR Path="/591E6415/591EA45A/591F0A89" Ref="R13"  Part="1"
-AR Path="/591E6415/591EA46C/591F0A89" Ref="R18"  Part="1"
-AR Path="/591E6415/591EA47E/591F0A89" Ref="R23"  Part="1"
-AR Path="/591E6415/591EA490/591F0A89" Ref="R28"  Part="1"
-AR Path="/591E6415/591EA4A2/591F0A89" Ref="R33"  Part="1"
-AR Path="/591E6415/591EA4B4/591F0A89" Ref="R38"  Part="1"
-AR Path="/591E6415/591EA4C6/591F0A89" Ref="R43"  Part="1"
-AR Path="/591E6415/591EA4D8/591F0A89" Ref="R48"  Part="1"
-AR Path="/591E6415/591EA4EA/591F0A89" Ref="R53"  Part="1"
-AR Path="/591E6415/591EA4FC/591F0A89" Ref="R58"  Part="1"
-AR Path="/591E6415/591EA50E/591F0A89" Ref="R63"  Part="1"
-F 0 "R63" V 3230 2800 50  0000 C CNN
+AR Path="/591E6415/591EA448/591F0A89" Ref="R1"  Part="1"
+AR Path="/591E6415/591EA45A/591F0A89" Ref="R3"  Part="1"
+AR Path="/591E6415/591EA46C/591F0A89" Ref="R5"  Part="1"
+AR Path="/591E6415/591EA47E/591F0A89" Ref="R7"  Part="1"
+AR Path="/591E6415/591EA490/591F0A89" Ref="R9"  Part="1"
+AR Path="/591E6415/591EA4A2/591F0A89" Ref="R11"  Part="1"
+AR Path="/591E6415/591EA4B4/591F0A89" Ref="R13"  Part="1"
+AR Path="/591E6415/591EA4C6/591F0A89" Ref="R15"  Part="1"
+AR Path="/591E6415/591EA4D8/591F0A89" Ref="R17"  Part="1"
+AR Path="/591E6415/591EA4EA/591F0A89" Ref="R19"  Part="1"
+AR Path="/591E6415/591EA4FC/591F0A89" Ref="R21"  Part="1"
+AR Path="/591E6415/591EA50E/591F0A89" Ref="R23"  Part="1"
+F 0 "R5" V 3230 2800 50  0000 C CNN
 F 1 "10K" V 3150 2800 50  0000 C CNN
 F 2 "Resistors_SMD:R_0603_HandSoldering" V 3080 2800 50  0001 C CNN
@@
 	1    0    0    -1
 $EndComp
-Wire Wire Line
-	3150 3200 3550 3200
-Wire Wire Line
-	3150 2950 3150 3200
 Wire Wire Line
 	3150 2650 3150 2450
@@
 AR Path="/591E6415/591EA4FC/591F0CEF" Ref="TP35"  Part="1"
 AR Path="/591E6415/591EA50E/591F0CEF" Ref="TP38"  Part="1"
-F 0 "TP38" H 4000 2900 50  0000 C BNN
+F 0 "TP11" H 4000 2900 50  0000 C BNN
 F 1 "TEST" H 4000 2850 50  0000 C CNN
 F 2 "Measurement_Points:Measurement_Point_Round-SMD-Pad_Big" H 4000 2600 50  0001 C CNN
@@
 Wire Wire Line
 	5100 2400 5100 1950
-Connection ~ 3350 3200
 Wire Wire Line
 	5100 2400 4900 2400
@@
 AR Path="/591E6415/591EA4FC/592CAEE3" Ref="TP34"  Part="1"
 AR Path="/591E6415/591EA50E/592CAEE3" Ref="TP37"  Part="1"
-F 0 "TP37" H 3900 2350 50  0000 C BNN
+F 0 "TP10" H 3900 2350 50  0000 C BNN
 F 1 "TEST" H 3900 2300 50  0000 C CNN
 F 2 "Measurement_Points:Measurement_Point_Round-SMD-Pad_Big" H 3900 2050 50  0001 C CNN
@@
 AR Path="/591E6415/591EA4FC/592CAF2C" Ref="TP33"  Part="1"
 AR Path="/591E6415/591EA50E/592CAF2C" Ref="TP36"  Part="1"
-F 0 "TP36" H 3700 2350 50  0000 C BNN
+F 0 "TP9" H 3700 2350 50  0000 C BNN
 F 1 "TEST" H 3700 2300 50  0000 C CNN
 F 2 "Measurement_Points:Measurement_Point_Round-SMD-Pad_Big" H 3700 2050 50  0001 C CNN
@@
 L GND #PWR05
 U 1 1 594EDAD2
-P 3350 3250
+P 3150 3000
 AR Path="/591E6415/591EA448/594EDAD2" Ref="#PWR05"  Part="1"
 AR Path="/591E6415/591EA45A/594EDAD2" Ref="#PWR07"  Part="1"
@@
 AR Path="/591E6415/591EA4FC/594EDAD2" Ref="#PWR025"  Part="1"
 AR Path="/591E6415/591EA50E/594EDAD2" Ref="#PWR027"  Part="1"
-F 0 "#PWR027" H 3350 3000 50  0001 C CNN
-F 1 "GND" H 3350 3100 50  0000 C CNN
-F 2 "" H 3350 3250 50  0001 C CNN
-F 3 "" H 3350 3250 50  0001 C CNN
-	1    3350 3250
-	1    0    0    -1
-$EndComp
-Wire Wire Line
-	3350 3250 3350 3200
+F 0 "#PWR027" H 3150 2750 50  0001 C CNN
+F 1 "GND" H 3150 2850 50  0000 C CNN
+F 2 "" H 3150 3000 50  0001 C CNN
+F 3 "" H 3150 3000 50  0001 C CNN
+	1    3150 3000
+	1    0    0    -1
+$EndComp
+Wire Wire Line
+	3150 3000 3150 2950
 $Comp
 L NLAS4599 U1
@@
 AR Path="/591E6415/591EA4FC/595F3F52" Ref="U11"  Part="1"
 AR Path="/591E6415/591EA50E/595F3F52" Ref="U12"  Part="1"
-F 0 "U12" H 4500 3250 60  0000 C CNN
+F 0 "U3" H 4500 3250 60  0000 C CNN
 F 1 "NLAS4599" H 4550 2500 60  0000 C CNN
 F 2 "TO_SOT_Packages_SMD:SOT-363_SC-70-6_Handsoldering" H 4300 2350 60  0001 C CNN
