File: Hardware/PWM.sch (KiCad schematic (older format))
At the start: 6 parts, among them J2 PWM, U1 NLAS4599

Commit message: routed PWM and SEL bus
Parts:
- TP3, TP4, TP5: footprint Measurement_Points:Measurement_Point_Round-SMD-Pad_Big -> Measurement_Points:Measurement_Point_Round-SMD-Pad_Small
Changed lines of the file:
@@
 AR Path="/591E6415/591EA4FC/5917D576" Ref="J12"  Part="1"
 AR Path="/591E6415/591EA50E/5917D576" Ref="J13"  Part="1"
-F 0 "J4" H 6350 2600 50  0001 C CNN
+F 0 "J2" H 6350 2600 50  0001 C CNN
 F 1 "PWM" V 6450 2400 50  0000 C CNN
 F 2 "Pin_Headers:Pin_Header_Straight_1x03_Pitch2.54mm" H 6350 2400 50  0001 C CNN
@@
 AR Path="/591E6415/591EA4FC/591F0A89" Ref="R21"  Part="1"
 AR Path="/591E6415/591EA50E/591F0A89" Ref="R23"  Part="1"
-F 0 "R5" V 3230 2800 50  0000 C CNN
+F 0 "R1" V 3230 2800 50  0000 C CNN
 F 1 "10K" V 3150 2800 50  0000 C CNN
 F 2 "Resistors_SMD:R_0603_HandSoldering" V 3080 2800 50  0001 C CNN
@@
 AR Path="/591E6415/591EA4FC/591F0CEF" Ref="TP35"  Part="1"
 AR Path="/591E6415/591EA50E/591F0CEF" Ref="TP38"  Part="1"
-F 0 "TP11" H 4000 2900 50  0000 C BNN
+F 0 "TP5" H 4000 2900 50  0000 C BNN
 F 1 "TEST" H 4000 2850 50  0000 C CNN
-F 2 "Measurement_Points:Measurement_Point_Round-SMD-Pad_Big" H 4000 2600 50  0001 C CNN
+F 2 "Measurement_Points:Measurement_Point_Round-SMD-Pad_Small" H 4000 2600 50  0001 C CNN
 F 3 "" H 4000 2600 50  0000 C CNN
 	1    4000 2600
@@
 AR Path="/591E6415/591EA4FC/592CAEE3" Ref="TP34"  Part="1"
 AR Path="/591E6415/591EA50E/592CAEE3" Ref="TP37"  Part="1"
-F 0 "TP10" H 3900 2350 50  0000 C BNN
+F 0 "TP4" H 3900 2350 50  0000 C BNN
 F 1 "TEST" H 3900 2300 50  0000 C CNN
-F 2 "Measurement_Points:Measurement_Point_Round-SMD-Pad_Big" H 3900 2050 50  0001 C CNN
+F 2 "Measurement_Points:Measurement_Point_Round-SMD-Pad_Small" H 3900 2050 50  0001 C CNN
 F 3 "" H 3900 2050 50  0000 C CNN
 	1    3900 2050
@@
 AR Path="/591E6415/591EA4FC/592CAF2C" Ref="TP33"  Part="1"
 AR Path="/591E6415/591EA50E/592CAF2C" Ref="TP36"  Part="1"
-F 0 "TP9" H 3700 2350 50  0000 C BNN
+F 0 "TP3" H 3700 2350 50  0000 C BNN
 F 1 "TEST" H 3700 2300 50  0000 C CNN
-F 2 "Measurement_Points:Measurement_Point_Round-SMD-Pad_Big" H 3700 2050 50  0001 C CNN
+F 2 "Measurement_Points:Measurement_Point_Round-SMD-Pad_Small" H 3700 2050 50  0001 C CNN
 F 3 "" H 3700 2050 50  0000 C CNN
 	1    3700 2050
@@
 AR Path="/591E6415/591EA4FC/594E7E73" Ref="#PWR024"  Part="1"
 AR Path="/591E6415/591EA50E/594E7E73" Ref="#PWR026"  Part="1"
-F 0 "#PWR026" H 5100 2450 50  0001 C CNN
+F 0 "#PWR04" H 5100 2450 50  0001 C CNN
 F 1 "GND" H 5100 2550 50  0000 C CNN
 F 2 "" H 5100 2700 50  0001 C CNN
@@
 AR Path="/591E6415/591EA4FC/594EDAD2" Ref="#PWR025"  Part="1"
 AR Path="/591E6415/591EA50E/594EDAD2" Ref="#PWR027"  Part="1"
-F 0 "#PWR027" H 3150 2750 50  0001 C CNN
+F 0 "#PWR05" H 3150 2750 50  0001 C CNN
 F 1 "GND" H 3150 2850 50  0000 C CNN
 F 2 "" H 3150 3000 50  0001 C CNN
@@
 AR Path="/591E6415/591EA4FC/595F3F52" Ref="U11"  Part="1"
 AR Path="/591E6415/591EA50E/595F3F52" Ref="U12"  Part="1"
-F 0 "U3" H 4500 3250 60  0000 C CNN
+F 0 "U1" H 4500 3250 60  0000 C CNN
 F 1 "NLAS4599" H 4550 2500 60  0000 C CNN
 F 2 "TO_SOT_Packages_SMD:SOT-363_SC-70-6_Handsoldering" H 4300 2350 60  0001 C CNN

Commit message: finished safety controller routing
Changed lines of the file:
@@
 $Descr A4 11693 8268
 encoding utf-8
-Sheet 3 21
+Sheet 5 21
 Title "PWM Switching Circuit"
 Date "2017-05-13"
@@
 AR Path="/591E6415/591EA4FC/5917D576" Ref="J12"  Part="1"
 AR Path="/591E6415/591EA50E/5917D576" Ref="J13"  Part="1"
-F 0 "J2" H 6350 2600 50  0001 C CNN
+F 0 "J13" H 6350 2600 50  0001 C CNN
 F 1 "PWM" V 6450 2400 50  0000 C CNN
 F 2 "Pin_Headers:Pin_Header_Straight_1x03_Pitch2.54mm" H 6350 2400 50  0001 C CNN
@@
 AR Path="/591E6415/591EA4FC/591F0A89" Ref="R21"  Part="1"
 AR Path="/591E6415/591EA50E/591F0A89" Ref="R23"  Part="1"
-F 0 "R1" V 3230 2800 50  0000 C CNN
+F 0 "R23" V 3230 2800 50  0000 C CNN
 F 1 "10K" V 3150 2800 50  0000 C CNN
 F 2 "Resistors_SMD:R_0603_HandSoldering" V 3080 2800 50  0001 C CNN
@@
 AR Path="/591E6415/591EA4FC/591F0CEF" Ref="TP35"  Part="1"
 AR Path="/591E6415/591EA50E/591F0CEF" Ref="TP38"  Part="1"
-F 0 "TP5" H 4000 2900 50  0000 C BNN
+F 0 "TP38" H 4000 2900 50  0000 C BNN
 F 1 "TEST" H 4000 2850 50  0000 C CNN
 F 2 "Measurement_Points:Measurement_Point_Round-SMD-Pad_Small" H 4000 2600 50  0001 C CNN
@@
 AR Path="/591E6415/591EA4FC/592CAEE3" Ref="TP34"  Part="1"
 AR Path="/591E6415/591EA50E/592CAEE3" Ref="TP37"  Part="1"
-F 0 "TP4" H 3900 2350 50  0000 C BNN
+F 0 "TP37" H 3900 2350 50  0000 C BNN
 F 1 "TEST" H 3900 2300 50  0000 C CNN
 F 2 "Measurement_Points:Measurement_Point_Round-SMD-Pad_Small" H 3900 2050 50  0001 C CNN
@@
 AR Path="/591E6415/591EA4FC/592CAF2C" Ref="TP33"  Part="1"
 AR Path="/591E6415/591EA50E/592CAF2C" Ref="TP36"  Part="1"
-F 0 "TP3" H 3700 2350 50  0000 C BNN
+F 0 "TP36" H 3700 2350 50  0000 C BNN
 F 1 "TEST" H 3700 2300 50  0000 C CNN
 F 2 "Measurement_Points:Measurement_Point_Round-SMD-Pad_Small" H 3700 2050 50  0001 C CNN
@@
 AR Path="/591E6415/591EA4FC/594E7E73" Ref="#PWR024"  Part="1"
 AR Path="/591E6415/591EA50E/594E7E73" Ref="#PWR026"  Part="1"
-F 0 "#PWR04" H 5100 2450 50  0001 C CNN
+F 0 "#PWR026" H 5100 2450 50  0001 C CNN
 F 1 "GND" H 5100 2550 50  0000 C CNN
 F 2 "" H 5100 2700 50  0001 C CNN
@@
 AR Path="/591E6415/591EA4FC/594EDAD2" Ref="#PWR025"  Part="1"
 AR Path="/591E6415/591EA50E/594EDAD2" Ref="#PWR027"  Part="1"
-F 0 "#PWR05" H 3150 2750 50  0001 C CNN
+F 0 "#PWR027" H 3150 2750 50  0001 C CNN
 F 1 "GND" H 3150 2850 50  0000 C CNN
 F 2 "" H 3150 3000 50  0001 C CNN
@@
 AR Path="/591E6415/591EA4FC/595F3F52" Ref="U11"  Part="1"
 AR Path="/591E6415/591EA50E/595F3F52" Ref="U12"  Part="1"
-F 0 "U1" H 4500 3250 60  0000 C CNN
+F 0 "U12" H 4500 3250 60  0000 C CNN
 F 1 "NLAS4599" H 4550 2500 60  0000 C CNN
 F 2 "TO_SOT_Packages_SMD:SOT-363_SC-70-6_Handsoldering" H 4300 2350 60  0001 C CNN
