File: Hardware/ZeroPilot.sch (KiCad schematic (older format))
At the start: 12 parts, among them J1 CONN_01X03, J2 CONN_01X04

Commit message: Added ressistor footprint
Parts:
- R1, R2, R3, R4, R5, R6: footprint (none) -> Resistors_SMD:R_0603_HandSoldering
Changed lines of the file:
@@
 F 0 "R5" V 11030 3550 50  0000 C CNN
 F 1 "10K" V 10950 3550 50  0000 C CNN
-F 2 "" V 10880 3550 50  0001 C CNN
+F 2 "Resistors_SMD:R_0603_HandSoldering" V 10880 3550 50  0001 C CNN
 F 3 "" H 10950 3550 50  0001 C CNN
 F 4 "RESS-005" V 10950 3550 60  0001 C CNN "part_num"
@@
 F 0 "R6" V 11030 3950 50  0000 C CNN
 F 1 "3k" V 10950 3950 50  0000 C CNN
-F 2 "" V 10880 3950 50  0001 C CNN
+F 2 "Resistors_SMD:R_0603_HandSoldering" V 10880 3950 50  0001 C CNN
 F 3 "" H 10950 3950 50  0001 C CNN
 F 4 "RESS-004" V 10950 3950 60  0001 C CNN "part_num"
@@
 F 0 "R3" V 10530 4100 50  0000 C CNN
 F 1 "100K" V 10450 4100 50  0000 C CNN
-F 2 "" V 10380 4100 50  0001 C CNN
+F 2 "Resistors_SMD:R_0603_HandSoldering" V 10380 4100 50  0001 C CNN
 F 3 "" H 10450 4100 50  0001 C CNN
 F 4 "RESS-003" V 10450 4100 60  0001 C CNN "part_num"
@@
 F 0 "R4" V 10530 4500 50  0000 C CNN
 F 1 "22K" V 10450 4500 50  0000 C CNN
-F 2 "" V 10380 4500 50  0001 C CNN
+F 2 "Resistors_SMD:R_0603_HandSoldering" V 10380 4500 50  0001 C CNN
 F 3 "" H 10450 4500 50  0001 C CNN
 F 4 "RESS-002" V 10450 4500 60  0001 C CNN "part_num"
@@
 F 0 "R1" V 4130 2000 50  0000 C CNN
 F 1 "0" V 4050 2000 50  0000 C CNN
-F 2 "" V 3980 2000 50  0001 C CNN
+F 2 "Resistors_SMD:R_0603_HandSoldering" V 3980 2000 50  0001 C CNN
 F 3 "" H 4050 2000 50  0001 C CNN
 F 4 "RESS-001" V 4050 2000 60  0001 C CNN "part_num"
@@
 F 0 "R2" V 4130 2100 50  0000 C CNN
 F 1 "0" V 4050 2100 50  0000 C CNN
-F 2 "" V 3980 2100 50  0001 C CNN
+F 2 "Resistors_SMD:R_0603_HandSoldering" V 3980 2100 50  0001 C CNN
 F 3 "" H 4050 2100 50  0001 C CNN
 F 4 "RESS-001" V 4050 2100 60  0001 C CNN "part_num"

Commit message: PCB?!
Added initial PCB file with ratsnest. footprint library still needs to
be setup.
Parts:
- D1, D2: footprint (none) -> Diodes_SMD:D_SOD-523
- J1: footprint (none) -> Pin_Headers:Pin_Header_Straight_1x03_Pitch2.54mm
- J2: footprint (none) -> Pin_Headers:Pin_Header_Straight_1x04_Pitch2.54mm
- TP1, TP2: footprint (none) -> Measurement_Points:Measurement_Point_Round-SMD-Pad_Big
Changed lines of the file:
@@
 $EndComp
 $Comp
-L GND #PWR01
+L GND #PWR5
 U 1 1 5921B8F8
 P 10950 4200
-F 0 "#PWR01" H 10950 3950 50  0001 C CNN
+F 0 "#PWR5" H 10950 3950 50  0001 C CNN
 F 1 "GND" H 10950 4050 50  0000 C CNN
 F 2 "" H 10950 4200 50  0001 C CNN
@@
 $EndComp
 $Comp
-L GND #PWR02
+L GND #PWR3
 U 1 1 59287255
 P 10450 4750
-F 0 "#PWR02" H 10450 4500 50  0001 C CNN
+F 0 "#PWR3" H 10450 4500 50  0001 C CNN
 F 1 "GND" H 10450 4600 50  0000 C CNN
 F 2 "" H 10450 4750 50  0001 C CNN
@@
 F 0 "TP1" H 2300 1600 50  0000 C BNN
 F 1 "TEST" H 2300 1550 50  0000 C CNN
-F 2 "" H 2300 1300 50  0001 C CNN
+F 2 "Measurement_Points:Measurement_Point_Round-SMD-Pad_Big" H 2300 1300 50  0001 C CNN
 F 3 "" H 2300 1300 50  0001 C CNN
 	1    2300 1300
@@
 F 0 "TP2" H 2450 1800 50  0000 C BNN
 F 1 "TEST" H 2450 1750 50  0000 C CNN
-F 2 "" H 2450 1500 50  0001 C CNN
+F 2 "Measurement_Points:Measurement_Point_Round-SMD-Pad_Big" H 2450 1500 50  0001 C CNN
 F 3 "" H 2450 1500 50  0001 C CNN
 	1    2450 1500
@@
 F 0 "J1" H 3450 2300 50  0000 C CNN
 F 1 "CONN_01X03" V 3550 2100 50  0000 C CNN
-F 2 "" H 3450 2100 50  0001 C CNN
+F 2 "Pin_Headers:Pin_Header_Straight_1x03_Pitch2.54mm" H 3450 2100 50  0001 C CNN
 F 3 "" H 3450 2100 50  0001 C CNN
 F 4 "CONN-007" H 3450 2100 60  0001 C CNN "part_num"
@@
 $EndComp
 $Comp
-L GND #PWR03
+L GND #PWR1
 U 1 1 592DF11B
 P 3750 2300
-F 0 "#PWR03" H 3750 2050 50  0001 C CNN
+F 0 "#PWR1" H 3750 2050 50  0001 C CNN
 F 1 "GND" H 3750 2150 50  0000 C CNN
 F 2 "" H 3750 2300 50  0001 C CNN
@@
 F 0 "D1" H 10000 3650 50  0000 C CNN
 F 1 "D" H 10000 3450 50  0000 C CNN
-F 2 "" H 10000 3550 50  0001 C CNN
+F 2 "Diodes_SMD:D_SOD-523" H 10000 3550 50  0001 C CNN
 F 3 "" H 10000 3550 50  0001 C CNN
 F 4 "DIOD-004" H 10000 3550 60  0001 C CNN "part_num"
@@
 F 0 "D2" H 10200 3650 50  0000 C CNN
 F 1 "D" H 10200 3450 50  0000 C CNN
-F 2 "" H 10200 3550 50  0001 C CNN
+F 2 "Diodes_SMD:D_SOD-523" H 10200 3550 50  0001 C CNN
 F 3 "" H 10200 3550 50  0001 C CNN
 F 4 "DIOD-004" H 10200 3550 60  0001 C CNN "part_num"
@@
 F 0 "J2" H 10450 3000 50  0000 C CNN
 F 1 "CONN_01X04" V 10550 2750 50  0000 C CNN
-F 2 "" H 10450 2750 50  0001 C CNN
+F 2 "Pin_Headers:Pin_Header_Straight_1x04_Pitch2.54mm" H 10450 2750 50  0001 C CNN
 F 3 "" H 10450 2750 50  0001 C CNN
 F 4 "CONN-008" H 10450 2750 60  0001 C CNN "part_num"
 	1    10450 2750
-	1    0    0    -1
+	1    0    0    1
 $EndComp
 Wire Wire Line
@@
 	9650 2800 10250 2800
 $Comp
-L GND #PWR04
+L GND #PWR2
 U 1 1 594DF6EB
 P 10150 3000
-F 0 "#PWR04" H 10150 2750 50  0001 C CNN
+F 0 "#PWR2" H 10150 2750 50  0001 C CNN
 F 1 "GND" H 10150 2850 50  0000 C CNN
 F 2 "" H 10150 3000 50  0001 C CNN
@@
 	10150 2900 10150 3000
 $Comp
-L GND #PWR05
+L GND #PWR4
 U 1 1 594F2D3B
 P 10450 6000
-F 0 "#PWR05" H 10450 5750 50  0001 C CNN
+F 0 "#PWR4" H 10450 5750 50  0001 C CNN
 F 1 "GND" H 10450 5850 50  0000 C CNN
 F 2 "" H 10450 6000 50  0001 C CNN
@@
 $EndComp
 $Comp
-L PWR_FLAG #FLG06
+L PWR_FLAG #FLG1
 U 1 1 594F3124
 P 10450 6000
-F 0 "#FLG06" H 10450 6075 50  0001 C CNN
+F 0 "#FLG1" H 10450 6075 50  0001 C CNN
 F 1 "PWR_FLAG" H 10450 6150 50  0000 C CNN
 F 2 "" H 10450 6000 50  0001 C CNN
