File: Hardware/STM32F0 RELAY.sch (KiCad schematic (older format))
At the start: 12 parts, among them U20 STM32F030R8T6, Y1 32.768kHz, Y2 8MHz

Commit message: Fixed some BOM stuff
fixed BOM for non RLC components
Parts:
- added D20: LED, symbol LED
- added R59: 100, symbol R
- U44: renamed from U20; part_num (none) -> CHIP-003
- Y1: part_num (none) -> XTAL-001
- Y2: part_num (none) -> XTAL-002
Connections:
- wire segments 79 -> 83
- no-connect marks 17 -> 16
Other:
- note removed: "\n\n\nTODO: How do you program this thing?\n"
Changed lines of the file:
@@
 $EndDescr
 $Comp
-L STM32F030R8T6 U20
+L STM32F030R8T6 U44
 U 1 1 5919370B
 P 4400 3200
-F 0 "U20" H 4400 4200 60  0000 C CNN
+F 0 "U44" H 4400 4200 60  0000 C CNN
 F 1 "STM32F030R8T6" H 4400 4100 60  0000 C CNN
 F 2 "" H 4150 3700 60  0001 C CNN
 F 3 "" H 4150 3700 60  0001 C CNN
+F 4 "CHIP-003" H 4400 3200 60  0001 C CNN "part_num"
 	1    4400 3200
 	1    0    0    -1
 $EndComp
 $Comp
-L STM32F030R8T6 U20
+L STM32F030R8T6 U44
 U 2 1 59193786
 P 4400 4600
-F 0 "U20" H 4400 5600 60  0000 C CNN
+F 0 "U44" H 4400 5600 60  0000 C CNN
 F 1 "STM32F030R8T6" H 4400 5500 60  0000 C CNN
 F 2 "" H 4150 5100 60  0001 C CNN
 F 3 "" H 4150 5100 60  0001 C CNN
+F 4 "CHIP-003" H 4400 4600 60  0001 C CNN "part_num"
 	2    4400 4600
 	1    0    0    -1
 $EndComp
 $Comp
-L STM32F030R8T6 U20
+L STM32F030R8T6 U44
 U 3 1 591937E7
 P 4400 5850
-F 0 "U20" H 4400 6850 60  0000 C CNN
+F 0 "U44" H 4400 6850 60  0000 C CNN
 F 1 "STM32F030R8T6" H 4400 6750 60  0000 C CNN
 F 2 "" H 4150 6350 60  0001 C CNN
 F 3 "" H 4150 6350 60  0001 C CNN
+F 4 "CHIP-003" H 4400 5850 60  0001 C CNN "part_num"
 	3    4400 5850
 	1    0    0    -1
 $EndComp
 $Comp
-L STM32F030R8T6 U20
+L STM32F030R8T6 U44
 U 4 1 59193842
 P 8000 3000
-F 0 "U20" H 8000 4000 60  0000 C CNN
+F 0 "U44" H 8000 4000 60  0000 C CNN
 F 1 "STM32F030R8T6" H 8000 3900 60  0000 C CNN
 F 2 "" H 7750 3500 60  0001 C CNN
 F 3 "" H 7750 3500 60  0001 C CNN
+F 4 "CHIP-003" H 8000 3000 60  0001 C CNN "part_num"
 	4    8000 3000
 	1    0    0    -1
 $EndComp
 $Comp
-L STM32F030R8T6 U20
+L STM32F030R8T6 U44
 U 5 1 591938AB
 P 9500 5150
-F 0 "U20" H 9500 6150 60  0000 C CNN
+F 0 "U44" H 9500 6150 60  0000 C CNN
 F 1 "STM32F030R8T6" H 9500 6050 60  0000 C CNN
 F 2 "" H 9250 5650 60  0001 C CNN
 F 3 "" H 9250 5650 60  0001 C CNN
+F 4 "CHIP-003" H 9500 5150 60  0001 C CNN "part_num"
 	5    9500 5150
 	1    0    0    -1
@@
 Text Label 4900 3150 0    60   ~ 0
 SWCLK
-Text Notes 5050 1150 0    60   ~ 0
-\n\n\nTODO: How do you program this thing?\n
 Entry Wire Line
 	2800 5000 2900 5100
@@
 Connection ~ 8350 5350
 $Comp
-L GND #PWR42
+L GND #PWR051
 U 1 1 59199AA1
 P 8600 5350
-F 0 "#PWR42" H 8600 5100 50  0001 C CNN
+F 0 "#PWR051" H 8600 5100 50  0001 C CNN
 F 1 "GND" H 8600 5200 50  0000 C CNN
 F 2 "" H 8600 5350 50  0001 C CNN
@@
 F 2 "" H 7000 2300 50  0001 C CNN
 F 3 "" H 7000 2300 50  0001 C CNN
+F 4 "XTAL-001" H 7000 2300 60  0001 C CNN "part_num"
 	1    7000 2300
 	0    1    1    0
@@
 F 2 "" H 7000 2850 50  0001 C CNN
 F 3 "" H 7000 2850 50  0001 C CNN
+F 4 "XTAL-002" H 7000 2850 60  0001 C CNN "part_num"
 	1    7000 2850
 	0    1    1    0
@@
 Connection ~ 6350 2300
 $Comp
-L GND #PWR41
+L GND #PWR052
 U 1 1 5919B18A
 P 6150 2650
-F 0 "#PWR41" H 6150 2400 50  0001 C CNN
+F 0 "#PWR052" H 6150 2400 50  0001 C CNN
 F 1 "GND" H 6150 2500 50  0000 C CNN
 F 2 "" H 6150 2650 50  0001 C CNN
@@
 NoConn ~ 8800 2950
 NoConn ~ 8800 2850
-NoConn ~ 8800 2750
 NoConn ~ 8800 2550
 Text HLabel 5300 3350 2    60   BiDi ~ 0
@@
 Wire Notes Line
 	2350 2700 3050 2700
+$Comp
+L LED D20
+U 1 1 59531E55
+P 9050 3000
+F 0 "D20" H 9050 3100 50  0000 C CNN
+F 1 "LED" H 9050 2900 50  0000 C CNN
+F 2 "" H 9050 3000 50  0001 C CNN
+F 3 "" H 9050 3000 50  0001 C CNN
+F 4 "DIOD-002" H 9050 3000 60  0001 C CNN "part_num"
+	1    9050 3000
+	0    -1   -1   0
+$EndComp
+$Comp
+L R R59
+U 1 1 59531EA2
+P 9050 3400
+F 0 "R59" V 9130 3400 50  0000 C CNN
+F 1 "100" V 9050 3400 50  0000 C CNN
+F 2 "" V 8980 3400 50  0001 C CNN
+F 3 "" H 9050 3400 50  0001 C CNN
+	1    9050 3400
+	1    0    0    -1
+$EndComp
+$Comp
+L GND #PWR053
+U 1 1 59531EED
+P 9050 3650
+F 0 "#PWR053" H 9050 3400 50  0001 C CNN
+F 1 "GND" H 9050 3500 50  0000 C CNN
+F 2 "" H 9050 3650 50  0001 C CNN
+F 3 "" H 9050 3650 50  0001 C CNN
+	1    9050 3650
+	1    0    0    -1
+$EndComp
+Wire Wire Line
+	9050 3550 9050 3650
+Wire Wire Line
+	9050 3250 9050 3150
+Wire Wire Line
+	9050 2850 9050 2750
+Wire Wire Line
+	9050 2750 8800 2750
+Text Label 8400 4850 0    59   ~ 0
+VDD
 $EndSCHEMATC

Commit message: Finished RLC bom stuff
Parts:
- C29, C30: value C -> 14pF; part_num (none) -> CAPP-008
- C31, C32: value C -> 7pF; part_num (none) -> CAPP-009
- C33, C34: part_num (none) -> CAPP-005
- C35: part_num (none) -> CAPP-006
- C36: part_num (none) -> CAPP-010
- C37: part_num (none) -> CAPP-004
- R59: part_num (none) -> RESS-006
- renumbered U44 to U19
Changed lines of the file:
@@
 $EndDescr
 $Comp
-L STM32F030R8T6 U44
+L STM32F030R8T6 U19
 U 1 1 5919370B
 P 4400 3200
-F 0 "U44" H 4400 4200 60  0000 C CNN
+F 0 "U19" H 4400 4200 60  0000 C CNN
 F 1 "STM32F030R8T6" H 4400 4100 60  0000 C CNN
 F 2 "" H 4150 3700 60  0001 C CNN
@@
 $EndComp
 $Comp
-L STM32F030R8T6 U44
+L STM32F030R8T6 U19
 U 2 1 59193786
 P 4400 4600
-F 0 "U44" H 4400 5600 60  0000 C CNN
+F 0 "U19" H 4400 5600 60  0000 C CNN
 F 1 "STM32F030R8T6" H 4400 5500 60  0000 C CNN
 F 2 "" H 4150 5100 60  0001 C CNN
@@
 $EndComp
 $Comp
-L STM32F030R8T6 U44
+L STM32F030R8T6 U19
 U 3 1 591937E7
 P 4400 5850
-F 0 "U44" H 4400 6850 60  0000 C CNN
+F 0 "U19" H 4400 6850 60  0000 C CNN
 F 1 "STM32F030R8T6" H 4400 6750 60  0000 C CNN
 F 2 "" H 4150 6350 60  0001 C CNN
@@
 $EndComp
 $Comp
-L STM32F030R8T6 U44
+L STM32F030R8T6 U19
 U 4 1 59193842
 P 8000 3000
-F 0 "U44" H 8000 4000 60  0000 C CNN
+F 0 "U19" H 8000 4000 60  0000 C CNN
 F 1 "STM32F030R8T6" H 8000 3900 60  0000 C CNN
 F 2 "" H 7750 3500 60  0001 C CNN
@@
 $EndComp
 $Comp
-L STM32F030R8T6 U44
+L STM32F030R8T6 U19
 U 5 1 591938AB
 P 9500 5150
-F 0 "U44" H 9500 6150 60  0000 C CNN
+F 0 "U19" H 9500 6150 60  0000 C CNN
 F 1 "STM32F030R8T6" H 9500 6050 60  0000 C CNN
 F 2 "" H 9250 5650 60  0001 C CNN
@@
 F 2 "" H 8388 4950 50  0001 C CNN
 F 3 "" H 8350 5100 50  0001 C CNN
+F 4 "CAPP-005" H 8350 5100 60  0001 C CNN "part_num"
 	1    8350 5100
 	1    0    0    -1
@@
 F 2 "" H 8638 4950 50  0001 C CNN
 F 3 "" H 8600 5100 50  0001 C CNN
+F 4 "CAPP-006" H 8600 5100 60  0001 C CNN "part_num"
 	1    8600 5100
 	1    0    0    -1
@@
 F 2 "" H 8888 4950 50  0001 C CNN
 F 3 "" H 8850 5100 50  0001 C CNN
+F 4 "CAPP-010" H 8850 5100 60  0001 C CNN "part_num"
 	1    8850 5100
 	1    0    0    -1
@@
 F 2 "" H 8138 4950 50  0001 C CNN
 F 3 "" H 8100 5100 50  0001 C CNN
+F 4 "CAPP-005" H 8100 5100 60  0001 C CNN "part_num"
 	1    8100 5100
 	1    0    0    -1
@@
 F 2 "" H 9138 4950 50  0001 C CNN
 F 3 "" H 9100 5100 50  0001 C CNN
+F 4 "CAPP-004" H 9100 5100 60  0001 C CNN "part_num"
 	1    9100 5100
 	1    0    0    -1
@@
 P 6550 2700
 F 0 "C31" H 6575 2800 50  0000 L CNN
-F 1 "C" H 6575 2600 50  0000 L CNN
+F 1 "7pF" H 6575 2600 50  0000 L CNN
 F 2 "" H 6588 2550 50  0001 C CNN
 F 3 "" H 6550 2700 50  0001 C CNN
+F 4 "CAPP-009" H 6550 2700 60  0001 C CNN "part_num"
 	1    6550 2700
 	0    -1   -1   0
@@
 P 6550 3000
 F 0 "C32" H 6575 3100 50  0000 L CNN
-F 1 "C" H 6575 2900 50  0000 L CNN
+F 1 "7pF" H 6575 2900 50  0000 L CNN
 F 2 "" H 6588 2850 50  0001 C CNN
 F 3 "" H 6550 3000 50  0001 C CNN
+F 4 "CAPP-009" H 6550 3000 60  0001 C CNN "part_num"
 	1    6550 3000
 	0    -1   -1   0
@@
 P 6550 2450
 F 0 "C30" H 6575 2550 50  0000 L CNN
-F 1 "C" H 6575 2350 50  0000 L CNN
+F 1 "14pF" H 6575 2350 50  0000 L CNN
 F 2 "" H 6588 2300 50  0001 C CNN
 F 3 "" H 6550 2450 50  0001 C CNN
+F 4 "CAPP-008" H 6550 2450 60  0001 C CNN "part_num"
 	1    6550 2450
 	0    -1   -1   0
@@
 P 6550 2150
 F 0 "C29" H 6575 2250 50  0000 L CNN
-F 1 "C" H 6575 2050 50  0000 L CNN
+F 1 "14pF" H 6575 2050 50  0000 L CNN
 F 2 "" H 6588 2000 50  0001 C CNN
 F 3 "" H 6550 2150 50  0001 C CNN
+F 4 "CAPP-008" H 6550 2150 60  0001 C CNN "part_num"
 	1    6550 2150
 	0    -1   -1   0
@@
 F 2 "" V 8980 3400 50  0001 C CNN
 F 3 "" H 9050 3400 50  0001 C CNN
+F 4 "RESS-006" V 9050 3400 60  0001 C CNN "part_num"
 	1    9050 3400
 	1    0    0    -1

Commit message: Added ressistor footprint
Parts:
- C29, C30, C31, C32, C33, C34, C35, C36, C37, R59: footprint (none) -> Resistors_SMD:R_0603_HandSoldering
Changed lines of the file:
@@
 F 0 "C34" H 8375 5200 50  0000 L CNN
 F 1 "100nF" H 8375 5000 50  0000 L CNN
-F 2 "" H 8388 4950 50  0001 C CNN
+F 2 "Resistors_SMD:R_0603_HandSoldering" H 8388 4950 50  0001 C CNN
 F 3 "" H 8350 5100 50  0001 C CNN
 F 4 "CAPP-005" H 8350 5100 60  0001 C CNN "part_num"
@@
 F 0 "C35" H 8625 5200 50  0000 L CNN
 F 1 "4.7uF" H 8625 5000 50  0000 L CNN
-F 2 "" H 8638 4950 50  0001 C CNN
+F 2 "Resistors_SMD:R_0603_HandSoldering" H 8638 4950 50  0001 C CNN
 F 3 "" H 8600 5100 50  0001 C CNN
 F 4 "CAPP-006" H 8600 5100 60  0001 C CNN "part_num"
@@
 F 0 "C36" H 8875 5200 50  0000 L CNN
 F 1 "10nF" H 8875 5000 50  0000 L CNN
-F 2 "" H 8888 4950 50  0001 C CNN
+F 2 "Resistors_SMD:R_0603_HandSoldering" H 8888 4950 50  0001 C CNN
 F 3 "" H 8850 5100 50  0001 C CNN
 F 4 "CAPP-010" H 8850 5100 60  0001 C CNN "part_num"
@@
 F 0 "C33" H 8125 5200 50  0000 L CNN
 F 1 "100nF" H 8125 5000 50  0000 L CNN
-F 2 "" H 8138 4950 50  0001 C CNN
+F 2 "Resistors_SMD:R_0603_HandSoldering" H 8138 4950 50  0001 C CNN
 F 3 "" H 8100 5100 50  0001 C CNN
 F 4 "CAPP-005" H 8100 5100 60  0001 C CNN "part_num"
@@
 F 0 "C37" H 9125 5200 50  0000 L CNN
 F 1 "1uF" H 9125 5000 50  0000 L CNN
-F 2 "" H 9138 4950 50  0001 C CNN
+F 2 "Resistors_SMD:R_0603_HandSoldering" H 9138 4950 50  0001 C CNN
 F 3 "" H 9100 5100 50  0001 C CNN
 F 4 "CAPP-004" H 9100 5100 60  0001 C CNN "part_num"
@@
 F 0 "C31" H 6575 2800 50  0000 L CNN
 F 1 "7pF" H 6575 2600 50  0000 L CNN
-F 2 "" H 6588 2550 50  0001 C CNN
+F 2 "Resistors_SMD:R_0603_HandSoldering" H 6588 2550 50  0001 C CNN
 F 3 "" H 6550 2700 50  0001 C CNN
 F 4 "CAPP-009" H 6550 2700 60  0001 C CNN "part_num"
@@
 F 0 "C32" H 6575 3100 50  0000 L CNN
 F 1 "7pF" H 6575 2900 50  0000 L CNN
-F 2 "" H 6588 2850 50  0001 C CNN
+F 2 "Resistors_SMD:R_0603_HandSoldering" H 6588 2850 50  0001 C CNN
 F 3 "" H 6550 3000 50  0001 C CNN
 F 4 "CAPP-009" H 6550 3000 60  0001 C CNN "part_num"
@@
 F 0 "C30" H 6575 2550 50  0000 L CNN
 F 1 "14pF" H 6575 2350 50  0000 L CNN
-F 2 "" H 6588 2300 50  0001 C CNN
+F 2 "Resistors_SMD:R_0603_HandSoldering" H 6588 2300 50  0001 C CNN
 F 3 "" H 6550 2450 50  0001 C CNN
 F 4 "CAPP-008" H 6550 2450 60  0001 C CNN "part_num"
@@
 F 0 "C29" H 6575 2250 50  0000 L CNN
 F 1 "14pF" H 6575 2050 50  0000 L CNN
-F 2 "" H 6588 2000 50  0001 C CNN
+F 2 "Resistors_SMD:R_0603_HandSoldering" H 6588 2000 50  0001 C CNN
 F 3 "" H 6550 2150 50  0001 C CNN
 F 4 "CAPP-008" H 6550 2150 60  0001 C CNN "part_num"
@@
 F 0 "R59" V 9130 3400 50  0000 C CNN
 F 1 "100" V 9050 3400 50  0000 C CNN
-F 2 "" V 8980 3400 50  0001 C CNN
+F 2 "Resistors_SMD:R_0603_HandSoldering" V 8980 3400 50  0001 C CNN
 F 3 "" H 9050 3400 50  0001 C CNN
 F 4 "RESS-006" V 9050 3400 60  0001 C CNN "part_num"

Commit message: PCB?!
Added initial PCB file with ratsnest. footprint library still needs to
be setup.
Parts:
- D20: footprint (none) -> LEDs:LED_0603
- U19: footprint (none) -> Housings_QFP:LQFP-64_10x10mm_Pitch0.5mm
- Y1: footprint (none) -> Crystals:Crystal_SMD_MicroCrystal_CC7V-T1A-2pin_3.2x1.5mm_HandSoldering
- Y2: footprint (none) -> Crystals:Crystal_SMD_5032-2pin_5.0x3.2mm_HandSoldering
- renumbered R59 to R84
Changed lines of the file:
@@
 Comment4 ""
 $EndDescr
-$Comp
-L STM32F030R8T6 U19
-U 1 1 5919370B
-P 4400 3200
-F 0 "U19" H 4400 4200 60  0000 C CNN
-F 1 "STM32F030R8T6" H 4400 4100 60  0000 C CNN
-F 2 "" H 4150 3700 60  0001 C CNN
-F 3 "" H 4150 3700 60  0001 C CNN
-F 4 "CHIP-003" H 4400 3200 60  0001 C CNN "part_num"
-	1    4400 3200
-	1    0    0    -1
-$EndComp
-$Comp
-L STM32F030R8T6 U19
-U 2 1 59193786
-P 4400 4600
-F 0 "U19" H 4400 5600 60  0000 C CNN
-F 1 "STM32F030R8T6" H 4400 5500 60  0000 C CNN
-F 2 "" H 4150 5100 60  0001 C CNN
-F 3 "" H 4150 5100 60  0001 C CNN
-F 4 "CHIP-003" H 4400 4600 60  0001 C CNN "part_num"
-	2    4400 4600
-	1    0    0    -1
-$EndComp
-$Comp
-L STM32F030R8T6 U19
-U 3 1 591937E7
-P 4400 5850
-F 0 "U19" H 4400 6850 60  0000 C CNN
-F 1 "STM32F030R8T6" H 4400 6750 60  0000 C CNN
-F 2 "" H 4150 6350 60  0001 C CNN
-F 3 "" H 4150 6350 60  0001 C CNN
-F 4 "CHIP-003" H 4400 5850 60  0001 C CNN "part_num"
-	3    4400 5850
-	1    0    0    -1
-$EndComp
-$Comp
-L STM32F030R8T6 U19
-U 4 1 59193842
-P 8000 3000
-F 0 "U19" H 8000 4000 60  0000 C CNN
-F 1 "STM32F030R8T6" H 8000 3900 60  0000 C CNN
-F 2 "" H 7750 3500 60  0001 C CNN
-F 3 "" H 7750 3500 60  0001 C CNN
-F 4 "CHIP-003" H 8000 3000 60  0001 C CNN "part_num"
-	4    8000 3000
-	1    0    0    -1
-$EndComp
-$Comp
-L STM32F030R8T6 U19
-U 5 1 591938AB
-P 9500 5150
-F 0 "U19" H 9500 6150 60  0000 C CNN
-F 1 "STM32F030R8T6" H 9500 6050 60  0000 C CNN
-F 2 "" H 9250 5650 60  0001 C CNN
-F 3 "" H 9250 5650 60  0001 C CNN
-F 4 "CHIP-003" H 9500 5150 60  0001 C CNN "part_num"
-	5    9500 5150
-	1    0    0    -1
-$EndComp
 Text HLabel 8850 4500 0    60   Input ~ 0
 VDD
@@
 Connection ~ 8350 5350
 $Comp
-L GND #PWR051
+L GND #PWR50
 U 1 1 59199AA1
 P 8600 5350
-F 0 "#PWR051" H 8600 5100 50  0001 C CNN
+F 0 "#PWR50" H 8600 5100 50  0001 C CNN
 F 1 "GND" H 8600 5200 50  0000 C CNN
 F 2 "" H 8600 5350 50  0001 C CNN
@@
 F 0 "Y1" H 7000 2450 50  0000 C CNN
 F 1 "32.768kHz" H 7000 2150 50  0000 C CNN
-F 2 "" H 7000 2300 50  0001 C CNN
+F 2 "Crystals:Crystal_SMD_MicroCrystal_CC7V-T1A-2pin_3.2x1.5mm_HandSoldering" H 7000 2300 50  0001 C CNN
 F 3 "" H 7000 2300 50  0001 C CNN
 F 4 "XTAL-001" H 7000 2300 60  0001 C CNN "part_num"
@@
 F 0 "Y2" H 7000 3000 50  0000 C CNN
 F 1 "8MHz" H 7000 2700 50  0000 C CNN
-F 2 "" H 7000 2850 50  0001 C CNN
+F 2 "Crystals:Crystal_SMD_5032-2pin_5.0x3.2mm_HandSoldering" H 7000 2850 50  0001 C CNN
 F 3 "" H 7000 2850 50  0001 C CNN
 F 4 "XTAL-002" H 7000 2850 60  0001 C CNN "part_num"
@@
 Connection ~ 6350 2300
 $Comp
-L GND #PWR052
+L GND #PWR49
 U 1 1 5919B18A
 P 6150 2650
-F 0 "#PWR052" H 6150 2400 50  0001 C CNN
+F 0 "#PWR49" H 6150 2400 50  0001 C CNN
 F 1 "GND" H 6150 2500 50  0000 C CNN
 F 2 "" H 6150 2650 50  0001 C CNN
@@
 F 0 "D20" H 9050 3100 50  0000 C CNN
 F 1 "LED" H 9050 2900 50  0000 C CNN
-F 2 "" H 9050 3000 50  0001 C CNN
+F 2 "LEDs:LED_0603" H 9050 3000 50  0001 C CNN
 F 3 "" H 9050 3000 50  0001 C CNN
 F 4 "DIOD-002" H 9050 3000 60  0001 C CNN "part_num"
@@
 $EndComp
 $Comp
-L R R59
+L R R84
 U 1 1 59531EA2
 P 9050 3400
-F 0 "R59" V 9130 3400 50  0000 C CNN
+F 0 "R84" V 9130 3400 50  0000 C CNN
 F 1 "100" V 9050 3400 50  0000 C CNN
 F 2 "Resistors_SMD:R_0603_HandSoldering" V 8980 3400 50  0001 C CNN
@@
 $EndComp
 $Comp
-L GND #PWR053
+L GND #PWR51
 U 1 1 59531EED
 P 9050 3650
-F 0 "#PWR053" H 9050 3400 50  0001 C CNN
+F 0 "#PWR51" H 9050 3400 50  0001 C CNN
 F 1 "GND" H 9050 3500 50  0000 C CNN
 F 2 "" H 9050 3650 50  0001 C CNN
@@
 Text Label 8400 4850 0    59   ~ 0
 VDD
+$Comp
+L STM32F030R8T6 U19
+U 1 1 595FA412
+P 4400 3200
+F 0 "U19" H 4400 4200 60  0000 C CNN
+F 1 "STM32F030R8T6" H 4400 4100 60  0000 C CNN
+F 2 "Housings_QFP:LQFP-64_10x10mm_Pitch0.5mm" H 4150 3700 60  0001 C CNN
+F 3 "" H 4150 3700 60  0001 C CNN
+F 4 "CHIP-003" H 4500 4300 60  0001 C CNN "part_num"
+	1    4400 3200
+	1    0    0    -1
+$EndComp
+$Comp
+L STM32F030R8T6 U19
+U 2 1 595FA45A
+P 4400 4600
+F 0 "U19" H 4400 5600 60  0000 C CNN
+F 1 "STM32F030R8T6" H 4400 5500 60  0000 C CNN
+F 2 "Housings_QFP:LQFP-64_10x10mm_Pitch0.5mm" H 4150 5100 60  0001 C CNN
+F 3 "" H 4150 5100 60  0001 C CNN
+F 4 "CHIP-003" H 4500 5700 60  0001 C CNN "part_num"
+	2    4400 4600
+	1    0    0    -1
+$EndComp
+$Comp
+L STM32F030R8T6 U19
+U 3 1 595FA4A8
+P 4400 5850
+F 0 "U19" H 4400 6850 60  0000 C CNN
+F 1 "STM32F030R8T6" H 4400 6750 60  0000 C CNN
+F 2 "Housings_QFP:LQFP-64_10x10mm_Pitch0.5mm" H 4150 6350 60  0001 C CNN
+F 3 "" H 4150 6350 60  0001 C CNN
+F 4 "CHIP-003" H 4500 6950 60  0001 C CNN "part_num"
+	3    4400 5850
+	1    0    0    -1
+$EndComp
+$Comp
+L STM32F030R8T6 U19
+U 4 1 595FA4F2
+P 8000 3000
+F 0 "U19" H 8000 4000 60  0000 C CNN
+F 1 "STM32F030R8T6" H 8000 3900 60  0000 C CNN
+F 2 "Housings_QFP:LQFP-64_10x10mm_Pitch0.5mm" H 7750 3500 60  0001 C CNN
+F 3 "" H 7750 3500 60  0001 C CNN
+F 4 "CHIP-003" H 8100 4100 60  0001 C CNN "part_num"
+	4    8000 3000
+	1    0    0    -1
+$EndComp
+$Comp
+L STM32F030R8T6 U19
+U 5 1 595FA680
+P 9500 5150
+F 0 "U19" H 9500 6150 60  0000 C CNN
+F 1 "STM32F030R8T6" H 9500 6050 60  0000 C CNN
+F 2 "Housings_QFP:LQFP-64_10x10mm_Pitch0.5mm" H 9250 5650 60  0001 C CNN
+F 3 "" H 9250 5650 60  0001 C CNN
+F 4 "CHIP-003" H 9600 6250 60  0001 C CNN "part_num"
+	5    9500 5150
+	1    0    0    -1
+$EndComp
 $EndSCHEMATC

Commit message: Fixed serge suggestions
Parts:
- added TP?: TEST, Measurement_Points:Measurement_Point_Round-SMD-Pad_Big, symbol TEST
Connections:
- wire segments 83 -> 85
Changed lines of the file:
@@
 $Descr A4 11693 8268
 encoding utf-8
-Sheet 19 20
+Sheet 19 21
 Title "Safety Switch Controller/ PPM Converter"
 Date "2017-05-14"
@@
 Connection ~ 8350 5350
 $Comp
-L GND #PWR50
+L GND #PWR049
 U 1 1 59199AA1
 P 8600 5350
-F 0 "#PWR50" H 8600 5100 50  0001 C CNN
+F 0 "#PWR049" H 8600 5100 50  0001 C CNN
 F 1 "GND" H 8600 5200 50  0000 C CNN
 F 2 "" H 8600 5350 50  0001 C CNN
@@
 Connection ~ 6350 2300
 $Comp
-L GND #PWR49
+L GND #PWR050
 U 1 1 5919B18A
 P 6150 2650
-F 0 "#PWR49" H 6150 2400 50  0001 C CNN
+F 0 "#PWR050" H 6150 2400 50  0001 C CNN
 F 1 "GND" H 6150 2500 50  0000 C CNN
 F 2 "" H 6150 2650 50  0001 C CNN
@@
 $EndComp
 $Comp
-L GND #PWR51
+L GND #PWR051
 U 1 1 59531EED
 P 9050 3650
-F 0 "#PWR51" H 9050 3400 50  0001 C CNN
+F 0 "#PWR051" H 9050 3400 50  0001 C CNN
 F 1 "GND" H 9050 3500 50  0000 C CNN
 F 2 "" H 9050 3650 50  0001 C CNN
@@
 	1    0    0    -1
 $EndComp
+$Comp
+L TEST TP?
+U 1 1 596A3495
+P 7200 3200
+F 0 "TP?" H 7200 3500 50  0000 C BNN
+F 1 "TEST" H 7200 3450 50  0000 C CNN
+F 2 "Measurement_Points:Measurement_Point_Round-SMD-Pad_Big" H 7200 3200 50  0001 C CNN
+F 3 "" H 7200 3200 50  0001 C CNN
+	1    7200 3200
+	-1   0    0    1
+$EndComp
+Wire Wire Line
+	7200 3200 7200 3150
+Wire Wire Line
+	7200 3150 7400 3150
 $EndSCHEMATC

Commit message: commit before my computer restarts
Parts:
- gave numbers to parts that had none: 1
- renumbered D20 to D18, R84 to R40
Changed lines of the file:
@@
 	2350 2700 3050 2700
 $Comp
-L LED D20
+L LED D18
 U 1 1 59531E55
 P 9050 3000
-F 0 "D20" H 9050 3100 50  0000 C CNN
+F 0 "D18" H 9050 3100 50  0000 C CNN
 F 1 "LED" H 9050 2900 50  0000 C CNN
 F 2 "LEDs:LED_0603" H 9050 3000 50  0001 C CNN
@@
 $EndComp
 $Comp
-L R R84
+L R R40
 U 1 1 59531EA2
 P 9050 3400
-F 0 "R84" V 9130 3400 50  0000 C CNN
+F 0 "R40" V 9130 3400 50  0000 C CNN
 F 1 "100" V 9050 3400 50  0000 C CNN
 F 2 "Resistors_SMD:R_0603_HandSoldering" V 8980 3400 50  0001 C CNN
@@
 $EndComp
 $Comp
-L TEST TP?
+L TEST TP40
 U 1 1 596A3495
 P 7200 3200
-F 0 "TP?" H 7200 3500 50  0000 C BNN
+F 0 "TP40" H 7200 3500 50  0000 C BNN
 F 1 "TEST" H 7200 3450 50  0000 C CNN
 F 2 "Measurement_Points:Measurement_Point_Round-SMD-Pad_Big" H 7200 3200 50  0001 C CNN
