File: Hardware/STM32F0 RELAY.sch (KiCad schematic (older format))
At the start: 22 parts, among them Q2 Q_NMOS_GSD, U19 STM32F030RCT6, Y1 32.768kHz, Y2 8MHz

Commit message: Fixed merge issues
Parts:
- renumbered C29 to C46, C30 to C47, C31 to C48, C32 to C49, C33 to C50, C34 to C51, C35 to C52, C36 to C53, C37 to C54, D1 to D7, D18 to D8, D2 to D9, R2 to R20, R1 to R21, R40 to R22, R4 to R23, TP40 to TP4, U19 to U10, Y1 to Y3, Y2 to Y4
Changed lines of the file:
@@
 LIBS:contrib
 LIBS:valves
+LIBS:ZeroPilot-cache
 EELAYER 25 0
 EELAYER END
@@
 Connection ~ 8900 4650
 $Comp
-L C C34
+L C C51
 U 1 1 5919967A
 P 7200 5050
-F 0 "C34" H 7225 5150 50  0000 L CNN
+F 0 "C51" H 7225 5150 50  0000 L CNN
 F 1 "100nF" H 7225 4950 50  0000 L CNN
 F 2 "Resistors_SMD:R_0603_HandSoldering" H 7238 4900 50  0001 C CNN
@@
 $EndComp
 $Comp
-L C C35
+L C C52
 U 1 1 591996BB
 P 7450 5050
-F 0 "C35" H 7475 5150 50  0000 L CNN
+F 0 "C52" H 7475 5150 50  0000 L CNN
 F 1 "4.7uF" H 7475 4950 50  0000 L CNN
 F 2 "Resistors_SMD:R_0603_HandSoldering" H 7488 4900 50  0001 C CNN
@@
 $EndComp
 $Comp
-L C C36
+L C C53
 U 1 1 591996E8
 P 7700 5050
-F 0 "C36" H 7725 5150 50  0000 L CNN
+F 0 "C53" H 7725 5150 50  0000 L CNN
 F 1 "10nF" H 7725 4950 50  0000 L CNN
 F 2 "Resistors_SMD:R_0603_HandSoldering" H 7738 4900 50  0001 C CNN
@@
 $EndComp
 $Comp
-L C C33
+L C C50
 U 1 1 5919971A
 P 6950 5050
-F 0 "C33" H 6975 5150 50  0000 L CNN
+F 0 "C50" H 6975 5150 50  0000 L CNN
 F 1 "100nF" H 6975 4950 50  0000 L CNN
 F 2 "Resistors_SMD:R_0603_HandSoldering" H 6988 4900 50  0001 C CNN
@@
 $EndComp
 $Comp
-L C C37
+L C C54
 U 1 1 5919974F
 P 7950 5050
-F 0 "C37" H 7975 5150 50  0000 L CNN
+F 0 "C54" H 7975 5150 50  0000 L CNN
 F 1 "1uF" H 7975 4950 50  0000 L CNN
 F 2 "Resistors_SMD:R_0603_HandSoldering" H 7988 4900 50  0001 C CNN
@@
 Connection ~ 7200 5300
 $Comp
-L GND #PWR39
+L GND #PWR029
 U 1 1 59199AA1
 P 7450 5300
-F 0 "#PWR39" H 7450 5050 50  0001 C CNN
+F 0 "#PWR029" H 7450 5050 50  0001 C CNN
 F 1 "GND" H 7450 5150 50  0000 C CNN
 F 2 "" H 7450 5300 50  0001 C CNN
@@
 Connection ~ 7950 5300
 $Comp
-L Crystal Y1
+L Crystal Y3
 U 1 1 5919A616
 P 7000 2300
-F 0 "Y1" H 7000 2450 50  0000 C CNN
+F 0 "Y3" H 7000 2450 50  0000 C CNN
 F 1 "32.768kHz" H 7000 2150 50  0000 C CNN
 F 2 "Crystals:Crystal_SMD_MicroCrystal_CC7V-T1A-2pin_3.2x1.5mm_HandSoldering" H 7000 2300 50  0001 C CNN
@@
 $EndComp
 $Comp
-L Crystal Y2
+L Crystal Y4
 U 1 1 5919A668
 P 7000 2850
-F 0 "Y2" H 7000 3000 50  0000 C CNN
+F 0 "Y4" H 7000 3000 50  0000 C CNN
 F 1 "8MHz" H 7000 2700 50  0000 C CNN
 F 2 "Crystals:Crystal_SMD_5032-2pin_5.0x3.2mm_HandSoldering" H 7000 2850 50  0001 C CNN
@@
 	7400 2150 7400 2350
 $Comp
-L C C31
+L C C48
 U 1 1 5919AAC2
 P 6550 2700
-F 0 "C31" H 6575 2800 50  0000 L CNN
+F 0 "C48" H 6575 2800 50  0000 L CNN
 F 1 "7pF" H 6575 2600 50  0000 L CNN
 F 2 "Resistors_SMD:R_0603_HandSoldering" H 6588 2550 50  0001 C CNN
@@
 $EndComp
 $Comp
-L C C32
+L C C49
 U 1 1 5919AB20
 P 6550 3000
-F 0 "C32" H 6575 3100 50  0000 L CNN
+F 0 "C49" H 6575 3100 50  0000 L CNN
 F 1 "7pF" H 6575 2900 50  0000 L CNN
 F 2 "Resistors_SMD:R_0603_HandSoldering" H 6588 2850 50  0001 C CNN
@@
 $EndComp
 $Comp
-L C C30
+L C C47
 U 1 1 5919ABF0
 P 6550 2450
-F 0 "C30" H 6575 2550 50  0000 L CNN
+F 0 "C47" H 6575 2550 50  0000 L CNN
 F 1 "14pF" H 6575 2350 50  0000 L CNN
 F 2 "Resistors_SMD:R_0603_HandSoldering" H 6588 2300 50  0001 C CNN
@@
 $EndComp
 $Comp
-L C C29
+L C C46
 U 1 1 5919AC3B
 P 6550 2150
-F 0 "C29" H 6575 2250 50  0000 L CNN
+F 0 "C46" H 6575 2250 50  0000 L CNN
 F 1 "14pF" H 6575 2050 50  0000 L CNN
 F 2 "Resistors_SMD:R_0603_HandSoldering" H 6588 2000 50  0001 C CNN
@@
 Connection ~ 6350 2300
 $Comp
-L GND #PWR36
+L GND #PWR030
 U 1 1 5919B18A
 P 6150 2650
-F 0 "#PWR36" H 6150 2400 50  0001 C CNN
+F 0 "#PWR030" H 6150 2400 50  0001 C CNN
 F 1 "GND" H 6150 2500 50  0000 C CNN
 F 2 "" H 6150 2650 50  0001 C CNN
@@
 	2350 2700 3050 2700
 $Comp
-L LED D18
+L LED D8
 U 1 1 59531E55
 P 5800 5750
-F 0 "D18" H 5800 5850 50  0000 C CNN
+F 0 "D8" H 5800 5850 50  0000 C CNN
 F 1 "LED" H 5800 5650 50  0000 C CNN
 F 2 "LEDs:LED_0603" H 5800 5750 50  0001 C CNN
@@
 $EndComp
 $Comp
-L R R40
+L R R22
 U 1 1 59531EA2
 P 5800 6150
-F 0 "R40" V 5880 6150 50  0000 C CNN
+F 0 "R22" V 5880 6150 50  0000 C CNN
 F 1 "100" V 5800 6150 50  0000 C CNN
 F 2 "Resistors_SMD:R_0603_HandSoldering" V 5730 6150 50  0001 C CNN
@@
 $EndComp
 $Comp
-L GND #PWR35
+L GND #PWR031
 U 1 1 59531EED
 P 5800 6400
-F 0 "#PWR35" H 5800 6150 50  0001 C CNN
+F 0 "#PWR031" H 5800 6150 50  0001 C CNN
 F 1 "GND" H 5800 6250 50  0000 C CNN
 F 2 "" H 5800 6400 50  0001 C CNN
@@
 VDD
 $Comp
-L TEST TP40
+L TEST TP4
 U 1 1 596A3495
 P 7200 3200
-F 0 "TP40" H 7200 3500 50  0000 C BNN
+F 0 "TP4" H 7200 3500 50  0000 C BNN
 F 1 "TEST" H 7200 3450 50  0000 C CNN
 F 2 "Measurement_Points:Measurement_Point_Round-SMD-Pad_Small" H 7200 3200 50  0001 C CNN
@@
 NoConn ~ 4900 4250
 $Comp
-L LED D1
+L LED D7
 U 1 1 592CEFDB
 P 5450 5750
-F 0 "D1" H 5450 5850 50  0000 C CNN
+F 0 "D7" H 5450 5850 50  0000 C CNN
 F 1 "LED" H 5450 5650 50  0000 C CNN
 F 2 "LEDs:LED_0603" H 5450 5750 50  0001 C CNN
@@
 $EndComp
 $Comp
-L R R2
+L R R20
 U 1 1 592CEFE3
 P 5450 6150
-F 0 "R2" V 5530 6150 50  0000 C CNN
+F 0 "R20" V 5530 6150 50  0000 C CNN
 F 1 "100" V 5450 6150 50  0000 C CNN
 F 2 "Resistors_SMD:R_0603_HandSoldering" V 5380 6150 50  0001 C CNN
@@
 $EndComp
 $Comp
-L GND #PWR33
+L GND #PWR032
 U 1 1 592CEFEA
 P 5450 6400
-F 0 "#PWR33" H 5450 6150 50  0001 C CNN
+F 0 "#PWR032" H 5450 6150 50  0001 C CNN
 F 1 "GND" H 5450 6250 50  0000 C CNN
 F 2 "" H 5450 6400 50  0001 C CNN
@@
 	5450 6000 5450 5900
 $Comp
-L LED D2
+L LED D9
 U 1 1 592CF150
 P 6150 5750
-F 0 "D2" H 6150 5850 50  0000 C CNN
+F 0 "D9" H 6150 5850 50  0000 C CNN
 F 1 "LED" H 6150 5650 50  0000 C CNN
 F 2 "LEDs:LED_0603" H 6150 5750 50  0001 C CNN
@@
 $EndComp
 $Comp
-L R R4
+L R R23
 U 1 1 592CF158
 P 6150 6150
-F 0 "R4" V 6230 6150 50  0000 C CNN
+F 0 "R23" V 6230 6150 50  0000 C CNN
 F 1 "100" V 6150 6150 50  0000 C CNN
 F 2 "Resistors_SMD:R_0603_HandSoldering" V 6080 6150 50  0001 C CNN
@@
 $EndComp
 $Comp
-L GND #PWR37
+L GND #PWR033
 U 1 1 592CF15F
 P 6150 6400
-F 0 "#PWR37" H 6150 6150 50  0001 C CNN
+F 0 "#PWR033" H 6150 6150 50  0001 C CNN
 F 1 "GND" H 6150 6250 50  0000 C CNN
 F 2 "" H 6150 6400 50  0001 C CNN
@@
 	3200 4150 3900 4150
 $Comp
-L GND #PWR34
+L GND #PWR034
 U 1 1 594F28B6
 P 5800 5000
-F 0 "#PWR34" H 5800 4750 50  0001 C CNN
+F 0 "#PWR034" H 5800 4750 50  0001 C CNN
 F 1 "GND" H 5800 4850 50  0000 C CNN
 F 2 "" H 5800 5000 50  0001 C CNN
@@
 $EndComp
 $Comp
-L STM32F030RCT6 U19
+L STM32F030RCT6 U10
 U 1 1 599C1943
 P 4400 3200
-F 0 "U19" H 4400 4200 60  0000 C CNN
+F 0 "U10" H 4400 4200 60  0000 C CNN
 F 1 "STM32F030RCT6" H 4400 4100 60  0000 C CNN
 F 2 "Housings_QFP:LQFP-64_10x10mm_Pitch0.5mm" H 4150 3700 60  0001 C CNN
@@
 $EndComp
 $Comp
-L STM32F030RCT6 U19
+L STM32F030RCT6 U10
 U 2 1 599C19BB
 P 4400 4600
-F 0 "U19" H 4400 5600 60  0000 C CNN
+F 0 "U10" H 4400 5600 60  0000 C CNN
 F 1 "STM32F030RCT6" H 4400 5500 60  0000 C CNN
 F 2 "Housings_QFP:LQFP-64_10x10mm_Pitch0.5mm" H 4150 5100 60  0001 C CNN
@@
 $EndComp
 $Comp
-L STM32F030RCT6 U19
+L STM32F030RCT6 U10
 U 3 1 599C1A21
 P 4400 5850
-F 0 "U19" H 4400 6850 60  0000 C CNN
+F 0 "U10" H 4400 6850 60  0000 C CNN
 F 1 "STM32F030RCT6" H 4400 6750 60  0000 C CNN
 F 2 "Housings_QFP:LQFP-64_10x10mm_Pitch0.5mm" H 4150 6350 60  0001 C CNN
@@
 $EndComp
 $Comp
-L STM32F030RCT6 U19
+L STM32F030RCT6 U10
 U 4 1 599C1A7B
 P 8000 3000
-F 0 "U19" H 8000 4000 60  0000 C CNN
+F 0 "U10" H 8000 4000 60  0000 C CNN
 F 1 "STM32F030RCT6" H 8000 3900 60  0000 C CNN
 F 2 "Housings_QFP:LQFP-64_10x10mm_Pitch0.5mm" H 7750 3500 60  0001 C CNN
@@
 $EndComp
 $Comp
-L STM32F030RCT6 U19
+L STM32F030RCT6 U10
 U 5 1 599C1AE4
 P 8350 4900
-F 0 "U19" H 8350 5900 60  0000 C CNN
+F 0 "U10" H 8350 5900 60  0000 C CNN
 F 1 "STM32F030RCT6" H 8350 5800 60  0000 C CNN
 F 2 "Housings_QFP:LQFP-64_10x10mm_Pitch0.5mm" H 8100 5400 60  0001 C CNN
@@
 	5800 4350 4900 4350
 $Comp
-L R R1
+L R R21
 U 1 1 599C8783
 P 5800 4750
-F 0 "R1" V 5880 4750 50  0000 C CNN
+F 0 "R21" V 5880 4750 50  0000 C CNN
 F 1 "100K" V 5800 4750 50  0000 C CNN
 F 2 "Resistors_SMD:R_0603_HandSoldering" V 5730 4750 50  0001 C CNN
@@
 Connection ~ 5800 4500
 $Comp
-L GND #PWR38
+L GND #PWR035
 U 1 1 599C9676
 P 6500 4800
-F 0 "#PWR38" H 6500 4550 50  0001 C CNN
+F 0 "#PWR035" H 6500 4550 50  0001 C CNN
 F 1 "GND" H 6500 4650 50  0000 C CNN
 F 2 "" H 6500 4800 50  0001 C CNN

Commit message: Remapped symbols for KiCAD 5.0.x
Parts:
- BZ1: symbol Buzzer -> Device:Buzzer
- C46, C47, C48, C49, C50, C51, C52, C53, C54: symbol C -> Device:C
- D7, D8, D9: symbol LED -> Device:LED
- Q2: symbol Q_NMOS_GSD -> Device:Q_NMOS_GSD
- R20, R21, R22, R23: symbol R -> Device:R
- TP4: symbol TEST -> Connector:TestPoint
- U10: symbol STM32F030RCT6 -> WARG:STM32F030RCT6
- Y3, Y4: symbol Crystal -> Device:Crystal
Other:
- moved on the sheet: TP4
Changed lines of the file:
@@
-EESchema Schematic File Version 2
-LIBS:WARG
-LIBS:power
-LIBS:device
-LIBS:transistors
-LIBS:conn
-LIBS:linear
-LIBS:regul
-LIBS:74xx
-LIBS:cmos4000
-LIBS:adc-dac
-LIBS:memory
-LIBS:xilinx
-LIBS:microcontrollers
-LIBS:dsp
-LIBS:microchip
-LIBS:analog_switches
-LIBS:motorola
-LIBS:texas
-LIBS:intel
-LIBS:audio
-LIBS:interface
-LIBS:digital-audio
-LIBS:philips
-LIBS:display
-LIBS:cypress
-LIBS:siliconi
-LIBS:opto
-LIBS:atmel
-LIBS:contrib
-LIBS:valves
+EESchema Schematic File Version 4
 LIBS:ZeroPilot-cache
-EELAYER 25 0
+EELAYER 26 0
 EELAYER END
 $Descr A4 11693 8268
@@
 Wire Bus Line
 	1300 3600 1400 3700
-Wire Bus Line
-	1400 3700 1400 5350
 Entry Wire Line
 	1400 3700 1500 3800
@@
 	7650 4400 7850 4400
 Wire Wire Line
-	7850 4250 7850 4800
+	7850 4250 7850 4350
 Wire Wire Line
 	7850 4750 7900 4750
@@
 	8850 4450 8900 4450
 Wire Wire Line
-	8900 4250 8900 5300
+	8900 4250 8900 4350
 Wire Wire Line
 	8900 4650 8850 4650
@@
 Connection ~ 8900 4650
 $Comp
-L C C51
+L Device:C C51
 U 1 1 5919967A
 P 7200 5050
@@
 $EndComp
 $Comp
-L C C52
+L Device:C C52
 U 1 1 591996BB
 P 7450 5050
@@
 $EndComp
 $Comp
-L C C53
+L Device:C C53
 U 1 1 591996E8
 P 7700 5050
@@
 $EndComp
 $Comp
-L C C50
+L Device:C C50
 U 1 1 5919971A
 P 6950 5050
@@
 $EndComp
 $Comp
-L C C54
+L Device:C C54
 U 1 1 5919974F
 P 7950 5050
@@
 	7950 4800 7950 4900
 Wire Wire Line
-	6950 4800 7950 4800
+	6950 4800 7200 4800
 Wire Wire Line
 	6950 4800 6950 4900
@@
 	6950 5200 6950 5300
 Wire Wire Line
-	6950 5300 8900 5300
+	6950 5300 7200 5300
 Wire Wire Line
 	7950 5300 7950 5200
@@
 Connection ~ 7200 5300
 $Comp
-L GND #PWR029
+L power:GND #PWR029
 U 1 1 59199AA1
 P 7450 5300
@@
 Connection ~ 7950 5300
 $Comp
-L Crystal Y3
+L Device:Crystal Y3
 U 1 1 5919A616
 P 7000 2300
@@
 $EndComp
 $Comp
-L Crystal Y4
+L Device:Crystal Y4
 U 1 1 5919A668
 P 7000 2850
@@
 $EndComp
 Wire Wire Line
-	6700 2450 7400 2450
-Wire Wire Line
-	6700 2700 7400 2700
-Wire Wire Line
-	6700 3000 7400 3000
+	6700 2450 7000 2450
+Wire Wire Line
+	6700 2700 7000 2700
+Wire Wire Line
+	6700 3000 7000 3000
 Wire Wire Line
 	7400 3000 7400 2800
 Wire Wire Line
-	6700 2150 7400 2150
+	6700 2150 7000 2150
 Wire Wire Line
 	7400 2150 7400 2350
 $Comp
-L C C48
+L Device:C C48
 U 1 1 5919AAC2
 P 6550 2700
@@
 $EndComp
 $Comp
-L C C49
+L Device:C C49
 U 1 1 5919AB20
 P 6550 3000
@@
 $EndComp
 $Comp
-L C C47
+L Device:C C47
 U 1 1 5919ABF0
 P 6550 2450
@@
 $EndComp
 $Comp
-L C C46
+L Device:C C46
 U 1 1 5919AC3B
 P 6550 2150
@@
 	6400 2150 6350 2150
 Wire Wire Line
-	6350 2150 6350 2450
+	6350 2150 6350 2300
 Wire Wire Line
 	6350 2450 6400 2450
@@
 	6400 2700 6350 2700
 Wire Wire Line
-	6350 2700 6350 3000
+	6350 2700 6350 2850
 Wire Wire Line
 	6350 3000 6400 3000
@@
 	6350 2300 6300 2300
 Wire Wire Line
-	6300 2300 6300 2850
+	6300 2300 6300 2550
 Wire Wire Line
 	6300 2850 6350 2850
@@
 Connection ~ 6350 2300
 $Comp
-L GND #PWR030
+L power:GND #PWR030
 U 1 1 5919B18A
 P 6150 2650
@@
 	2350 2700 3050 2700
 $Comp
-L LED D8
+L Device:LED D8
 U 1 1 59531E55
 P 5800 5750
@@
 $EndComp
 $Comp
-L R R22
+L Device:R R22
 U 1 1 59531EA2
 P 5800 6150
@@
 $EndComp
 $Comp
-L GND #PWR031
+L power:GND #PWR031
 U 1 1 59531EED
 P 5800 6400
@@
 VDD
 $Comp
-L TEST TP4
+L Connector:TestPoint TP4
 U 1 1 596A3495
 P 7200 3200
@@
 NoConn ~ 4900 4250
 $Comp
-L LED D7
+L Device:LED D7
 U 1 1 592CEFDB
 P 5450 5750
@@
 $EndComp
 $Comp
-L R R20
+L Device:R R20
 U 1 1 592CEFE3
 P 5450 6150
@@
 $EndComp
 $Comp
-L GND #PWR032
+L power:GND #PWR032
 U 1 1 592CEFEA
 P 5450 6400
@@
 	5450 6000 5450 5900
 $Comp
-L LED D9
+L Device:LED D9
 U 1 1 592CF150
 P 6150 5750
@@
 $EndComp
 $Comp
-L R R23
+L Device:R R23
 U 1 1 592CF158
 P 6150 6150
@@
 $EndComp
 $Comp
-L GND #PWR033
+L power:GND #PWR033
 U 1 1 592CF15F
 P 6150 6400
@@
 	3200 4150 3900 4150
 $Comp
-L GND #PWR034
+L power:GND #PWR034
 U 1 1 594F28B6
 P 5800 5000
@@
 $EndComp
 $Comp
-L Buzzer BZ1
+L Device:Buzzer BZ1
 U 1 1 594F2B8D
 P 6600 3950
@@
 $EndComp
 $Comp
-L STM32F030RCT6 U10
+L WARG:STM32F030RCT6 U10
 U 1 1 599C1943
 P 4400 3200
@@
 F 1 "STM32F030RCT6" H 4400 4100 60  0000 C CNN
 F 2 "Housings_QFP:LQFP-64_10x10mm_Pitch0.5mm" H 4150 3700 60  0001 C CNN
-F 3 "" H 4150 3700 60  0001 C CNN
+F 3 "https://www.st.com/resource/en/datasheet/stm32f030rc.pdf" H 4150 3700 60  0001 C CNN
 F 4 "CHIP-003" H 4500 4300 60  0001 C CNN "part_num"
 	1    4400 3200
@@
 $EndComp
 $Comp
-L STM32F030RCT6 U10
+L WARG:STM32F030RCT6 U10
 U 2 1 599C19BB
 P 4400 4600
@@
 F 1 "STM32F030RCT6" H 4400 5500 60  0000 C CNN
 F 2 "Housings_QFP:LQFP-64_10x10mm_Pitch0.5mm" H 4150 5100 60  0001 C CNN
-F 3 "" H 4150 5100 60  0001 C CNN
+F 3 "https://www.st.com/resource/en/datasheet/stm32f030rc.pdf" H 4150 5100 60  0001 C CNN
 F 4 "CHIP-003" H 4500 5700 60  0001 C CNN "part_num"
 	2    4400 4600
@@
 $EndComp
 $Comp
-L STM32F030RCT6 U10
+L WARG:STM32F030RCT6 U10
 U 3 1 599C1A21
 P 4400 5850
@@
 F 1 "STM32F030RCT6" H 4400 6750 60  0000 C CNN
 F 2 "Housings_QFP:LQFP-64_10x10mm_Pitch0.5mm" H 4150 6350 60  0001 C CNN
-F 3 "" H 4150 6350 60  0001 C CNN
+F 3 "https://www.st.com/resource/en/datasheet/stm32f030rc.pdf" H 4150 6350 60  0001 C CNN
 F 4 "CHIP-003" H 4500 6950 60  0001 C CNN "part_num"
 	3    4400 5850
@@
 $EndComp
 $Comp
-L STM32F030RCT6 U10
+L WARG:STM32F030RCT6 U10
 U 4 1 599C1A7B
 P 8000 3000
@@
 F 1 "STM32F030RCT6" H 8000 3900 60  0000 C CNN
 F 2 "Housings_QFP:LQFP-64_10x10mm_Pitch0.5mm" H 7750 3500 60  0001 C CNN
-F 3 "" H 7750 3500 60  0001 C CNN
+F 3 "https://www.st.com/resource/en/datasheet/stm32f030rc.pdf" H 7750 3500 60  0001 C CNN
 F 4 "CHIP-003" H 8100 4100 60  0001 C CNN "part_num"
 	4    8000 3000
@@
 $EndComp
 $Comp
-L STM32F030RCT6 U10
+L WARG:STM32F030RCT6 U10
 U 5 1 599C1AE4
 P 8350 4900
@@
 F 1 "STM32F030RCT6" H 8350 5800 60  0000 C CNN
 F 2 "Housings_QFP:LQFP-64_10x10mm_Pitch0.5mm" H 8100 5400 60  0001 C CNN
-F 3 "" H 8100 5400 60  0001 C CNN
+F 3 "https://www.st.com/resource/en/datasheet/stm32f030rc.pdf" H 8100 5400 60  0001 C CNN
 F 4 "CHIP-003" H 8450 6000 60  0001 C CNN "part_num"
 	5    8350 4900
@@
 	5800 4350 4900 4350
 $Comp
-L R R21
+L Device:R R21
 U 1 1 599C8783
 P 5800 4750
@@
 V_SPK
 Wire Wire Line
-	5800 4350 5800 4600
+	5800 4350 5800 4500
 Wire Wire Line
 	5800 5000 5800 4900
 Connection ~ 5800 4500
 $Comp
-L GND #PWR035
+L power:GND #PWR035
 U 1 1 599C9676
 P 6500 4800
@@
 	6500 3650 6350 3650
 $Comp
-L Q_NMOS_GSD Q2
+L Device:Q_NMOS_GSD Q2
 U 1 1 599C9998
 P 6400 4500
@@
 	1    0    0    -1
 $EndComp
+Wire Wire Line
+	7850 4650 7850 4750
+Wire Wire Line
+	7850 4550 7850 4650
+Wire Wire Line
+	7850 4450 7850 4550
+Wire Wire Line
+	8900 4550 8900 4650
+Wire Wire Line
+	8900 4650 8900 5300
+Wire Wire Line
+	7200 4800 7450 4800
+Wire Wire Line
+	7450 4800 7700 4800
+Wire Wire Line
+	7700 4800 7850 4800
+Wire Wire Line
+	7850 4800 7950 4800
+Wire Wire Line
+	7850 4750 7850 4800
+Wire Wire Line
+	7700 5300 7950 5300
+Wire Wire Line
+	7450 5300 7700 5300
+Wire Wire Line
+	7200 5300 7450 5300
+Wire Wire Line
+	7950 5300 8900 5300
+Wire Wire Line
+	6350 2850 6350 3000
+Wire Wire Line
+	6350 2300 6350 2450
+Wire Wire Line
+	6300 2550 6300 2850
+Wire Wire Line
+	7000 2150 7400 2150
+Wire Wire Line
+	7000 2450 7400 2450
+Wire Wire Line
+	7000 2700 7400 2700
+Wire Wire Line
+	7000 3000 7400 3000
+Wire Wire Line
+	7850 4400 7850 4450
+Wire Wire Line
+	8900 4450 8900 4550
+Wire Wire Line
+	8900 4350 8900 4450
+Wire Wire Line
+	5800 4500 5800 4600
+Wire Bus Line
+	1400 3700 1400 5350
 $EndSCHEMATC
