File: Hardware/_saved_STM32F0 RELAY.sch (KiCad schematic (older format))
At the start: 20 parts, among them U19 STM32F030R8T6, Y1 32.768kHz, Y2 8MHz

Commit message: added speaker
Parts:
- gave numbers to parts that had none: 1
Changed lines of the file:
@@
 	5000 5600 5000 5850
 $Comp
-L GND #PWR?
+L GND #PWR056
 U 1 1 594F28B6
 P 5000 6150
-F 0 "#PWR?" H 5000 5900 50  0001 C CNN
+F 0 "#PWR056" H 5000 5900 50  0001 C CNN
 F 1 "GND" H 5000 6000 50  0000 C CNN
 F 2 "" H 5000 6150 50  0001 C CNN
@@
 	5000 6150 5000 6050
 $Comp
-L Buzzer BZ?
+L Buzzer BZ1
 U 1 1 594F2B8D
 P 5100 5950
-F 0 "BZ?" H 5250 6000 50  0000 L CNN
+F 0 "BZ1" H 5250 6000 50  0000 L CNN
 F 1 "Buzzer" H 5250 5900 50  0000 L CNN
 F 2 "WARG:AI-1027-TWT-3V-R" V 5075 6050 50  0001 C CNN
