File: Hardware/HEADERS.sch (KiCad schematic (older format))
At the start: 46 parts, among them J16 SPOX-3, J17 SPOX-3, J18 SPOX-4, J19 SPOX-2, J22 SPOX-4, J23 SPOX-4, J24 SPOX-6, J25 SPOX-6, J26 SPOX-6, J28 SPOX-6, J29 SPOX-6, J30 SPOX-6

Commit message: Updated pcb
Parts:
- TP19, TP22: footprint (none) -> Measurement_Points:Measurement_Point_Round-SMD-Pad_Small
Changed lines of the file:
@@
 F 0 "TP19" H 1550 5100 50  0000 C BNN
 F 1 "TEST" H 1550 5050 50  0000 C CNN
-F 2 "" H 1550 4800 50  0001 C CNN
+F 2 "Measurement_Points:Measurement_Point_Round-SMD-Pad_Small" H 1550 4800 50  0001 C CNN
 F 3 "" H 1550 4800 50  0001 C CNN
 	1    1550 4800
@@
 F 0 "TP22" H 1550 5200 50  0000 C BNN
 F 1 "TEST" H 1550 5150 50  0000 C CNN
-F 2 "" H 1550 4900 50  0001 C CNN
+F 2 "Measurement_Points:Measurement_Point_Round-SMD-Pad_Small" H 1550 4900 50  0001 C CNN
 F 3 "" H 1550 4900 50  0001 C CNN
 	1    1550 4900

Commit message: Remapped symbols for KiCAD 5.0.x
Parts:
- J16, J17: symbol SPOX-3 -> WARG:SPOX-3
- J18, J22, J23: symbol SPOX-4 -> WARG:SPOX-4
- J19: symbol SPOX-2 -> WARG:SPOX-2
- J24, J25, J26, J28, J29, J30: symbol SPOX-6 -> WARG:SPOX-6
- R47, R48, R49, R50, R51, R52: symbol R -> Device:R
- TP10, TP11, TP12, TP13, TP14, TP15, TP16, TP17, TP18, TP19, TP20, TP21, TP22, TP23, TP24, TP25, TP26, TP30, TP31, TP32, TP33, TP34, TP35, TP5, TP6, TP7, TP8, TP9: symbol TEST -> Connector:TestPoint
Other:
- moved on the sheet: TP10, TP11, TP12, TP13, TP14, TP15, TP16, TP17, TP18, TP19, TP20, TP21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

Commit message: Added RSSI, datasheets, INDU-004
Added RSSI input to PPM connector. Added datasheets for most of the components. The filter inductors for the FTDI were labeled as INDU-002, which is a 15uH smps inductor.
Parts:
- removed TP19, TP22: TEST, Measurement_Points:Measurement_Point_Round-SMD-Pad_Small, symbol Connector:TestPoint
- added H? (x4): MountingHole_M3, Mounting_Holes:MountingHole_3.2mm_M3_Pad, symbol Mechanical:MountingHole
- added J?: SPOX-4, Connectors_Molex:Molex_SPOX-5267_22-03-5045_04x2.54mm_Straight, symbol WARG:SPOX-4
- J16: value SPOX-3 -> SPOX-4; footprint Connectors_Molex:Molex_SPOX-5267_22-03-5035_03x2.54mm_Straight -> Connectors_Molex:Molex_SPOX-5267_22-03-5045_04x2.54mm_Straight; symbol WARG:SPOX-3 -> WARG:SPOX-4
Connections:
- net labels added: RSSI, V_UHF
- wire segments 133 -> 137
Other:
- moved on the sheet: J19
Changed lines of the file:
@@
 Text HLabel 1700 1900 2    60   Input ~ 0
 AIRSPD
-Text HLabel 1650 1400 2    60   Input ~ 0
+Text HLabel 1650 1200 2    60   Input ~ 0
 V_PPM
 Text HLabel 1650 1300 2    60   Input ~ 0
@@
 F 1 "SPOX-3" H 1350 1800 60  0000 C CNN
 F 2 "Connectors_Molex:Molex_SPOX-5267_22-03-5035_03x2.54mm_Straight" H 1250 2150 60  0001 C CNN
-F 3 "" H 1350 2250 60  0001 C CNN
+F 3 "https://www.molex.com/pdm_docs/sd/022035035_sd.pdf" H 1350 2250 60  0001 C CNN
 F 4 "CONN-002" H 1450 2350 60  0001 C CNN "part_num"
 	1    1250 2000
@@
 F 1 "SPOX-6" H 5500 2300 60  0000 C CNN
 F 2 "Connectors_Molex:Molex_SPOX-5267_22-03-5065_06x2.54mm_Straight" H 5400 2800 60  0001 C CNN
-F 3 "" H 5400 2800 60  0001 C CNN
+F 3 "https://www.molex.com/pdm_docs/sd/022035065_sd.pdf" H 5400 2800 60  0001 C CNN
 F 4 "CONN-005" H 5600 3100 60  0001 C CNN "part_num"
 	1    5400 2650
@@
 F 1 "SPOX-6" H 5500 3150 60  0000 C CNN
 F 2 "Connectors_Molex:Molex_SPOX-5267_22-03-5065_06x2.54mm_Straight" H 5400 3650 60  0001 C CNN
-F 3 "" H 5400 3650 60  0001 C CNN
+F 3 "https://www.molex.com/pdm_docs/sd/022035065_sd.pdf" H 5400 3650 60  0001 C CNN
 F 4 "CONN-005" H 5600 3950 60  0001 C CNN "part_num"
 	1    5400 3500
@@
 F 1 "SPOX-6" H 5500 5000 60  0000 C CNN
 F 2 "Connectors_Molex:Molex_SPOX-5267_22-03-5065_06x2.54mm_Straight" H 5400 5500 60  0001 C CNN
-F 3 "" H 5400 5500 60  0001 C CNN
+F 3 "https://www.molex.com/pdm_docs/sd/022035065_sd.pdf" H 5400 5500 60  0001 C CNN
 F 4 "CONN-005" H 5600 5800 60  0001 C CNN "part_num"
 	1    5400 5350
@@
 F 1 "SPOX-6" H 9100 3400 60  0000 C CNN
 F 2 "Connectors_Molex:Molex_SPOX-5267_22-03-5065_06x2.54mm_Straight" H 9000 3900 60  0001 C CNN
-F 3 "" H 9000 3900 60  0001 C CNN
+F 3 "https://www.molex.com/pdm_docs/sd/022035065_sd.pdf" H 9000 3900 60  0001 C CNN
 F 4 "CONN-005" H 9200 4200 60  0001 C CNN "part_num"
 	1    9000 3750
@@
 F 1 "SPOX-6" H 9100 4200 60  0000 C CNN
 F 2 "Connectors_Molex:Molex_SPOX-5267_22-03-5065_06x2.54mm_Straight" H 9000 4700 60  0001 C CNN
-F 3 "" H 9000 4700 60  0001 C CNN
+F 3 "https://www.molex.com/pdm_docs/sd/022035065_sd.pdf" H 9000 4700 60  0001 C CNN
 F 4 "CONN-005" H 9200 5000 60  0001 C CNN "part_num"
 	1    9000 4550
@@
 F 1 "SPOX-6" H 9100 5050 60  0000 C CNN
 F 2 "Connectors_Molex:Molex_SPOX-5267_22-03-5065_06x2.54mm_Straight" H 9000 5550 60  0001 C CNN
-F 3 "" H 9000 5550 60  0001 C CNN
+F 3 "https://www.molex.com/pdm_docs/sd/022035065_sd.pdf" H 9000 5550 60  0001 C CNN
 F 4 "CONN-005" H 9200 5850 60  0001 C CNN "part_num"
 	1    9000 5400
@@
 F 1 "SPOX-4" H 3800 4200 60  0000 C CNN
 F 2 "Connectors_Molex:Molex_SPOX-5267_22-03-5045_04x2.54mm_Straight" H 3700 4500 60  0001 C CNN
-F 3 "" H 3700 4500 60  0001 C CNN
+F 3 "https://www.molex.com/pdm_docs/sd/022035045_sd.pdf" H 3700 4500 60  0001 C CNN
 F 4 "CONN-003" H 3900 4800 60  0001 C CNN "part_num"
 	1    3700 4450
@@
 F 1 "SPOX-4" H 3800 4750 60  0000 C CNN
 F 2 "Connectors_Molex:Molex_SPOX-5267_22-03-5045_04x2.54mm_Straight" H 3700 5050 60  0001 C CNN
-F 3 "" H 3700 5050 60  0001 C CNN
+F 3 "https://www.molex.com/pdm_docs/sd/022035045_sd.pdf" H 3700 5050 60  0001 C CNN
 F 4 "CONN-003" H 3900 5350 60  0001 C CNN "part_num"
 	1    3700 5000
@@
 $EndComp
 $Comp
-L WARG:SPOX-3 J16
+L WARG:SPOX-4 J16
 U 1 1 5966BE07
-P 1200 1400
-F 0 "J16" H 1300 1650 60  0000 C CNN
-F 1 "SPOX-3" H 1300 1200 60  0000 C CNN
-F 2 "Connectors_Molex:Molex_SPOX-5267_22-03-5035_03x2.54mm_Straight" H 1200 1550 60  0001 C CNN
-F 3 "" H 1300 1650 60  0001 C CNN
-F 4 "CONN-002" H 1400 1750 60  0001 C CNN "part_num"
-	1    1200 1400
+P 1250 1350
+F 0 "J16" H 1350 1650 60  0000 C CNN
+F 1 "SPOX-4" H 1350 1100 60  0000 C CNN
+F 2 "Connectors_Molex:Molex_SPOX-5267_22-03-5045_04x2.54mm_Straight" H 1250 1500 60  0001 C CNN
+F 3 "https://www.molex.com/pdm_docs/sd/022035045_sd.pdf" H 1350 1600 60  0001 C CNN
+F 4 "CONN-002" H 1450 1700 60  0001 C CNN "part_num"
+	1    1250 1350
 	1    0    0    -1
 $EndComp
@@
 F 1 "SPOX-4" H 1350 2350 60  0000 C CNN
 F 2 "Connectors_Molex:Molex_SPOX-5267_22-03-5045_04x2.54mm_Straight" H 1250 2650 60  0001 C CNN
-F 3 "" H 1250 2650 60  0001 C CNN
+F 3 "https://www.molex.com/pdm_docs/sd/022035045_sd.pdf" H 1250 2650 60  0001 C CNN
 F 4 "CONN-003" H 1450 2950 60  0001 C CNN "part_num"
 	1    1250 2600
@@
 L WARG:SPOX-2 J19
 U 1 1 597D9B19
-P 1300 3250
-F 0 "J19" H 1400 3400 60  0000 C CNN
-F 1 "SPOX-2" H 1400 3100 60  0000 C CNN
-F 2 "Connectors_Molex:Molex_SPOX-5267_22-03-5025_02x2.54mm_Straight" H 1300 3200 60  0001 C CNN
-F 3 "" H 1300 3200 60  0001 C CNN
-F 4 "CONN-001" H 1500 3500 60  0001 C CNN "part_num"
-	1    1300 3250
+P 1250 3250
+F 0 "J19" H 1350 3400 60  0000 C CNN
+F 1 "SPOX-2" H 1350 3100 60  0000 C CNN
+F 2 "Connectors_Molex:Molex_SPOX-5267_22-03-5025_02x2.54mm_Straight" H 1250 3200 60  0001 C CNN
+F 3 "https://www.molex.com/pdm_docs/sd/022035025_sd.pdf" H 1250 3200 60  0001 C CNN
+F 4 "CONN-001" H 1450 3500 60  0001 C CNN "part_num"
+	1    1250 3250
 	1    0    0    -1
 $EndComp
@@
 I2C_PULLUP
 Wire Wire Line
-	1600 3300 1500 3300
-Wire Wire Line
-	1700 3200 1500 3200
+	1600 3300 1450 3300
+Wire Wire Line
+	1700 3200 1450 3200
 Wire Wire Line
 	1750 3700 1500 3700
@@
 	1600 1500 1600 2100
 Wire Wire Line
-	1400 1500 1600 1500
+	1450 1500 1600 1500
 Connection ~ 1600 2100
 Wire Wire Line
@@
 	5600 5500 5700 5500
 Wire Wire Line
-	1750 4800 1550 4800
-Wire Wire Line
-	1750 4900 1550 4900
+	1750 4800 1500 4800
+Wire Wire Line
+	1750 4900 1500 4900
 Wire Wire Line
 	6600 2400 5600 2400
@@
 Connection ~ 3350 3150
 Wire Wire Line
-	1650 1300 1400 1300
-Wire Wire Line
-	1400 1400 1650 1400
+	1650 1300 1450 1300
+Wire Wire Line
+	1450 1400 1650 1400
 Wire Wire Line
 	9300 5550 9200 5550
@@
 L power:GND #PWR064
 U 1 1 5923F1BC
-P 1600 5000
-F 0 "#PWR064" H 1600 4750 50  0001 C CNN
-F 1 "GND" H 1600 4850 50  0000 C CNN
-F 2 "" H 1600 5000 50  0001 C CNN
-F 3 "" H 1600 5000 50  0001 C CNN
-	1    1600 5000
-	1    0    0    -1
-$EndComp
-$Comp
-L Connector:TestPoint TP19
-U 1 1 5B4E2465
-P 1550 4800
-F 0 "TP19" H 1550 5100 50  0000 C BNN
-F 1 "TEST" H 1550 5050 50  0000 C CNN
-F 2 "Measurement_Points:Measurement_Point_Round-SMD-Pad_Small" H 1550 4800 50  0001 C CNN
-F 3 "" H 1550 4800 50  0001 C CNN
-	1    1550 4800
-	0    -1   -1   0
-$EndComp
-$Comp
-L Connector:TestPoint TP22
-U 1 1 5B4E251E
-P 1550 4900
-F 0 "TP22" H 1550 5200 50  0000 C BNN
-F 1 "TEST" H 1550 5150 50  0000 C CNN
-F 2 "Measurement_Points:Measurement_Point_Round-SMD-Pad_Small" H 1550 4900 50  0001 C CNN
-F 3 "" H 1550 4900 50  0001 C CNN
-	1    1550 4900
-	0    -1   -1   0
+P 1600 5200
+F 0 "#PWR064" H 1600 4950 50  0001 C CNN
+F 1 "GND" H 1600 5050 50  0000 C CNN
+F 2 "" H 1600 5200 50  0001 C CNN
+F 3 "" H 1600 5200 50  0001 C CNN
+	1    1600 5200
+	1    0    0    -1
 $EndComp
 Wire Wire Line
@@
 Wire Wire Line
 	6600 3250 6600 5100
+Text HLabel 1650 1400 2    60   Input ~ 0
+RSSI
+Wire Wire Line
+	1450 1200 1650 1200
+$Comp
+L WARG:SPOX-4 J?
+U 1 1 5CB789D7
+P 1300 4850
+F 0 "J?" H 1400 5150 60  0000 C CNN
+F 1 "SPOX-4" H 1400 4600 60  0000 C CNN
+F 2 "Connectors_Molex:Molex_SPOX-5267_22-03-5045_04x2.54mm_Straight" H 1300 5000 60  0001 C CNN
+F 3 "https://www.molex.com/pdm_docs/sd/022035045_sd.pdf" H 1400 5100 60  0001 C CNN
+F 4 "CONN-002" H 1500 5200 60  0001 C CNN "part_num"
+	1    1300 4850
+	1    0    0    -1
+$EndComp
+Wire Wire Line
+	1500 5000 1600 5000
+Connection ~ 1600 5000
+Wire Wire Line
+	1600 5000 1600 5200
+Wire Wire Line
+	1500 4700 1750 4700
+Text HLabel 1750 4700 2    60   Input ~ 0
+V_UHF
+$Comp
+L Mechanical:MountingHole H?
+U 1 1 5CCE10BC
+P 9450 1100
+F 0 "H?" H 9550 1146 50  0000 L CNN
+F 1 "MountingHole_M3" H 9550 1055 50  0000 L CNN
+F 2 "Mounting_Holes:MountingHole_3.2mm_M3_Pad" H 9450 1100 50  0001 C CNN
+F 3 "~" H 9450 1100 50  0001 C CNN
+	1    9450 1100
+	1    0    0    -1
+$EndComp
+$Comp
+L Mechanical:MountingHole H?
+U 1 1 5CCE1241
+P 10350 1100
+F 0 "H?" H 10450 1146 50  0000 L CNN
+F 1 "MountingHole_M3" H 10450 1055 50  0000 L CNN
+F 2 "Mounting_Holes:MountingHole_3.2mm_M3_Pad" H 10350 1100 50  0001 C CNN
+F 3 "~" H 10350 1100 50  0001 C CNN
+	1    10350 1100
+	1    0    0    -1
+$EndComp
+$Comp
+L Mechanical:MountingHole H?
+U 1 1 5CCE706E
+P 9450 850
+F 0 "H?" H 9550 896 50  0000 L CNN
+F 1 "MountingHole_M3" H 9550 805 50  0000 L CNN
+F 2 "Mounting_Holes:MountingHole_3.2mm_M3_Pad" H 9450 850 50  0001 C CNN
+F 3 "~" H 9450 850 50  0001 C CNN
+	1    9450 850
+	1    0    0    -1
+$EndComp
+$Comp
+L Mechanical:MountingHole H?
+U 1 1 5CCE70E0
+P 10350 850
+F 0 "H?" H 10450 896 50  0000 L CNN
+F 1 "MountingHole_M3" H 10450 805 50  0000 L CNN
+F 2 "Mounting_Holes:MountingHole_3.2mm_M3_Pad" H 10350 850 50  0001 C CNN
+F 3 "~" H 10350 850 50  0001 C CNN
+	1    10350 850
+	1    0    0    -1
+$EndComp
 $EndSCHEMATC

Commit message: Finished Datasheets
Parts:
- removed H? (x3): MountingHole_M3, Mounting_Holes:MountingHole_3.2mm_M3_Pad, symbol Mechanical:MountingHole
- added H? (x3): MountingHole_M4, Mounting_Holes:MountingHole_4.3mm_M4_Pad, symbol Mechanical:MountingHole
- H?: value MountingHole_M3 -> MountingHole_M4; footprint Mounting_Holes:MountingHole_3.2mm_M3_Pad -> Mounting_Holes:MountingHole_4.3mm_M4_Pad
Changed lines of the file:
@@
 F 1 "10K" V 3350 3350 50  0000 C CNN
 F 2 "Resistors_SMD:R_0603_HandSoldering" V 3280 3350 50  0001 C CNN
-F 3 "" H 3350 3350 50  0001 C CNN
+F 3 "http://industrial.panasonic.com/www-cgi/jvcr13pz.cgi?E+PZ+3+AOA0001+ERJ3GEYJ103V+7+WW" H 3350 3350 50  0001 C CNN
 F 4 "RESS-005" V 3350 3350 60  0001 C CNN "part_num"
 	1    3350 3350
@@
 F 1 "10K" V 3550 3350 50  0000 C CNN
 F 2 "Resistors_SMD:R_0603_HandSoldering" V 3480 3350 50  0001 C CNN
-F 3 "" H 3550 3350 50  0001 C CNN
+F 3 "http://industrial.panasonic.com/www-cgi/jvcr13pz.cgi?E+PZ+3+AOA0001+ERJ3GEYJ103V+7+WW" H 3550 3350 50  0001 C CNN
 F 4 "RESS-005" V 3550 3350 60  0001 C CNN "part_num"
 	1    3550 3350
@@
 F 1 "10K" V 3550 3950 50  0000 C CNN
 F 2 "Resistors_SMD:R_0603_HandSoldering" V 3480 3950 50  0001 C CNN
-F 3 "" H 3550 3950 50  0001 C CNN
+F 3 "http://industrial.panasonic.com/www-cgi/jvcr13pz.cgi?E+PZ+3+AOA0001+ERJ3GEYJ103V+7+WW" H 3550 3950 50  0001 C CNN
 F 4 "RESS-005" V 3550 3950 60  0001 C CNN "part_num"
 	1    3550 3950
@@
 F 1 "10K" V 3350 3950 50  0000 C CNN
 F 2 "Resistors_SMD:R_0603_HandSoldering" V 3280 3950 50  0001 C CNN
-F 3 "" H 3350 3950 50  0001 C CNN
+F 3 "http://industrial.panasonic.com/www-cgi/jvcr13pz.cgi?E+PZ+3+AOA0001+ERJ3GEYJ103V+7+WW" H 3350 3950 50  0001 C CNN
 F 4 "RESS-005" V 3350 3950 60  0001 C CNN "part_num"
 	1    3350 3950
@@
 F 1 "10K" V 3350 4500 50  0000 C CNN
 F 2 "Resistors_SMD:R_0603_HandSoldering" V 3280 4500 50  0001 C CNN
-F 3 "" H 3350 4500 50  0001 C CNN
+F 3 "http://industrial.panasonic.com/www-cgi/jvcr13pz.cgi?E+PZ+3+AOA0001+ERJ3GEYJ103V+7+WW" H 3350 4500 50  0001 C CNN
 F 4 "RESS-005" V 3350 4500 60  0001 C CNN "part_num"
 	1    3350 4500
@@
 F 1 "10K" V 3550 4500 50  0000 C CNN
 F 2 "Resistors_SMD:R_0603_HandSoldering" V 3480 4500 50  0001 C CNN
-F 3 "" H 3550 4500 50  0001 C CNN
+F 3 "http://industrial.panasonic.com/www-cgi/jvcr13pz.cgi?E+PZ+3+AOA0001+ERJ3GEYJ103V+7+WW" H 3550 4500 50  0001 C CNN
 F 4 "RESS-005" V 3550 4500 60  0001 C CNN "part_num"
 	1    3550 4500
@@
 $Comp
 L Mechanical:MountingHole H?
-U 1 1 5CCE10BC
-P 9450 1100
-F 0 "H?" H 9550 1146 50  0000 L CNN
-F 1 "MountingHole_M3" H 9550 1055 50  0000 L CNN
-F 2 "Mounting_Holes:MountingHole_3.2mm_M3_Pad" H 9450 1100 50  0001 C CNN
-F 3 "~" H 9450 1100 50  0001 C CNN
-	1    9450 1100
-	1    0    0    -1
-$EndComp
-$Comp
-L Mechanical:MountingHole H?
 U 1 1 5CCE1241
 P 10350 1100
 F 0 "H?" H 10450 1146 50  0000 L CNN
-F 1 "MountingHole_M3" H 10450 1055 50  0000 L CNN
-F 2 "Mounting_Holes:MountingHole_3.2mm_M3_Pad" H 10350 1100 50  0001 C CNN
+F 1 "MountingHole_M4" H 10450 1055 50  0000 L CNN
+F 2 "Mounting_Holes:MountingHole_4.3mm_M4_Pad" H 10350 1100 50  0001 C CNN
 F 3 "~" H 10350 1100 50  0001 C CNN
 	1    10350 1100
@@
 $Comp
 L Mechanical:MountingHole H?
-U 1 1 5CCE706E
-P 9450 850
-F 0 "H?" H 9550 896 50  0000 L CNN
-F 1 "MountingHole_M3" H 9550 805 50  0000 L CNN
-F 2 "Mounting_Holes:MountingHole_3.2mm_M3_Pad" H 9450 850 50  0001 C CNN
-F 3 "~" H 9450 850 50  0001 C CNN
-	1    9450 850
+U 1 1 5CB39751
+P 10350 900
+F 0 "H?" H 10450 946 50  0000 L CNN
+F 1 "MountingHole_M4" H 10450 855 50  0000 L CNN
+F 2 "Mounting_Holes:MountingHole_4.3mm_M4_Pad" H 10350 900 50  0001 C CNN
+F 3 "~" H 10350 900 50  0001 C CNN
+	1    10350 900
 	1    0    0    -1
 $EndComp
 $Comp
 L Mechanical:MountingHole H?
-U 1 1 5CCE70E0
-P 10350 850
-F 0 "H?" H 10450 896 50  0000 L CNN
-F 1 "MountingHole_M3" H 10450 805 50  0000 L CNN
-F 2 "Mounting_Holes:MountingHole_3.2mm_M3_Pad" H 10350 850 50  0001 C CNN
-F 3 "~" H 10350 850 50  0001 C CNN
-	1    10350 850
-	1    0    0    -1
-$EndComp
+U 1 1 5CB39892
+P 9450 1100
+F 0 "H?" H 9550 1146 50  0000 L CNN
+F 1 "MountingHole_M4" H 9550 1055 50  0000 L CNN
+F 2 "Mounting_Holes:MountingHole_4.3mm_M4_Pad" H 9450 1100 50  0001 C CNN
+F 3 "~" H 9450 1100 50  0001 C CNN
+	1    9450 1100
+	1    0    0    -1
+$EndComp
+$Comp
+L Mechanical:MountingHole H?
+U 1 1 5CB39899
+P 9450 900
+F 0 "H?" H 9550 946 50  0000 L CNN
+F 1 "MountingHole_M4" H 9550 855 50  0000 L CNN
+F 2 "Mounting_Holes:MountingHole_4.3mm_M4_Pad" H 9450 900 50  0001 C CNN
+F 3 "~" H 9450 900 50  0001 C CNN
+	1    9450 900
+	1    0    0    -1
+$EndComp

Commit message: Bug fixes, added Isense, changed conn to JST-GH
Added boot0 pull-down resistors. Changed ext_batt to current sense line. Changed spox conn to JST-GH, this will dramatically reduce the required size of the board.
Parts:
- J16, J?: value SPOX-4 -> GH-4; footprint Connectors_Molex:Molex_SPOX-5267_22-03-5045_04x2.54mm_Straight -> Connectors_JST:JST_GH_BM04B-GHS-TBT_04x1.25mm_Straight; symbol WARG:SPOX-4 -> conn:Conn_01x04; part_num CONN-002 -> CONN-015
- J17: value SPOX-3 -> GH-3; footprint Connectors_Molex:Molex_SPOX-5267_22-03-5035_03x2.54mm_Straight -> Connectors_JST:JST_GH_BM03B-GHS-TBT_03x1.25mm_Straight; symbol WARG:SPOX-3 -> conn:Conn_01x03; part_num CONN-002 -> CONN-014
- J18, J22, J23: value SPOX-4 -> GH-4; footprint Connectors_Molex:Molex_SPOX-5267_22-03-5045_04x2.54mm_Straight -> Connectors_JST:JST_GH_BM04B-GHS-TBT_04x1.25mm_Straight; symbol WARG:SPOX-4 -> conn:Conn_01x04; part_num CONN-003 -> CONN-015
- J19: value SPOX-2 -> GH-2; footprint Connectors_Molex:Molex_SPOX-5267_22-03-5025_02x2.54mm_Straight -> Connectors_JST:JST_GH_BM02B-GHS-TBT_02x1.25mm_Straight; symbol WARG:SPOX-2 -> conn:Conn_01x02; part_num CONN-001 -> CONN-013
- J24, J25, J26, J28, J29, J30: value SPOX-6 -> GH-6; footprint Connectors_Molex:Molex_SPOX-5267_22-03-5065_06x2.54mm_Straight -> Connectors_JST:JST_GH_BM06B-GHS-TBT_06x1.25mm_Straight; symbol WARG:SPOX-6 -> conn:Conn_01x06; part_num CONN-005 -> CONN-017
Connections:
- net labels added: V_ISENSE
- net labels removed: EXT_BATT
- wire segments 137 -> 139

Commit message: Added protection diode to USB
Connections:
- wire segments 139 -> 137
Changed lines of the file:
@@
 	4050 4600 4050 5150
-Wire Wire Line
-	4050 5150 3950 5150
 Wire Wire Line
 	3900 4600 4050 4600
 Connection ~ 4050 5150
-Wire Wire Line
-	4200 5050 3950 5050
 Wire Wire Line
 	4200 3250 4200 4500
@@
 	1    0    0    -1
 $EndComp
-Connection ~ 3950 5050
-Wire Wire Line
-	3950 5050 3900 5050
-Connection ~ 3950 5150
-Wire Wire Line
-	3950 5150 3900 5150
+Wire Wire Line
+	3900 5150 4050 5150
+Wire Wire Line
+	3900 5050 4200 5050
 $EndSCHEMATC

Commit message: Removed F0 SPI, gave Baro its own I2C line, changed IMU to SPI1
Parts:
- removed J22: GH-4, Connectors_JST:JST_GH_BM04B-GHS-TBT_04x1.25mm_Straight, symbol conn:Conn_01x04
- added TP? (x2): TEST, Measurement_Points:Measurement_Point_Round-SMD-Pad_Small, symbol Connector:TestPoint
Connections:
- wire segments 137 -> 133
Changed lines of the file:
@@
 EESchema Schematic File Version 4
-LIBS:ZeroPilot-cache
 EELAYER 26 0
 EELAYER END
@@
 $EndComp
 $Comp
-L conn:Conn_01x04 J22
-U 1 1 595C306F
-P 3700 4500
-F 0 "J22" H 3800 4750 60  0000 C CNN
-F 1 "GH-4" H 3800 4250 60  0000 C CNN
-F 2 "Connectors_JST:JST_GH_BM04B-GHS-TBT_04x1.25mm_Straight" H 3700 4550 60  0001 C CNN
-F 3 "http://www.jst-mfg.com/product/pdf/eng/eGH.pdf" H 3700 4550 60  0001 C CNN
-F 4 "CONN-015" H 3900 4850 60  0001 C CNN "part_num"
-	1    3700 4500
-	-1   0    0    1
-$EndComp
-$Comp
 L conn:Conn_01x04 J23
 U 1 1 595C30C3
@@
 L conn:Conn_01x04 J18
 U 1 1 5966BE8B
-P 1250 2600
-F 0 "J18" H 1350 2850 60  0000 C CNN
-F 1 "GH-4" H 1350 2350 60  0000 C CNN
-F 2 "Connectors_JST:JST_GH_BM04B-GHS-TBT_04x1.25mm_Straight" H 1250 2650 60  0001 C CNN
-F 3 "http://www.jst-mfg.com/product/pdf/eng/eGH.pdf" H 1250 2650 60  0001 C CNN
-F 4 "CONN-015" H 1450 2950 60  0001 C CNN "part_num"
-	1    1250 2600
-	1    0    0    -1
+P 1250 2650
+F 0 "J18" H 1350 2900 60  0000 C CNN
+F 1 "GH-4" H 1350 2400 60  0000 C CNN
+F 2 "Connectors_JST:JST_GH_BM04B-GHS-TBT_04x1.25mm_Straight" H 1250 2700 60  0001 C CNN
+F 3 "http://www.jst-mfg.com/product/pdf/eng/eGH.pdf" H 1250 2700 60  0001 C CNN
+F 4 "CONN-015" H 1450 3000 60  0001 C CNN "part_num"
+	1    1250 2650
+	-1   0    0    1
 $EndComp
 Text HLabel 1750 4300 2    60   Input ~ 0
@@
 	1750 3800 1500 3800
 Wire Wire Line
-	4050 4600 4050 5150
-Wire Wire Line
-	3900 4600 4050 4600
-Connection ~ 4050 5150
-Wire Wire Line
-	4200 3250 4200 4500
-Wire Wire Line
-	3900 4500 4200 4500
-Connection ~ 4200 4500
-Wire Wire Line
 	3900 3700 4050 3700
 Wire Wire Line
 	3900 3800 3950 3800
-Wire Wire Line
-	3900 4300 4000 4300
-Wire Wire Line
-	3900 4400 3950 4400
 Wire Wire Line
 	3900 4850 4000 4850
@@
 Wire Wire Line
 	4000 4150 4000 4300
-Connection ~ 4000 4300
 Wire Wire Line
 	3350 4100 3350 4200
@@
 Wire Wire Line
 	3950 4200 3950 4400
-Connection ~ 3950 4400
 Wire Wire Line
 	3550 4650 3550 4750
@@
 	4050 5150 4050 5300
 Wire Wire Line
-	4200 4500 4200 5050
-Wire Wire Line
 	6600 2400 6600 3250
 Wire Wire Line
@@
 Wire Wire Line
 	3900 5050 4200 5050
+Wire Wire Line
+	4200 3250 4200 5050
+$Comp
+L Connector:TestPoint TP?
+U 1 1 5CBD2553
+P 3900 4300
+F 0 "TP?" H 3900 4600 50  0000 C BNN
+F 1 "TEST" H 3900 4550 50  0000 C CNN
+F 2 "Measurement_Points:Measurement_Point_Round-SMD-Pad_Small" H 3900 4300 50  0001 C CNN
+F 3 "" H 3900 4300 50  0001 C CNN
+	1    3900 4300
+	0    -1   -1   0
+$EndComp
+$Comp
+L Connector:TestPoint TP?
+U 1 1 5CBD25D5
+P 3900 4400
+F 0 "TP?" H 3900 4700 50  0000 C BNN
+F 1 "TEST" H 3900 4650 50  0000 C CNN
+F 2 "Measurement_Points:Measurement_Point_Round-SMD-Pad_Small" H 3900 4400 50  0001 C CNN
+F 3 "" H 3900 4400 50  0001 C CNN
+	1    3900 4400
+	0    -1   -1   0
+$EndComp
+Wire Wire Line
+	3900 4400 3950 4400
+Connection ~ 3950 4400
+Wire Wire Line
+	3900 4300 4000 4300
+Connection ~ 4000 4300
 $EndSCHEMATC
