File: Hardware/POWER.sch (KiCad schematic (older format))
At the start: 20 parts, among them U13 TS30013-M050QFNR, U14 TS30013-M050QFNR, U15 MCP1826S-3302E/DB

Commit message: Fixed some BOM stuff
fixed BOM for non RLC components
Parts:
- removed BATT1: SPOX-2, symbol SPOX-2
- removed TP?: TEST, symbol TEST
- added J15: SPOX-2, symbol SPOX-2
- added J16: CONN_02X05, symbol CONN_02X05
- added Q1: Q_PMOS_DGS, symbol Q_PMOS_DGS
- added R43, R44, R45, R46: 0, symbol R
- D15: renamed from D?; part_num (none) -> DIOD-001
- D16: renamed from D?; part_num (none) -> DIOD-003
- U37: renamed from U13; part_num (none) -> REGU-001
- U38: renamed from U14; part_num (none) -> REGU-001
- U39: renamed from U15; Digikey # MCP1826S-3302E/DB-ND -> (none); part_num (none) -> REGU-002
- gave numbers to parts that had none: 1
Connections:
- net labels added: 3V3_JMP, 5V_EXT_JMP, 5V_INT_JMP, VBATT_JMP
- wire segments 100 -> 85
Other:
- note removed: "TODO: add\nprotection circuit"
- moved on the sheet: C5, C6, C7, C8

Commit message: Finished RLC bom stuff
Parts:
- C1, C2: part_num (none) -> CAPP-001
- C10: value 0.1uF -> 100nF; part_num (none) -> CAPP-005
- C3, C4: part_num (none) -> CAPP-002
- C5, C6, C7, C8: part_num (none) -> CAPP-003
- C9: part_num (none) -> CAPP-004
- L1, L2: part_num (none) -> INDU-001
- R43, R44, R45, R46: part_num (none) -> RESS-001
- R47: part_num (none) -> RESS-006
- renumbered U37 to U13, U38 to U14, U39 to U15
Changed lines of the file:
@@
 $EndDescr
 $Comp
-L MCP1826S-3302E/DB U39
+L MCP1826S-3302E/DB U15
 U 1 1 59180881
 P 8050 4850
-F 0 "U39" H 8000 5250 60  0000 C CNN
+F 0 "U15" H 8000 5250 60  0000 C CNN
 F 1 "MCP1826S-3302E/DB" H 8050 4400 60  0000 C CNN
 F 2 "" H 8050 4850 60  0001 C CNN
@@
 F 2 "" H 5850 2050 50  0000 C CNN
 F 3 "" H 5850 2050 50  0000 C CNN
+F 4 "INDU-001" V 5850 2050 60  0001 C CNN "part_num"
 	1    5850 2050
 	0    -1   -1   0
@@
 F 2 "" H 6638 2100 50  0000 C CNN
 F 3 "" H 6600 2250 50  0000 C CNN
+F 4 "CAPP-003" H 6600 2250 60  0001 C CNN "part_num"
 	1    6600 2250
 	1    0    0    -1
@@
 F 2 "" H 3988 2350 50  0000 C CNN
 F 3 "" H 3950 2500 50  0000 C CNN
+F 4 "CAPP-001" H 3950 2500 60  0001 C CNN "part_num"
 	1    3950 2500
 	1    0    0    -1
@@
 5V External Reg
 $Comp
-L TS30013-M050QFNR U37
+L TS30013-M050QFNR U13
 U 1 1 591820DA
 P 4700 2300
-F 0 "U37" H 4650 3250 60  0000 C CNN
+F 0 "U13" H 4650 3250 60  0000 C CNN
 F 1 "TS30013-M050QFNR" H 4700 1700 60  0000 C CNN
 F 2 "" H 4850 2300 60  0001 C CNN
@@
 F 2 "" H 5588 1600 50  0000 C CNN
 F 3 "" H 5550 1750 50  0000 C CNN
+F 4 "CAPP-002" H 5550 1750 60  0001 C CNN "part_num"
 	1    5550 1750
-	1    0    0    -1
-$EndComp
-$Comp
-L C C7
-U 1 1 591829F4
-P 6850 2250
-F 0 "C7" H 6875 2350 50  0000 L CNN
-F 1 "22uF" H 6875 2150 50  0000 L CNN
-F 2 "" H 6888 2100 50  0000 C CNN
-F 3 "" H 6850 2250 50  0000 C CNN
-	1    6850 2250
 	1    0    0    -1
 $EndComp
@@
 F 2 "" H 5850 4700 50  0000 C CNN
 F 3 "" H 5850 4700 50  0000 C CNN
+F 4 "INDU-001" V 5850 4700 60  0001 C CNN "part_num"
 	1    5850 4700
 	0    -1   -1   0
-$EndComp
-$Comp
-L C C6
-U 1 1 59184627
-P 6650 4900
-F 0 "C6" H 6675 5000 50  0000 L CNN
-F 1 "22uF" H 6675 4800 50  0000 L CNN
-F 2 "" H 6688 4750 50  0000 C CNN
-F 3 "" H 6650 4900 50  0000 C CNN
-	1    6650 4900
-	1    0    0    -1
 $EndComp
 $Comp
@@
 F 2 "" H 3988 5000 50  0000 C CNN
 F 3 "" H 3950 5150 50  0000 C CNN
+F 4 "CAPP-001" H 3950 5150 60  0001 C CNN "part_num"
 	1    3950 5150
 	1    0    0    -1
@@
 5V Internal Reg
 $Comp
-L TS30013-M050QFNR U38
+L TS30013-M050QFNR U14
 U 1 1 5918463C
 P 4700 4950
-F 0 "U38" H 4650 5900 60  0000 C CNN
+F 0 "U14" H 4650 5900 60  0000 C CNN
 F 1 "TS30013-M050QFNR" H 4700 4350 60  0000 C CNN
 F 2 "" H 4850 4950 60  0001 C CNN
@@
 F 2 "" H 5588 4250 50  0000 C CNN
 F 3 "" H 5550 4400 50  0000 C CNN
+F 4 "CAPP-002" H 5550 4400 60  0001 C CNN "part_num"
 	1    5550 4400
-	1    0    0    -1
-$EndComp
-$Comp
-L C C8
-U 1 1 59184650
-P 6900 4900
-F 0 "C8" H 6925 5000 50  0000 L CNN
-F 1 "22uF" H 6925 4800 50  0000 L CNN
-F 2 "" H 6938 4750 50  0000 C CNN
-F 3 "" H 6900 4900 50  0000 C CNN
-	1    6900 4900
 	1    0    0    -1
 $EndComp
@@
 F 2 "" H 8688 4750 50  0000 C CNN
 F 3 "" H 8650 4900 50  0000 C CNN
+F 4 "CAPP-004" H 8650 4900 60  0001 C CNN "part_num"
 	1    8650 4900
 	1    0    0    -1
@@
 P 8850 4900
 F 0 "C10" H 8875 5000 50  0000 L CNN
-F 1 "0.1uF" H 8875 4800 50  0000 L CNN
+F 1 "100nF" H 8875 4800 50  0000 L CNN
 F 2 "" H 8888 4750 50  0000 C CNN
 F 3 "" H 8850 4900 50  0000 C CNN
+F 4 "CAPP-005" H 8850 4900 60  0001 C CNN "part_num"
 	1    8850 4900
 	1    0    0    -1
@@
 F 2 "" V 9130 4950 50  0001 C CNN
 F 3 "" H 9200 4950 50  0001 C CNN
+F 4 "RESS-006" V 9200 4950 60  0001 C CNN "part_num"
 	1    9200 4950
 	1    0    0    -1
@@
 F 2 "" V 5930 2250 50  0001 C CNN
 F 3 "" H 6000 2250 50  0001 C CNN
+F 4 "RESS-001" V 6000 2250 60  0001 C CNN "part_num"
 	1    6000 2250
 	0    1    1    0
@@
 F 2 "" V 5730 2550 50  0001 C CNN
 F 3 "" H 5800 2550 50  0001 C CNN
+F 4 "RESS-001" V 5800 2550 60  0001 C CNN "part_num"
 	1    5800 2550
 	-1   0    0    1
@@
 F 2 "" V 6130 4900 50  0001 C CNN
 F 3 "" H 6200 4900 50  0001 C CNN
+F 4 "RESS-001" V 6200 4900 60  0001 C CNN "part_num"
 	1    6200 4900
 	0    1    1    0
@@
 F 2 "" V 5880 5200 50  0001 C CNN
 F 3 "" H 5950 5200 50  0001 C CNN
+F 4 "RESS-001" V 5950 5200 60  0001 C CNN "part_num"
 	1    5950 5200
 	-1   0    0    1
@@
 	1    0    0    -1
 $EndComp
+$Comp
+L C C7
+U 1 1 595A1C8B
+P 6850 2250
+F 0 "C7" H 6875 2350 50  0000 L CNN
+F 1 "22uF" H 6875 2150 50  0000 L CNN
+F 2 "" H 6888 2100 50  0000 C CNN
+F 3 "" H 6850 2250 50  0000 C CNN
+F 4 "CAPP-003" H 6850 2250 60  0001 C CNN "part_num"
+	1    6850 2250
+	1    0    0    -1
+$EndComp
+$Comp
+L C C6
+U 1 1 595A1CD1
+P 6650 4900
+F 0 "C6" H 6675 5000 50  0000 L CNN
+F 1 "22uF" H 6675 4800 50  0000 L CNN
+F 2 "" H 6688 4750 50  0000 C CNN
+F 3 "" H 6650 4900 50  0000 C CNN
+F 4 "CAPP-003" H 6650 4900 60  0001 C CNN "part_num"
+	1    6650 4900
+	1    0    0    -1
+$EndComp
+$Comp
+L C C8
+U 1 1 595A1D31
+P 6900 4900
+F 0 "C8" H 6925 5000 50  0000 L CNN
+F 1 "22uF" H 6925 4800 50  0000 L CNN
+F 2 "" H 6938 4750 50  0000 C CNN
+F 3 "" H 6900 4900 50  0000 C CNN
+F 4 "CAPP-003" H 6900 4900 60  0001 C CNN "part_num"
+	1    6900 4900
+	1    0    0    -1
+$EndComp

Commit message: Added ressistor footprint
Parts:
- C1, C10, C2, C3, C4, C5, C6, C7, C8, C9, R43, R44, R45, R46, R47: footprint (none) -> Resistors_SMD:R_0603_HandSoldering
Changed lines of the file:
@@
 F 0 "C5" H 6625 2350 50  0000 L CNN
 F 1 "22uF" H 6625 2150 50  0000 L CNN
-F 2 "" H 6638 2100 50  0000 C CNN
+F 2 "Resistors_SMD:R_0603_HandSoldering" H 6638 2100 50  0001 C CNN
 F 3 "" H 6600 2250 50  0000 C CNN
 F 4 "CAPP-003" H 6600 2250 60  0001 C CNN "part_num"
@@
 F 0 "C1" H 3975 2600 50  0000 L CNN
 F 1 "10uF" H 3975 2400 50  0000 L CNN
-F 2 "" H 3988 2350 50  0000 C CNN
+F 2 "Resistors_SMD:R_0603_HandSoldering" H 3988 2350 50  0001 C CNN
 F 3 "" H 3950 2500 50  0000 C CNN
 F 4 "CAPP-001" H 3950 2500 60  0001 C CNN "part_num"
@@
 F 0 "C3" H 5575 1850 50  0000 L CNN
 F 1 "22nF" H 5575 1650 50  0000 L CNN
-F 2 "" H 5588 1600 50  0000 C CNN
+F 2 "Resistors_SMD:R_0603_HandSoldering" H 5588 1600 50  0001 C CNN
 F 3 "" H 5550 1750 50  0000 C CNN
 F 4 "CAPP-002" H 5550 1750 60  0001 C CNN "part_num"
@@
 F 0 "C2" H 3975 5250 50  0000 L CNN
 F 1 "10uF" H 3975 5050 50  0000 L CNN
-F 2 "" H 3988 5000 50  0000 C CNN
+F 2 "Resistors_SMD:R_0603_HandSoldering" H 3988 5000 50  0001 C CNN
 F 3 "" H 3950 5150 50  0000 C CNN
 F 4 "CAPP-001" H 3950 5150 60  0001 C CNN "part_num"
@@
 F 0 "C4" H 5575 4500 50  0000 L CNN
 F 1 "22nF" H 5575 4300 50  0000 L CNN
-F 2 "" H 5588 4250 50  0000 C CNN
+F 2 "Resistors_SMD:R_0603_HandSoldering" H 5588 4250 50  0001 C CNN
 F 3 "" H 5550 4400 50  0000 C CNN
 F 4 "CAPP-002" H 5550 4400 60  0001 C CNN "part_num"
@@
 F 0 "C9" H 8675 5000 50  0000 L CNN
 F 1 "1uF" H 8675 4800 50  0000 L CNN
-F 2 "" H 8688 4750 50  0000 C CNN
+F 2 "Resistors_SMD:R_0603_HandSoldering" H 8688 4750 50  0001 C CNN
 F 3 "" H 8650 4900 50  0000 C CNN
 F 4 "CAPP-004" H 8650 4900 60  0001 C CNN "part_num"
@@
 F 0 "C10" H 8875 5000 50  0000 L CNN
 F 1 "100nF" H 8875 4800 50  0000 L CNN
-F 2 "" H 8888 4750 50  0000 C CNN
+F 2 "Resistors_SMD:R_0603_HandSoldering" H 8888 4750 50  0001 C CNN
 F 3 "" H 8850 4900 50  0000 C CNN
 F 4 "CAPP-005" H 8850 4900 60  0001 C CNN "part_num"
@@
 F 0 "R47" V 9280 4950 50  0000 C CNN
 F 1 "100" V 9200 4950 50  0000 C CNN
-F 2 "" V 9130 4950 50  0001 C CNN
+F 2 "Resistors_SMD:R_0603_HandSoldering" V 9130 4950 50  0001 C CNN
 F 3 "" H 9200 4950 50  0001 C CNN
 F 4 "RESS-006" V 9200 4950 60  0001 C CNN "part_num"
@@
 F 0 "R45" V 6080 2250 50  0000 C CNN
 F 1 "0" V 6000 2250 50  0000 C CNN
-F 2 "" V 5930 2250 50  0001 C CNN
+F 2 "Resistors_SMD:R_0603_HandSoldering" V 5930 2250 50  0001 C CNN
 F 3 "" H 6000 2250 50  0001 C CNN
 F 4 "RESS-001" V 6000 2250 60  0001 C CNN "part_num"
@@
 F 0 "R43" V 5880 2550 50  0000 C CNN
 F 1 "0" V 5800 2550 50  0000 C CNN
-F 2 "" V 5730 2550 50  0001 C CNN
+F 2 "Resistors_SMD:R_0603_HandSoldering" V 5730 2550 50  0001 C CNN
 F 3 "" H 5800 2550 50  0001 C CNN
 F 4 "RESS-001" V 5800 2550 60  0001 C CNN "part_num"
@@
 F 0 "R46" V 6280 4900 50  0000 C CNN
 F 1 "0" V 6200 4900 50  0000 C CNN
-F 2 "" V 6130 4900 50  0001 C CNN
+F 2 "Resistors_SMD:R_0603_HandSoldering" V 6130 4900 50  0001 C CNN
 F 3 "" H 6200 4900 50  0001 C CNN
 F 4 "RESS-001" V 6200 4900 60  0001 C CNN "part_num"
@@
 F 0 "R44" V 6030 5200 50  0000 C CNN
 F 1 "0" V 5950 5200 50  0000 C CNN
-F 2 "" V 5880 5200 50  0001 C CNN
+F 2 "Resistors_SMD:R_0603_HandSoldering" V 5880 5200 50  0001 C CNN
 F 3 "" H 5950 5200 50  0001 C CNN
 F 4 "RESS-001" V 5950 5200 60  0001 C CNN "part_num"
@@
 F 0 "C7" H 6875 2350 50  0000 L CNN
 F 1 "22uF" H 6875 2150 50  0000 L CNN
-F 2 "" H 6888 2100 50  0000 C CNN
+F 2 "Resistors_SMD:R_0603_HandSoldering" H 6888 2100 50  0001 C CNN
 F 3 "" H 6850 2250 50  0000 C CNN
 F 4 "CAPP-003" H 6850 2250 60  0001 C CNN "part_num"
@@
 F 0 "C6" H 6675 5000 50  0000 L CNN
 F 1 "22uF" H 6675 4800 50  0000 L CNN
-F 2 "" H 6688 4750 50  0000 C CNN
+F 2 "Resistors_SMD:R_0603_HandSoldering" H 6688 4750 50  0001 C CNN
 F 3 "" H 6650 4900 50  0000 C CNN
 F 4 "CAPP-003" H 6650 4900 60  0001 C CNN "part_num"
@@
 F 0 "C8" H 6925 5000 50  0000 L CNN
 F 1 "22uF" H 6925 4800 50  0000 L CNN
-F 2 "" H 6938 4750 50  0000 C CNN
+F 2 "Resistors_SMD:R_0603_HandSoldering" H 6938 4750 50  0001 C CNN
 F 3 "" H 6900 4900 50  0000 C CNN
 F 4 "CAPP-003" H 6900 4900 60  0001 C CNN "part_num"

Commit message: PCB?!
Added initial PCB file with ratsnest. footprint library still needs to
be setup.
Parts:
- D16: footprint (none) -> LEDs:LED_0603
- J15: footprint (none) -> Connectors_Molex:Molex_SPOX-5267_22-03-5025_02x2.54mm_Straight
- J16: footprint (none) -> Pin_Headers:Pin_Header_Straight_2x05_Pitch2.54mm
- Q1: footprint (none) -> TO_SOT_Packages_SMD:TSOT-23-6_MK06A_HandSoldering
- U13, U14: footprint (none) -> Housings_DFN_QFN:QFN-16-1EP_3x3mm_Pitch0.5mm; part_num REGU-001 -> (none)
- U15: footprint (none) -> TO_SOT_Packages_SMD:SOT-223
- renumbered R43 to R67, R44 to R68, R45 to R69, R46 to R70, R47 to R71
Changed lines of the file:
@@
 $EndDescr
-$Comp
-L MCP1826S-3302E/DB U15
-U 1 1 59180881
-P 8050 4850
-F 0 "U15" H 8000 5250 60  0000 C CNN
-F 1 "MCP1826S-3302E/DB" H 8050 4400 60  0000 C CNN
-F 2 "" H 8050 4850 60  0001 C CNN
-F 3 "" H 8050 4850 60  0001 C CNN
-F 4 "REGU-002" H 8050 4850 60  0001 C CNN "part_num"
-	1    8050 4850
-	1    0    0    -1
-$EndComp
 $Comp
 L L L1
@@
 $EndComp
 $Comp
-L GND #PWR031
+L GND #PWR35
 U 1 1 59180DCE
 P 6600 2550
-F 0 "#PWR031" H 6600 2300 50  0001 C CNN
+F 0 "#PWR35" H 6600 2300 50  0001 C CNN
 F 1 "GND" H 6600 2400 50  0000 C CNN
 F 2 "" H 6600 2550 50  0000 C CNN
@@
 5V External Reg
 $Comp
-L TS30013-M050QFNR U13
-U 1 1 591820DA
-P 4700 2300
-F 0 "U13" H 4650 3250 60  0000 C CNN
-F 1 "TS30013-M050QFNR" H 4700 1700 60  0000 C CNN
-F 2 "" H 4850 2300 60  0001 C CNN
-F 3 "" H 4850 2300 60  0001 C CNN
-F 4 "REGU-001" H 4700 2300 60  0001 C CNN "part_num"
-	1    4700 2300
-	1    0    0    -1
-$EndComp
-$Comp
-L GND #PWR032
+L GND #PWR31
 U 1 1 59182319
 P 4700 3000
-F 0 "#PWR032" H 4700 2750 50  0001 C CNN
+F 0 "#PWR31" H 4700 2750 50  0001 C CNN
 F 1 "GND" H 4700 2850 50  0000 C CNN
 F 2 "" H 4700 3000 50  0000 C CNN
@@
 	1600 2800 2400 2800
 $Comp
-L GND #PWR033
+L GND #PWR30
 U 1 1 59183E68
 P 1150 3250
-F 0 "#PWR033" H 1150 3000 50  0001 C CNN
+F 0 "#PWR30" H 1150 3000 50  0001 C CNN
 F 1 "GND" H 1150 3100 50  0000 C CNN
 F 2 "" H 1150 3250 50  0000 C CNN
@@
 $EndComp
 $Comp
-L GND #PWR034
+L GND #PWR36
 U 1 1 5918462E
 P 6650 5200
-F 0 "#PWR034" H 6650 4950 50  0001 C CNN
+F 0 "#PWR36" H 6650 4950 50  0001 C CNN
 F 1 "GND" H 6650 5050 50  0000 C CNN
 F 2 "" H 6650 5200 50  0000 C CNN
@@
 5V Internal Reg
 $Comp
-L TS30013-M050QFNR U14
-U 1 1 5918463C
-P 4700 4950
-F 0 "U14" H 4650 5900 60  0000 C CNN
-F 1 "TS30013-M050QFNR" H 4700 4350 60  0000 C CNN
-F 2 "" H 4850 4950 60  0001 C CNN
-F 3 "" H 4850 4950 60  0001 C CNN
-F 4 "REGU-001" H 4700 4950 60  0001 C CNN "part_num"
-	1    4700 4950
-	1    0    0    -1
-$EndComp
-$Comp
-L GND #PWR035
+L GND #PWR32
 U 1 1 59184643
 P 4700 5650
-F 0 "#PWR035" H 4700 5400 50  0001 C CNN
+F 0 "#PWR32" H 4700 5400 50  0001 C CNN
 F 1 "GND" H 4700 5500 50  0000 C CNN
 F 2 "" H 4700 5650 50  0000 C CNN
@@
 	7450 5000 7550 5000
 $Comp
-L GND #PWR036
+L GND #PWR37
 U 1 1 591852CA
 P 7450 5150
-F 0 "#PWR036" H 7450 4900 50  0001 C CNN
+F 0 "#PWR37" H 7450 4900 50  0001 C CNN
 F 1 "GND" H 7450 5000 50  0000 C CNN
 F 2 "" H 7450 5150 50  0000 C CNN
@@
 	8650 4700 8650 4750
 $Comp
-L GND #PWR037
+L GND #PWR38
 U 1 1 59185849
 P 8650 5150
-F 0 "#PWR037" H 8650 4900 50  0001 C CNN
+F 0 "#PWR38" H 8650 4900 50  0001 C CNN
 F 1 "GND" H 8650 5000 50  0000 C CNN
 F 2 "" H 8650 5150 50  0000 C CNN
@@
 F 0 "D16" H 9200 5350 50  0000 C CNN
 F 1 "PWR_LED" H 9200 5150 50  0000 C CNN
-F 2 "" H 9200 5250 50  0001 C CNN
+F 2 "LEDs:LED_0603" H 9200 5250 50  0001 C CNN
 F 3 "" H 9200 5250 50  0001 C CNN
 F 4 "DIOD-003" H 9200 5250 60  0001 C CNN "part_num"
@@
 $EndComp
 $Comp
-L R R47
+L R R71
 U 1 1 592C1353
 P 9200 4950
-F 0 "R47" V 9280 4950 50  0000 C CNN
+F 0 "R71" V 9280 4950 50  0000 C CNN
 F 1 "100" V 9200 4950 50  0000 C CNN
 F 2 "Resistors_SMD:R_0603_HandSoldering" V 9130 4950 50  0001 C CNN
@@
 	9200 4700 9200 4800
 $Comp
-L GND #PWR038
+L GND #PWR40
 U 1 1 592C1537
 P 9200 5400
-F 0 "#PWR038" H 9200 5150 50  0001 C CNN
+F 0 "#PWR40" H 9200 5150 50  0001 C CNN
 F 1 "GND" H 9200 5250 50  0000 C CNN
 F 2 "" H 9200 5400 50  0000 C CNN
@@
 F 0 "Q1" H 1600 2950 50  0000 L CNN
 F 1 "Q_PMOS_DGS" H 1600 2850 50  0000 L CNN
-F 2 "" H 1600 3000 50  0001 C CNN
+F 2 "TO_SOT_Packages_SMD:TSOT-23-6_MK06A_HandSoldering" H 1600 3000 50  0001 C CNN
 F 3 "" H 1400 2900 50  0001 C CNN
 F 4 "TRAN-001" H 1400 2900 60  0001 C CNN "part_num"
@@
 	1400 3200 1400 3100
 $Comp
-L PWR_FLAG #FLG039
+L PWR_FLAG #FLG2
 U 1 1 594F4062
 P 1850 2750
-F 0 "#FLG039" H 1850 2825 50  0001 C CNN
+F 0 "#FLG2" H 1850 2825 50  0001 C CNN
 F 1 "PWR_FLAG" H 1850 2900 50  0000 C CNN
 F 2 "" H 1850 2750 50  0001 C CNN
@@
 Connection ~ 1850 2800
 $Comp
-L R R45
+L R R69
 U 1 1 595015EF
 P 6000 2250
-F 0 "R45" V 6080 2250 50  0000 C CNN
+F 0 "R69" V 6080 2250 50  0000 C CNN
 F 1 "0" V 6000 2250 50  0000 C CNN
 F 2 "Resistors_SMD:R_0603_HandSoldering" V 5930 2250 50  0001 C CNN
@@
 Connection ~ 5800 2250
 $Comp
-L R R43
+L R R67
 U 1 1 5950186D
 P 5800 2550
-F 0 "R43" V 5880 2550 50  0000 C CNN
+F 0 "R67" V 5880 2550 50  0000 C CNN
 F 1 "0" V 5800 2550 50  0000 C CNN
 F 2 "Resistors_SMD:R_0603_HandSoldering" V 5730 2550 50  0001 C CNN
@@
 $EndComp
 $Comp
-L GND #PWR040
+L GND #PWR33
 U 1 1 595018DF
 P 5800 2800
-F 0 "#PWR040" H 5800 2550 50  0001 C CNN
+F 0 "#PWR33" H 5800 2550 50  0001 C CNN
 F 1 "GND" H 5800 2650 50  0000 C CNN
 F 2 "" H 5800 2800 50  0000 C CNN
@@
 Connection ~ 6200 2050
 $Comp
-L R R46
+L R R70
 U 1 1 595024E6
 P 6200 4900
-F 0 "R46" V 6280 4900 50  0000 C CNN
+F 0 "R70" V 6280 4900 50  0000 C CNN
 F 1 "0" V 6200 4900 50  0000 C CNN
 F 2 "Resistors_SMD:R_0603_HandSoldering" V 6130 4900 50  0001 C CNN
@@
 $EndComp
 $Comp
-L R R44
+L R R68
 U 1 1 59502557
 P 5950 5200
-F 0 "R44" V 6030 5200 50  0000 C CNN
+F 0 "R68" V 6030 5200 50  0000 C CNN
 F 1 "0" V 5950 5200 50  0000 C CNN
 F 2 "Resistors_SMD:R_0603_HandSoldering" V 5880 5200 50  0001 C CNN
@@
 $EndComp
 $Comp
-L GND #PWR041
+L GND #PWR34
 U 1 1 595025C5
 P 5950 5500
-F 0 "#PWR041" H 5950 5250 50  0001 C CNN
+F 0 "#PWR34" H 5950 5250 50  0001 C CNN
 F 1 "GND" H 5950 5350 50  0000 C CNN
 F 2 "" H 5950 5500 50  0000 C CNN
@@
 F 0 "J16" H 9200 2750 50  0000 C CNN
 F 1 "CONN_02X05" H 9200 2150 50  0000 C CNN
-F 2 "" H 9200 1250 50  0001 C CNN
+F 2 "Pin_Headers:Pin_Header_Straight_2x05_Pitch2.54mm" H 9200 1250 50  0001 C CNN
 F 3 "" H 9200 1250 50  0001 C CNN
 F 4 "CONN-010" H 9200 2450 60  0001 C CNN "part_num"
@@
 	9550 2650 9450 2650
 $Comp
-L GND #PWR042
+L GND #PWR39
 U 1 1 595132A0
 P 9200 2900
-F 0 "#PWR042" H 9200 2650 50  0001 C CNN
+F 0 "#PWR39" H 9200 2650 50  0001 C CNN
 F 1 "GND" H 9200 2750 50  0000 C CNN
 F 2 "" H 9200 2900 50  0000 C CNN
@@
 	1150 3250 1150 3200
 Connection ~ 1150 3200
-$Comp
-L SPOX-2 J15
-U 1 1 5955D6CC
-P 750 2850
-F 0 "J15" H 850 3000 60  0000 C CNN
-F 1 "SPOX-2" H 850 2700 60  0000 C CNN
-F 2 "" H 750 2800 60  0001 C CNN
-F 3 "" H 750 2800 60  0001 C CNN
-F 4 "CONN-001" H 950 3100 60  0001 C CNN "part_num"
-	1    750  2850
-	1    0    0    -1
-$EndComp
 $Comp
 L C C7
@@
 	1    0    0    -1
 $EndComp
+$Comp
+L SPOX-2 J15
+U 1 1 595BCAC3
+P 750 2850
+F 0 "J15" H 850 3000 60  0000 C CNN
+F 1 "SPOX-2" H 850 2700 60  0000 C CNN
+F 2 "Connectors_Molex:Molex_SPOX-5267_22-03-5025_02x2.54mm_Straight" H 750 2800 60  0001 C CNN
+F 3 "" H 750 2800 60  0001 C CNN
+F 4 "CONN-001" H 950 3100 60  0001 C CNN "part_num"
+	1    750  2850
+	1    0    0    -1
+$EndComp
+$Comp
+L TS30013-M050QFNR U13
+U 1 1 595F6A2F
+P 4700 2300
+F 0 "U13" H 4650 3250 60  0000 C CNN
+F 1 "TS30013-M050QFNR" H 4700 1700 60  0000 C CNN
+F 2 "Housings_DFN_QFN:QFN-16-1EP_3x3mm_Pitch0.5mm" H 4850 2300 60  0001 C CNN
+F 3 "REGU-001" H 4850 2300 60  0001 C CNN
+	1    4700 2300
+	1    0    0    -1
+$EndComp
+$Comp
+L TS30013-M050QFNR U14
+U 1 1 595F6BE5
+P 4700 4950
+F 0 "U14" H 4650 5900 60  0000 C CNN
+F 1 "TS30013-M050QFNR" H 4700 4350 60  0000 C CNN
+F 2 "Housings_DFN_QFN:QFN-16-1EP_3x3mm_Pitch0.5mm" H 4850 4950 60  0001 C CNN
+F 3 "REGU-001" H 4850 4950 60  0001 C CNN
+	1    4700 4950
+	1    0    0    -1
+$EndComp
+$Comp
+L MCP1826S-3302E/DB U15
+U 1 1 595F71A4
+P 8050 4850
+F 0 "U15" H 8000 5250 60  0000 C CNN
+F 1 "MCP1826S-3302E/DB" H 8050 4400 60  0000 C CNN
+F 2 "TO_SOT_Packages_SMD:SOT-223" H 7900 5150 60  0001 C CNN
+F 3 "" H 8000 5250 60  0001 C CNN
+F 4 "REGU-002" H 8100 5350 60  0001 C CNN "part_num"
+	1    8050 4850
+	1    0    0    -1
+$EndComp
