File: Hardware/POWER.sch (KiCad schematic (older format))
At the start: 25 parts, among them J15 SPOX-2, J16 CONN_02X05, Q1 Q_PMOS_DGS, U13 TS30013-M050QFNR, U14 TS30013-M050QFNR, U15 MCP1826S-3302E/DB

Commit message: Fixed serge suggestions
Parts:
- removed D15: D_Schottky, symbol D_Schottky
- added D21: D_Zener, symbol D_Zener
- added F1, F2: 3A, symbol Fuse
Connections:
- wire segments 85 -> 87
Changed lines of the file:
@@
 $Descr A4 11693 8268
 encoding utf-8
-Sheet 15 20
+Sheet 15 21
 Title ""
 Date ""
@@
 $EndComp
 $Comp
-L GND #PWR35
+L GND #PWR028
 U 1 1 59180DCE
 P 6600 2550
-F 0 "#PWR35" H 6600 2300 50  0001 C CNN
+F 0 "#PWR028" H 6600 2300 50  0001 C CNN
 F 1 "GND" H 6600 2400 50  0000 C CNN
 F 2 "" H 6600 2550 50  0000 C CNN
@@
 5V External Reg
 $Comp
-L GND #PWR31
+L GND #PWR029
 U 1 1 59182319
 P 4700 3000
-F 0 "#PWR31" H 4700 2750 50  0001 C CNN
+F 0 "#PWR029" H 4700 2750 50  0001 C CNN
 F 1 "GND" H 4700 2850 50  0000 C CNN
 F 2 "" H 4700 3000 50  0000 C CNN
@@
 Connection ~ 5550 2050
 Wire Wire Line
-	6000 2050 7050 2050
-Wire Wire Line
 	6600 2400 6600 2550
 Connection ~ 6600 2050
@@
 	1600 2800 2400 2800
 $Comp
-L GND #PWR30
+L GND #PWR030
 U 1 1 59183E68
 P 1150 3250
-F 0 "#PWR30" H 1150 3000 50  0001 C CNN
+F 0 "#PWR030" H 1150 3000 50  0001 C CNN
 F 1 "GND" H 1150 3100 50  0000 C CNN
 F 2 "" H 1150 3250 50  0000 C CNN
@@
 $EndComp
 $Comp
-L GND #PWR36
+L GND #PWR031
 U 1 1 5918462E
 P 6650 5200
-F 0 "#PWR36" H 6650 4950 50  0001 C CNN
+F 0 "#PWR031" H 6650 4950 50  0001 C CNN
 F 1 "GND" H 6650 5050 50  0000 C CNN
 F 2 "" H 6650 5200 50  0000 C CNN
@@
 5V Internal Reg
 $Comp
-L GND #PWR32
+L GND #PWR032
 U 1 1 59184643
 P 4700 5650
-F 0 "#PWR32" H 4700 5400 50  0001 C CNN
+F 0 "#PWR032" H 4700 5400 50  0001 C CNN
 F 1 "GND" H 4700 5500 50  0000 C CNN
 F 2 "" H 4700 5650 50  0000 C CNN
@@
 Connection ~ 5550 4700
 Wire Wire Line
-	6000 4700 7550 4700
-Wire Wire Line
 	6650 5050 6650 5200
 Wire Wire Line
@@
 5V_EXT
 Wire Wire Line
-	7550 4900 7450 4900
+	7650 4900 7450 4900
 Wire Wire Line
 	7450 4900 7450 5150
 Wire Wire Line
-	7450 5000 7550 5000
-$Comp
-L GND #PWR37
+	7450 5000 7650 5000
+$Comp
+L GND #PWR033
 U 1 1 591852CA
 P 7450 5150
-F 0 "#PWR37" H 7450 4900 50  0001 C CNN
+F 0 "#PWR033" H 7450 4900 50  0001 C CNN
 F 1 "GND" H 7450 5000 50  0000 C CNN
 F 2 "" H 7450 5150 50  0000 C CNN
@@
 $EndComp
 Wire Wire Line
-	8450 4700 9200 4700
+	8550 4700 9200 4700
 Wire Wire Line
 	8650 4700 8650 4750
 $Comp
-L GND #PWR38
+L GND #PWR034
 U 1 1 59185849
 P 8650 5150
-F 0 "#PWR38" H 8650 4900 50  0001 C CNN
+F 0 "#PWR034" H 8650 4900 50  0001 C CNN
 F 1 "GND" H 8650 5000 50  0000 C CNN
 F 2 "" H 8650 5150 50  0000 C CNN
@@
 VBATT
 Wire Wire Line
-	7350 2050 7850 2050
-Wire Wire Line
 	6600 2050 6600 2100
-$Comp
-L D_Schottky D15
-U 1 1 592A4A96
-P 7200 2050
-F 0 "D15" H 7200 2150 50  0000 C CNN
-F 1 "D_Schottky" H 7200 1950 50  0000 C CNN
-F 2 "" H 7200 2050 50  0001 C CNN
-F 3 "" H 7200 2050 50  0001 C CNN
-F 4 "DIOD-001" H 7200 2050 60  0001 C CNN "part_num"
-	1    7200 2050
-	-1   0    0    1
-$EndComp
 $Comp
 L LED D16
@@
 	9200 4700 9200 4800
 $Comp
-L GND #PWR40
+L GND #PWR035
 U 1 1 592C1537
 P 9200 5400
-F 0 "#PWR40" H 9200 5150 50  0001 C CNN
+F 0 "#PWR035" H 9200 5150 50  0001 C CNN
 F 1 "GND" H 9200 5250 50  0000 C CNN
 F 2 "" H 9200 5400 50  0000 C CNN
@@
 	1400 3200 1400 3100
 $Comp
-L PWR_FLAG #FLG2
+L PWR_FLAG #FLG036
 U 1 1 594F4062
 P 1850 2750
-F 0 "#FLG2" H 1850 2825 50  0001 C CNN
+F 0 "#FLG036" H 1850 2825 50  0001 C CNN
 F 1 "PWR_FLAG" H 1850 2900 50  0000 C CNN
 F 2 "" H 1850 2750 50  0001 C CNN
@@
 $EndComp
 $Comp
-L GND #PWR33
+L GND #PWR037
 U 1 1 595018DF
 P 5800 2800
-F 0 "#PWR33" H 5800 2550 50  0001 C CNN
+F 0 "#PWR037" H 5800 2550 50  0001 C CNN
 F 1 "GND" H 5800 2650 50  0000 C CNN
 F 2 "" H 5800 2800 50  0000 C CNN
@@
 $EndComp
 $Comp
-L GND #PWR34
+L GND #PWR038
 U 1 1 595025C5
 P 5950 5500
-F 0 "#PWR34" H 5950 5250 50  0001 C CNN
+F 0 "#PWR038" H 5950 5250 50  0001 C CNN
 F 1 "GND" H 5950 5350 50  0000 C CNN
 F 2 "" H 5950 5500 50  0000 C CNN
@@
 Wire Wire Line
 	9800 2350 9450 2350
-Text Label 7350 2050 0    59   ~ 0
+Text Label 7500 2050 0    59   ~ 0
 5V_EXT_JMP
 Text Label 9500 2350 0    59   ~ 0
@@
 Text Label 8950 2450 2    59   ~ 0
 5V_INT_JMP
-Text Label 7200 4700 2    59   ~ 0
+Text Label 7300 4700 0    59   ~ 0
 5V_INT_JMP
 Wire Wire Line
@@
 	9550 2650 9450 2650
 $Comp
-L GND #PWR39
+L GND #PWR039
 U 1 1 595132A0
 P 9200 2900
-F 0 "#PWR39" H 9200 2650 50  0001 C CNN
+F 0 "#PWR039" H 9200 2650 50  0001 C CNN
 F 1 "GND" H 9200 2750 50  0000 C CNN
 F 2 "" H 9200 2900 50  0000 C CNN
@@
 L MCP1826S-3302E/DB U15
 U 1 1 595F71A4
-P 8050 4850
-F 0 "U15" H 8000 5250 60  0000 C CNN
-F 1 "MCP1826S-3302E/DB" H 8050 4400 60  0000 C CNN
-F 2 "TO_SOT_Packages_SMD:SOT-223" H 7900 5150 60  0001 C CNN
-F 3 "" H 8000 5250 60  0001 C CNN
-F 4 "REGU-002" H 8100 5350 60  0001 C CNN "part_num"
-	1    8050 4850
-	1    0    0    -1
-$EndComp
+P 8150 4850
+F 0 "U15" H 8100 5250 60  0000 C CNN
+F 1 "MCP1826S-3302E/DB" H 8150 4400 60  0000 C CNN
+F 2 "TO_SOT_Packages_SMD:SOT-223" H 8000 5150 60  0001 C CNN
+F 3 "" H 8100 5250 60  0001 C CNN
+F 4 "REGU-002" H 8200 5350 60  0001 C CNN "part_num"
+	1    8150 4850
+	1    0    0    -1
+$EndComp
+$Comp
+L D_Zener D21
+U 1 1 5962B2F8
+P 7700 2350
+F 0 "D21" H 7700 2450 50  0000 C CNN
+F 1 "D_Zener" H 7700 2250 50  0000 C CNN
+F 2 "" H 7700 2350 50  0001 C CNN
+F 3 "" H 7700 2350 50  0001 C CNN
+F 4 "DIOD-001" H 7700 2350 60  0001 C CNN "part_num"
+	1    7700 2350
+	0    1    1    0
+$EndComp
+Wire Wire Line
+	7700 2200 7700 2050
+Connection ~ 7700 2050
+$Comp
+L GND #PWR040
+U 1 1 5962B870
+P 7700 2500
+F 0 "#PWR040" H 7700 2250 50  0001 C CNN
+F 1 "GND" H 7700 2350 50  0000 C CNN
+F 2 "" H 7700 2500 50  0001 C CNN
+F 3 "" H 7700 2500 50  0001 C CNN
+	1    7700 2500
+	1    0    0    -1
+$EndComp
+$Comp
+L Fuse F2
+U 1 1 59684814
+P 7200 2050
+F 0 "F2" V 7280 2050 50  0000 C CNN
+F 1 "3A" V 7125 2050 50  0000 C CNN
+F 2 "" V 7130 2050 50  0001 C CNN
+F 3 "" H 7200 2050 50  0001 C CNN
+F 4 "FUSE-001" V 7200 2050 60  0001 C CNN "part_num"
+	1    7200 2050
+	0    1    1    0
+$EndComp
+Wire Wire Line
+	6000 2050 7050 2050
+$Comp
+L Fuse F1
+U 1 1 59684AE1
+P 7100 4700
+F 0 "F1" V 7180 4700 50  0000 C CNN
+F 1 "3A" V 7025 4700 50  0000 C CNN
+F 2 "" V 7030 4700 50  0001 C CNN
+F 3 "" H 7100 4700 50  0001 C CNN
+F 4 "FUSE-001" V 7100 4700 60  0001 C CNN "part_num"
+	1    7100 4700
+	0    1    1    0
+$EndComp
+Wire Wire Line
+	7700 2050 7350 2050
+Wire Wire Line
+	6000 4700 6950 4700
+Wire Wire Line
+	7250 4700 7650 4700
 $EndSCHEMATC

Commit message: commit before my computer restarts
Parts:
- D13: renamed from D21; footprint (none) -> Diodes_SMD:D_SOD-123
- F1, F2: footprint (none) -> Resistors_SMD:R_0603_HandSoldering
- L1, L2: footprint (none) -> WARG:5.1x6.5
- Q1: footprint TO_SOT_Packages_SMD:TSOT-23-6_MK06A_HandSoldering -> WARG:TSOT-23-6_MK06A_HandSoldering
- renumbered D16 to D14, J15 to J14, J16 to J15, R67 to R25, R68 to R26, R69 to R27, R70 to R28, R71 to R29
Connections:
- wire segments 87 -> 89
Changed lines of the file:
@@
 F 0 "L1" V 5800 2050 50  0000 C CNN
 F 1 "4.7 uH" V 5925 2050 50  0000 C CNN
-F 2 "" H 5850 2050 50  0000 C CNN
+F 2 "WARG:5.1x6.5" H 5850 2050 50  0001 C CNN
 F 3 "" H 5850 2050 50  0000 C CNN
 F 4 "INDU-001" V 5850 2050 60  0001 C CNN "part_num"
@@
 	4550 2800 4550 2900
 Wire Wire Line
-	3950 2900 4800 2900
+	3950 2900 4900 2900
 Wire Wire Line
 	4800 2900 4800 2800
@@
 F 0 "L2" V 5800 4700 50  0000 C CNN
 F 1 "4.7 uH" V 5925 4700 50  0000 C CNN
-F 2 "" H 5850 4700 50  0000 C CNN
+F 2 "WARG:5.1x6.5" H 5850 4700 50  0001 C CNN
 F 3 "" H 5850 4700 50  0000 C CNN
 F 4 "INDU-001" V 5850 4700 60  0001 C CNN "part_num"
@@
 	4550 5450 4550 5550
 Wire Wire Line
-	3950 5550 4800 5550
+	3950 5550 4900 5550
 Wire Wire Line
 	4800 5550 4800 5450
@@
 	6600 2050 6600 2100
 $Comp
-L LED D16
+L LED D14
 U 1 1 592C12E2
 P 9200 5250
-F 0 "D16" H 9200 5350 50  0000 C CNN
+F 0 "D14" H 9200 5350 50  0000 C CNN
 F 1 "PWR_LED" H 9200 5150 50  0000 C CNN
 F 2 "LEDs:LED_0603" H 9200 5250 50  0001 C CNN
@@
 $EndComp
 $Comp
-L R R71
+L R R29
 U 1 1 592C1353
 P 9200 4950
-F 0 "R71" V 9280 4950 50  0000 C CNN
+F 0 "R29" V 9280 4950 50  0000 C CNN
 F 1 "100" V 9200 4950 50  0000 C CNN
 F 2 "Resistors_SMD:R_0603_HandSoldering" V 9130 4950 50  0001 C CNN
@@
 F 0 "Q1" H 1600 2950 50  0000 L CNN
 F 1 "Q_PMOS_DGS" H 1600 2850 50  0000 L CNN
-F 2 "TO_SOT_Packages_SMD:TSOT-23-6_MK06A_HandSoldering" H 1600 3000 50  0001 C CNN
+F 2 "WARG:TSOT-23-6_MK06A_HandSoldering" H 1600 3000 50  0001 C CNN
 F 3 "" H 1400 2900 50  0001 C CNN
 F 4 "TRAN-001" H 1400 2900 60  0001 C CNN "part_num"
@@
 Connection ~ 1850 2800
 $Comp
-L R R69
+L R R27
 U 1 1 595015EF
 P 6000 2250
-F 0 "R69" V 6080 2250 50  0000 C CNN
+F 0 "R27" V 6080 2250 50  0000 C CNN
 F 1 "0" V 6000 2250 50  0000 C CNN
 F 2 "Resistors_SMD:R_0603_HandSoldering" V 5930 2250 50  0001 C CNN
@@
 Connection ~ 5800 2250
 $Comp
-L R R67
+L R R25
 U 1 1 5950186D
 P 5800 2550
-F 0 "R67" V 5880 2550 50  0000 C CNN
+F 0 "R25" V 5880 2550 50  0000 C CNN
 F 1 "0" V 5800 2550 50  0000 C CNN
 F 2 "Resistors_SMD:R_0603_HandSoldering" V 5730 2550 50  0001 C CNN
@@
 Connection ~ 6200 2050
 $Comp
-L R R70
+L R R28
 U 1 1 595024E6
 P 6200 4900
-F 0 "R70" V 6280 4900 50  0000 C CNN
+F 0 "R28" V 6280 4900 50  0000 C CNN
 F 1 "0" V 6200 4900 50  0000 C CNN
 F 2 "Resistors_SMD:R_0603_HandSoldering" V 6130 4900 50  0001 C CNN
@@
 $EndComp
 $Comp
-L R R68
+L R R26
 U 1 1 59502557
 P 5950 5200
-F 0 "R68" V 6030 5200 50  0000 C CNN
+F 0 "R26" V 6030 5200 50  0000 C CNN
 F 1 "0" V 5950 5200 50  0000 C CNN
 F 2 "Resistors_SMD:R_0603_HandSoldering" V 5880 5200 50  0001 C CNN
@@
 Connection ~ 6850 2050
 $Comp
-L CONN_02X05 J16
+L CONN_02X05 J15
 U 1 1 59512411
 P 9200 2450
-F 0 "J16" H 9200 2750 50  0000 C CNN
+F 0 "J15" H 9200 2750 50  0000 C CNN
 F 1 "CONN_02X05" H 9200 2150 50  0000 C CNN
 F 2 "Pin_Headers:Pin_Header_Straight_2x05_Pitch2.54mm" H 9200 1250 50  0001 C CNN
@@
 $EndComp
 $Comp
-L SPOX-2 J15
+L SPOX-2 J14
 U 1 1 595BCAC3
 P 750 2850
-F 0 "J15" H 850 3000 60  0000 C CNN
+F 0 "J14" H 850 3000 60  0000 C CNN
 F 1 "SPOX-2" H 850 2700 60  0000 C CNN
 F 2 "Connectors_Molex:Molex_SPOX-5267_22-03-5025_02x2.54mm_Straight" H 750 2800 60  0001 C CNN
@@
 $EndComp
 $Comp
-L D_Zener D21
+L D_Zener D13
 U 1 1 5962B2F8
 P 7700 2350
-F 0 "D21" H 7700 2450 50  0000 C CNN
+F 0 "D13" H 7700 2450 50  0000 C CNN
 F 1 "D_Zener" H 7700 2250 50  0000 C CNN
-F 2 "" H 7700 2350 50  0001 C CNN
+F 2 "Diodes_SMD:D_SOD-123" H 7700 2350 50  0001 C CNN
 F 3 "" H 7700 2350 50  0001 C CNN
 F 4 "DIOD-001" H 7700 2350 60  0001 C CNN "part_num"
@@
 F 0 "F2" V 7280 2050 50  0000 C CNN
 F 1 "3A" V 7125 2050 50  0000 C CNN
-F 2 "" V 7130 2050 50  0001 C CNN
+F 2 "Resistors_SMD:R_0603_HandSoldering" V 7130 2050 50  0001 C CNN
 F 3 "" H 7200 2050 50  0001 C CNN
 F 4 "FUSE-001" V 7200 2050 60  0001 C CNN "part_num"
@@
 F 0 "F1" V 7180 4700 50  0000 C CNN
 F 1 "3A" V 7025 4700 50  0000 C CNN
-F 2 "" V 7030 4700 50  0001 C CNN
+F 2 "Resistors_SMD:R_0603_HandSoldering" V 7030 4700 50  0001 C CNN
 F 3 "" H 7100 4700 50  0001 C CNN
 F 4 "FUSE-001" V 7100 4700 60  0001 C CNN "part_num"
@@
 Wire Wire Line
 	7250 4700 7650 4700
+Wire Wire Line
+	4900 5550 4900 5450
+Connection ~ 4800 5550
+Wire Wire Line
+	4900 2900 4900 2800
+Connection ~ 4800 2900
 $EndSCHEMATC

Commit message: This power is HUGE
Made some big traces and pours for power. Need to do some ground layer
stiching to fix the ground plane still
Connections:
- net labels added: 5V_EXT_FB, 5V_EXT_OUT, 5V_EXT_PREFUSE, 5V_INT_FB, 5V_INT_OUT, 5V_INT_PREFUSE, BATT_IN
Changed lines of the file:
@@
 	4900 2900 4900 2800
 Connection ~ 4800 2900
+Text Label 950  2800 0    60   ~ 0
+BATT_IN
+Text Label 5350 2050 0    60   ~ 0
+5V_EXT_OUT
+Text Label 6200 2050 0    60   ~ 0
+5V_EXT_PREFUSE
+Text Label 5400 4700 0    60   ~ 0
+5V_INT_OUT
+Text Label 6150 4700 0    60   ~ 0
+5V_INT_PREFUSE
+Text Label 5500 4900 0    60   ~ 0
+5V_INT_FB
+Text Label 5300 2250 0    60   ~ 0
+5V_EXT_FB
 $EndSCHEMATC

Commit message: Restarted work
Removed OC and SEL busses. Still need to add clocks.
Parts:
- removed J14: SPOX-2, Connectors_Molex:Molex_SPOX-5267_22-03-5025_02x2.54mm_Straight, symbol SPOX-2
- removed U13, U14: TS30013-M050QFNR, Housings_DFN_QFN:QFN-16-1EP_3x3mm_Pitch0.5mm, symbol TS30013-M050QFNR
- added J?: SPOX-2, Connectors_Molex:Molex_SPOX-5267_22-03-5025_02x2.54mm_Straight, symbol SPOX-2
- added U? (x2): TS30013-M050QFNR, Housings_DFN_QFN:QFN-16-1EP_3x3mm_Pitch0.5mm, symbol TS30013-M050QFNR
Other:
- note added: "Power jumper\nUse to measure current and\ndebug power"
- note added: "Reverse polarity protection"
Changed lines of the file:
@@
 EESchema Schematic File Version 2
+LIBS:ZeroPilot-rescue
 LIBS:WARG
 LIBS:power
@@
 $Descr A4 11693 8268
 encoding utf-8
-Sheet 15 21
+Sheet 3 8
 Title ""
 Date ""
@@
 $EndComp
 $Comp
-L SPOX-2 J14
-U 1 1 595BCAC3
-P 750 2850
-F 0 "J14" H 850 3000 60  0000 C CNN
-F 1 "SPOX-2" H 850 2700 60  0000 C CNN
-F 2 "Connectors_Molex:Molex_SPOX-5267_22-03-5025_02x2.54mm_Straight" H 750 2800 60  0001 C CNN
-F 3 "" H 750 2800 60  0001 C CNN
-F 4 "CONN-001" H 950 3100 60  0001 C CNN "part_num"
-	1    750  2850
-	1    0    0    -1
-$EndComp
-$Comp
-L TS30013-M050QFNR U13
-U 1 1 595F6A2F
-P 4700 2300
-F 0 "U13" H 4650 3250 60  0000 C CNN
-F 1 "TS30013-M050QFNR" H 4700 1700 60  0000 C CNN
-F 2 "Housings_DFN_QFN:QFN-16-1EP_3x3mm_Pitch0.5mm" H 4850 2300 60  0001 C CNN
-F 3 "REGU-001" H 4850 2300 60  0001 C CNN
-	1    4700 2300
-	1    0    0    -1
-$EndComp
-$Comp
-L TS30013-M050QFNR U14
-U 1 1 595F6BE5
-P 4700 4950
-F 0 "U14" H 4650 5900 60  0000 C CNN
-F 1 "TS30013-M050QFNR" H 4700 4350 60  0000 C CNN
-F 2 "Housings_DFN_QFN:QFN-16-1EP_3x3mm_Pitch0.5mm" H 4850 4950 60  0001 C CNN
-F 3 "REGU-001" H 4850 4950 60  0001 C CNN
-	1    4700 4950
-	1    0    0    -1
-$EndComp
-$Comp
 L MCP1826S-3302E/DB U15
 U 1 1 595F71A4
@@
 $EndComp
 Wire Wire Line
-	7700 2050 7350 2050
+	7350 2050 8050 2050
 Wire Wire Line
 	6000 4700 6950 4700
@@
 Text Label 5300 2250 0    60   ~ 0
 5V_EXT_FB
+$Comp
+L SPOX-2 J?
+U 1 1 597DA04D
+P 750 2850
+F 0 "J?" H 850 3000 60  0000 C CNN
+F 1 "SPOX-2" H 850 2700 60  0000 C CNN
+F 2 "Connectors_Molex:Molex_SPOX-5267_22-03-5025_02x2.54mm_Straight" H 750 2800 60  0001 C CNN
+F 3 "" H 750 2800 60  0001 C CNN
+F 4 "CONN-001" H 950 3100 60  0001 C CNN "part_num"
+	1    750  2850
+	1    0    0    -1
+$EndComp
+Text Notes 8900 2050 0    60   ~ 0
+Power jumper\nUse to measure current and\ndebug power
+Text Notes 850  2150 0    60   ~ 0
+Reverse polarity protection
+$Comp
+L TS30013-M050QFNR U?
+U 1 1 597EBED9
+P 4700 4950
+F 0 "U?" H 4650 5900 60  0000 C CNN
+F 1 "TS30013-M050QFNR" H 4700 4350 60  0000 C CNN
+F 2 "Housings_DFN_QFN:QFN-16-1EP_3x3mm_Pitch0.5mm" H 4850 4950 60  0001 C CNN
+F 3 "" H 4850 4950 60  0001 C CNN
+F 4 "REGU-001" H 4750 6000 60  0000 C CNN "part_num"
+	1    4700 4950
+	1    0    0    -1
+$EndComp
+$Comp
+L TS30013-M050QFNR U?
+U 1 1 597EBF5F
+P 4700 2300
+F 0 "U?" H 4650 3250 60  0000 C CNN
+F 1 "TS30013-M050QFNR" H 4700 1700 60  0000 C CNN
+F 2 "Housings_DFN_QFN:QFN-16-1EP_3x3mm_Pitch0.5mm" H 4850 2300 60  0001 C CNN
+F 3 "" H 4850 2300 60  0001 C CNN
+F 4 "REGU-001" H 4750 3350 60  0000 C CNN "part_num"
+	1    4700 2300
+	1    0    0    -1
+$EndComp
 $EndSCHEMATC
