File: Hardware/POWER.sch (KiCad schematic (older format))
At the start: 54 parts, among them J14 SPOX-2, Q1 Q_PMOS_DGS, U1 TPS54308, U15 MCP1826S-3302E/DB, U2 TPS54308DDCT, U3 NC7S04P5X, U5 TPS22810DRV, U6 TPS22810DRV, U7 TPS22810DRV, U8 TPS22810DRV

Commit message: Fixed merge issues
Parts:
- C9: renamed from C25; part_num (none) -> CAPP-005
- R10: renamed from R13; NO LOAD NO LOAD -> (none)
- R11: renamed from R16; NO LOAD NO LOAD -> (none)
- R12: renamed from R15; NO LOAD NO LOAD -> (none)
- R13: renamed from R17; NO LOAD NO LOAD -> (none)
- R14: renamed from R18; NO LOAD NO LOAD -> (none)
- R9: renamed from R12; NO LOAD NO LOAD -> (none)
- renumbered C26 to C10, C43 to C11, C44 to C12, C45 to C13, C46 to C14, C47 to C15, C48 to C16, C53 to C17, C50 to C18, C54 to C19, C51 to C20, C49 to C21, C52 to C22, C9 to C23, C10 to C24, D3 to D1, D4 to D2, D14 to D3, J14 to J13, R3 to R1, R29 to R15, R5 to R2, R6 to R3, R7 to R4, R8 to R5, R9 to R6, R10 to R7, R11 to R8, U5 to U4, U6 to U5, U7 to U6, U8 to U7, U15 to U8
Connections:
- wire segments 206 -> 150

Commit message: Removed unused connectors, started placements of components on new board
Parts:
- C1: footprint Capacitors_SMD:C_0603_HandSoldering -> Resistors_SMD:R_0603_HandSoldering
- C11, C12, C13, C14, C15, C16, C17, C18, C19, C20, C21, C22: footprint Capacitor_SMD:C_0603_1608Metric_Pad0.84x1.00mm_HandSolder -> Resistors_SMD:R_0603_HandSoldering
- C2: footprint Capacitor_SMD:C_0805_2012Metric_Pad1.15x1.50mm_HandSolder -> Resistors_SMD:R_0603_HandSoldering
- C3, C4, C5, C6, C7, C8: footprint Capacitor_SMD:C_0805_2012Metric_Pad1.15x1.50mm_HandSolder -> Resistors_SMD:R_0805_HandSoldering
- C9, R6: footprint (none) -> Resistors_SMD:R_0603_HandSoldering
- D1, D2: footprint Diode_SMD:D_SMA_Handsoldering -> Diodes_SMD:D_SMA_Handsoldering
Changed lines of the file:
@@
 F 0 "C12" H 5475 6500 50  0000 L CNN
 F 1 "22uF" H 5475 6300 50  0000 L CNN
-F 2 "Capacitor_SMD:C_0603_1608Metric_Pad0.84x1.00mm_HandSolder" H 5488 6250 50  0001 C CNN
+F 2 "Resistors_SMD:R_0603_HandSoldering" H 5488 6250 50  0001 C CNN
 F 3 "" H 5450 6400 50  0001 C CNN
 F 4 "CAPP-003" H 5450 6400 60  0001 C CNN "part_num"
@@
 F 0 "C9" H 4425 2250 50  0000 L CNN
 F 1 "100nF" H 4425 2050 50  0000 L CNN
-F 2 "" H 4438 2000 50  0001 C CNN
+F 2 "Resistors_SMD:R_0603_HandSoldering" H 4438 2000 50  0001 C CNN
 F 3 "" H 4400 2150 50  0001 C CNN
 F 4 "CAPP-005" H 4400 2150 60  0001 C CNN "part_num"
@@
 F 0 "R6" V 5030 3200 50  0000 C CNN
 F 1 "11k" V 4950 3200 50  0000 C CNN
-F 2 "" V 4880 3200 50  0001 C CNN
+F 2 "Resistors_SMD:R_0603_HandSoldering" V 4880 3200 50  0001 C CNN
 F 3 "" H 4950 3200 50  0001 C CNN
 F 4 "RESS-004" V 4950 3200 60  0001 C CNN "part_num"
@@
 F 0 "C14" H 5725 6500 50  0000 L CNN
 F 1 "22uF" H 5725 6300 50  0000 L CNN
-F 2 "Capacitor_SMD:C_0603_1608Metric_Pad0.84x1.00mm_HandSolder" H 5738 6250 50  0001 C CNN
+F 2 "Resistors_SMD:R_0603_HandSoldering" H 5738 6250 50  0001 C CNN
 F 3 "" H 5700 6400 50  0001 C CNN
 F 4 "CAPP-003" H 5700 6400 60  0001 C CNN "part_num"
@@
 F 0 "C16" H 5975 6500 50  0000 L CNN
 F 1 "22uF" H 5975 6300 50  0000 L CNN
-F 2 "Capacitor_SMD:C_0603_1608Metric_Pad0.84x1.00mm_HandSolder" H 5988 6250 50  0001 C CNN
+F 2 "Resistors_SMD:R_0603_HandSoldering" H 5988 6250 50  0001 C CNN
 F 3 "" H 5950 6400 50  0001 C CNN
 F 4 "CAPP-003" H 5950 6400 60  0001 C CNN "part_num"
@@
 F 0 "C11" H 5275 2750 50  0000 L CNN
 F 1 "22uF" H 5275 2550 50  0000 L CNN
-F 2 "Capacitor_SMD:C_0603_1608Metric_Pad0.84x1.00mm_HandSolder" H 5288 2500 50  0001 C CNN
+F 2 "Resistors_SMD:R_0603_HandSoldering" H 5288 2500 50  0001 C CNN
 F 3 "" H 5250 2650 50  0001 C CNN
 F 4 "CAPP-003" H 5250 2650 60  0001 C CNN "part_num"
@@
 F 0 "C13" H 5525 2750 50  0000 L CNN
 F 1 "22uF" H 5525 2550 50  0000 L CNN
-F 2 "Capacitor_SMD:C_0603_1608Metric_Pad0.84x1.00mm_HandSolder" H 5538 2500 50  0001 C CNN
+F 2 "Resistors_SMD:R_0603_HandSoldering" H 5538 2500 50  0001 C CNN
 F 3 "" H 5500 2650 50  0001 C CNN
 F 4 "CAPP-003" H 5500 2650 60  0001 C CNN "part_num"
@@
 F 0 "C15" H 5825 2750 50  0000 L CNN
 F 1 "22uF" H 5825 2550 50  0000 L CNN
-F 2 "Capacitor_SMD:C_0603_1608Metric_Pad0.84x1.00mm_HandSolder" H 5838 2500 50  0001 C CNN
+F 2 "Resistors_SMD:R_0603_HandSoldering" H 5838 2500 50  0001 C CNN
 F 3 "" H 5800 2650 50  0001 C CNN
 F 4 "CAPP-003" H 5800 2650 60  0001 C CNN "part_num"
@@
 F 0 "C3" H 1425 2300 50  0000 L CNN
 F 1 "6.8uF" H 1425 2100 50  0000 L CNN
-F 2 "Capacitor_SMD:C_0805_2012Metric_Pad1.15x1.50mm_HandSolder" H 1438 2050 50  0001 C CNN
+F 2 "Resistors_SMD:R_0805_HandSoldering" H 1438 2050 50  0001 C CNN
 F 3 "" H 1400 2200 50  0001 C CNN
 F 4 "CAPP-013" H 1400 2200 60  0001 C CNN "part_num"
@@
 F 0 "C21" H 8675 6150 50  0000 L CNN
 F 1 "1uF" H 8675 5950 50  0000 L CNN
-F 2 "Capacitor_SMD:C_0603_1608Metric_Pad0.84x1.00mm_HandSolder" H 8688 5900 50  0001 C CNN
+F 2 "Resistors_SMD:R_0603_HandSoldering" H 8688 5900 50  0001 C CNN
 F 3 "" H 8650 6050 50  0001 C CNN
 F 4 "CAPP-004" H 8650 6050 60  0001 C CNN "part_num"
@@
 F 0 "C5" H 1725 2300 50  0000 L CNN
 F 1 "6.8uF" H 1725 2100 50  0000 L CNN
-F 2 "Capacitor_SMD:C_0805_2012Metric_Pad1.15x1.50mm_HandSolder" H 1738 2050 50  0001 C CNN
+F 2 "Resistors_SMD:R_0805_HandSoldering" H 1738 2050 50  0001 C CNN
 F 3 "" H 1700 2200 50  0001 C CNN
 F 4 "CAPP-013" H 1700 2200 60  0001 C CNN "part_num"
@@
 F 0 "C7" H 2075 2300 50  0000 L CNN
 F 1 "6.8uF" H 2075 2100 50  0000 L CNN
-F 2 "Capacitor_SMD:C_0805_2012Metric_Pad1.15x1.50mm_HandSolder" H 2088 2050 50  0001 C CNN
+F 2 "Resistors_SMD:R_0805_HandSoldering" H 2088 2050 50  0001 C CNN
 F 3 "" H 2050 2200 50  0001 C CNN
 F 4 "CAPP-013" H 2050 2200 60  0001 C CNN "part_num"
@@
 F 0 "C4" H 1625 6000 50  0000 L CNN
 F 1 "6.8uF" H 1625 5800 50  0000 L CNN
-F 2 "Capacitor_SMD:C_0805_2012Metric_Pad1.15x1.50mm_HandSolder" H 1638 5750 50  0001 C CNN
+F 2 "Resistors_SMD:R_0805_HandSoldering" H 1638 5750 50  0001 C CNN
 F 3 "" H 1600 5900 50  0001 C CNN
 F 4 "CAPP-013" H 1600 5900 60  0001 C CNN "part_num"
@@
 F 0 "C6" H 1925 6000 50  0000 L CNN
 F 1 "6.8uF" H 1925 5800 50  0000 L CNN
-F 2 "Capacitor_SMD:C_0805_2012Metric_Pad1.15x1.50mm_HandSolder" H 1938 5750 50  0001 C CNN
+F 2 "Resistors_SMD:R_0805_HandSoldering" H 1938 5750 50  0001 C CNN
 F 3 "" H 1900 5900 50  0001 C CNN
 F 4 "CAPP-013" H 1900 5900 60  0001 C CNN "part_num"
@@
 F 0 "C8" H 2275 6000 50  0000 L CNN
 F 1 "6.8uF" H 2275 5800 50  0000 L CNN
-F 2 "Capacitor_SMD:C_0805_2012Metric_Pad1.15x1.50mm_HandSolder" H 2288 5750 50  0001 C CNN
+F 2 "Resistors_SMD:R_0805_HandSoldering" H 2288 5750 50  0001 C CNN
 F 3 "" H 2250 5900 50  0001 C CNN
 F 4 "CAPP-013" H 2250 5900 60  0001 C CNN "part_num"
@@
 F 0 "C2" H 1325 6000 50  0000 L CNN
 F 1 "0.1uF" H 1325 5800 50  0000 L CNN
-F 2 "Capacitor_SMD:C_0805_2012Metric_Pad1.15x1.50mm_HandSolder" H 1338 5750 50  0001 C CNN
+F 2 "Resistors_SMD:R_0603_HandSoldering" H 1338 5750 50  0001 C CNN
 F 3 "" H 1300 5900 50  0001 C CNN
 F 4 "CAPP-014" H 1300 5900 60  0001 C CNN "part_num"
@@
 F 0 "C1" H 1025 2300 50  0000 L CNN
 F 1 "0.1uF" H 1025 2100 50  0000 L CNN
-F 2 "Capacitors_SMD:C_0603_HandSoldering" H 1038 2050 50  0001 C CNN
+F 2 "Resistors_SMD:R_0603_HandSoldering" H 1038 2050 50  0001 C CNN
 F 3 "" H 1000 2200 50  0001 C CNN
 F 4 "CAPP-014" H 1000 2200 60  0001 C CNN "part_num"
@@
 F 0 "D2" H 7000 5500 50  0000 C CNN
 F 1 "S1B-13-F" H 7000 5600 50  0001 C CNN
-F 2 "Diode_SMD:D_SMA_Handsoldering" H 7000 5400 50  0001 C CNN
+F 2 "Diodes_SMD:D_SMA_Handsoldering" H 7000 5400 50  0001 C CNN
 F 3 "" H 7000 5400 50  0001 C CNN
 F 4 "DIOD-005" H 7000 5400 60  0001 C CNN "part_num"
@@
 F 0 "C20" H 8625 2650 50  0000 L CNN
 F 1 "10nF" H 8625 2450 50  0000 L CNN
-F 2 "Capacitor_SMD:C_0603_1608Metric_Pad0.84x1.00mm_HandSolder" H 8638 2400 50  0001 C CNN
+F 2 "Resistors_SMD:R_0603_HandSoldering" H 8638 2400 50  0001 C CNN
 F 3 "" H 8600 2550 50  0001 C CNN
 F 4 "CAPP-010" H 8600 2550 60  0001 C CNN "part_num"
@@
 F 0 "C22" H 9125 2500 50  0000 L CNN
 F 1 "1uF" H 9125 2300 50  0000 L CNN
-F 2 "Capacitor_SMD:C_0603_1608Metric_Pad0.84x1.00mm_HandSolder" H 9138 2250 50  0001 C CNN
+F 2 "Resistors_SMD:R_0603_HandSoldering" H 9138 2250 50  0001 C CNN
 F 3 "" H 9100 2400 50  0001 C CNN
 F 4 "CAPP-004" H 9100 2400 60  0001 C CNN "part_num"
@@
 F 0 "C18" H 8125 6350 50  0000 L CNN
 F 1 "10nF" H 8125 6150 50  0000 L CNN
-F 2 "Capacitor_SMD:C_0603_1608Metric_Pad0.84x1.00mm_HandSolder" H 8138 6100 50  0001 C CNN
+F 2 "Resistors_SMD:R_0603_HandSoldering" H 8138 6100 50  0001 C CNN
 F 3 "" H 8100 6250 50  0001 C CNN
 F 4 "CAPP-010" H 8100 6250 60  0001 C CNN "part_num"
@@
 F 0 "C19" H 8575 1350 50  0000 L CNN
 F 1 "10nF" H 8550 1150 50  0000 L CNN
-F 2 "Capacitor_SMD:C_0603_1608Metric_Pad0.84x1.00mm_HandSolder" H 8588 1100 50  0001 C CNN
+F 2 "Resistors_SMD:R_0603_HandSoldering" H 8588 1100 50  0001 C CNN
 F 3 "" H 8550 1250 50  0001 C CNN
 F 4 "CAPP-010" H 8550 1250 60  0001 C CNN "part_num"
@@
 F 0 "C17" H 8075 5000 50  0000 L CNN
 F 1 "10nF" H 8050 4800 50  0000 L CNN
-F 2 "Capacitor_SMD:C_0603_1608Metric_Pad0.84x1.00mm_HandSolder" H 8088 4750 50  0001 C CNN
+F 2 "Resistors_SMD:R_0603_HandSoldering" H 8088 4750 50  0001 C CNN
 F 3 "" H 8050 4900 50  0001 C CNN
 F 4 "CAPP-010" H 8050 4900 60  0001 C CNN "part_num"
@@
 F 0 "D1" H 7000 4900 50  0000 C CNN
 F 1 "S1B-13-F" H 7000 5000 50  0001 C CNN
-F 2 "Diode_SMD:D_SMA_Handsoldering" H 7000 4800 50  0001 C CNN
+F 2 "Diodes_SMD:D_SMA_Handsoldering" H 7000 4800 50  0001 C CNN
 F 3 "" H 7000 4800 50  0001 C CNN
 F 4 "DIOD-005" H 7000 4800 60  0001 C CNN "part_num"

Commit message: Removed J20, added smaller inductor, updated placements
Parts:
- L1, L2: footprint Inductors_SMD:L_12x12mm_h8mm -> WARG:SRP6060FA-150M; part_num INDU-002 -> INDU-003
Changed lines of the file:
@@
 6V External Reg - Servo Supply
 $Comp
-L GND #PWR5
+L GND #PWR06
 U 1 1 59183E68
 P 1300 4850
-F 0 "#PWR5" H 1300 4600 50  0001 C CNN
+F 0 "#PWR06" H 1300 4600 50  0001 C CNN
 F 1 "GND" H 1300 4700 50  0000 C CNN
 F 2 "" H 1300 4850 50  0000 C CNN
@@
 6V_EXT
 $Comp
-L GND #PWR18
+L GND #PWR07
 U 1 1 591852CA
 P 8850 6300
-F 0 "#PWR18" H 8850 6050 50  0001 C CNN
+F 0 "#PWR07" H 8850 6050 50  0001 C CNN
 F 1 "GND" H 8850 6150 50  0000 C CNN
 F 2 "" H 8850 6300 50  0000 C CNN
@@
 $EndComp
 $Comp
-L GND #PWR20
+L GND #PWR08
 U 1 1 59185849
 P 9900 6300
-F 0 "#PWR20" H 9900 6050 50  0001 C CNN
+F 0 "#PWR08" H 9900 6050 50  0001 C CNN
 F 1 "GND" H 9900 6150 50  0000 C CNN
 F 2 "" H 9900 6300 50  0000 C CNN
@@
 $EndComp
 $Comp
-L GND #PWR21
+L GND #PWR09
 U 1 1 592C1537
 P 10450 5250
-F 0 "#PWR21" H 10450 5000 50  0001 C CNN
+F 0 "#PWR09" H 10450 5000 50  0001 C CNN
 F 1 "GND" H 10450 5100 50  0000 C CNN
 F 2 "" H 10450 5250 50  0000 C CNN
@@
 $EndComp
 $Comp
-L PWR_FLAG #FLG2
+L PWR_FLAG #FLG010
 U 1 1 594F4062
 P 2000 4350
-F 0 "#FLG2" H 2000 4425 50  0001 C CNN
+F 0 "#FLG010" H 2000 4425 50  0001 C CNN
 F 1 "PWR_FLAG" H 2000 4500 50  0000 C CNN
 F 2 "" H 2000 4350 50  0001 C CNN
@@
 $EndComp
 $Comp
-L GND #PWR7
+L GND #PWR011
 U 1 1 5B0F7994
 P 1900 6200
-F 0 "#PWR7" H 1900 5950 50  0001 C CNN
+F 0 "#PWR011" H 1900 5950 50  0001 C CNN
 F 1 "GND" H 1900 6050 50  0000 C CNN
 F 2 "" H 1900 6200 50  0000 C CNN
@@
 $EndComp
 $Comp
-L GND #PWR9
+L GND #PWR012
 U 1 1 5B145441
 P 2600 6600
-F 0 "#PWR9" H 2600 6350 50  0001 C CNN
+F 0 "#PWR012" H 2600 6350 50  0001 C CNN
 F 1 "GND" H 2600 6450 50  0000 C CNN
 F 2 "" H 2600 6600 50  0001 C CNN
@@
 $EndComp
 $Comp
-L GND #PWR11
+L GND #PWR013
 U 1 1 5B146E7C
 P 5150 7250
-F 0 "#PWR11" H 5150 7000 50  0001 C CNN
+F 0 "#PWR013" H 5150 7000 50  0001 C CNN
 F 1 "GND" H 5150 7100 50  0000 C CNN
 F 2 "" H 5150 7250 50  0001 C CNN
@@
 $EndComp
 $Comp
-L GND #PWR6
+L GND #PWR014
 U 1 1 5B160FEE
 P 1700 2500
-F 0 "#PWR6" H 1700 2250 50  0001 C CNN
+F 0 "#PWR014" H 1700 2250 50  0001 C CNN
 F 1 "GND" H 1700 2350 50  0000 C CNN
 F 2 "" H 1700 2500 50  0000 C CNN
@@
 F 0 "L1" V 4500 2350 50  0000 C CNN
 F 1 "15uH" V 4625 2350 50  0000 C CNN
-F 2 "Inductors_SMD:L_12x12mm_h8mm" H 4550 2350 50  0001 C CNN
+F 2 "WARG:SRP6060FA-150M" H 4550 2350 50  0001 C CNN
 F 3 "" H 4550 2350 50  0001 C CNN
-F 4 "INDU-002" V 4550 2350 60  0001 C CNN "part_num"
+F 4 "INDU-003" V 4550 2350 60  0001 C CNN "part_num"
 	1    4550 2350
 	0    1    1    0
 $EndComp
 $Comp
-L GND #PWR8
+L GND #PWR015
 U 1 1 5B16100A
 P 2400 2900
-F 0 "#PWR8" H 2400 2650 50  0001 C CNN
+F 0 "#PWR015" H 2400 2650 50  0001 C CNN
 F 1 "GND" H 2400 2750 50  0000 C CNN
 F 2 "" H 2400 2900 50  0001 C CNN
@@
 $EndComp
 $Comp
-L GND #PWR10
+L GND #PWR016
 U 1 1 5B161017
 P 4950 3500
-F 0 "#PWR10" H 4950 3250 50  0001 C CNN
+F 0 "#PWR016" H 4950 3250 50  0001 C CNN
 F 1 "GND" H 4950 3350 50  0000 C CNN
 F 2 "" H 4950 3500 50  0001 C CNN
@@
 F 0 "L2" V 4700 6050 50  0000 C CNN
 F 1 "15uH" V 4825 6050 50  0000 C CNN
-F 2 "Inductors_SMD:L_12x12mm_h8mm" H 4750 6050 50  0001 C CNN
+F 2 "WARG:SRP6060FA-150M" H 4750 6050 50  0001 C CNN
 F 3 "" H 4750 6050 50  0001 C CNN
-F 4 "INDU-002" V 4750 6050 60  0001 C CNN "part_num"
+F 4 "INDU-003" V 4750 6050 60  0001 C CNN "part_num"
 	1    4750 6050
 	0    1    1    0
@@
 $EndComp
 $Comp
-L GND #PWR12
+L GND #PWR017
 U 1 1 5B223354
 P 5850 5300
-F 0 "#PWR12" H 5850 5050 50  0001 C CNN
+F 0 "#PWR017" H 5850 5050 50  0001 C CNN
 F 1 "GND" H 5850 5150 50  0000 C CNN
 F 2 "" H 5850 5300 50  0001 C CNN
@@
 $EndComp
 $Comp
-L GND #PWR15
+L GND #PWR018
 U 1 1 5B28DFBE
 P 7550 2800
-F 0 "#PWR15" H 7550 2550 50  0001 C CNN
+F 0 "#PWR018" H 7550 2550 50  0001 C CNN
 F 1 "GND" H 7550 2650 50  0000 C CNN
 F 2 "" H 7550 2800 50  0001 C CNN
@@
 $EndComp
 $Comp
-L GND #PWR14
+L GND #PWR019
 U 1 1 5B29EF8B
 P 7350 900
-F 0 "#PWR14" H 7350 650 50  0001 C CNN
+F 0 "#PWR019" H 7350 650 50  0001 C CNN
 F 1 "GND" H 7350 750 50  0000 C CNN
 F 2 "" H 7350 900 50  0001 C CNN
@@
 $EndComp
 $Comp
-L GND #PWR13
+L GND #PWR020
 U 1 1 5B29FB49
 P 6850 4600
-F 0 "#PWR13" H 6850 4350 50  0001 C CNN
+F 0 "#PWR020" H 6850 4350 50  0001 C CNN
 F 1 "GND" H 6850 4450 50  0000 C CNN
 F 2 "" H 6850 4600 50  0001 C CNN
@@
 $EndComp
 $Comp
-L GND #PWR19
+L GND #PWR021
 U 1 1 5B2F8DF1
 P 9100 2650
-F 0 "#PWR19" H 9100 2400 50  0001 C CNN
+F 0 "#PWR021" H 9100 2400 50  0001 C CNN
 F 1 "GND" H 9100 2500 50  0000 C CNN
 F 2 "" H 9100 2650 50  0000 C CNN
@@
 $EndComp
 $Comp
-L GND #PWR17
+L GND #PWR022
 U 1 1 5B308240
 P 8550 1500
-F 0 "#PWR17" H 8550 1250 50  0001 C CNN
+F 0 "#PWR022" H 8550 1250 50  0001 C CNN
 F 1 "GND" H 8550 1350 50  0000 C CNN
 F 2 "" H 8550 1500 50  0001 C CNN
@@
 $EndComp
 $Comp
-L GND #PWR16
+L GND #PWR023
 U 1 1 5B308C3B
 P 8050 5150
-F 0 "#PWR16" H 8050 4900 50  0001 C CNN
+F 0 "#PWR023" H 8050 4900 50  0001 C CNN
 F 1 "GND" H 8050 5000 50  0000 C CNN
 F 2 "" H 8050 5150 50  0000 C CNN

Commit message: Updated schematic
-Changed diode to 0603 diodes
-Changed SD card to proper pinout
-Fixed SPI1 conflict
-Renamed some power nets
-Fixed naming error in IMU NSS
Connections:
- net labels removed: INT_INT_VCC
Changed lines of the file:
@@
 	0    1    1    0
 $EndComp
-Text Label 7000 5250 0    60   ~ 0
-INT_INT_VCC
 Text Label 7000 800  0    60   ~ 0
 5V_USB+
@@
 	1600 6050 1600 6200
 Wire Wire Line
-	8000 5850 8500 5850
-Wire Wire Line
 	6400 4500 7150 4500
 Connection ~ 5700 7200
@@
 Wire Wire Line
 	7500 2150 7500 2150
-Text Label 8500 5850 2    60   ~ 0
+Text Label 8200 5800 1    60   ~ 0
 5V_INT_JMP
+Wire Wire Line
+	8000 5850 8200 5850
 $EndSCHEMATC

Commit message: Remapped symbols for KiCAD 5.0.x
Parts:
- C?: renamed from C23; symbol C -> Device:C
- C?: renamed from C24; symbol C -> Device:C
- C?: renamed from C10; symbol C -> Device:C
- C?: renamed from C12; symbol C -> Device:C
- C?: renamed from C9; symbol C -> Device:C
- C?: renamed from C14; symbol C -> Device:C
- C?: renamed from C16; symbol C -> Device:C
- C?: renamed from C11; symbol C -> Device:C
- C?: renamed from C13; symbol C -> Device:C
- C?: renamed from C15; symbol C -> Device:C
- C?: renamed from C3; symbol C -> Device:C
- C?: renamed from C21; symbol C -> Device:C
- C?: renamed from C5; symbol C -> Device:C
- C?: renamed from C7; symbol C -> Device:C
- C?: renamed from C4; symbol C -> Device:C
- C?: renamed from C6; symbol C -> Device:C
- C?: renamed from C8; symbol C -> Device:C
- C?: renamed from C2; symbol C -> Device:C
- C?: renamed from C1; symbol C -> Device:C
- C?: renamed from C20; symbol C -> Device:C
- C?: renamed from C22; symbol C -> Device:C
- C?: renamed from C18; symbol C -> Device:C
- C?: renamed from C19; symbol C -> Device:C
- C?: renamed from C17; symbol C -> Device:C
- D?: renamed from D3; symbol LED -> Device:LED
- D?: renamed from D2; symbol D -> Device:D
- D?: renamed from D1; symbol D -> Device:D
- J?: renamed from J13; symbol SPOX-2 -> WARG:SPOX-2
- L?: renamed from L1; symbol L -> Device:L
- L?: renamed from L2; symbol L -> Device:L
- Q?: renamed from Q1; symbol Q_PMOS_DGS -> Device:Q_PMOS_DGS
- R?: renamed from R15; symbol R -> Device:R
- R?: renamed from R3; symbol R -> Device:R
- R?: renamed from R4; symbol R -> Device:R
- R?: renamed from R8; symbol R -> Device:R
- R?: renamed from R7; symbol R -> Device:R
- R?: renamed from R1; symbol R -> Device:R
- R?: renamed from R2; symbol R -> Device:R
- R?: renamed from R6; symbol R -> Device:R
- R?: renamed from R9; symbol R -> Device:R
- R?: renamed from R5; symbol R -> Device:R
- R?: renamed from R12; symbol R -> Device:R
- R?: renamed from R10; symbol R -> Device:R
- R?: renamed from R14; symbol R -> Device:R
- R?: renamed from R11; symbol R -> Device:R
- R?: renamed from R13; symbol R -> Device:R
- U?: renamed from U8; symbol MCP1826S-3302E/DB -> WARG:MCP1826S-3302E_DB
- U?: renamed from U2; symbol TPS54308 -> WARG:TPS54308
- U?: renamed from U1; symbol TPS54308 -> WARG:TPS54308
- U?: renamed from U4; symbol TPS22810DRV -> WARG:TPS22810DRV
- U?: renamed from U5; symbol TPS22810DRV -> WARG:TPS22810DRV
- U?: renamed from U3; symbol NC7S04P5X -> WARG:NC7S04P5X
- U?: renamed from U6; symbol TPS22810DRV -> WARG:TPS22810DRV
- U?: renamed from U7; symbol TPS22810DRV -> WARG:TPS22810DRV
Connections:
- wire segments 150 -> 202

Commit message: Added RSSI, datasheets, INDU-004
Added RSSI input to PPM connector. Added datasheets for most of the components. The filter inductors for the FTDI were labeled as INDU-002, which is a 15uH smps inductor.
Parts:
- added D?: PWR_LED, LEDs:LED_0603, symbol Device:LED
- added R? (x2): 100, Resistors_SMD:R_0603_HandSoldering, symbol Device:R
- C? (x18): footprint Resistors_SMD:R_0603_HandSoldering -> Capacitors_SMD:C_0603_HandSoldering
- C? (x6): footprint Resistors_SMD:R_0805_HandSoldering -> Capacitors_SMD:C_0805_HandSoldering
- D? (x2): value S1B-13-F -> D
- R?: value 226k -> 226K
- R?: value 56k -> 56K
- R?: value 13.7k -> 13.7K
- R? (x2): value 100k -> 100K
- R?: value 210k -> 210K
- R?: value 43.2k -> 43.2K
- R?: value 11k -> 11K
Connections:
- wire segments 202 -> 211
Other:
- moved on the sheet: C?, D?, R?
