File: Hardware/POWER.sch (KiCad schematic (older format))
At the start: 57 parts

Commit message: Bug fixes, added Isense, changed conn to JST-GH
Added boot0 pull-down resistors. Changed ext_batt to current sense line. Changed spox conn to JST-GH, this will dramatically reduce the required size of the board.
Parts:
- J?: value SPOX-2 -> GH-2; footprint Connectors_Molex:Molex_SPOX-5267_22-03-5025_02x2.54mm_Straight -> Connectors_JST:JST_GH_BM02B-GHS-TBT_02x1.25mm_Straight; symbol WARG:SPOX-2 -> conn:Conn_01x02; part_num CONN-001 -> CONN-013
Changed lines of the file:
@@
 BATT_IN
 $Comp
-L WARG:SPOX-2 J?
+L conn:Conn_01x02 J?
 U 1 1 597DA04D
-P 900 4450
-F 0 "J?" H 1000 4600 60  0000 C CNN
-F 1 "SPOX-2" H 1000 4300 60  0000 C CNN
-F 2 "Connectors_Molex:Molex_SPOX-5267_22-03-5025_02x2.54mm_Straight" H 900 4400 60  0001 C CNN
-F 3 "https://www.molex.com/pdm_docs/sd/022035025_sd.pdf" H 900 4400 60  0001 C CNN
-F 4 "CONN-001" H 1100 4700 60  0001 C CNN "part_num"
-	1    900  4450
-	1    0    0    -1
+P 900 4500
+F 0 "J?" H 1000 4650 60  0000 C CNN
+F 1 "GH-2" H 1000 4350 60  0000 C CNN
+F 2 "Connectors_JST:JST_GH_BM02B-GHS-TBT_02x1.25mm_Straight" H 900 4450 60  0001 C CNN
+F 3 "http://www.jst-mfg.com/product/pdf/eng/eGH.pdf" H 900 4450 60  0001 C CNN
+F 4 "CONN-013" H 1100 4750 60  0001 C CNN "part_num"
+	1    900  4500
+	-1   0    0    1
 $EndComp
 Text Notes 9450 3150 0    60   ~ 0

Commit message: Added protection diode to USB
Changed lines of the file:
@@
 	-1   0    0    1
 $EndComp
-Text Notes 9450 3150 0    60   ~ 0
+Text Notes 9450 3200 0    60   ~ 0
 Power jumper\nUse to measure current and\ndebug power
 Text Notes 800  3700 0    60   ~ 0
@@
 	7550 2750 7550 2800
 Wire Wire Line
-	9100 2150 9900 2150
-Wire Wire Line
 	6150 2150 7650 2150
 Wire Wire Line
@@
 Wire Wire Line
 	10600 3650 10800 3650
+Wire Wire Line
+	9100 2150 9900 2150
 $EndSCHEMATC

Commit message: Removed F0 SPI, gave Baro its own I2C line, changed IMU to SPI1
Parts:
- removed J?: GH-2, Connectors_JST:JST_GH_BM02B-GHS-TBT_02x1.25mm_Straight, symbol conn:Conn_01x02
- added J?: SPOX-2, Connectors_Molex:Molex_SPOX-5267_22-03-5025_02x2.54mm_Straight, symbol WARG:SPOX-2
Changed lines of the file:
@@
 EESchema Schematic File Version 4
-LIBS:ZeroPilot-cache
 EELAYER 26 0
 EELAYER END
@@
 Text Label 1100 4400 0    60   ~ 0
 BATT_IN
-$Comp
-L conn:Conn_01x02 J?
-U 1 1 597DA04D
-P 900 4500
-F 0 "J?" H 1000 4650 60  0000 C CNN
-F 1 "GH-2" H 1000 4350 60  0000 C CNN
-F 2 "Connectors_JST:JST_GH_BM02B-GHS-TBT_02x1.25mm_Straight" H 900 4450 60  0001 C CNN
-F 3 "http://www.jst-mfg.com/product/pdf/eng/eGH.pdf" H 900 4450 60  0001 C CNN
-F 4 "CONN-013" H 1100 4750 60  0001 C CNN "part_num"
-	1    900  4500
-	-1   0    0    1
-$EndComp
 Text Notes 9450 3200 0    60   ~ 0
 Power jumper\nUse to measure current and\ndebug power
@@
 Wire Wire Line
 	9100 2150 9900 2150
+$Comp
+L WARG:SPOX-2 J?
+U 1 1 5CB5E0BD
+P 900 4450
+F 0 "J?" H 981 4747 60  0000 C CNN
+F 1 "SPOX-2" H 981 4641 60  0000 C CNN
+F 2 "Connectors_Molex:Molex_SPOX-5267_22-03-5025_02x2.54mm_Straight" H 900 4400 60  0001 C CNN
+F 3 "https://www.molex.com/pdm_docs/sd/022035025_sd.pdf" H 900 4400 60  0001 C CNN
+F 4 "CONN-001" H 1100 4700 60  0001 C CNN "part_num"
+	1    900  4450
+	1    0    0    -1
+$EndComp
 $EndSCHEMATC

Commit message: Generated netlist and board outline
Parts:
- gave numbers to parts that had none: 57

Commit message: Initial Routing of Zeropilot Rev1
This is the initial routing of the board. It needs to be cleaned up slightly, but library references are screwed up so they will be fixed first.
Parts:
- removed C18, C19, C20: 10nF, Capacitors_SMD:C_0603_HandSoldering, symbol Device:C
- removed R10, R9: 0, Resistors_SMD:R_0603_HandSoldering, symbol Device:R
- removed U3: NC7S04P5X, TO_SOT_Packages_SMD:SOT-353_SC-70-5_Handsoldering, symbol WARG:NC7S04P5X
- removed U4, U5, U6, U7: TPS22810DRV, WARG:TPS22810DRV, symbol WARG:TPS22810DRV
- C17: value 10nF -> 1uF; NO LOAD NO LOAD -> (none); part_num CAPP-010 -> CAPP-004
- C3, C4, C5, C6, C7, C8: footprint Capacitors_SMD:C_0805_HandSoldering -> Capacitors_SMD:C_0603_HandSoldering
- D1, D2: footprint Diodes_SMD:D_SMA_Handsoldering -> Diodes_SMD:D_PowerDI-123; part_num DIOD-005 -> DIOD-007
Connections:
- net labels removed: EXT_JMP1, INT_JMP1, USB_EN
- wire segments 211 -> 154
- no-connect marks 1 -> 0
Other:
- moved on the sheet: C22, R11, R12

Commit message: Updated Footprints
Updated the footprints to 5.1, added 3D models to all components.
Parts:
- C1, C10, C11, C12, C13, C14, C15, C16, C17, C2, C21, C22, C23, C24, C3, C4, C5, C6, C7, C8, C9: footprint Capacitors_SMD:C_0603_HandSoldering -> Capacitor_SMD:C_0603_1608Metric_Pad1.05x0.95mm_HandSolder
- D1, D2: footprint Diodes_SMD:D_PowerDI-123 -> Diode_SMD:D_PowerDI-123
- D3, D4: footprint LEDs:LED_0603 -> LED_SMD:LED_0603_1608Metric_Pad1.05x0.95mm_HandSolder
- J7: footprint Connectors_Molex:Molex_SPOX-5267_22-03-5025_02x2.54mm_Straight -> Connector_Molex:Molex_SPOX_5267-02A_1x02_P2.50mm_Vertical
- Q1: footprint WARG:TSOT-23-6_MK06A_HandSoldering -> WARG-kicad:IRF5806
- R1, R11, R12, R13, R14, R15, R16, R17, R2, R3, R4, R5, R6, R7, R8: footprint Resistors_SMD:R_0603_HandSoldering -> Resistor_SMD:R_0603_1608Metric_Pad1.05x0.95mm_HandSolder
- U1, U2: footprint WARG:TPS54308DDCT -> Package_TO_SOT_SMD:TSOT-23-6_HandSoldering
- U8: footprint TO_SOT_Packages_SMD:SOT-223 -> Package_TO_SOT_SMD:SOT-223

Commit message: HW Bootcamp for Zeropilot R1
Changed the board to R1.
Parts:
- removed D1, D2: D, Diode_SMD:D_PowerDI-123, symbol Device:D
- added H3, H4: MountingHole, MountingHole:MountingHole_3.2mm_M3_ISO14580_Pad, symbol Mechanical:MountingHole
- renumbered C22 to C18, C21 to C19, C23 to C20, C24 to C21, D3 to D1, R12 to R10, R13 to R11, R14 to R12, R15 to R13, R16 to R14, R17 to R15, R11 to R9, U8 to U3
Connections:
- net labels removed: 5V_USB+
- wire segments 154 -> 152
Changed lines of the file:
@@
 EESchema Schematic File Version 4
-LIBS:ZeroPilot-cache
 EELAYER 29 0
 EELAYER END
 $Descr A4 11693 8268
 encoding utf-8
-Sheet 3 10
+Sheet 2 2
 Title ""
 Date ""
@@
 6V_EXT
 $Comp
-L power:GND #PWR018
+L power:GND #PWR014
 U 1 1 591852CA
 P 8850 6300
-F 0 "#PWR018" H 8850 6050 50  0001 C CNN
+F 0 "#PWR014" H 8850 6050 50  0001 C CNN
 F 1 "GND" H 8850 6150 50  0000 C CNN
 F 2 "" H 8850 6300 50  0000 C CNN
@@
 $EndComp
 $Comp
-L Device:C C23
+L Device:C C20
 U 1 1 59185746
 P 9900 6050
-F 0 "C23" H 9925 6150 50  0000 L CNN
+F 0 "C20" H 9925 6150 50  0000 L CNN
 F 1 "1uF" H 9925 5950 50  0000 L CNN
 F 2 "Capacitor_SMD:C_0603_1608Metric_Pad1.05x0.95mm_HandSolder" H 9938 5900 50  0001 C CNN
@@
 $EndComp
 $Comp
-L power:GND #PWR020
+L power:GND #PWR015
 U 1 1 59185849
 P 9900 6300
-F 0 "#PWR020" H 9900 6050 50  0001 C CNN
+F 0 "#PWR015" H 9900 6050 50  0001 C CNN
 F 1 "GND" H 9900 6150 50  0000 C CNN
 F 2 "" H 9900 6300 50  0000 C CNN
@@
 $EndComp
 $Comp
-L Device:C C24
+L Device:C C21
 U 1 1 591858E8
 P 10100 6050
-F 0 "C24" H 10125 6150 50  0000 L CNN
+F 0 "C21" H 10125 6150 50  0000 L CNN
 F 1 "100nF" H 10125 5950 50  0000 L CNN
 F 2 "Capacitor_SMD:C_0603_1608Metric_Pad1.05x0.95mm_HandSolder" H 10138 5900 50  0001 C CNN
@@
 VBATT
 $Comp
-L Device:LED D3
+L Device:LED D1
 U 1 1 592C12E2
 P 10250 5100
-F 0 "D3" H 10250 5200 50  0000 C CNN
+F 0 "D1" H 10250 5200 50  0000 C CNN
 F 1 "PWR_LED" H 10250 5000 50  0000 C CNN
 F 2 "LED_SMD:LED_0603_1608Metric_Pad1.05x0.95mm_HandSolder" H 10250 5100 50  0001 C CNN
@@
 $EndComp
 $Comp
-L Device:R R15
+L Device:R R13
 U 1 1 592C1353
 P 10250 4800
-F 0 "R15" V 10330 4800 50  0000 C CNN
+F 0 "R13" V 10330 4800 50  0000 C CNN
 F 1 "100" V 10250 4800 50  0000 C CNN
 F 2 "Resistor_SMD:R_0603_1608Metric_Pad1.05x0.95mm_HandSolder" V 10180 4800 50  0001 C CNN
@@
 $EndComp
 $Comp
-L power:GND #PWR021
+L power:GND #PWR016
 U 1 1 592C1537
 P 10250 5250
-F 0 "#PWR021" H 10250 5000 50  0001 C CNN
+F 0 "#PWR016" H 10250 5000 50  0001 C CNN
 F 1 "GND" H 10250 5100 50  0000 C CNN
 F 2 "" H 10250 5250 50  0000 C CNN
@@
 3V3_JMP
 $Comp
-L WARG:MCP1826S-3302E_DB U8
+L WARG:MCP1826S-3302E_DB U3
 U 1 1 595F71A4
 P 9400 6000
-F 0 "U8" H 9350 6400 60  0000 C CNN
+F 0 "U3" H 9350 6400 60  0000 C CNN
 F 1 "MCP1826S-3302E/DB" H 9300 6600 60  0000 C CNN
 F 2 "Package_TO_SOT_SMD:SOT-223" H 9250 6300 60  0001 C CNN
@@
 $EndComp
 $Comp
-L Device:C C21
+L Device:C C19
 U 1 1 5B21EBD0
 P 8650 6050
-F 0 "C21" H 8675 6150 50  0000 L CNN
+F 0 "C19" H 8675 6150 50  0000 L CNN
 F 1 "1uF" H 8675 5950 50  0000 L CNN
 F 2 "Capacitor_SMD:C_0603_1608Metric_Pad1.05x0.95mm_HandSolder" H 8688 5900 50  0001 C CNN
@@
 Text Label 850  1950 0    60   ~ 0
 VBATT
-Text HLabel 10300 3100 0    60   Input ~ 0
-5V_USB+
-$Comp
-L Device:R R12
+$Comp
+L Device:R R10
 U 1 1 5B295982
 P 9800 3400
-F 0 "R12" V 9700 3400 50  0000 C CNN
+F 0 "R10" V 9700 3400 50  0000 C CNN
 F 1 "0" V 9800 3400 50  0000 C CNN
 F 2 "Resistor_SMD:R_0603_1608Metric_Pad1.05x0.95mm_HandSolder" V 9730 3400 50  0001 C CNN
@@
 $EndComp
 $Comp
-L Device:R R14
+L Device:R R12
 U 1 1 5B2B489A
 P 9800 4250
-F 0 "R14" V 9700 4250 50  0000 C CNN
+F 0 "R12" V 9700 4250 50  0000 C CNN
 F 1 "0" V 9800 4250 50  0000 C CNN
 F 2 "Resistor_SMD:R_0603_1608Metric_Pad1.05x0.95mm_HandSolder" V 9730 4250 50  0001 C CNN
@@
 3V3_JMP
 $Comp
-L Device:R R11
+L Device:R R9
 U 1 1 5B2ED738
 P 9800 2850
-F 0 "R11" V 9700 2850 50  0000 C CNN
+F 0 "R9" V 9700 2850 50  0000 C CNN
 F 1 "0" V 9800 2850 50  0000 C CNN
 F 2 "Resistor_SMD:R_0603_1608Metric_Pad1.05x0.95mm_HandSolder" V 9730 2850 50  0001 C CNN
@@
 $EndComp
 $Comp
-L Device:R R13
+L Device:R R11
 U 1 1 5B2EE677
 P 9800 3950
-F 0 "R13" V 9700 3950 50  0000 C CNN
+F 0 "R11" V 9700 3950 50  0000 C CNN
 F 1 "0" V 9800 3950 50  0000 C CNN
 F 2 "Resistor_SMD:R_0603_1608Metric_Pad1.05x0.95mm_HandSolder" V 9730 3950 50  0001 C CNN
@@
 $EndComp
 $Comp
-L Device:C C22
+L Device:C C18
 U 1 1 5B2F8C14
 P 8250 2400
-F 0 "C22" H 8275 2500 50  0000 L CNN
+F 0 "C18" H 8275 2500 50  0000 L CNN
 F 1 "1uF" H 8275 2300 50  0000 L CNN
 F 2 "Capacitor_SMD:C_0603_1608Metric_Pad1.05x0.95mm_HandSolder" H 8288 2250 50  0001 C CNN
@@
 $EndComp
 $Comp
-L power:GND #PWR019
+L power:GND #PWR013
 U 1 1 5B2F8DF1
 P 8250 2650
-F 0 "#PWR019" H 8250 2400 50  0001 C CNN
+F 0 "#PWR013" H 8250 2400 50  0001 C CNN
 F 1 "GND" H 8250 2500 50  0000 C CNN
 F 2 "" H 8250 2650 50  0000 C CNN
@@
 $EndComp
 $Comp
-L Device:R R17
+L Device:R R15
 U 1 1 5CBD97C2
 P 10900 4650
-F 0 "R17" V 10980 4650 50  0000 C CNN
+F 0 "R15" V 10980 4650 50  0000 C CNN
 F 1 "100" V 10900 4650 50  0000 C CNN
 F 2 "Resistor_SMD:R_0603_1608Metric_Pad1.05x0.95mm_HandSolder" V 10830 4650 50  0001 C CNN
@@
 	10900 4800 10900 4950
 $Comp
-L power:GND #PWR022
+L power:GND #PWR017
 U 1 1 5CC21AE8
 P 10900 5250
-F 0 "#PWR022" H 10900 5000 50  0001 C CNN
+F 0 "#PWR017" H 10900 5000 50  0001 C CNN
 F 1 "GND" H 10900 5100 50  0000 C CNN
 F 2 "" H 10900 5250 50  0000 C CNN
@@
 $EndComp
 $Comp
-L Device:R R16
+L Device:R R14
 U 1 1 5CC233BF
 P 10900 4350
-F 0 "R16" V 10980 4350 50  0000 C CNN
+F 0 "R14" V 10980 4350 50  0000 C CNN
 F 1 "100" V 10900 4350 50  0000 C CNN
 F 2 "Resistor_SMD:R_0603_1608Metric_Pad1.05x0.95mm_HandSolder" V 10830 4350 50  0001 C CNN
@@
 Connection ~ 8250 2150
 $Comp
-L Device:D D2
-U 1 1 5CF5F66A
-P 10400 3800
-F 0 "D2" V 10446 3721 50  0000 R CNN
-F 1 "D" V 10355 3721 50  0000 R CNN
-F 2 "Diode_SMD:D_PowerDI-123" H 10400 3800 50  0001 C CNN
-F 3 "https://www.diodes.com/assets/Datasheets/ds30492.pdf" H 10400 3800 50  0001 C CNN
-F 4 "DIOD-007" V 10400 3800 50  0001 C CNN "part_num"
-	1    10400 3800
-	0    -1   -1   0
-$EndComp
-$Comp
-L Device:D D1
-U 1 1 5CF5FEF3
-P 10600 3250
-F 0 "D1" V 10646 3171 50  0000 R CNN
-F 1 "D" V 10555 3171 50  0000 R CNN
-F 2 "Diode_SMD:D_PowerDI-123" H 10600 3250 50  0001 C CNN
-F 3 "https://www.diodes.com/assets/Datasheets/ds30492.pdf" H 10600 3250 50  0001 C CNN
-F 4 "DIOD-007" H 10600 3250 50  0001 C CNN "part_num"
-	1    10600 3250
-	0    -1   -1   0
-$EndComp
-$Comp
 L Device:C C17
 U 1 1 5CF610BB
@@
 $EndComp
 $Comp
-L power:GND #PWR0101
+L power:GND #PWR012
 U 1 1 5CF610C1
 P 7750 6350
-F 0 "#PWR0101" H 7750 6100 50  0001 C CNN
+F 0 "#PWR012" H 7750 6100 50  0001 C CNN
 F 1 "GND" H 7750 6200 50  0000 C CNN
 F 2 "" H 7750 6350 50  0000 C CNN
@@
 	4950 2150 5250 2150
 Wire Wire Line
-	10300 3100 10600 3100
-Text HLabel 10100 3650 0    60   Input ~ 0
-5V_USB+
-Wire Wire Line
-	10100 3650 10400 3650
-Wire Wire Line
 	7750 5950 7750 5850
 Connection ~ 7750 5850
@@
 Wire Wire Line
 	10600 3550 10900 3550
+$Comp
+L Mechanical:MountingHole H3
+U 1 1 5CE1E8FF
+P 9800 700
+F 0 "H3" H 9900 746 50  0000 L CNN
+F 1 "MountingHole" H 9900 655 50  0000 L CNN
+F 2 "MountingHole:MountingHole_3.2mm_M3_ISO14580_Pad" H 9800 700 50  0001 C CNN
+F 3 "~" H 9800 700 50  0001 C CNN
+	1    9800 700
+	1    0    0    -1
+$EndComp
+$Comp
+L Mechanical:MountingHole H4
+U 1 1 5CE1F752
+P 10500 700
+F 0 "H4" H 10600 746 50  0000 L CNN
+F 1 "MountingHole" H 10600 655 50  0000 L CNN
+F 2 "MountingHole:MountingHole_3.2mm_M3_ISO14580_Pad" H 10500 700 50  0001 C CNN
+F 3 "~" H 10500 700 50  0001 C CNN
+	1    10500 700
+	1    0    0    -1
+$EndComp
 $EndSCHEMATC
