File: Hardware/ADC_voltage_dividers.sch (KiCad schematic (older format))
At the start: 8 parts

Commit message: commit before my computer restarts
Parts:
- renumbered D1 to D19, D2 to D20, R1 to R48, R2 to R49, R3 to R50, R4 to R51, R5 to R52, R6 to R53
Changed lines of the file:
@@
 $EndComp
 $Comp
-L D D1
+L D D19
 U 1 1 596892D3
 P 4050 1450
-F 0 "D1" H 4050 1550 50  0000 C CNN
+F 0 "D19" H 4050 1550 50  0000 C CNN
 F 1 "D" H 4050 1350 50  0000 C CNN
 F 2 "Diodes_SMD:D_SOD-523" H 4050 1450 50  0001 C CNN
@@
 $EndComp
 $Comp
-L D D2
+L D D20
 U 1 1 596892DB
 P 4050 2450
-F 0 "D2" H 4050 2550 50  0000 C CNN
+F 0 "D20" H 4050 2550 50  0000 C CNN
 F 1 "D" H 4050 2350 50  0000 C CNN
 F 2 "Diodes_SMD:D_SOD-523" H 4050 2450 50  0001 C CNN
@@
 	3850 3050 3850 3150
 $Comp
-L R R5
+L R R52
 U 1 1 596892FC
 P 3850 2900
-F 0 "R5" V 3930 2900 50  0000 C CNN
+F 0 "R52" V 3930 2900 50  0000 C CNN
 F 1 "22K" V 3850 2900 50  0000 C CNN
 F 2 "Resistors_SMD:R_0603_HandSoldering" V 3780 2900 50  0001 C CNN
@@
 $EndComp
 $Comp
-L R R2
+L R R49
 U 1 1 59689304
 P 3400 2700
-F 0 "R2" V 3480 2700 50  0000 C CNN
+F 0 "R49" V 3480 2700 50  0000 C CNN
 F 1 "100K" V 3400 2700 50  0000 C CNN
 F 2 "Resistors_SMD:R_0603_HandSoldering" V 3330 2700 50  0001 C CNN
@@
 Connection ~ 4050 2700
 $Comp
-L R R1
+L R R48
 U 1 1 59689BEB
 P 3400 1800
-F 0 "R1" V 3480 1800 50  0000 C CNN
+F 0 "R48" V 3480 1800 50  0000 C CNN
 F 1 "100K" V 3400 1800 50  0000 C CNN
 F 2 "Resistors_SMD:R_0603_HandSoldering" V 3330 1800 50  0001 C CNN
@@
 	3800 2200 3800 2300
 $Comp
-L R R4
+L R R51
 U 1 1 59689CB5
 P 3800 2050
-F 0 "R4" V 3880 2050 50  0000 C CNN
+F 0 "R51" V 3880 2050 50  0000 C CNN
 F 1 "22K" V 3800 2050 50  0000 C CNN
 F 2 "Resistors_SMD:R_0603_HandSoldering" V 3730 2050 50  0001 C CNN
@@
 	3850 4050 3850 4150
 $Comp
-L R R6
+L R R53
 U 1 1 59689D93
 P 3850 3900
-F 0 "R6" V 3930 3900 50  0000 C CNN
+F 0 "R53" V 3930 3900 50  0000 C CNN
 F 1 "22K" V 3850 3900 50  0000 C CNN
 F 2 "Resistors_SMD:R_0603_HandSoldering" V 3780 3900 50  0001 C CNN
@@
 	3600 3600 4400 3600
 $Comp
-L R R3
+L R R50
 U 1 1 59689DC9
 P 3450 3600
-F 0 "R3" V 3530 3600 50  0000 C CNN
+F 0 "R50" V 3530 3600 50  0000 C CNN
 F 1 "11K" V 3450 3600 50  0000 C CNN
 F 2 "Resistors_SMD:R_0603_HandSoldering" V 3380 3600 50  0001 C CNN
