File: Hardware/ADC_voltage_dividers.sch (KiCad schematic (older format))
At the start: 8 parts

Commit message: Fixed merge issues
Parts:
- renumbered D19 to D10, D20 to D11, R48 to R31, R49 to R32, R50 to R33, R51 to R34, R52 to R35, R53 to R36
Changed lines of the file:
@@
 LIBS:contrib
 LIBS:valves
+LIBS:ZeroPilot-cache
 EELAYER 25 0
 EELAYER END
@@
 $EndDescr
 $Comp
-L GND #PWR45
+L GND #PWR040
 U 1 1 596892B4
 P 3850 3150
-F 0 "#PWR45" H 3850 2900 50  0001 C CNN
+F 0 "#PWR040" H 3850 2900 50  0001 C CNN
 F 1 "GND" H 3850 3000 50  0000 C CNN
 F 2 "" H 3850 3150 50  0001 C CNN
@@
 $EndComp
 $Comp
-L D D19
+L D D10
 U 1 1 596892D3
 P 4050 1450
-F 0 "D19" H 4050 1550 50  0000 C CNN
+F 0 "D10" H 4050 1550 50  0000 C CNN
 F 1 "D" H 4050 1350 50  0000 C CNN
 F 2 "Diodes_SMD:D_SOD-523" H 4050 1450 50  0001 C CNN
@@
 $EndComp
 $Comp
-L D D20
+L D D11
 U 1 1 596892DB
 P 4050 2450
-F 0 "D20" H 4050 2550 50  0000 C CNN
+F 0 "D11" H 4050 2550 50  0000 C CNN
 F 1 "D" H 4050 2350 50  0000 C CNN
 F 2 "Diodes_SMD:D_SOD-523" H 4050 2450 50  0001 C CNN
@@
 	3850 3050 3850 3150
 $Comp
-L R R52
+L R R35
 U 1 1 596892FC
 P 3850 2900
-F 0 "R52" V 3930 2900 50  0000 C CNN
+F 0 "R35" V 3930 2900 50  0000 C CNN
 F 1 "22K" V 3850 2900 50  0000 C CNN
 F 2 "Resistors_SMD:R_0603_HandSoldering" V 3780 2900 50  0001 C CNN
@@
 $EndComp
 $Comp
-L R R49
+L R R32
 U 1 1 59689304
 P 3400 2700
-F 0 "R49" V 3480 2700 50  0000 C CNN
+F 0 "R32" V 3480 2700 50  0000 C CNN
 F 1 "150K" V 3400 2700 50  0000 C CNN
 F 2 "Resistors_SMD:R_0603_HandSoldering" V 3330 2700 50  0001 C CNN
@@
 Connection ~ 3850 2700
 $Comp
-L GND #PWR44
+L GND #PWR041
 U 1 1 59689CAD
 P 3800 2300
-F 0 "#PWR44" H 3800 2050 50  0001 C CNN
+F 0 "#PWR041" H 3800 2050 50  0001 C CNN
 F 1 "GND" H 3800 2150 50  0000 C CNN
 F 2 "" H 3800 2300 50  0001 C CNN
@@
 	3800 2200 3800 2300
 $Comp
-L R R51
+L R R34
 U 1 1 59689CB5
 P 3800 2050
-F 0 "R51" V 3880 2050 50  0000 C CNN
+F 0 "R34" V 3880 2050 50  0000 C CNN
 F 1 "22K" V 3800 2050 50  0000 C CNN
 F 2 "Resistors_SMD:R_0603_HandSoldering" V 3730 2050 50  0001 C CNN
@@
 AIRSPD_OUT
 $Comp
-L GND #PWR46
+L GND #PWR042
 U 1 1 59689D8B
 P 3850 4150
-F 0 "#PWR46" H 3850 3900 50  0001 C CNN
+F 0 "#PWR042" H 3850 3900 50  0001 C CNN
 F 1 "GND" H 3850 4000 50  0000 C CNN
 F 2 "" H 3850 4150 50  0001 C CNN
@@
 	3850 4050 3850 4150
 $Comp
-L R R53
+L R R36
 U 1 1 59689D93
 P 3850 3900
-F 0 "R53" V 3930 3900 50  0000 C CNN
+F 0 "R36" V 3930 3900 50  0000 C CNN
 F 1 "22K" V 3850 3900 50  0000 C CNN
 F 2 "Resistors_SMD:R_0603_HandSoldering" V 3780 3900 50  0001 C CNN
@@
 	3600 3600 4400 3600
 $Comp
-L R R50
+L R R33
 U 1 1 59689DC9
 P 3450 3600
-F 0 "R50" V 3530 3600 50  0000 C CNN
+F 0 "R33" V 3530 3600 50  0000 C CNN
 F 1 "11K" V 3450 3600 50  0000 C CNN
 F 2 "Resistors_SMD:R_0603_HandSoldering" V 3380 3600 50  0001 C CNN
@@
 	3300 3600 2950 3600
 $Comp
-L R R48
+L R R31
 U 1 1 599BFDE6
 P 3400 1800
-F 0 "R48" V 3480 1800 50  0000 C CNN
+F 0 "R31" V 3480 1800 50  0000 C CNN
 F 1 "150K" V 3400 1800 50  0000 C CNN
 F 2 "Resistors_SMD:R_0603_HandSoldering" V 3330 1800 50  0001 C CNN

Commit message: Updated schematic
-Changed diode to 0603 diodes
-Changed SD card to proper pinout
-Fixed SPI1 conflict
-Renamed some power nets
-Fixed naming error in IMU NSS
Parts:
- D10, D11: footprint Diodes_SMD:D_SOD-523 -> Diodes_SMD:D_SMA_Handsoldering; part_num DIOD-004 -> DIOD-005
Changed lines of the file:
@@
 F 0 "D10" H 4050 1550 50  0000 C CNN
 F 1 "D" H 4050 1350 50  0000 C CNN
-F 2 "Diodes_SMD:D_SOD-523" H 4050 1450 50  0001 C CNN
+F 2 "Diodes_SMD:D_SMA_Handsoldering" H 4050 1450 50  0001 C CNN
 F 3 "" H 4050 1450 50  0001 C CNN
-F 4 "DIOD-004" H 4050 1450 60  0001 C CNN "part_num"
+F 4 "DIOD-005" H 4050 1450 60  0001 C CNN "part_num"
 	1    4050 1450
 	0    1    1    0
@@
 F 0 "D11" H 4050 2550 50  0000 C CNN
 F 1 "D" H 4050 2350 50  0000 C CNN
-F 2 "Diodes_SMD:D_SOD-523" H 4050 2450 50  0001 C CNN
+F 2 "Diodes_SMD:D_SMA_Handsoldering" H 4050 2450 50  0001 C CNN
 F 3 "" H 4050 2450 50  0001 C CNN
-F 4 "DIOD-004" H 4050 2450 60  0001 C CNN "part_num"
+F 4 "DIOD-005" H 4050 2450 60  0001 C CNN "part_num"
 	1    4050 2450
 	0    1    1    0

Commit message: Remapped symbols for KiCAD 5.0.x
Parts:
- D?: renamed from D10; symbol D -> Device:D
- D?: renamed from D11; symbol D -> Device:D
- R?: renamed from R35; symbol R -> Device:R
- R?: renamed from R32; symbol R -> Device:R
- R?: renamed from R34; symbol R -> Device:R
- R?: renamed from R36; symbol R -> Device:R
- R?: renamed from R33; symbol R -> Device:R
- R?: renamed from R31; symbol R -> Device:R
Changed lines of the file:
@@
-EESchema Schematic File Version 2
-LIBS:WARG
-LIBS:power
-LIBS:device
-LIBS:transistors
-LIBS:conn
-LIBS:linear
-LIBS:regul
-LIBS:74xx
-LIBS:cmos4000
-LIBS:adc-dac
-LIBS:memory
-LIBS:xilinx
-LIBS:microcontrollers
-LIBS:dsp
-LIBS:microchip
-LIBS:analog_switches
-LIBS:motorola
-LIBS:texas
-LIBS:intel
-LIBS:audio
-LIBS:interface
-LIBS:digital-audio
-LIBS:philips
-LIBS:display
-LIBS:cypress
-LIBS:siliconi
-LIBS:opto
-LIBS:atmel
-LIBS:contrib
-LIBS:valves
+EESchema Schematic File Version 4
 LIBS:ZeroPilot-cache
-EELAYER 25 0
+EELAYER 26 0
 EELAYER END
 $Descr A4 11693 8268
@@
 $EndDescr
 $Comp
-L GND #PWR040
+L power:GND #PWR?
 U 1 1 596892B4
 P 3850 3150
-F 0 "#PWR040" H 3850 2900 50  0001 C CNN
+F 0 "#PWR?" H 3850 2900 50  0001 C CNN
 F 1 "GND" H 3850 3000 50  0000 C CNN
 F 2 "" H 3850 3150 50  0001 C CNN
@@
 $EndComp
 $Comp
-L D D10
+L Device:D D?
 U 1 1 596892D3
 P 4050 1450
-F 0 "D10" H 4050 1550 50  0000 C CNN
+F 0 "D?" H 4050 1550 50  0000 C CNN
 F 1 "D" H 4050 1350 50  0000 C CNN
 F 2 "Diodes_SMD:D_SMA_Handsoldering" H 4050 1450 50  0001 C CNN
@@
 $EndComp
 $Comp
-L D D11
+L Device:D D?
 U 1 1 596892DB
 P 4050 2450
-F 0 "D11" H 4050 2550 50  0000 C CNN
+F 0 "D?" H 4050 2550 50  0000 C CNN
 F 1 "D" H 4050 2350 50  0000 C CNN
 F 2 "Diodes_SMD:D_SMA_Handsoldering" H 4050 2450 50  0001 C CNN
@@
 	3850 3050 3850 3150
 $Comp
-L R R35
+L Device:R R?
 U 1 1 596892FC
 P 3850 2900
-F 0 "R35" V 3930 2900 50  0000 C CNN
+F 0 "R?" V 3930 2900 50  0000 C CNN
 F 1 "22K" V 3850 2900 50  0000 C CNN
 F 2 "Resistors_SMD:R_0603_HandSoldering" V 3780 2900 50  0001 C CNN
@@
 $EndComp
 $Comp
-L R R32
+L Device:R R?
 U 1 1 59689304
 P 3400 2700
-F 0 "R32" V 3480 2700 50  0000 C CNN
+F 0 "R?" V 3480 2700 50  0000 C CNN
 F 1 "150K" V 3400 2700 50  0000 C CNN
 F 2 "Resistors_SMD:R_0603_HandSoldering" V 3330 2700 50  0001 C CNN
@@
 	4050 1600 4050 1800
 Wire Wire Line
-	3550 1800 4400 1800
+	3550 1800 3800 1800
 Wire Wire Line
 	4050 2600 4050 2700
 Wire Wire Line
-	3550 2700 4400 2700
+	3550 2700 3850 2700
 Wire Wire Line
 	4050 2300 4050 2200
@@
 Connection ~ 3850 2700
 $Comp
-L GND #PWR041
+L power:GND #PWR?
 U 1 1 59689CAD
 P 3800 2300
-F 0 "#PWR041" H 3800 2050 50  0001 C CNN
+F 0 "#PWR?" H 3800 2050 50  0001 C CNN
 F 1 "GND" H 3800 2150 50  0000 C CNN
 F 2 "" H 3800 2300 50  0001 C CNN
@@
 	3800 2200 3800 2300
 $Comp
-L R R34
+L Device:R R?
 U 1 1 59689CB5
 P 3800 2050
-F 0 "R34" V 3880 2050 50  0000 C CNN
+F 0 "R?" V 3880 2050 50  0000 C CNN
 F 1 "22K" V 3800 2050 50  0000 C CNN
 F 2 "Resistors_SMD:R_0603_HandSoldering" V 3730 2050 50  0001 C CNN
@@
 AIRSPD_OUT
 $Comp
-L GND #PWR042
+L power:GND #PWR?
 U 1 1 59689D8B
 P 3850 4150
-F 0 "#PWR042" H 3850 3900 50  0001 C CNN
+F 0 "#PWR?" H 3850 3900 50  0001 C CNN
 F 1 "GND" H 3850 4000 50  0000 C CNN
 F 2 "" H 3850 4150 50  0001 C CNN
@@
 	3850 4050 3850 4150
 $Comp
-L R R36
+L Device:R R?
 U 1 1 59689D93
 P 3850 3900
-F 0 "R36" V 3930 3900 50  0000 C CNN
+F 0 "R?" V 3930 3900 50  0000 C CNN
 F 1 "22K" V 3850 3900 50  0000 C CNN
 F 2 "Resistors_SMD:R_0603_HandSoldering" V 3780 3900 50  0001 C CNN
@@
 	3850 3750 3850 3600
 Wire Wire Line
-	3600 3600 4400 3600
-$Comp
-L R R33
+	3600 3600 3850 3600
+$Comp
+L Device:R R?
 U 1 1 59689DC9
 P 3450 3600
-F 0 "R33" V 3530 3600 50  0000 C CNN
+F 0 "R?" V 3530 3600 50  0000 C CNN
 F 1 "11K" V 3450 3600 50  0000 C CNN
 F 2 "Resistors_SMD:R_0603_HandSoldering" V 3380 3600 50  0001 C CNN
@@
 	3300 3600 2950 3600
 $Comp
-L R R31
+L Device:R R?
 U 1 1 599BFDE6
 P 3400 1800
-F 0 "R31" V 3480 1800 50  0000 C CNN
+F 0 "R?" V 3480 1800 50  0000 C CNN
 F 1 "150K" V 3400 1800 50  0000 C CNN
 F 2 "Resistors_SMD:R_0603_HandSoldering" V 3330 1800 50  0001 C CNN
@@
 	0    1    1    0
 $EndComp
+Wire Wire Line
+	4050 2700 4400 2700
+Wire Wire Line
+	4050 1800 4400 1800
+Wire Wire Line
+	3850 2700 4050 2700
+Wire Wire Line
+	3800 1800 4050 1800
+Wire Wire Line
+	3850 3600 4400 3600
 $EndSCHEMATC

Commit message: Bug fixes, added Isense, changed conn to JST-GH
Added boot0 pull-down resistors. Changed ext_batt to current sense line. Changed spox conn to JST-GH, this will dramatically reduce the required size of the board.
Connections:
- net EXT_BATT_IN renamed V_ISENSE_IN
- net EXT_BATT_OUT renamed V_ISENSE_OUT
Changed lines of the file:
@@
 $EndComp
 Text HLabel 2950 2700 0    60   Input ~ 0
-EXT_BATT_IN
+V_ISENSE_IN
 Text HLabel 4400 2700 2    60   Output ~ 0
-EXT_BATT_OUT
+V_ISENSE_OUT
 Text HLabel 2950 1800 0    60   Input ~ 0
 VBATT_IN
