File: Hardware/_saved_POWER.sch (KiCad schematic (older format))
At the start: 28 parts, among them J14 SPOX-2, J15 CONN_02X05, Q1 Q_PMOS_DGS, U1 TS30013-M050QFNR, U15 LM2576D2TR4-3.3GOSTR-ND, U2 TS30013-M050QFNR

Commit message: I think this is everything
Parts:
- C9: footprint (none) -> Resistors_SMD:R_0603_HandSoldering
- D30: footprint (none) -> Diodes_SMD:D_SOD-123
- L3: footprint (none) -> WARG:5.1x6.5
Changed lines of the file:
@@
 EESchema Schematic File Version 2
 LIBS:ZeroPilot-rescue
+LIBS:WARG
 LIBS:power
 LIBS:device
@@
 LIBS:contrib
 LIBS:valves
-LIBS:WARG
 LIBS:ZeroPilot-cache
 EELAYER 25 0
@@
 F 0 "L3" V 2550 4550 50  0000 C CNN
 F 1 "100 uH" V 2675 4550 50  0000 C CNN
-F 2 "" H 2600 4550 50  0001 C CNN
+F 2 "WARG:5.1x6.5" H 2600 4550 50  0001 C CNN
 F 3 "" H 2600 4550 50  0001 C CNN
 	1    2600 4550
@@
 F 0 "D30" H 2300 4850 50  0000 C CNN
 F 1 "D" H 2300 4650 50  0000 C CNN
-F 2 "" H 2300 4750 50  0001 C CNN
+F 2 "Diodes_SMD:D_SOD-123" H 2300 4750 50  0001 C CNN
 F 3 "" H 2300 4750 50  0001 C CNN
 	1    2300 4750
@@
 F 0 "C9" H 2825 4850 50  0000 L CNN
 F 1 "100 uF" H 2825 4650 50  0000 L CNN
-F 2 "" H 2800 4750 50  0001 C CNN
+F 2 "Resistors_SMD:R_0603_HandSoldering" H 2800 4750 50  0001 C CNN
 F 3 "" H 2800 4750 50  0001 C CNN
 	1    2800 4750
