File: Hardware/sensors.sch (KiCad schematic (older format))
At the start: 6 parts, among them U3 ICM-20602, U4 MS5637-02BA03

Commit message: Fixed altimeter schematic
Parts:
- added C45: 100nF, symbol C
- added R6, R7: 10k, symbol R
Connections:
- wire segments 12 -> 22
Changed lines of the file:
@@
 U 1 1 5B0F962E
 P 6200 3650
-F 0 "U4" H 6200 4270 118 0000 C CNN
-F 1 "MS5637-02BA03" H 6200 2990 118 0000 C CNN
+F 0 "U4" H 6200 4600 118 0000 C CNN
+F 1 "MS5637-02BA03" H 6200 2425 118 0000 C CNN
 F 2 "" H 6218 3462 60  0001 C CNN
 F 3 "" H 6218 3462 60  0001 C CNN
@@
 Connection ~ 2400 2800
 Connection ~ 2700 2800
+$Comp
+L C C45
+U 1 1 5B1017C9
+P 6200 2975
+F 0 "C45" H 6225 3075 50  0000 L CNN
+F 1 "100nF" H 6225 2875 50  0000 L CNN
+F 2 "" H 6238 2825 50  0001 C CNN
+F 3 "" H 6200 2975 50  0001 C CNN
+	1    6200 2975
+	0    1    1    0
+$EndComp
+Wire Wire Line
+	6350 2975 6780 2975
+Wire Wire Line
+	6780 2975 6780 3500
+Wire Wire Line
+	6050 2975 5620 2975
+Wire Wire Line
+	5620 2975 5620 3640
+$Comp
+L R R6
+U 1 1 5B1091F6
+P 5620 3950
+F 0 "R6" V 5700 3950 50  0000 C CNN
+F 1 "10k" V 5620 3950 50  0000 C CNN
+F 2 "" V 5550 3950 50  0001 C CNN
+F 3 "" H 5620 3950 50  0001 C CNN
+	1    5620 3950
+	-1   0    0    1
+$EndComp
+$Comp
+L R R7
+U 1 1 5B109293
+P 5770 4260
+F 0 "R7" V 5850 4260 50  0000 C CNN
+F 1 "10k" V 5770 4260 50  0000 C CNN
+F 2 "" V 5700 4260 50  0001 C CNN
+F 3 "" H 5770 4260 50  0001 C CNN
+	1    5770 4260
+	0    1    1    0
+$EndComp
+Wire Wire Line
+	6780 3800 6780 4265
+Wire Wire Line
+	6780 4265 5920 4260
+Wire Wire Line
+	5620 3640 5080 3640
+Connection ~ 5620 3500
+Wire Wire Line
+	5620 4260 5620 4100
+Wire Wire Line
+	5620 4260 5080 4260
+Wire Wire Line
+	5080 4260 5080 3640
 $EndSCHEMATC

Commit message: Removed pull up resistors from altimeter
Parts:
- removed R6, R7: 10k, symbol R
Connections:
- wire segments 22 -> 16
Changed lines of the file:
@@
 EESchema Schematic File Version 2
-LIBS:ZeroPilot-rescue
 LIBS:WARG
 LIBS:power
@@
 	1    0    0    -1
 $EndComp
-$Comp
-L MS5637-02BA03 U4
-U 1 1 5B0F962E
-P 6200 3650
-F 0 "U4" H 6200 4600 118 0000 C CNN
-F 1 "MS5637-02BA03" H 6200 2425 118 0000 C CNN
-F 2 "" H 6218 3462 60  0001 C CNN
-F 3 "" H 6218 3462 60  0001 C CNN
-	1    6200 3650
-	1    0    0    -1
-$EndComp
 Wire Wire Line
 	1950 2800 3075 2800
@@
 	6050 2975 5620 2975
 Wire Wire Line
-	5620 2975 5620 3640
-$Comp
-L R R6
-U 1 1 5B1091F6
-P 5620 3950
-F 0 "R6" V 5700 3950 50  0000 C CNN
-F 1 "10k" V 5620 3950 50  0000 C CNN
-F 2 "" V 5550 3950 50  0001 C CNN
-F 3 "" H 5620 3950 50  0001 C CNN
-	1    5620 3950
-	-1   0    0    1
-$EndComp
-$Comp
-L R R7
-U 1 1 5B109293
-P 5770 4260
-F 0 "R7" V 5850 4260 50  0000 C CNN
-F 1 "10k" V 5770 4260 50  0000 C CNN
-F 2 "" V 5700 4260 50  0001 C CNN
-F 3 "" H 5770 4260 50  0001 C CNN
-	1    5770 4260
-	0    1    1    0
-$EndComp
-Wire Wire Line
-	6780 3800 6780 4265
-Wire Wire Line
-	6780 4265 5920 4260
-Wire Wire Line
-	5620 3640 5080 3640
-Connection ~ 5620 3500
-Wire Wire Line
-	5620 4260 5620 4100
-Wire Wire Line
-	5620 4260 5080 4260
-Wire Wire Line
-	5080 4260 5080 3640
+	5620 2975 5620 3500
+$Comp
+L MS5637-02BA03 U4
+U 1 1 5B0F962E
+P 6200 3650
+F 0 "U4" H 6200 4600 118 0000 C CNN
+F 1 "MS5637-02BA03" H 6200 2425 118 0000 C CNN
+F 2 "" H 6218 3462 60  0001 C CNN
+F 3 "" H 6218 3462 60  0001 C CNN
+	1    6200 3650
+	1    0    0    -1
+$EndComp
 $EndSCHEMATC

Commit message: Added part nums to IMU and altimeter, updated csv file
Connections:
- wire segments 16 -> 25
Changed lines of the file:
@@
 $EndComp
 Wire Wire Line
-	1950 2800 3075 2800
+	1950 2800 2150 2800
+Wire Wire Line
+	2150 2800 2400 2800
+Wire Wire Line
+	2400 2800 2700 2800
+Wire Wire Line
+	2700 2800 3075 2800
 Wire Wire Line
 	3075 2800 3075 3075
@@
 	3725 3450 3925 3450
 Wire Wire Line
-	3925 3450 3925 4100
+	3925 3450 3925 3550
+Wire Wire Line
+	3925 3550 3925 3650
+Wire Wire Line
+	3925 3650 3925 3750
+Wire Wire Line
+	3925 3750 3925 3850
+Wire Wire Line
+	3925 3850 3925 4100
 Wire Wire Line
 	3725 3550 3925 3550
@@
 VDC
 Wire Wire Line
-	1700 3450 2575 3450
+	1700 3450 2150 3450
+Wire Wire Line
+	2150 3450 2575 3450
 NoConn ~ 3150 3075
 Wire Wire Line
-	2150 2800 2150 3425
+	2150 2800 2150 3450
+Wire Wire Line
+	2150 3450 2150 3455
 NoConn ~ 3150 4225
 Text HLabel 2575 3850 0    60   Input ~ 0

Commit message: Added footprint values and part nums to capacitors
Also added part nums on the sheet to the sensors, however they already exist in the footprint editor
Parts:
- C25: footprint (none) -> CAP-010; part_num (none) -> CAPP-010
- C26, C44, C45: footprint (none) -> CAPP-005; part_num (none) -> CAPP-005
- C43: footprint (none) -> CAPP-007; part_num (none) -> CAPP-007
- U3: footprint (none) -> SENS-001; part_num (none) -> SENS-001
- U4: footprint (none) -> SENS-002; part_num (none) -> SENS-002
Connections:
- wire segments 25 -> 16
Changed lines of the file:
@@
 U 1 1 5B0F92D3
 P 3150 3650
-F 0 "U3" H 3150 4650 118 0000 C CNN
+F 0 "U3" H 3150 4870 118 0000 C CNN
 F 1 "ICM-20602" H 3150 2400 118 0000 C CNN
-F 2 "" H 3125 4664 60  0001 C CNN
+F 2 "SENS-001" H 3125 4664 60  0000 C CNN
 F 3 "" H 3125 4664 60  0001 C CNN
+F 4 "SENS-001" H 3150 3650 60  0001 C CNN "part_num"
 	1    3150 3650
 	1    0    0    -1
 $EndComp
 Wire Wire Line
-	1950 2800 2150 2800
-Wire Wire Line
-	2150 2800 2400 2800
-Wire Wire Line
-	2400 2800 2700 2800
-Wire Wire Line
-	2700 2800 3075 2800
+	1950 2800 3075 2800
 Wire Wire Line
 	3075 2800 3075 3075
@@
 F 0 "C25" H 1725 3700 50  0000 L CNN
 F 1 "10nF" H 1725 3500 50  0000 L CNN
-F 2 "" H 1738 3450 50  0001 C CNN
+F 2 "CAP-010" H 2040 3600 50  0001 C CNN
 F 3 "" H 1700 3600 50  0001 C CNN
+F 4 "CAPP-010" H 1700 3600 60  0001 C CNN "part_num"
 	1    1700 3600
 	-1   0    0    1
@@
 F 0 "C26" H 2425 3050 50  0000 L CNN
 F 1 "0.1uF" H 2425 2850 50  0000 L CNN
-F 2 "" H 2438 2800 50  0001 C CNN
+F 2 "CAPP-005" H 2438 2800 50  0001 C CNN
 F 3 "" H 2400 2950 50  0001 C CNN
+F 4 "CAPP-005" H 2400 2950 60  0001 C CNN "part_num"
 	1    2400 2950
 	1    0    0    -1
@@
 F 0 "C43" H 2725 3050 50  0000 L CNN
 F 1 "2.2uF" H 2725 2850 50  0000 L CNN
-F 2 "" H 2738 2800 50  0001 C CNN
+F 2 "CAPP-007" H 2738 2800 50  0001 C CNN
 F 3 "" H 2700 2950 50  0001 C CNN
+F 4 "CAPP-007" H 2700 2950 60  0001 C CNN "part_num"
 	1    2700 2950
 	1    0    0    -1
@@
 F 0 "C44" H 3750 3125 50  0000 L CNN
 F 1 "0.1uF" H 3750 2925 50  0000 L CNN
-F 2 "" H 3763 2875 50  0001 C CNN
+F 2 "CAPP-005" H 3763 2875 50  0001 C CNN
 F 3 "" H 3725 3025 50  0001 C CNN
+F 4 "CAPP-005" H 3725 3025 60  0001 C CNN "part_num"
 	1    3725 3025
 	1    0    0    -1
@@
 	3725 3450 3925 3450
 Wire Wire Line
-	3925 3450 3925 3550
-Wire Wire Line
-	3925 3550 3925 3650
-Wire Wire Line
-	3925 3650 3925 3750
-Wire Wire Line
-	3925 3750 3925 3850
-Wire Wire Line
-	3925 3850 3925 4100
+	3925 3450 3925 4100
 Wire Wire Line
 	3725 3550 3925 3550
@@
 VDC
 Wire Wire Line
-	1700 3450 2150 3450
-Wire Wire Line
-	2150 3450 2575 3450
+	1700 3450 2575 3450
 NoConn ~ 3150 3075
 Wire Wire Line
-	2150 2800 2150 3450
-Wire Wire Line
-	2150 3450 2150 3455
+	2150 2800 2150 3455
 NoConn ~ 3150 4225
 Text HLabel 2575 3850 0    60   Input ~ 0
@@
 F 0 "C45" H 6225 3075 50  0000 L CNN
 F 1 "100nF" H 6225 2875 50  0000 L CNN
-F 2 "" H 6238 2825 50  0001 C CNN
+F 2 "CAPP-005" H 6238 2825 50  0001 C CNN
 F 3 "" H 6200 2975 50  0001 C CNN
+F 4 "CAPP-005" H 6200 2975 60  0001 C CNN "part_num"
 	1    6200 2975
 	0    1    1    0
@@
 U 1 1 5B0F962E
 P 6200 3650
-F 0 "U4" H 6200 4600 118 0000 C CNN
-F 1 "MS5637-02BA03" H 6200 2425 118 0000 C CNN
-F 2 "" H 6218 3462 60  0001 C CNN
+F 0 "U4" H 6200 4890 118 0000 C CNN
+F 1 "MS5637-02BA03" H 6200 2860 118 0000 C CNN
+F 2 "SENS-002" H 6200 4640 60  0000 C CNN
 F 3 "" H 6218 3462 60  0001 C CNN
+F 4 "SENS-002" H 6200 3650 60  0001 C CNN "part_num"
 	1    6200 3650
 	1    0    0    -1

Commit message: Added test points, updated footprint values, fixed J1, replaced connectors
Parts:
- U3: footprint SENS-001 -> WARG:ICM-20602
- U4: footprint SENS-002 -> WARG:MS5637-02BA03
Changed lines of the file:
@@
 F 0 "U3" H 3150 4870 118 0000 C CNN
 F 1 "ICM-20602" H 3150 2400 118 0000 C CNN
-F 2 "SENS-001" H 3125 4664 60  0000 C CNN
+F 2 "WARG:ICM-20602" H 3125 4664 60  0000 C CNN
 F 3 "" H 3125 4664 60  0001 C CNN
 F 4 "SENS-001" H 3150 3650 60  0001 C CNN "part_num"
@@
 F 0 "U4" H 6200 4890 118 0000 C CNN
 F 1 "MS5637-02BA03" H 6200 2860 118 0000 C CNN
-F 2 "SENS-002" H 6200 4640 60  0000 C CNN
+F 2 "WARG:MS5637-02BA03" H 6200 4640 60  0000 C CNN
 F 3 "" H 6218 3462 60  0001 C CNN
 F 4 "SENS-002" H 6200 3650 60  0001 C CNN "part_num"

Commit message: Updated footprint field for capacitors in sensors sheet
Parts:
- C25: footprint CAP-010 -> Resistors_SMD:R_0603_HandSoldering
- C26, C44, C45: footprint CAPP-005 -> Resistors_SMD:R_0603_HandSoldering
- C43: footprint CAPP-007 -> Resistors_SMD:R_0603_HandSoldering
Changed lines of the file:
@@
 F 0 "C25" H 1725 3700 50  0000 L CNN
 F 1 "10nF" H 1725 3500 50  0000 L CNN
-F 2 "CAP-010" H 2040 3600 50  0001 C CNN
+F 2 "Resistors_SMD:R_0603_HandSoldering" H 2040 3600 50  0001 C CNN
 F 3 "" H 1700 3600 50  0001 C CNN
 F 4 "CAPP-010" H 1700 3600 60  0001 C CNN "part_num"
@@
 F 0 "C26" H 2425 3050 50  0000 L CNN
 F 1 "0.1uF" H 2425 2850 50  0000 L CNN
-F 2 "CAPP-005" H 2438 2800 50  0001 C CNN
+F 2 "Resistors_SMD:R_0603_HandSoldering" H 2438 2800 50  0001 C CNN
 F 3 "" H 2400 2950 50  0001 C CNN
 F 4 "CAPP-005" H 2400 2950 60  0001 C CNN "part_num"
@@
 F 0 "C43" H 2725 3050 50  0000 L CNN
 F 1 "2.2uF" H 2725 2850 50  0000 L CNN
-F 2 "CAPP-007" H 2738 2800 50  0001 C CNN
+F 2 "Resistors_SMD:R_0603_HandSoldering" H 2738 2800 50  0001 C CNN
 F 3 "" H 2700 2950 50  0001 C CNN
 F 4 "CAPP-007" H 2700 2950 60  0001 C CNN "part_num"
@@
 F 0 "C44" H 3750 3125 50  0000 L CNN
 F 1 "0.1uF" H 3750 2925 50  0000 L CNN
-F 2 "CAPP-005" H 3763 2875 50  0001 C CNN
+F 2 "Resistors_SMD:R_0603_HandSoldering" H 3763 2875 50  0001 C CNN
 F 3 "" H 3725 3025 50  0001 C CNN
 F 4 "CAPP-005" H 3725 3025 60  0001 C CNN "part_num"
@@
 F 0 "C45" H 6225 3075 50  0000 L CNN
 F 1 "100nF" H 6225 2875 50  0000 L CNN
-F 2 "CAPP-005" H 6238 2825 50  0001 C CNN
+F 2 "Resistors_SMD:R_0603_HandSoldering" H 6238 2825 50  0001 C CNN
 F 3 "" H 6200 2975 50  0001 C CNN
 F 4 "CAPP-005" H 6200 2975 60  0001 C CNN "part_num"
