File: Hardware/USB INTERFACE.sch (KiCad schematic (older format))
At the start: 14 parts

Commit message: Added more components
Parts:
- added C?: 8pF, Resistors_SMD:R_0603_HandSoldering, symbol C
- C? (x2): footprint Capacitors_SMD:C_0603 -> Resistors_SMD:R_0603_HandSoldering
- D? (x2): footprint Diodes_SMD:D_0603 -> Resistors_SMD:R_0603_HandSoldering
- R? (x4): footprint Resistors_SMD:R_0603 -> Resistors_SMD:R_0603_HandSoldering
- Y?: footprint (none) -> Crystals:Crystal_SMD_2520-4pin_2.5x2.0mm
Changed lines of the file:
@@
 L FT4232H U?
 U 3 1 5B18AA4E
-P 8800 4100
-F 0 "U?" H 8800 5000 60  0000 C CNN
-F 1 "FT4232H" H 8800 5150 60  0000 C CNN
-F 2 "Housings_QFP:LQFP-64_10x10mm_Pitch0.5mm" H 8800 3350 60  0001 C CNN
-F 3 "" H 8200 3750 60  0001 C CNN
-F 4 "CHIP-005" H 8800 4850 60  0000 C CNN "part_num"
-	3    8800 4100
+P 3250 5100
+F 0 "U?" H 3250 6000 60  0000 C CNN
+F 1 "FT4232H" H 3250 6150 60  0000 C CNN
+F 2 "Housings_QFP:LQFP-64_10x10mm_Pitch0.5mm" H 3250 4350 60  0001 C CNN
+F 3 "" H 2650 4750 60  0001 C CNN
+F 4 "CHIP-005" H 3250 5850 60  0000 C CNN "part_num"
+	3    3250 5100
 	1    0    0    -1
 $EndComp
@@
 F 0 "D?" H 1600 2000 50  0000 C CNN
 F 1 "600R" H 1600 1800 50  0000 C CNN
-F 2 "Diodes_SMD:D_0603" H 1600 1900 50  0001 C CNN
+F 2 "Resistors_SMD:R_0603_HandSoldering" H 1600 1900 50  0001 C CNN
 F 3 "" H 1600 1900 50  0001 C CNN
 F 4 "INDU-002" H 1600 1900 60  0001 C CNN "part_num"
@@
 F 0 "R?" V 2280 1850 50  0000 C CNN
 F 1 "4.7k" V 2200 1850 50  0000 C CNN
-F 2 "Resistors_SMD:R_0603" V 2130 1850 50  0001 C CNN
+F 2 "Resistors_SMD:R_0603_HandSoldering" V 2130 1850 50  0001 C CNN
 F 3 "" H 2200 1850 50  0001 C CNN
 F 4 "RESS-010" V 2200 1850 60  0001 C CNN "part_num"
@@
 F 0 "Y?" V 4900 2000 50  0000 L CNN
 F 1 "12MHz" V 5000 1950 50  0000 L CNN
-F 2 "" H 4650 2050 50  0001 C CNN
+F 2 "Crystals:Crystal_SMD_2520-4pin_2.5x2.0mm" H 4650 2050 50  0001 C CNN
 F 3 "" H 4650 2050 50  0001 C CNN
 F 4 "XTAL-003" V 4650 2050 60  0001 C CNN "part_num"
@@
 F 0 "C?" H 5175 2650 50  0000 L CNN
 F 1 "8pF" H 5175 2450 50  0000 L CNN
-F 2 "Capacitors_SMD:C_0603" H 5188 2400 50  0001 C CNN
+F 2 "Resistors_SMD:R_0603_HandSoldering" H 5188 2400 50  0001 C CNN
 F 3 "" H 5150 2550 50  0001 C CNN
 F 4 "CAPP-011" H 5150 2550 60  0001 C CNN "part_num"
@@
 F 0 "D?" H 1900 2000 50  0000 C CNN
 F 1 "600R" H 1900 1800 50  0000 C CNN
-F 2 "Diodes_SMD:D_0603" H 1900 1900 50  0001 C CNN
+F 2 "Resistors_SMD:R_0603_HandSoldering" H 1900 1900 50  0001 C CNN
 F 3 "" H 1900 1900 50  0001 C CNN
 F 4 "INDU-002" H 1900 1900 60  0001 C CNN "part_num"
@@
 F 0 "R?" V 2280 2450 50  0000 C CNN
 F 1 "10k" V 2200 2450 50  0000 C CNN
-F 2 "Resistors_SMD:R_0603" V 2130 2450 50  0001 C CNN
+F 2 "Resistors_SMD:R_0603_HandSoldering" V 2130 2450 50  0001 C CNN
 F 3 "" H 2200 2450 50  0001 C CNN
 F 4 "RESS-005" V 2200 2450 60  0001 C CNN "part_num"
@@
 F 0 "R?" V 2580 2450 50  0000 C CNN
 F 1 "12k" V 2500 2450 50  0000 C CNN
-F 2 "Resistors_SMD:R_0603" V 2430 2450 50  0001 C CNN
+F 2 "Resistors_SMD:R_0603_HandSoldering" V 2430 2450 50  0001 C CNN
 F 3 "" H 2500 2450 50  0001 C CNN
 F 4 "RESS-011" V 2500 2450 60  0001 C CNN "part_num"
@@
 F 0 "R?" V 2930 2150 50  0000 C CNN
 F 1 "1k" V 2850 2150 50  0000 C CNN
-F 2 "Resistors_SMD:R_0603" V 2780 2150 50  0001 C CNN
+F 2 "Resistors_SMD:R_0603_HandSoldering" V 2780 2150 50  0001 C CNN
 F 3 "" H 2850 2150 50  0001 C CNN
 F 4 "RESS-009" V 2850 2150 60  0001 C CNN "part_num"
@@
 F 0 "C?" H 5425 2650 50  0000 L CNN
 F 1 "8pF" H 5425 2450 50  0000 L CNN
-F 2 "Capacitors_SMD:C_0603" H 5438 2400 50  0001 C CNN
+F 2 "Resistors_SMD:R_0603_HandSoldering" H 5438 2400 50  0001 C CNN
 F 3 "" H 5400 2550 50  0001 C CNN
 F 4 "CAPP-011" H 5400 2550 60  0001 C CNN "part_num"
@@
 	1    0    0    -1
 $EndComp
+$Comp
+L C C?
+U 1 1 5B19574E
+P 4250 4750
+F 0 "C?" H 4275 4850 50  0000 L CNN
+F 1 "8pF" H 4275 4650 50  0000 L CNN
+F 2 "Resistors_SMD:R_0603_HandSoldering" H 4288 4600 50  0001 C CNN
+F 3 "" H 4250 4750 50  0001 C CNN
+F 4 "CAPP-011" H 4250 4750 60  0001 C CNN "part_num"
+	1    4250 4750
+	1    0    0    -1
+$EndComp

Commit message: Almost Done USB Interface
Parts:
- added C? (x4): 4.7uF, Resistors_SMD:R_0603_HandSoldering, symbol C
- added C? (x10): 100nF, Resistors_SMD:R_0603_HandSoldering, symbol C
- added L? (x2): 600R, Resistors_SMD:R_0603_HandSoldering, symbol L_Core_Ferrite
- C?: value 8pF -> 100nF; part_num CAPP-011 -> CAPP-005
Connections:
- net labels added: VDD
- wire segments 46 -> 103
- no-connect marks 0 -> 27
Other:
- moved on the sheet: C?

Commit message: Finalized USB Interface
Added SWD line resistors
Parts:
- removed Y?: 12MHz, Crystals:Crystal_SMD_2520-4pin_2.5x2.0mm, symbol Crystal_GND23
- added R? (x2): 10R, Resistors_SMD:R_0603_HandSoldering, symbol R
- added R? (x2): 100R, Resistors_SMD:R_0603_HandSoldering, symbol R
- added R? (x2): 1K, Resistors_SMD:R_0603_HandSoldering, symbol R
- added Y?: Crystal_GND24, Crystals:Crystal_SMD_2520-4pin_2.5x2.0mm, symbol Crystal_GND24
Connections:
- net labels added: SWD1_TCK, SWD1_TDI, SWD2_TCK, SWD2_TDI, UART1_CTS, UART1_RTS, UART1_RX, UART1_TX, UART2_CTS, UART2_RTS, UART2_RX, UART2_TX
- wire segments 103 -> 122
- no-connect marks 27 -> 23
Other:
- moved on the sheet: C?, R?

Commit message: Fixed Missing Bits
Fixed missing crystal part_num and added hierarchical pin for VBUS.
Parts:
- Y?: part_num (none) -> XTAL-003
Connections:
- net labels added: USB_VBUS
- wire segments 122 -> 123
Other:
- moved on the sheet: C?
Changed lines of the file:
@@
 encoding utf-8
 Sheet 9 9
-Title ""
-Date ""
+Title "USB INTERFACE (SWD/UART)"
+Date "2018-06-18"
 Rev ""
-Comp ""
-Comment1 ""
+Comp "WARG"
+Comment1 "Author: Alex Petkovic"
 Comment2 ""
 Comment3 ""
@@
 L C C?
 U 1 1 5B19574E
-P 2350 5350
-F 0 "C?" H 2375 5450 50  0000 L CNN
-F 1 "100nF" H 2375 5250 50  0000 L CNN
-F 2 "Resistors_SMD:R_0603_HandSoldering" H 2388 5200 50  0001 C CNN
-F 3 "" H 2350 5350 50  0001 C CNN
-F 4 "CAPP-005" H 2350 5350 60  0001 C CNN "part_num"
-	1    2350 5350
+P 2450 5350
+F 0 "C?" H 2475 5450 50  0000 L CNN
+F 1 "100nF" H 2475 5250 50  0000 L CNN
+F 2 "Resistors_SMD:R_0603_HandSoldering" H 2488 5200 50  0001 C CNN
+F 3 "" H 2450 5350 50  0001 C CNN
+F 4 "CAPP-005" H 2450 5350 60  0001 C CNN "part_num"
+	1    2450 5350
 	1    0    0    -1
 $EndComp
@@
 L C C?
 U 1 1 5B1A4637
-P 2650 5350
-F 0 "C?" H 2675 5450 50  0000 L CNN
-F 1 "100nF" H 2675 5250 50  0000 L CNN
-F 2 "Resistors_SMD:R_0603_HandSoldering" H 2688 5200 50  0001 C CNN
-F 3 "" H 2650 5350 50  0001 C CNN
-F 4 "CAPP-005" H 2650 5350 60  0001 C CNN "part_num"
-	1    2650 5350
+P 2750 5350
+F 0 "C?" H 2775 5450 50  0000 L CNN
+F 1 "100nF" H 2775 5250 50  0000 L CNN
+F 2 "Resistors_SMD:R_0603_HandSoldering" H 2788 5200 50  0001 C CNN
+F 3 "" H 2750 5350 50  0001 C CNN
+F 4 "CAPP-005" H 2750 5350 60  0001 C CNN "part_num"
+	1    2750 5350
 	1    0    0    -1
 $EndComp
@@
 L C C?
 U 1 1 5B1A4690
-P 2950 5350
-F 0 "C?" H 2975 5450 50  0000 L CNN
-F 1 "100nF" H 2975 5250 50  0000 L CNN
-F 2 "Resistors_SMD:R_0603_HandSoldering" H 2988 5200 50  0001 C CNN
-F 3 "" H 2950 5350 50  0001 C CNN
-F 4 "CAPP-005" H 2950 5350 60  0001 C CNN "part_num"
-	1    2950 5350
+P 3050 5350
+F 0 "C?" H 3075 5450 50  0000 L CNN
+F 1 "100nF" H 3075 5250 50  0000 L CNN
+F 2 "Resistors_SMD:R_0603_HandSoldering" H 3088 5200 50  0001 C CNN
+F 3 "" H 3050 5350 50  0001 C CNN
+F 4 "CAPP-005" H 3050 5350 60  0001 C CNN "part_num"
+	1    3050 5350
 	1    0    0    -1
 $EndComp
@@
 L GND #PWR?
 U 1 1 5B1ACDD5
-P 2650 5650
-F 0 "#PWR?" H 2650 5400 50  0001 C CNN
-F 1 "GND" H 2650 5500 50  0000 C CNN
-F 2 "" H 2650 5650 50  0001 C CNN
-F 3 "" H 2650 5650 50  0001 C CNN
-	1    2650 5650
+P 2750 5650
+F 0 "#PWR?" H 2750 5400 50  0001 C CNN
+F 1 "GND" H 2750 5500 50  0000 C CNN
+F 2 "" H 2750 5650 50  0001 C CNN
+F 3 "" H 2750 5650 50  0001 C CNN
+	1    2750 5650
 	1    0    0    -1
 $EndComp
@@
 L C C?
 U 1 1 5B1AF6AA
-P 3400 5350
-F 0 "C?" H 3425 5450 50  0000 L CNN
-F 1 "100nF" H 3425 5250 50  0000 L CNN
-F 2 "Resistors_SMD:R_0603_HandSoldering" H 3438 5200 50  0001 C CNN
-F 3 "" H 3400 5350 50  0001 C CNN
-F 4 "CAPP-005" H 3400 5350 60  0001 C CNN "part_num"
-	1    3400 5350
+P 3500 5350
+F 0 "C?" H 3525 5450 50  0000 L CNN
+F 1 "100nF" H 3525 5250 50  0000 L CNN
+F 2 "Resistors_SMD:R_0603_HandSoldering" H 3538 5200 50  0001 C CNN
+F 3 "" H 3500 5350 50  0001 C CNN
+F 4 "CAPP-005" H 3500 5350 60  0001 C CNN "part_num"
+	1    3500 5350
 	1    0    0    -1
 $EndComp
@@
 L C C?
 U 1 1 5B1AF726
-P 3700 5350
-F 0 "C?" H 3725 5450 50  0000 L CNN
-F 1 "4.7uF" H 3725 5250 50  0000 L CNN
-F 2 "Resistors_SMD:R_0603_HandSoldering" H 3738 5200 50  0001 C CNN
-F 3 "" H 3700 5350 50  0001 C CNN
-F 4 "CAPP-006" H 3700 5350 60  0001 C CNN "part_num"
-	1    3700 5350
+P 3800 5350
+F 0 "C?" H 3825 5450 50  0000 L CNN
+F 1 "4.7uF" H 3825 5250 50  0000 L CNN
+F 2 "Resistors_SMD:R_0603_HandSoldering" H 3838 5200 50  0001 C CNN
+F 3 "" H 3800 5350 50  0001 C CNN
+F 4 "CAPP-006" H 3800 5350 60  0001 C CNN "part_num"
+	1    3800 5350
 	1    0    0    -1
 $EndComp
@@
 L GND #PWR?
 U 1 1 5B1AFA96
-P 3550 5650
-F 0 "#PWR?" H 3550 5400 50  0001 C CNN
-F 1 "GND" H 3550 5500 50  0000 C CNN
-F 2 "" H 3550 5650 50  0001 C CNN
-F 3 "" H 3550 5650 50  0001 C CNN
-	1    3550 5650
+P 3650 5650
+F 0 "#PWR?" H 3650 5400 50  0001 C CNN
+F 1 "GND" H 3650 5500 50  0000 C CNN
+F 2 "" H 3650 5650 50  0001 C CNN
+F 3 "" H 3650 5650 50  0001 C CNN
+	1    3650 5650
 	1    0    0    -1
 $EndComp
@@
 	2100 5050 2100 5250
 Wire Wire Line
-	2050 5150 2950 5150
+	2050 5150 3050 5150
 Wire Wire Line
 	2100 5250 2050 5250
@@
 Connection ~ 2100 6350
 Wire Wire Line
-	2650 5500 2650 5650
-Wire Wire Line
-	2350 5500 2350 5550
-Wire Wire Line
-	2350 5550 2950 5550
-Connection ~ 2650 5550
-Wire Wire Line
-	2950 5550 2950 5500
-Wire Wire Line
-	2350 5150 2350 5200
-Wire Wire Line
-	2650 5050 2650 5200
-Connection ~ 2350 5150
-Connection ~ 2650 5150
+	2750 5500 2750 5650
+Wire Wire Line
+	2450 5500 2450 5550
+Wire Wire Line
+	2450 5550 3050 5550
+Connection ~ 2750 5550
+Wire Wire Line
+	3050 5550 3050 5500
+Wire Wire Line
+	2450 5150 2450 5200
+Wire Wire Line
+	2750 5050 2750 5200
+Connection ~ 2450 5150
+Connection ~ 2750 5150
 Connection ~ 2100 5650
 Connection ~ 2100 5250
 Connection ~ 2100 5350
 Wire Wire Line
-	2950 5150 2950 5200
-Wire Wire Line
-	3400 5200 3400 5150
-Wire Wire Line
-	3400 5150 3700 5150
-Wire Wire Line
-	3700 5150 3700 5200
-Wire Wire Line
-	3550 4950 3550 5150
-Connection ~ 3550 5150
-Wire Wire Line
-	3400 5500 3400 5550
-Wire Wire Line
-	3400 5550 3700 5550
-Wire Wire Line
-	3700 5550 3700 5500
-Wire Wire Line
-	3550 5550 3550 5650
-Connection ~ 3550 5550
-Wire Wire Line
-	2050 4950 3550 4950
-Connection ~ 3550 4950
-Connection ~ 3550 5050
+	3050 5150 3050 5200
+Wire Wire Line
+	3500 5200 3500 5150
+Wire Wire Line
+	3500 5150 3800 5150
+Wire Wire Line
+	3800 5150 3800 5200
+Wire Wire Line
+	3650 4950 3650 5150
+Connection ~ 3650 5150
+Wire Wire Line
+	3500 5500 3500 5550
+Wire Wire Line
+	3500 5550 3800 5550
+Wire Wire Line
+	3800 5550 3800 5500
+Wire Wire Line
+	3650 5550 3650 5650
+Connection ~ 3650 5550
+Wire Wire Line
+	2050 4950 3650 4950
+Connection ~ 3650 5050
 Wire Wire Line
 	8450 4800 8350 4800
@@
 	3150 1800 3300 1800
 Wire Wire Line
-	3550 5050 2650 5050
+	3650 5050 2750 5050
 Wire Wire Line
 	8350 2000 8450 2000
@@
 	9450 1800 10350 1800
 Wire Wire Line
-	2350 1900 2350 1500
+	2350 1300 2350 1900
 Wire Wire Line
 	2350 1500 1500 1500
@@
 F 2 "Crystals:Crystal_SMD_2520-4pin_2.5x2.0mm" H 4650 2250 50  0001 C CNN
 F 3 "" H 4650 2250 50  0001 C CNN
+F 4 "XTAL-003" V 4650 2250 60  0001 C CNN "part_num"
 	1    4650 2250
 	0    1    1    0
@@
 Wire Wire Line
 	4400 2250 4450 2250
+Text HLabel 2550 1300 2    60   Output ~ 0
+USB_VBUS
+Wire Wire Line
+	2550 1300 2350 1300
+Connection ~ 2350 1500
 $EndSCHEMATC

Commit message: Bug Fixes
Fixed some missing connections related to the USB Interface.
Connections:
- net labels removed: UART1_CTS, UART1_RTS, UART2_CTS, UART2_RTS
- wire segments 123 -> 119
- no-connect marks 23 -> 28
Changed lines of the file:
@@
 	1    0    0    -1
 $EndComp
-Text HLabel 8350 5000 0    60   Input ~ 0
-UART1_RTS
-Text HLabel 8350 5100 0    60   Input ~ 0
-UART1_CTS
-Text HLabel 9550 5000 2    60   Input ~ 0
-UART2_RTS
-Text HLabel 9550 5100 2    60   Input ~ 0
-UART2_CTS
 $Comp
 L R R?
@@
 Wire Wire Line
 	9450 4900 9550 4900
-Wire Wire Line
-	9450 5000 9550 5000
-Wire Wire Line
-	9450 5100 9550 5100
-Wire Wire Line
-	8450 5000 8350 5000
-Wire Wire Line
-	8350 5100 8450 5100
 Wire Wire Line
 	3300 1700 3150 1700
@@
 	2550 1300 2350 1300
 Connection ~ 2350 1500
+NoConn ~ 9450 5000
+NoConn ~ 9450 5100
+NoConn ~ 8450 5100
+NoConn ~ 8450 5000
+NoConn ~ 1500 1900
 $EndSCHEMATC

Commit message: Updated Part Number
Parts:
- J?: part_num CONN-11 -> CONN-12
Changed lines of the file:
@@
 F 2 "WARG-kicad:USB_Micro-B_10118194-0001LF" H 1250 1200 50  0001 C CNN
 F 3 "" H 1350 1650 50  0001 C CNN
-F 4 "CONN-11" H 1200 2100 60  0000 C CNN "part_num"
+F 4 "CONN-12" H 1200 2100 60  0000 C CNN "part_num"
 	1    1200 1700
 	1    0    0    -1

Commit message: Added Test Points for USB Interface
Added JTAG and UART test points for the FT4232H
Connections:
- net labels added: GPIOL0_A, GPIOL0_B, TCK_A, TCK_B, TDI_A, TDI_B, TDO_A, TDO_B, TMS_A, TMS_B, UART1_CTS, UART1_RTS, UART2_CTS, UART2_RTS
- net labels removed: SWD1_TCK, SWD1_TDI, SWD2_TCK, SWD2_TDI
- wire segments 119 -> 129
- no-connect marks 28 -> 18
Changed lines of the file:
@@
-$Comp
-L FT4232H U?
-U 1 1 5B18A9C2
-P 8950 2150
-F 0 "U?" H 8950 3050 60  0000 C CNN
-F 1 "FT4232H" H 8950 3200 60  0000 C CNN
-F 2 "Housings_QFP:LQFP-64_10x10mm_Pitch0.5mm" H 8950 1400 60  0001 C CNN
-F 3 "" H 8350 1800 60  0001 C CNN
-F 4 "CHIP-005" H 8950 2900 60  0000 C CNN "part_num"
-	1    8950 2150
-	1    0    0    -1
-$EndComp
 $Comp
 L FT4232H U?
@@
 NoConn ~ 4300 1800
 NoConn ~ 4300 1900
-NoConn ~ 9450 2100
-NoConn ~ 9450 2200
-NoConn ~ 9450 2300
 NoConn ~ 9450 2400
 NoConn ~ 9450 2500
 NoConn ~ 8450 2500
 NoConn ~ 8450 2400
-NoConn ~ 8450 2300
-NoConn ~ 8450 2200
-NoConn ~ 8450 2100
 NoConn ~ 9450 5200
 NoConn ~ 9450 5300
@@
 $EndComp
 Text HLabel 7550 1800 0    60   Input ~ 0
-SWD1_TCK
+TCK_A
 Text HLabel 7550 1900 0    60   Input ~ 0
-SWD1_TDI
+TDI_A
 $Comp
 L R R?
@@
 $EndComp
 Text HLabel 10350 1800 2    60   Input ~ 0
-SWD2_TCK
+TCK_B
 Text HLabel 10350 1900 2    60   Input ~ 0
-SWD2_TDI
+TDI_B
 $Comp
 L R R?
@@
 	2550 1300 2350 1300
 Connection ~ 2350 1500
-NoConn ~ 9450 5000
-NoConn ~ 9450 5100
-NoConn ~ 8450 5100
-NoConn ~ 8450 5000
 NoConn ~ 1500 1900
+Text HLabel 7550 2100 0    60   Input ~ 0
+TDO_A
+Text HLabel 7550 2200 0    60   Input ~ 0
+TMS_A
+Text HLabel 10350 2100 2    60   Input ~ 0
+TDO_B
+Text HLabel 10350 2200 2    60   Input ~ 0
+TMS_B
+Wire Wire Line
+	10350 2100 9450 2100
+Wire Wire Line
+	9450 2200 10350 2200
+Wire Wire Line
+	8450 2100 7550 2100
+Wire Wire Line
+	7550 2200 8450 2200
+$Comp
+L FT4232H U?
+U 1 1 5B18A9C2
+P 8950 2150
+F 0 "U?" H 8950 3050 60  0000 C CNN
+F 1 "FT4232H" H 8950 3200 60  0000 C CNN
+F 2 "Housings_QFP:LQFP-64_10x10mm_Pitch0.5mm" H 8950 1400 60  0001 C CNN
+F 3 "" H 8350 1800 60  0001 C CNN
+F 4 "CHIP-005" H 8950 2900 60  0000 C CNN "part_num"
+	1    8950 2150
+	1    0    0    -1
+$EndComp
+Text HLabel 10350 2300 2    60   Input ~ 0
+GPIOL0_B
+Text HLabel 7550 2300 0    60   Input ~ 0
+GPIOL0_A
+Wire Wire Line
+	9450 2300 10350 2300
+Wire Wire Line
+	7550 2300 8450 2300
+Text HLabel 9550 5000 2    60   Output ~ 0
+UART2_RTS
+Text HLabel 9550 5100 2    60   Input ~ 0
+UART2_CTS
+Text HLabel 8350 5000 0    60   Output ~ 0
+UART1_RTS
+Text HLabel 8350 5100 0    60   Input ~ 0
+UART1_CTS
+Wire Wire Line
+	9450 5000 9550 5000
+Wire Wire Line
+	9450 5100 9550 5100
+Wire Wire Line
+	8450 5000 8350 5000
+Wire Wire Line
+	8350 5100 8450 5100
 $EndSCHEMATC
