File: Hardware/USB INTERFACE.sch (KiCad schematic (older format))
At the start: 34 parts, among them J15 USB_MICRO_B, U14 FT4232H, Y5 Crystal_GND24

Commit message: Updated Resistors
Changed 1K resistors on DBUS1 lines to 220R resistors and 100R resistors on DBUS2 lines to 0R resistors, on the FT4232H.
Parts:
- R43, R46: value 1K -> 220R; part_num RESS-012 -> RESS-014
- R44, R45: value 100R -> 0R; part_num RESS-006 -> RESS-001
Other:
- moved on the sheet: R43, R46

Commit message: Fixed Bugs
Noticed my part numbers in the library had been overwritten, so updated to reflect adding them back with new numbers. Also fixed typo with TVS diodes.
Parts:
- C73, C74: part_num CAPP-014 -> CAPP-011
- D12, D13: value 600R -> TVS; part_num INDU-002 -> DIOD-006
- R37: part_num RESS-013 -> RESS-015
- R39: part_num RESS-014 -> RESS-016
- R40, R41: part_num RESS-015 -> RESS-018
- R42: part_num RESS-012 -> RESS-017
Changed lines of the file:
@@
 P 1750 2100
 F 0 "D12" H 1750 2200 50  0000 C CNN
-F 1 "600R" H 1750 2000 50  0000 C CNN
+F 1 "TVS" H 1750 2000 50  0000 C CNN
 F 2 "Resistors_SMD:R_0603_HandSoldering" H 1750 2100 50  0001 C CNN
 F 3 "" H 1750 2100 50  0001 C CNN
-F 4 "INDU-002" H 1750 2100 60  0001 C CNN "part_num"
+F 4 "DIOD-006" H 1750 2100 60  0001 C CNN "part_num"
 	1    1750 2100
 	0    1    1    0
@@
 F 2 "Resistors_SMD:R_0603_HandSoldering" V 2280 2050 50  0001 C CNN
 F 3 "" H 2350 2050 50  0001 C CNN
-F 4 "RESS-013" V 2350 2050 60  0001 C CNN "part_num"
+F 4 "RESS-015" V 2350 2050 60  0001 C CNN "part_num"
 	1    2350 2050
 	1    0    0    -1
@@
 F 2 "Resistors_SMD:R_0603_HandSoldering" H 5338 2600 50  0001 C CNN
 F 3 "" H 5300 2750 50  0001 C CNN
-F 4 "CAPP-014" H 5300 2750 60  0001 C CNN "part_num"
+F 4 "CAPP-011" H 5300 2750 60  0001 C CNN "part_num"
 	1    5300 2750
 	1    0    0    -1
@@
 P 2050 2100
 F 0 "D13" H 2050 2200 50  0000 C CNN
-F 1 "600R" H 2050 2000 50  0000 C CNN
+F 1 "TVS" H 2050 2000 50  0000 C CNN
 F 2 "Resistors_SMD:R_0603_HandSoldering" H 2050 2100 50  0001 C CNN
 F 3 "" H 2050 2100 50  0001 C CNN
-F 4 "INDU-002" H 2050 2100 60  0001 C CNN "part_num"
+F 4 "DIOD-006" H 2050 2100 60  0001 C CNN "part_num"
 	1    2050 2100
 	0    1    1    0
@@
 F 2 "Resistors_SMD:R_0603_HandSoldering" V 2580 2650 50  0001 C CNN
 F 3 "" H 2650 2650 50  0001 C CNN
-F 4 "RESS-014" V 2650 2650 60  0001 C CNN "part_num"
+F 4 "RESS-016" V 2650 2650 60  0001 C CNN "part_num"
 	1    2650 2650
 	1    0    0    -1
@@
 F 2 "Resistors_SMD:R_0603_HandSoldering" V 2930 2350 50  0001 C CNN
 F 3 "" H 3000 2350 50  0001 C CNN
-F 4 "RESS-012" V 3000 2350 60  0001 C CNN "part_num"
+F 4 "RESS-017" V 3000 2350 60  0001 C CNN "part_num"
 	1    3000 2350
 	0    1    1    0
@@
 F 2 "Resistors_SMD:R_0603_HandSoldering" H 5588 2600 50  0001 C CNN
 F 3 "" H 5550 2750 50  0001 C CNN
-F 4 "CAPP-014" H 5550 2750 60  0001 C CNN "part_num"
+F 4 "CAPP-011" H 5550 2750 60  0001 C CNN "part_num"
 	1    5550 2750
 	1    0    0    -1
@@
 F 2 "Resistors_SMD:R_0603_HandSoldering" V 2930 1700 50  0001 C CNN
 F 3 "" H 3000 1700 50  0001 C CNN
-F 4 "RESS-015" V 3000 1700 60  0001 C CNN "part_num"
+F 4 "RESS-018" V 3000 1700 60  0001 C CNN "part_num"
 	1    3000 1700
 	0    1    1    0
@@
 F 2 "Resistors_SMD:R_0603_HandSoldering" V 2930 1800 50  0001 C CNN
 F 3 "" H 3000 1800 50  0001 C CNN
-F 4 "RESS-015" V 3000 1800 60  0001 C CNN "part_num"
+F 4 "RESS-018" V 3000 1800 60  0001 C CNN "part_num"
 	1    3000 1800
 	0    1    1    0

Commit message: Fixed one more bug
Fixed overwritten part num
Parts:
- J15: part_num CONN-011 -> CONN-012
Changed lines of the file:
@@
 F 2 "WARG:USB_Micro-B_10118194-0001LF" H 1250 1200 50  0001 C CNN
 F 3 "" H 1350 1650 50  0001 C CNN
-F 4 "CONN-011" H 1200 2100 60  0000 C CNN "part_num"
+F 4 "CONN-012" H 1200 2100 60  0000 C CNN "part_num"
 	1    1200 1700
 	1    0    0    -1

Commit message: Remapped symbols for KiCAD 5.0.x
Parts:
- C?: renamed from C73; symbol C -> Device:C
- C?: renamed from C74; symbol C -> Device:C
- C?: renamed from C63; symbol C -> Device:C
- C?: renamed from C71; symbol C -> Device:C
- C?: renamed from C65; symbol C -> Device:C
- C?: renamed from C66; symbol C -> Device:C
- C?: renamed from C60; symbol C -> Device:C
- C?: renamed from C61; symbol C -> Device:C
- C?: renamed from C62; symbol C -> Device:C
- C?: renamed from C72; symbol C -> Device:C
- C?: renamed from C69; symbol C -> Device:C
- C?: renamed from C70; symbol C -> Device:C
- C?: renamed from C76; symbol C -> Device:C
- C?: renamed from C75; symbol C -> Device:C
- C?: renamed from C64; symbol C -> Device:C
- C?: renamed from C67; symbol C -> Device:C
- C?: renamed from C68; symbol C -> Device:C
- D?: renamed from D12; symbol D_TVS -> Device:D_TVS
- D?: renamed from D13; symbol D_TVS -> Device:D_TVS
- J?: renamed from J15; symbol USB_MICRO_B -> Connector:USB_B_Micro
- L?: renamed from L4; symbol L_Core_Ferrite -> Device:L_Core_Ferrite
- L?: renamed from L3; symbol L_Core_Ferrite -> Device:L_Core_Ferrite
- R?: renamed from R37; symbol R -> Device:R
- R?: renamed from R38; symbol R -> Device:R
- R?: renamed from R39; symbol R -> Device:R
- R?: renamed from R42; symbol R -> Device:R
- R?: renamed from R40; symbol R -> Device:R
- R?: renamed from R41; symbol R -> Device:R
- R?: renamed from R44; symbol R -> Device:R
- R?: renamed from R43; symbol R -> Device:R
- R?: renamed from R45; symbol R -> Device:R
- R?: renamed from R46; symbol R -> Device:R
- U? (x4): renamed from U14; symbol FT4232H -> WARG:FT4232H
- Y?: renamed from Y5; symbol Crystal_GND24 -> Device:Crystal_GND24
Connections:
- wire segments 129 -> 182

Commit message: Added RSSI, datasheets, INDU-004
Added RSSI input to PPM connector. Added datasheets for most of the components. The filter inductors for the FTDI were labeled as INDU-002, which is a 15uH smps inductor.
Parts:
- C? (x17): footprint Resistors_SMD:R_0603_HandSoldering -> Capacitors_SMD:C_0603_HandSoldering
- D? (x2): footprint Resistors_SMD:R_0603_HandSoldering -> Diodes_SMD:D_0603
- L? (x2): footprint Resistors_SMD:R_0603_HandSoldering -> Inductors_SMD:L_0603_HandSoldering
- R?: value 4.7k -> 4.7K
- R?: value 10k -> 10K
- R?: value 12k -> 12K
- R?: value 1k -> 1K
- R? (x2): value 10R -> 10
- R? (x2): value 0R -> 0
- R? (x2): value 220R -> 220
Connections:
- wire segments 182 -> 183
Other:
- note added: "Add OV and OC protection."
- moved on the sheet: R?

Commit message: Added protection diode to USB
Parts:
- added D?: D_Schottky, Diodes_SMD:D_SOD-123F, symbol Device:D_Schottky
Connections:
- wire segments 183 -> 185
Changed lines of the file:
@@
 L Device:D_TVS D?
 U 1 1 5B18DE9F
-P 1750 2100
-F 0 "D?" H 1750 2200 50  0000 C CNN
-F 1 "TVS" H 1750 2000 50  0000 C CNN
-F 2 "Diodes_SMD:D_0603" H 1750 2100 50  0001 C CNN
-F 3 "https://www.littelfuse.com/data/en/data_sheets/littelfuse_pulseguard-esd_pgb1.pdf" H 1750 2100 50  0001 C CNN
-F 4 "DIOD-006" H 1750 2100 60  0001 C CNN "part_num"
-	1    1750 2100
+P 1650 2100
+F 0 "D?" H 1650 2200 50  0000 C CNN
+F 1 "TVS" H 1650 2000 50  0000 C CNN
+F 2 "Diodes_SMD:D_0603" H 1650 2100 50  0001 C CNN
+F 3 "https://www.littelfuse.com/data/en/data_sheets/littelfuse_pulseguard-esd_pgb1.pdf" H 1650 2100 50  0001 C CNN
+F 4 "DIOD-006" H 1650 2100 60  0001 C CNN "part_num"
+	1    1650 2100
 	0    1    1    0
 $EndComp
@@
 L Device:D_TVS D?
 U 1 1 5B192B88
-P 2050 2100
-F 0 "D?" H 2050 2200 50  0000 C CNN
-F 1 "TVS" H 2050 2000 50  0000 C CNN
-F 2 "Diodes_SMD:D_0603" H 2050 2100 50  0001 C CNN
-F 3 "https://www.littelfuse.com/data/en/data_sheets/littelfuse_pulseguard-esd_pgb1.pdf" H 2050 2100 50  0001 C CNN
-F 4 "DIOD-006" H 2050 2100 60  0001 C CNN "part_num"
-	1    2050 2100
+P 1950 2100
+F 0 "D?" H 1950 2200 50  0000 C CNN
+F 1 "TVS" H 1950 2000 50  0000 C CNN
+F 2 "Diodes_SMD:D_0603" H 1950 2100 50  0001 C CNN
+F 3 "https://www.littelfuse.com/data/en/data_sheets/littelfuse_pulseguard-esd_pgb1.pdf" H 1950 2100 50  0001 C CNN
+F 4 "DIOD-006" H 1950 2100 60  0001 C CNN "part_num"
+	1    1950 2100
 	0    1    1    0
 $EndComp
@@
 UART1_CTS
 Wire Wire Line
-	1500 1700 2050 1700
-Wire Wire Line
-	1500 1800 1750 1800
-Wire Wire Line
-	1750 1800 1750 1950
-Connection ~ 1750 1800
-Wire Wire Line
-	2050 1700 2050 1950
-Connection ~ 2050 1700
-Wire Wire Line
 	2550 2200 2550 2350
 Wire Wire Line
@@
 	2800 2000 3300 2000
 Wire Wire Line
-	2050 2350 2050 2250
-Wire Wire Line
 	1100 2350 1200 2350
 Wire Wire Line
-	1750 2250 1750 2350
-Wire Wire Line
 	1200 2350 1200 2100
-Connection ~ 1750 2350
 Wire Wire Line
 	1100 2100 1100 2350
@@
 	2350 1300 2350 1500
 Wire Wire Line
-	2350 1500 1500 1500
-Wire Wire Line
 	8050 2000 7650 2000
 Wire Wire Line
@@
 Connection ~ 7650 1900
 Wire Wire Line
-	1750 1800 2850 1800
-Wire Wire Line
-	2050 1700 2850 1700
-Wire Wire Line
 	2550 2350 2550 2500
 Wire Wire Line
-	1750 2350 2050 2350
-Wire Wire Line
 	1750 2350 1750 2600
 Wire Wire Line
-	1200 2350 1750 2350
+	1200 2350 1650 2350
 Wire Wire Line
 	5550 3000 5550 3100
@@
 Wire Wire Line
 	2550 1500 2550 1900
-Connection ~ 2350 1500
 Text Notes 1650 1100 0    60   ~ 0
 Add OV and OC protection.
+Wire Wire Line
+	1500 1700 1950 1700
+Wire Wire Line
+	1650 2250 1650 2350
+Wire Wire Line
+	1500 1800 1650 1800
+Connection ~ 1650 2350
+Wire Wire Line
+	1650 2350 1750 2350
+Wire Wire Line
+	1750 2350 1950 2350
+Wire Wire Line
+	1950 2350 1950 2250
+Connection ~ 1750 2350
+Wire Wire Line
+	1650 1950 1650 1800
+Connection ~ 1650 1800
+Wire Wire Line
+	1650 1800 2850 1800
+Wire Wire Line
+	1950 1950 1950 1700
+Connection ~ 1950 1700
+Wire Wire Line
+	1950 1700 2850 1700
+$Comp
+L Device:D_Schottky D?
+U 1 1 5CC2FB03
+P 1800 1500
+F 0 "D?" H 1800 1284 50  0000 C CNN
+F 1 "D_Schottky" H 1800 1375 50  0000 C CNN
+F 2 "Diodes_SMD:D_SOD-123F" H 1800 1500 50  0001 C CNN
+F 3 "http://www.onsemi.com/pub/Collateral/MBR120VLSFT1-D.PDF" H 1800 1500 50  0001 C CNN
+F 4 "DIOD-007" H 0   0   50  0001 C CNN "part_num"
+	1    1800 1500
+	-1   0    0    1
+$EndComp
+Wire Wire Line
+	1500 1500 1650 1500
+Wire Wire Line
+	1950 1500 2350 1500
+Connection ~ 2350 1500
 $EndSCHEMATC
