File: Hardware/USB INTERFACE.sch (KiCad schematic (older format))
At the start: 38 parts

Commit message: Generated netlist and board outline
Parts:
- gave numbers to parts that had none: 35

Commit message: Initial Routing of Zeropilot Rev1
This is the initial routing of the board. It needs to be cleaned up slightly, but library references are screwed up so they will be fixed first.
Parts:
- removed D14: D_Schottky, Diodes_SMD:D_SOD-123F, symbol Device:D_Schottky
Connections:
- wire segments 185 -> 183
Other:
- note removed: "Add OV and OC protection."
Changed lines of the file:
@@
 EESchema Schematic File Version 4
-LIBS:ZeroPilot-cache
-EELAYER 26 0
+EELAYER 29 0
 EELAYER END
 $Descr A4 11693 8268
@@
 TDI1
 $Comp
-L Device:R R48
-U 1 1 5B25A964
-P 8200 2000
-F 0 "R48" V 8250 1800 50  0000 C CNN
-F 1 "0" V 8200 2000 50  0000 C CNN
-F 2 "Resistors_SMD:R_0603_HandSoldering" V 8130 2000 50  0001 C CNN
-F 3 "http://www.yageo.com/documents/recent/PYu-RC_Group_51_RoHS_L_10.pdf" H 8200 2000 50  0001 C CNN
-F 4 "RESS-001" V 8200 2000 60  0001 C CNN "part_num"
-	1    8200 2000
-	0    1    1    0
-$EndComp
-$Comp
 L Device:R R47
 U 1 1 5B25BD92
@@
 TDI2
 $Comp
-L Device:R R49
-U 1 1 5B25CA6C
-P 9700 2000
-F 0 "R49" V 9750 1800 50  0000 C CNN
-F 1 "0" V 9700 2000 50  0000 C CNN
-F 2 "Resistors_SMD:R_0603_HandSoldering" V 9630 2000 50  0001 C CNN
-F 3 "http://www.yageo.com/documents/recent/PYu-RC_Group_51_RoHS_L_10.pdf" H 9700 2000 50  0001 C CNN
-F 4 "RESS-001" V 9700 2000 60  0001 C CNN "part_num"
-	1    9700 2000
-	0    -1   1    0
-$EndComp
-$Comp
 L Device:R R50
 U 1 1 5B25CA74
@@
 	1    0    0    -1
 $EndComp
-Text HLabel 2550 1300 2    60   Output ~ 0
+Text HLabel 2750 1300 2    60   Output ~ 0
 USB_VBUS
 NoConn ~ 1500 1900
@@
 	8350 2000 8450 2000
 Wire Wire Line
-	8100 1900 8450 1900
-Wire Wire Line
 	7550 1800 8450 1800
 Wire Wire Line
@@
 	9450 1800 10350 1800
 Wire Wire Line
-	2350 1300 2350 1500
+	2550 1300 2550 1500
 Wire Wire Line
 	8050 2000 7650 2000
@@
 	4400 2250 4450 2250
 Wire Wire Line
-	2550 1300 2350 1300
+	2750 1300 2550 1300
 Wire Wire Line
 	10350 2100 9450 2100
@@
 	7650 1900 7800 1900
 Wire Wire Line
-	2350 1500 2550 1500
-Wire Wire Line
-	2550 1500 2550 1900
-Text Notes 1650 1100 0    60   ~ 0
-Add OV and OC protection.
-Wire Wire Line
 	1500 1700 1950 1700
 Wire Wire Line
@@
 Wire Wire Line
 	1950 1700 2850 1700
-$Comp
-L Device:D_Schottky D14
-U 1 1 5CC2FB03
-P 1800 1500
-F 0 "D14" H 1800 1284 50  0000 C CNN
-F 1 "D_Schottky" H 1800 1375 50  0000 C CNN
-F 2 "Diodes_SMD:D_SOD-123F" H 1800 1500 50  0001 C CNN
-F 3 "http://www.onsemi.com/pub/Collateral/MBR120VLSFT1-D.PDF" H 1800 1500 50  0001 C CNN
-F 4 "DIOD-007" H 0   0   50  0001 C CNN "part_num"
-	1    1800 1500
-	-1   0    0    1
-$EndComp
-Wire Wire Line
-	1500 1500 1650 1500
-Wire Wire Line
-	1950 1500 2350 1500
-Connection ~ 2350 1500
+Wire Wire Line
+	8100 1900 8450 1900
+$Comp
+L Device:R R49
+U 1 1 5B25CA6C
+P 9700 2000
+F 0 "R49" V 9750 1800 50  0000 C CNN
+F 1 "0" V 9700 2000 50  0000 C CNN
+F 2 "Resistors_SMD:R_0603_HandSoldering" V 9630 2000 50  0001 C CNN
+F 3 "http://www.yageo.com/documents/recent/PYu-RC_Group_51_RoHS_L_10.pdf" H 9700 2000 50  0001 C CNN
+F 4 "RESS-001" V 9700 2000 60  0001 C CNN "part_num"
+	1    9700 2000
+	0    -1   1    0
+$EndComp
+$Comp
+L Device:R R48
+U 1 1 5B25A964
+P 8200 2000
+F 0 "R48" V 8250 1800 50  0000 C CNN
+F 1 "0" V 8200 2000 50  0000 C CNN
+F 2 "Resistors_SMD:R_0603_HandSoldering" V 8130 2000 50  0001 C CNN
+F 3 "http://www.yageo.com/documents/recent/PYu-RC_Group_51_RoHS_L_10.pdf" H 8200 2000 50  0001 C CNN
+F 4 "RESS-001" V 8200 2000 60  0001 C CNN "part_num"
+	1    8200 2000
+	0    1    1    0
+$EndComp
+Wire Wire Line
+	2550 1900 2550 1500
+Wire Wire Line
+	1500 1500 2550 1500
+Connection ~ 2550 1500
 $EndSCHEMATC

Commit message: Updated Footprints
Updated the footprints to 5.1, added 3D models to all components.
Parts:
- C60, C61, C62, C63, C64, C65, C66, C67, C68, C69, C70, C71, C72, C73, C74, C75, C76: footprint Capacitors_SMD:C_0603_HandSoldering -> Capacitor_SMD:C_0603_1608Metric_Pad1.05x0.95mm_HandSolder
- D13, D15: footprint Diodes_SMD:D_0603 -> Diode_SMD:D_0603_1608Metric_Pad1.05x0.95mm_HandSolder
- L3, L4: footprint Inductors_SMD:L_0603_HandSoldering -> Inductor_SMD:L_0603_1608Metric_Pad1.05x0.95mm_HandSolder; part_num INDU-002 -> INDU-004
- R41, R42, R43, R44, R45, R46, R47, R48, R49, R50: footprint Resistors_SMD:R_0603_HandSoldering -> Resistor_SMD:R_0603_1608Metric_Pad1.05x0.95mm_HandSolder
- U14: footprint Housings_QFP:LQFP-64_10x10mm_Pitch0.5mm -> Package_QFP:LQFP-64_10x10mm_P0.5mm
- Y5: footprint Crystals:Crystal_SMD_2520-4pin_2.5x2.0mm -> Crystal:Crystal_SMD_2520-4Pin_2.5x2.0mm

Commit message: Bug fixes
Parts:
- C68: value 4.7uF -> 3.3uF; part_num CAPP-006 -> CAPP-015
Connections:
- wire segments 183 -> 184
Changed lines of the file:
@@
-$EndComp
-$Comp
-L power:GND #PWR053
-U 1 1 5B1ACB05
-P 2100 6500
-F 0 "#PWR053" H 2100 6250 50  0001 C CNN
-F 1 "GND" H 2100 6350 50  0000 C CNN
-F 2 "" H 2100 6500 50  0001 C CNN
-F 3 "" H 2100 6500 50  0001 C CNN
-	1    2100 6500
-	1    0    0    -1
 $EndComp
 $Comp
@@
 P 3800 5350
 F 0 "C68" H 3825 5450 50  0000 L CNN
-F 1 "4.7uF" H 3825 5250 50  0000 L CNN
+F 1 "3.3uF" H 3825 5250 50  0000 L CNN
 F 2 "Capacitor_SMD:C_0603_1608Metric_Pad1.05x0.95mm_HandSolder" H 3838 5200 50  0001 C CNN
-F 3 "http://www.samsungsem.com/kr/support/product-search/mlcc/CL10A475MP5LNNC.jsp" H 3800 5350 50  0001 C CNN
-F 4 "CAPP-006" H 3800 5350 60  0001 C CNN "part_num"
+F 3 "http://www.samsungsem.com/kr/support/product-search/mlcc/CL10A335KP8NNNC.jsp" H 3800 5350 50  0001 C CNN
+F 4 "CAPP-015" H 3800 5350 60  0001 C CNN "part_num"
 	1    3800 5350
 	1    0    0    -1
@@
 Connection ~ 2250 6350
 Wire Wire Line
-	2100 6350 2100 6500
-Connection ~ 2100 6350
-Wire Wire Line
 	2750 5500 2750 5550
 Wire Wire Line
@@
 	2250 5950 2550 5950
 Wire Wire Line
-	1950 6350 2100 6350
-Wire Wire Line
 	2250 6350 2550 6350
-Wire Wire Line
-	2100 6350 2250 6350
 Wire Wire Line
 	2750 5550 2750 5650
@@
 	1500 1500 2550 1500
 Connection ~ 2550 1500
+Wire Wire Line
+	2100 6350 2250 6350
+Wire Wire Line
+	1950 6350 2100 6350
+Connection ~ 2100 6350
+Wire Wire Line
+	2100 6350 2100 6500
+$Comp
+L power:GND #PWR053
+U 1 1 5B1ACB05
+P 2100 6500
+F 0 "#PWR053" H 2100 6250 50  0001 C CNN
+F 1 "GND" H 2100 6350 50  0000 C CNN
+F 2 "" H 2100 6500 50  0001 C CNN
+F 3 "" H 2100 6500 50  0001 C CNN
+	1    2100 6500
+	1    0    0    -1
+$EndComp
+Wire Wire Line
+	2550 5950 3050 5950
+Connection ~ 2550 5950
+Text HLabel 3050 5950 2    60   Input ~ 0
+VDD
 $EndSCHEMATC

Commit message: Fixes
Parts:
- renumbered C60 to C48, C61 to C49, C62 to C50, C63 to C51, C64 to C52, C65 to C53, C66 to C54, C67 to C55, C68 to C56, C69 to C57, C70 to C58, C71 to C59, C72 to C60, C73 to C61, C74 to C62, C75 to C63, C76 to C64, D13 to D10, D15 to D11, R41 to R34, R42 to R35, R43 to R36, R44 to R37, R45 to R38, R46 to R39, R47 to R40, R48 to R41, R49 to R42, R50 to R43, U14 to U8, Y5 to Y3
