File: Hardware/PWM_1-12.sch (KiCad schematic (older format))
At the start: 12 parts, among them J10 74099-0603, J11 74099-0603, J12 74099-0603, J13 74099-0603, J2 74099-0603, J3 74099-0603, J4 74099-0603, J5 74099-0603, J6 74099-0603, J7 74099-0603, J8 74099-0603, J9 74099-0603

Commit message: Fixed merge issues
Parts:
- renumbered J2 to J1, J11 to J10, J12 to J11, J13 to J12, J3 to J2, J4 to J3, J5 to J4, J6 to J5, J7 to J6, J8 to J7, J9 to J8, J10 to J9
Changed lines of the file:
@@
 LIBS:contrib
 LIBS:valves
+LIBS:ZeroPilot-cache
 EELAYER 25 0
 EELAYER END
@@
 PWM_5V
 $Comp
-L Conn_01x03 J2
+L Conn_01x03 J1
 U 1 1 597DAC0F
 P 2900 1150
-AR Path="/597DAC0F" Ref="J2"  Part="1"
-AR Path="/591E6415/597DAC0F" Ref="J2"  Part="1"
-F 0 "J2" H 2900 1350 50  0000 C CNN
+F 0 "J1" H 2900 1350 50  0000 C CNN
 F 1 "74099-0603" V 3000 1150 50  0000 C CNN
 F 2 "WARG:74099-0603" H 2900 1150 50  0001 C CNN
@@
 $EndComp
 $Comp
-L Conn_01x03 J3
+L Conn_01x03 J2
 U 1 1 597DAC47
 P 2900 2600
-AR Path="/597DAC47" Ref="J3"  Part="1"
-AR Path="/591E6415/597DAC47" Ref="J3"  Part="1"
-F 0 "J3" H 2900 2800 50  0000 C CNN
+F 0 "J2" H 2900 2800 50  0000 C CNN
 F 1 "74099-0603" V 3000 2600 50  0000 C CNN
 F 2 "WARG:74099-0603" H 2900 2600 50  0001 C CNN
@@
 $EndComp
 $Comp
-L GND #PWR3
+L GND #PWR03
 U 1 1 597DB10B
 P 2300 5900
-F 0 "#PWR3" H 2300 5650 50  0001 C CNN
+F 0 "#PWR03" H 2300 5650 50  0001 C CNN
 F 1 "GND" H 2300 5750 50  0000 C CNN
 F 2 "" H 2300 5900 50  0001 C CNN
@@
 Connection ~ 2300 5450
 $Comp
-L GND #PWR4
+L GND #PWR04
 U 1 1 597DB1D3
 P 5000 5900
-F 0 "#PWR4" H 5000 5650 50  0001 C CNN
+F 0 "#PWR04" H 5000 5650 50  0001 C CNN
 F 1 "GND" H 5000 5750 50  0000 C CNN
 F 2 "" H 5000 5900 50  0001 C CNN
@@
 $EndComp
 $Comp
-L GND #PWR5
+L GND #PWR05
 U 1 1 597DB202
 P 7850 5800
-F 0 "#PWR5" H 7850 5550 50  0001 C CNN
+F 0 "#PWR05" H 7850 5550 50  0001 C CNN
 F 1 "GND" H 7850 5650 50  0000 C CNN
 F 2 "" H 7850 5800 50  0001 C CNN
@@
 Connection ~ 5000 2500
 $Comp
-L Conn_01x03 J4
+L Conn_01x03 J3
 U 1 1 5B1918E4
 P 2900 4100
-F 0 "J4" H 2900 4300 50  0000 C CNN
+F 0 "J3" H 2900 4300 50  0000 C CNN
 F 1 "74099-0603" V 3000 4100 50  0000 C CNN
 F 2 "WARG:74099-0603" H 2900 4100 50  0001 C CNN
@@
 $EndComp
 $Comp
-L Conn_01x03 J5
+L Conn_01x03 J4
 U 1 1 5B191B06
 P 2900 5550
-F 0 "J5" H 2900 5750 50  0000 C CNN
+F 0 "J4" H 2900 5750 50  0000 C CNN
 F 1 "74099-0603" V 3000 5550 50  0000 C CNN
 F 2 "WARG:74099-0603" H 2900 5550 50  0001 C CNN
@@
 $EndComp
 $Comp
-L Conn_01x03 J6
+L Conn_01x03 J5
 U 1 1 5B191E1C
 P 5600 1150
-F 0 "J6" H 5600 1350 50  0000 C CNN
+F 0 "J5" H 5600 1350 50  0000 C CNN
 F 1 "74099-0603" V 5700 1150 50  0000 C CNN
 F 2 "WARG:74099-0603" H 5600 1150 50  0001 C CNN
@@
 $EndComp
 $Comp
-L Conn_01x03 J7
+L Conn_01x03 J6
 U 1 1 5B191E94
 P 5600 2600
-F 0 "J7" H 5600 2800 50  0000 C CNN
+F 0 "J6" H 5600 2800 50  0000 C CNN
 F 1 "74099-0603" V 5700 2600 50  0000 C CNN
 F 2 "WARG:74099-0603" H 5600 2600 50  0001 C CNN
@@
 $EndComp
 $Comp
-L Conn_01x03 J8
+L Conn_01x03 J7
 U 1 1 5B191F57
 P 5600 4100
-F 0 "J8" H 5600 4300 50  0000 C CNN
+F 0 "J7" H 5600 4300 50  0000 C CNN
 F 1 "74099-0603" V 5700 4100 50  0000 C CNN
 F 2 "WARG:74099-0603" H 5600 4100 50  0001 C CNN
@@
 $EndComp
 $Comp
-L Conn_01x03 J9
+L Conn_01x03 J8
 U 1 1 5B1920C6
 P 5600 5550
-F 0 "J9" H 5600 5750 50  0000 C CNN
+F 0 "J8" H 5600 5750 50  0000 C CNN
 F 1 "74099-0603" V 5700 5550 50  0000 C CNN
 F 2 "WARG:74099-0603" H 5600 5550 50  0001 C CNN
@@
 $EndComp
 $Comp
-L Conn_01x03 J10
+L Conn_01x03 J9
 U 1 1 5B192277
 P 8450 1150
-F 0 "J10" H 8450 1350 50  0000 C CNN
+F 0 "J9" H 8450 1350 50  0000 C CNN
 F 1 "74099-0603" V 8550 1150 50  0000 C CNN
 F 2 "WARG:74099-0603" H 8450 1150 50  0001 C CNN
@@
 $EndComp
 $Comp
-L Conn_01x03 J11
+L Conn_01x03 J10
 U 1 1 5B1922FD
 P 8450 2600
-F 0 "J11" H 8450 2800 50  0000 C CNN
+F 0 "J10" H 8450 2800 50  0000 C CNN
 F 1 "74099-0603" V 8550 2600 50  0000 C CNN
 F 2 "WARG:74099-0603" H 8450 2600 50  0001 C CNN
@@
 $EndComp
 $Comp
-L Conn_01x03 J12
+L Conn_01x03 J11
 U 1 1 5B1923B5
 P 8450 4100
-F 0 "J12" H 8450 4300 50  0000 C CNN
+F 0 "J11" H 8450 4300 50  0000 C CNN
 F 1 "74099-0603" V 8550 4100 50  0000 C CNN
 F 2 "WARG:74099-0603" H 8450 4100 50  0001 C CNN
@@
 $EndComp
 $Comp
-L Conn_01x03 J13
+L Conn_01x03 J12
 U 1 1 5B1924AD
 P 8450 5550
-F 0 "J13" H 8450 5750 50  0000 C CNN
+F 0 "J12" H 8450 5750 50  0000 C CNN
 F 1 "74099-0603" V 8550 5550 50  0000 C CNN
 F 2 "WARG:74099-0603" H 8450 5550 50  0001 C CNN

Commit message: Capacitors where they should be on the pcb, usb interface moved
Parts:
- J1, J10, J11, J12, J2, J3, J4, J5, J6, J7, J8, J9: value 74099-0603 -> Conn_01x03; footprint WARG:74099-0603 -> Pin_Headers:Pin_Header_Straight_1x03_Pitch2.54mm; part_num CONN-011 -> CONN-007
Changed lines of the file:
@@
 P 2900 1150
 F 0 "J1" H 2900 1350 50  0000 C CNN
-F 1 "74099-0603" V 3000 1150 50  0000 C CNN
-F 2 "WARG:74099-0603" H 2900 1150 50  0001 C CNN
+F 1 "Conn_01x03" V 3000 1150 50  0000 C CNN
+F 2 "Pin_Headers:Pin_Header_Straight_1x03_Pitch2.54mm" H 2900 1150 50  0001 C CNN
 F 3 "" H 2900 1150 50  0001 C CNN
-F 4 "CONN-011" H 2900 1150 60  0001 C CNN "part_num"
+F 4 "CONN-007" H 2900 1150 60  0001 C CNN "part_num"
 	1    2900 1150
 	1    0    0    -1
 $EndComp
 $Comp
-L Conn_01x03 J2
-U 1 1 597DAC47
-P 2900 2600
-F 0 "J2" H 2900 2800 50  0000 C CNN
-F 1 "74099-0603" V 3000 2600 50  0000 C CNN
-F 2 "WARG:74099-0603" H 2900 2600 50  0001 C CNN
-F 3 "" H 2900 2600 50  0001 C CNN
-F 4 "CONN-011" H 2900 2600 60  0001 C CNN "part_num"
-	1    2900 2600
-	1    0    0    -1
-$EndComp
-$Comp
-L GND #PWR03
+L GND #PWR2
 U 1 1 597DB10B
 P 2300 5900
-F 0 "#PWR03" H 2300 5650 50  0001 C CNN
+F 0 "#PWR2" H 2300 5650 50  0001 C CNN
 F 1 "GND" H 2300 5750 50  0000 C CNN
 F 2 "" H 2300 5900 50  0001 C CNN
@@
 Connection ~ 2300 5450
 $Comp
-L GND #PWR04
+L GND #PWR3
 U 1 1 597DB1D3
 P 5000 5900
-F 0 "#PWR04" H 5000 5650 50  0001 C CNN
+F 0 "#PWR3" H 5000 5650 50  0001 C CNN
 F 1 "GND" H 5000 5750 50  0000 C CNN
 F 2 "" H 5000 5900 50  0001 C CNN
@@
 $EndComp
 $Comp
-L GND #PWR05
+L GND #PWR4
 U 1 1 597DB202
 P 7850 5800
-F 0 "#PWR05" H 7850 5550 50  0001 C CNN
+F 0 "#PWR4" H 7850 5550 50  0001 C CNN
 F 1 "GND" H 7850 5650 50  0000 C CNN
 F 2 "" H 7850 5800 50  0001 C CNN
@@
 Connection ~ 5000 2500
 $Comp
+L Conn_01x03 J2
+U 1 1 5B47A50A
+P 2900 2600
+F 0 "J2" H 2900 2800 50  0000 C CNN
+F 1 "Conn_01x03" V 3000 2600 50  0000 C CNN
+F 2 "Pin_Headers:Pin_Header_Straight_1x03_Pitch2.54mm" H 2900 2600 50  0001 C CNN
+F 3 "" H 2900 2600 50  0001 C CNN
+F 4 "CONN-007" H 2900 2600 60  0001 C CNN "part_num"
+	1    2900 2600
+	1    0    0    -1
+$EndComp
+$Comp
 L Conn_01x03 J3
-U 1 1 5B1918E4
+U 1 1 5B47A572
 P 2900 4100
 F 0 "J3" H 2900 4300 50  0000 C CNN
-F 1 "74099-0603" V 3000 4100 50  0000 C CNN
-F 2 "WARG:74099-0603" H 2900 4100 50  0001 C CNN
+F 1 "Conn_01x03" V 3000 4100 50  0000 C CNN
+F 2 "Pin_Headers:Pin_Header_Straight_1x03_Pitch2.54mm" H 2900 4100 50  0001 C CNN
 F 3 "" H 2900 4100 50  0001 C CNN
-F 4 "CONN-011" H 2900 4100 60  0001 C CNN "part_num"
+F 4 "CONN-007" H 2900 4100 60  0001 C CNN "part_num"
 	1    2900 4100
 	1    0    0    -1
@@
 $Comp
 L Conn_01x03 J4
-U 1 1 5B191B06
+U 1 1 5B47A5CD
 P 2900 5550
 F 0 "J4" H 2900 5750 50  0000 C CNN
-F 1 "74099-0603" V 3000 5550 50  0000 C CNN
-F 2 "WARG:74099-0603" H 2900 5550 50  0001 C CNN
+F 1 "Conn_01x03" V 3000 5550 50  0000 C CNN
+F 2 "Pin_Headers:Pin_Header_Straight_1x03_Pitch2.54mm" H 2900 5550 50  0001 C CNN
 F 3 "" H 2900 5550 50  0001 C CNN
-F 4 "CONN-011" H 2900 5550 60  0001 C CNN "part_num"
+F 4 "CONN-007" H 2900 5550 60  0001 C CNN "part_num"
 	1    2900 5550
 	1    0    0    -1
 $EndComp
 $Comp
+L Conn_01x03 J8
+U 1 1 5B47A679
+P 5600 5550
+F 0 "J8" H 5600 5750 50  0000 C CNN
+F 1 "Conn_01x03" V 5700 5550 50  0000 C CNN
+F 2 "Pin_Headers:Pin_Header_Straight_1x03_Pitch2.54mm" H 5600 5550 50  0001 C CNN
+F 3 "" H 5600 5550 50  0001 C CNN
+F 4 "CONN-007" H 5600 5550 60  0001 C CNN "part_num"
+	1    5600 5550
+	1    0    0    -1
+$EndComp
+$Comp
+L Conn_01x03 J7
+U 1 1 5B47A6F6
+P 5600 4100
+F 0 "J7" H 5600 4300 50  0000 C CNN
+F 1 "Conn_01x03" V 5700 4100 50  0000 C CNN
+F 2 "Pin_Headers:Pin_Header_Straight_1x03_Pitch2.54mm" H 5600 4100 50  0001 C CNN
+F 3 "" H 5600 4100 50  0001 C CNN
+F 4 "CONN-007" H 5600 4100 60  0001 C CNN "part_num"
+	1    5600 4100
+	1    0    0    -1
+$EndComp
+$Comp
+L Conn_01x03 J6
+U 1 1 5B47A774
+P 5600 2600
+F 0 "J6" H 5600 2800 50  0000 C CNN
+F 1 "Conn_01x03" V 5700 2600 50  0000 C CNN
+F 2 "Pin_Headers:Pin_Header_Straight_1x03_Pitch2.54mm" H 5600 2600 50  0001 C CNN
+F 3 "" H 5600 2600 50  0001 C CNN
+F 4 "CONN-007" H 5600 2600 60  0001 C CNN "part_num"
+	1    5600 2600
+	1    0    0    -1
+$EndComp
+$Comp
 L Conn_01x03 J5
-U 1 1 5B191E1C
+U 1 1 5B47A831
 P 5600 1150
 F 0 "J5" H 5600 1350 50  0000 C CNN
-F 1 "74099-0603" V 5700 1150 50  0000 C CNN
-F 2 "WARG:74099-0603" H 5600 1150 50  0001 C CNN
+F 1 "Conn_01x03" V 5700 1150 50  0000 C CNN
+F 2 "Pin_Headers:Pin_Header_Straight_1x03_Pitch2.54mm" H 5600 1150 50  0001 C CNN
 F 3 "" H 5600 1150 50  0001 C CNN
-F 4 "CONN-011" H 5600 1150 60  0001 C CNN "part_num"
+F 4 "CONN-007" H 5600 1150 60  0001 C CNN "part_num"
 	1    5600 1150
 	1    0    0    -1
 $EndComp
 $Comp
-L Conn_01x03 J6
-U 1 1 5B191E94
-P 5600 2600
-F 0 "J6" H 5600 2800 50  0000 C CNN
-F 1 "74099-0603" V 5700 2600 50  0000 C CNN
-F 2 "WARG:74099-0603" H 5600 2600 50  0001 C CNN
-F 3 "" H 5600 2600 50  0001 C CNN
-F 4 "CONN-011" H 5600 2600 60  0001 C CNN "part_num"
-	1    5600 2600
-	1    0    0    -1
-$EndComp
-$Comp
-L Conn_01x03 J7
-U 1 1 5B191F57
-P 5600 4100
-F 0 "J7" H 5600 4300 50  0000 C CNN
-F 1 "74099-0603" V 5700 4100 50  0000 C CNN
-F 2 "WARG:74099-0603" H 5600 4100 50  0001 C CNN
-F 3 "" H 5600 4100 50  0001 C CNN
-F 4 "CONN-011" H 5600 4100 60  0001 C CNN "part_num"
-	1    5600 4100
-	1    0    0    -1
-$EndComp
-$Comp
-L Conn_01x03 J8
-U 1 1 5B1920C6
-P 5600 5550
-F 0 "J8" H 5600 5750 50  0000 C CNN
-F 1 "74099-0603" V 5700 5550 50  0000 C CNN
-F 2 "WARG:74099-0603" H 5600 5550 50  0001 C CNN
-F 3 "" H 5600 5550 50  0001 C CNN
-F 4 "CONN-011" H 5600 5550 60  0001 C CNN "part_num"
-	1    5600 5550
-	1    0    0    -1
-$EndComp
-$Comp
 L Conn_01x03 J9
-U 1 1 5B192277
+U 1 1 5B47A8FB
 P 8450 1150
 F 0 "J9" H 8450 1350 50  0000 C CNN
-F 1 "74099-0603" V 8550 1150 50  0000 C CNN
-F 2 "WARG:74099-0603" H 8450 1150 50  0001 C CNN
+F 1 "Conn_01x03" V 8550 1150 50  0000 C CNN
+F 2 "Pin_Headers:Pin_Header_Straight_1x03_Pitch2.54mm" H 8450 1150 50  0001 C CNN
 F 3 "" H 8450 1150 50  0001 C CNN
-F 4 "CONN-011" H 8450 1150 60  0001 C CNN "part_num"
+F 4 "CONN-007" H 8450 1150 60  0001 C CNN "part_num"
 	1    8450 1150
 	1    0    0    -1
@@
 $Comp
 L Conn_01x03 J10
-U 1 1 5B1922FD
+U 1 1 5B47AA06
 P 8450 2600
 F 0 "J10" H 8450 2800 50  0000 C CNN
-F 1 "74099-0603" V 8550 2600 50  0000 C CNN
-F 2 "WARG:74099-0603" H 8450 2600 50  0001 C CNN
+F 1 "Conn_01x03" V 8550 2600 50  0000 C CNN
+F 2 "Pin_Headers:Pin_Header_Straight_1x03_Pitch2.54mm" H 8450 2600 50  0001 C CNN
 F 3 "" H 8450 2600 50  0001 C CNN
-F 4 "CONN-011" H 8450 2600 60  0001 C CNN "part_num"
+F 4 "CONN-007" H 8450 2600 60  0001 C CNN "part_num"
 	1    8450 2600
 	1    0    0    -1
@@
 $Comp
 L Conn_01x03 J11
-U 1 1 5B1923B5
+U 1 1 5B47AB32
 P 8450 4100
 F 0 "J11" H 8450 4300 50  0000 C CNN
-F 1 "74099-0603" V 8550 4100 50  0000 C CNN
-F 2 "WARG:74099-0603" H 8450 4100 50  0001 C CNN
+F 1 "Conn_01x03" V 8550 4100 50  0000 C CNN
+F 2 "Pin_Headers:Pin_Header_Straight_1x03_Pitch2.54mm" H 8450 4100 50  0001 C CNN
 F 3 "" H 8450 4100 50  0001 C CNN
-F 4 "CONN-011" H 8450 4100 60  0001 C CNN "part_num"
+F 4 "CONN-007" H 8450 4100 60  0001 C CNN "part_num"
 	1    8450 4100
 	1    0    0    -1
@@
 $Comp
 L Conn_01x03 J12
-U 1 1 5B1924AD
+U 1 1 5B47AC5F
 P 8450 5550
 F 0 "J12" H 8450 5750 50  0000 C CNN
-F 1 "74099-0603" V 8550 5550 50  0000 C CNN
-F 2 "WARG:74099-0603" H 8450 5550 50  0001 C CNN
+F 1 "Conn_01x03" V 8550 5550 50  0000 C CNN
+F 2 "Pin_Headers:Pin_Header_Straight_1x03_Pitch2.54mm" H 8450 5550 50  0001 C CNN
 F 3 "" H 8450 5550 50  0001 C CNN
-F 4 "CONN-011" H 8450 5550 60  0001 C CNN "part_num"
+F 4 "CONN-007" H 8450 5550 60  0001 C CNN "part_num"
 	1    8450 5550
 	1    0    0    -1

Commit message: Remapped symbols for KiCAD 5.0.x
Parts:
- J1, J10, J11, J12, J2, J3, J4, J5, J6, J7, J8, J9: symbol Conn_01x03 -> conn:Conn_01x03
Connections:
- wire segments 28 -> 35
Changed lines of the file:
@@
-EESchema Schematic File Version 2
-LIBS:WARG
-LIBS:power
-LIBS:device
-LIBS:transistors
-LIBS:conn
-LIBS:linear
-LIBS:regul
-LIBS:74xx
-LIBS:cmos4000
-LIBS:adc-dac
-LIBS:memory
-LIBS:xilinx
-LIBS:microcontrollers
-LIBS:dsp
-LIBS:microchip
-LIBS:analog_switches
-LIBS:motorola
-LIBS:texas
-LIBS:intel
-LIBS:audio
-LIBS:interface
-LIBS:digital-audio
-LIBS:philips
-LIBS:display
-LIBS:cypress
-LIBS:siliconi
-LIBS:opto
-LIBS:atmel
-LIBS:contrib
-LIBS:valves
+EESchema Schematic File Version 4
 LIBS:ZeroPilot-cache
-EELAYER 25 0
+EELAYER 26 0
 EELAYER END
 $Descr A4 11693 8268
@@
 Text Label 7900 5650 0    60   ~ 0
 PWM12
-Wire Bus Line
-	2150 900  2150 5550
 Wire Wire Line
 	2250 5650 2700 5650
@@
 Wire Wire Line
 	2250 1250 2700 1250
-Wire Bus Line
-	4850 900  4850 5550
 Wire Wire Line
 	4950 5650 5400 5650
@@
 Wire Wire Line
 	4950 1250 5400 1250
-Wire Bus Line
-	7700 900  7700 5550
 Wire Wire Line
 	7800 5650 8250 5650
@@
 PWM_5V
 $Comp
-L Conn_01x03 J1
+L conn:Conn_01x03 J1
 U 1 1 597DAC0F
 P 2900 1150
@@
 $EndComp
 $Comp
-L GND #PWR03
+L power:GND #PWR03
 U 1 1 597DB10B
 P 2300 5900
@@
 	2700 1050 2300 1050
 Wire Wire Line
-	2300 1050 2300 5900
+	2300 1050 2300 2500
 Wire Wire Line
 	2700 2500 2300 2500
@@
 Wire Wire Line
 	2700 4000 2300 4000
-Wire Wire Line
-	2300 4000 2300 3950
 Connection ~ 2300 3950
 Wire Wire Line
@@
 Connection ~ 2300 5450
 $Comp
-L GND #PWR04
+L power:GND #PWR04
 U 1 1 597DB1D3
 P 5000 5900
@@
 $EndComp
 $Comp
-L GND #PWR05
+L power:GND #PWR05
 U 1 1 597DB202
 P 7850 5800
@@
 $EndComp
 Wire Wire Line
-	7850 1050 7850 5800
+	7850 1050 7850 2500
 Wire Wire Line
 	7850 1050 8250 1050
@@
 	5400 4000 5000 4000
 Wire Wire Line
-	5000 1050 5000 5900
+	5000 1050 5000 2500
 Wire Wire Line
 	5400 1050 5000 1050
@@
 Connection ~ 5000 2500
 $Comp
-L Conn_01x03 J2
+L conn:Conn_01x03 J2
 U 1 1 5B47A50A
 P 2900 2600
@@
 $EndComp
 $Comp
-L Conn_01x03 J3
+L conn:Conn_01x03 J3
 U 1 1 5B47A572
 P 2900 4100
@@
 $EndComp
 $Comp
-L Conn_01x03 J4
+L conn:Conn_01x03 J4
 U 1 1 5B47A5CD
 P 2900 5550
@@
 $EndComp
 $Comp
-L Conn_01x03 J8
+L conn:Conn_01x03 J8
 U 1 1 5B47A679
 P 5600 5550
@@
 $EndComp
 $Comp
-L Conn_01x03 J7
+L conn:Conn_01x03 J7
 U 1 1 5B47A6F6
 P 5600 4100
@@
 $EndComp
 $Comp
-L Conn_01x03 J6
+L conn:Conn_01x03 J6
 U 1 1 5B47A774
 P 5600 2600
@@
 $EndComp
 $Comp
-L Conn_01x03 J5
+L conn:Conn_01x03 J5
 U 1 1 5B47A831
 P 5600 1150
@@
 $EndComp
 $Comp
-L Conn_01x03 J9
+L conn:Conn_01x03 J9
 U 1 1 5B47A8FB
 P 8450 1150
@@
 $EndComp
 $Comp
-L Conn_01x03 J10
+L conn:Conn_01x03 J10
 U 1 1 5B47AA06
 P 8450 2600
@@
 $EndComp
 $Comp
-L Conn_01x03 J11
+L conn:Conn_01x03 J11
 U 1 1 5B47AB32
 P 8450 4100
@@
 $EndComp
 $Comp
-L Conn_01x03 J12
+L conn:Conn_01x03 J12
 U 1 1 5B47AC5F
 P 8450 5550
@@
 	1    0    0    -1
 $EndComp
+Wire Wire Line
+	2300 5450 2300 5900
+Wire Wire Line
+	7850 2500 7850 4000
+Wire Wire Line
+	7850 4000 7850 5450
+Wire Wire Line
+	7850 5450 7850 5800
+Wire Wire Line
+	5000 4000 5000 5450
+Wire Wire Line
+	5000 5450 5000 5900
+Wire Wire Line
+	5000 2500 5000 4000
+Wire Wire Line
+	2300 2500 2300 5450
+Wire Bus Line
+	2150 900  2150 5550
+Wire Bus Line
+	4850 900  4850 5550
+Wire Bus Line
+	7700 900  7700 5550
 $EndSCHEMATC

Commit message: Added RSSI, datasheets, INDU-004
Added RSSI input to PPM connector. Added datasheets for most of the components. The filter inductors for the FTDI were labeled as INDU-002, which is a 15uH smps inductor.
Connections:
- net labels added: PWM_6V
- net labels removed: PWM_5V
Changed lines of the file:
@@
 PWM[1..12]
 Text HLabel 1100 650  0    60   Input ~ 0
-PWM_5V
+PWM_6V
 Wire Bus Line
 	1100 900  7700 900
@@
 PWM[1..12]
 Text Label 2700 1150 2    60   ~ 0
-PWM_5V
+PWM_6V
 Text Label 2700 4100 2    60   ~ 0
-PWM_5V
+PWM_6V
 Text Label 2700 5550 2    60   ~ 0
-PWM_5V
+PWM_6V
 Text Label 5400 1150 2    60   ~ 0
-PWM_5V
+PWM_6V
 Text Label 5400 2600 2    60   ~ 0
-PWM_5V
+PWM_6V
 Text Label 5400 4100 2    60   ~ 0
-PWM_5V
+PWM_6V
 Text Label 5400 5550 2    60   ~ 0
-PWM_5V
+PWM_6V
 Text Label 8250 1150 2    60   ~ 0
-PWM_5V
+PWM_6V
 Text Label 8250 2600 2    60   ~ 0
-PWM_5V
+PWM_6V
 Text Label 8250 4100 2    60   ~ 0
-PWM_5V
+PWM_6V
 Text Label 8250 5550 2    60   ~ 0
-PWM_5V
+PWM_6V
 Text Label 1100 650  0    60   ~ 0
-PWM_5V
+PWM_6V
 Text Label 2700 2600 2    60   ~ 0
-PWM_5V
+PWM_6V
 $Comp
 L conn:Conn_01x03 J1
@@
 Wire Wire Line
 	2700 4000 2300 4000
-Connection ~ 2300 3950
 Wire Wire Line
 	2700 5450 2300 5450

Commit message: Bug fixes, added Isense, changed conn to JST-GH
Added boot0 pull-down resistors. Changed ext_batt to current sense line. Changed spox conn to JST-GH, this will dramatically reduce the required size of the board.
Parts:
- removed J1, J10, J11, J12, J2, J3, J4, J5, J6, J7, J8, J9: Conn_01x03, Pin_Headers:Pin_Header_Straight_1x03_Pitch2.54mm, symbol conn:Conn_01x03
- added J? (x6): GH-6, Connectors_JST:JST_GH_BM06B-GHS-TBT_06x1.25mm_Straight, symbol conn:Conn_01x06
Connections:
- wire segments 35 -> 36

Commit message: Generated netlist and board outline
Parts:
- gave numbers to parts that had none: 6
Changed lines of the file:
@@
 PWM_6V
 $Comp
-L power:GND #PWR03
+L power:GND #PWR02
 U 1 1 597DB10B
 P 2300 2750
-F 0 "#PWR03" H 2300 2500 50  0001 C CNN
+F 0 "#PWR02" H 2300 2500 50  0001 C CNN
 F 1 "GND" H 2300 2600 50  0000 C CNN
 F 2 "" H 2300 2750 50  0001 C CNN
@@
 $EndComp
 $Comp
-L conn:Conn_01x06 J?
+L conn:Conn_01x06 J1
 U 1 1 5CBEBA42
 P 2900 1400
-F 0 "J?" H 2979 1392 50  0000 L CNN
+F 0 "J1" H 2979 1392 50  0000 L CNN
 F 1 "GH-6" H 2979 1301 50  0000 L CNN
 F 2 "Connectors_JST:JST_GH_BM06B-GHS-TBT_06x1.25mm_Straight" H 2900 1400 50  0001 C CNN
@@
 	2300 1600 2300 2400
 $Comp
-L conn:Conn_01x06 J?
+L conn:Conn_01x06 J2
 U 1 1 5CBF0512
 P 2900 2200
-F 0 "J?" H 2980 2192 50  0000 L CNN
+F 0 "J2" H 2980 2192 50  0000 L CNN
 F 1 "GH-6" H 2980 2101 50  0000 L CNN
 F 2 "Connectors_JST:JST_GH_BM06B-GHS-TBT_06x1.25mm_Straight" H 2900 2200 50  0001 C CNN
@@
 PWM_6V
 $Comp
-L power:GND #PWR?
+L power:GND #PWR03
 U 1 1 5CBF3F2F
 P 5000 2750
-F 0 "#PWR?" H 5000 2500 50  0001 C CNN
+F 0 "#PWR03" H 5000 2500 50  0001 C CNN
 F 1 "GND" H 5000 2600 50  0000 C CNN
 F 2 "" H 5000 2750 50  0001 C CNN
@@
 $EndComp
 $Comp
-L conn:Conn_01x06 J?
+L conn:Conn_01x06 J3
 U 1 1 5CBF3F35
 P 5600 1400
-F 0 "J?" H 5680 1392 50  0000 L CNN
+F 0 "J3" H 5680 1392 50  0000 L CNN
 F 1 "GH-6" H 5680 1301 50  0000 L CNN
 F 2 "Connectors_JST:JST_GH_BM06B-GHS-TBT_06x1.25mm_Straight" H 5600 1400 50  0001 C CNN
@@
 	5000 1600 5000 2400
 $Comp
-L conn:Conn_01x06 J?
+L conn:Conn_01x06 J4
 U 1 1 5CBF3F45
 P 5600 2200
-F 0 "J?" H 5680 2192 50  0000 L CNN
+F 0 "J4" H 5680 2192 50  0000 L CNN
 F 1 "GH-6" H 5680 2101 50  0000 L CNN
 F 2 "Connectors_JST:JST_GH_BM06B-GHS-TBT_06x1.25mm_Straight" H 5600 2200 50  0001 C CNN
@@
 PWM_6V
 $Comp
-L power:GND #PWR?
+L power:GND #PWR04
 U 1 1 5CBF4250
 P 7850 2750
-F 0 "#PWR?" H 7850 2500 50  0001 C CNN
+F 0 "#PWR04" H 7850 2500 50  0001 C CNN
 F 1 "GND" H 7850 2600 50  0000 C CNN
 F 2 "" H 7850 2750 50  0001 C CNN
@@
 $EndComp
 $Comp
-L conn:Conn_01x06 J?
+L conn:Conn_01x06 J5
 U 1 1 5CBF4256
 P 8450 1400
-F 0 "J?" H 8530 1392 50  0000 L CNN
+F 0 "J5" H 8530 1392 50  0000 L CNN
 F 1 "GH-6" H 8530 1301 50  0000 L CNN
 F 2 "Connectors_JST:JST_GH_BM06B-GHS-TBT_06x1.25mm_Straight" H 8450 1400 50  0001 C CNN
@@
 	7850 1600 7850 2400
 $Comp
-L conn:Conn_01x06 J?
+L conn:Conn_01x06 J6
 U 1 1 5CBF4266
 P 8450 2200
-F 0 "J?" H 8530 2192 50  0000 L CNN
+F 0 "J6" H 8530 2192 50  0000 L CNN
 F 1 "GH-6" H 8530 2101 50  0000 L CNN
 F 2 "Connectors_JST:JST_GH_BM06B-GHS-TBT_06x1.25mm_Straight" H 8450 2200 50  0001 C CNN
