File: Hardware/SENSORS.sch (KiCad schematic (older format))
At the start: 7 parts, among them U12 ICM-20602, U13 MS5637-02BA03

Commit message: Fixes
Parts:
- U6: renamed from U12; symbol ZeroPilot-rescue:ICM-20602-WARG -> WARG:ICM-20602
- U7: renamed from U13; symbol ZeroPilot-rescue:MS5637-02BA03-WARG -> WARG:MS5637-02BA03
- renumbered C55 to C43, C56 to C44, C57 to C45, C58 to C46, C59 to C47
Changed lines of the file:
@@
 EESchema Schematic File Version 4
+LIBS:ZeroPilot-cache
 EELAYER 29 0
 EELAYER END
 $Descr A4 11693 8268
 encoding utf-8
-Sheet 8 10
+Sheet 7 10
 Title ""
 Date ""
@@
 	1950 2800 2150 2800
 $Comp
-L power:GND #PWR044
+L power:GND #PWR031
 U 1 1 5B1268E9
 P 1700 3750
-F 0 "#PWR044" H 1700 3500 50  0001 C CNN
+F 0 "#PWR031" H 1700 3500 50  0001 C CNN
 F 1 "GND" H 1700 3600 50  0000 C CNN
 F 2 "" H 1700 3750 50  0001 C CNN
@@
 $EndComp
 $Comp
-L power:GND #PWR045
+L power:GND #PWR032
 U 1 1 5B1269F7
 P 2400 3100
-F 0 "#PWR045" H 2400 2850 50  0001 C CNN
+F 0 "#PWR032" H 2400 2850 50  0001 C CNN
 F 1 "GND" H 2400 2950 50  0000 C CNN
 F 2 "" H 2400 3100 50  0001 C CNN
@@
 $EndComp
 $Comp
-L power:GND #PWR046
+L power:GND #PWR033
 U 1 1 5B126A15
 P 2700 3100
-F 0 "#PWR046" H 2700 2850 50  0001 C CNN
+F 0 "#PWR033" H 2700 2850 50  0001 C CNN
 F 1 "GND" H 2700 2950 50  0000 C CNN
 F 2 "" H 2700 3100 50  0001 C CNN
@@
 $EndComp
 $Comp
-L power:GND #PWR048
+L power:GND #PWR035
 U 1 1 5B126E10
 P 3750 3200
-F 0 "#PWR048" H 3750 2950 50  0001 C CNN
+F 0 "#PWR035" H 3750 2950 50  0001 C CNN
 F 1 "GND" H 3750 3050 50  0000 C CNN
 F 2 "" H 3750 3200 50  0001 C CNN
@@
 $EndComp
 $Comp
-L power:GND #PWR049
+L power:GND #PWR036
 U 1 1 5B126ED4
 P 3800 4100
-F 0 "#PWR049" H 3800 3850 50  0001 C CNN
+F 0 "#PWR036" H 3800 3850 50  0001 C CNN
 F 1 "GND" H 3800 3950 50  0000 C CNN
 F 2 "" H 3800 4100 50  0001 C CNN
@@
 ALT_SDA
 $Comp
-L power:GND #PWR050
+L power:GND #PWR037
 U 1 1 5B159952
 P 6750 3500
-F 0 "#PWR050" H 6750 3250 50  0001 C CNN
+F 0 "#PWR037" H 6750 3250 50  0001 C CNN
 F 1 "GND" H 6750 3350 50  0000 C CNN
 F 2 "" H 6750 3500 50  0001 C CNN
@@
 	2400 2800 2700 2800
 $Comp
-L power:GND #PWR047
+L power:GND #PWR034
 U 1 1 5CB7EA67
 P 3150 2900
-F 0 "#PWR047" H 3150 2650 50  0001 C CNN
+F 0 "#PWR034" H 3150 2650 50  0001 C CNN
 F 1 "GND" H 3150 2750 50  0000 C CNN
 F 2 "" H 3150 2900 50  0001 C CNN
@@
 Connection ~ 2700 2800
 $Comp
-L ZeroPilot-rescue:MS5637-02BA03-WARG U13
+L WARG:MS5637-02BA03 U7
 U 1 1 5B0F962E
 P 6200 3650
-F 0 "U13" H 6200 4850 118 0000 C CNN
+F 0 "U7" H 6200 4850 118 0000 C CNN
 F 1 "MS5637-02BA03" H 6200 2850 118 0000 C CNN
 F 2 "WARG-kicad:MS5637-02BA03" H 6200 4640 60  0001 C CNN
@@
 $EndComp
 $Comp
-L Device:C C59
+L Device:C C47
 U 1 1 5B1017C9
 P 6200 3050
-F 0 "C59" H 6225 3150 50  0000 L CNN
+F 0 "C47" H 6225 3150 50  0000 L CNN
 F 1 "100nF" H 6225 2950 50  0000 L CNN
 F 2 "Capacitor_SMD:C_0603_1608Metric_Pad1.05x0.95mm_HandSolder" H 6238 2900 50  0001 C CNN
@@
 $EndComp
 $Comp
-L Device:C C58
+L Device:C C46
 U 1 1 5B126D43
 P 3750 3050
-F 0 "C58" H 3775 3150 50  0000 L CNN
+F 0 "C46" H 3775 3150 50  0000 L CNN
 F 1 "100nF" H 3775 2950 50  0000 L CNN
 F 2 "Capacitor_SMD:C_0603_1608Metric_Pad1.05x0.95mm_HandSolder" H 3788 2900 50  0001 C CNN
@@
 $EndComp
 $Comp
-L Device:C C57
+L Device:C C45
 U 1 1 5B126990
 P 2700 2950
-F 0 "C57" H 2725 3050 50  0000 L CNN
+F 0 "C45" H 2725 3050 50  0000 L CNN
 F 1 "2.2uF" H 2725 2850 50  0000 L CNN
 F 2 "Capacitor_SMD:C_0603_1608Metric_Pad1.05x0.95mm_HandSolder" H 2738 2800 50  0001 C CNN
@@
 $EndComp
 $Comp
-L Device:C C56
+L Device:C C44
 U 1 1 5B126921
 P 2400 2950
-F 0 "C56" H 2425 3050 50  0000 L CNN
+F 0 "C44" H 2425 3050 50  0000 L CNN
 F 1 "100nF" H 2425 2850 50  0000 L CNN
 F 2 "Capacitor_SMD:C_0603_1608Metric_Pad1.05x0.95mm_HandSolder" H 2438 2800 50  0001 C CNN
@@
 $EndComp
 $Comp
-L Device:C C55
+L Device:C C43
 U 1 1 5B12679C
 P 1700 3600
-F 0 "C55" H 1725 3700 50  0000 L CNN
+F 0 "C43" H 1725 3700 50  0000 L CNN
 F 1 "10nF" H 1725 3500 50  0000 L CNN
 F 2 "Capacitor_SMD:C_0603_1608Metric_Pad1.05x0.95mm_HandSolder" H 2040 3600 50  0001 C CNN
@@
 $EndComp
 $Comp
-L ZeroPilot-rescue:ICM-20602-WARG U12
+L WARG:ICM-20602 U?
 U 1 1 5B0F92D3
 P 3150 3650
-AR Path="/5B0F92D3" Ref="U12"  Part="1"
-AR Path="/5B0F2007/5B0F92D3" Ref="U12"  Part="1"
-F 0 "U12" H 3150 4850 118 0000 C CNN
+AR Path="/5B0F92D3" Ref="U?"  Part="1"
+AR Path="/5B0F2007/5B0F92D3" Ref="U6"  Part="1"
+F 0 "U6" H 3150 4850 118 0000 C CNN
 F 1 "ICM-20602" H 3150 2400 118 0000 C CNN
 F 2 "Package_LGA:LGA-16_3x3mm_P0.5mm" H 3125 4664 60  0001 C CNN

Commit message: Silkscreen and BOM update
Parts:
- U6: symbol WARG:ICM-20602 -> ZeroPilot-rescue:ICM-20602-WARG
- U7: symbol WARG:MS5637-02BA03 -> ZeroPilot-rescue:MS5637-02BA03-WARG
Changed lines of the file:
@@
 Connection ~ 2700 2800
 $Comp
-L WARG:MS5637-02BA03 U7
+L ZeroPilot-rescue:MS5637-02BA03-WARG U7
 U 1 1 5B0F962E
 P 6200 3650
+AR Path="/5B0F962E" Ref="U7"  Part="1"
+AR Path="/5B0F2007/5B0F962E" Ref="U7"  Part="1"
 F 0 "U7" H 6200 4850 118 0000 C CNN
 F 1 "MS5637-02BA03" H 6200 2850 118 0000 C CNN
@@
 $EndComp
 $Comp
-L WARG:ICM-20602 U?
+L ZeroPilot-rescue:ICM-20602-WARG U?
 U 1 1 5B0F92D3
 P 3150 3650
