File: Hardware/MEMORY.sch (KiCad schematic (older format))
At the start: 9 parts, among them J8 Micro_SD_Card, U11 M24C64-WDW6TP

Commit message: Initial Routing of Zeropilot Rev1
This is the initial routing of the board. It needs to be cleaned up slightly, but library references are screwed up so they will be fixed first.
Parts:
- J8: symbol conn:Micro_SD_Card -> Connector:Micro_SD_Card
Changed lines of the file:
@@
 EESchema Schematic File Version 4
-LIBS:ZeroPilot-cache
-EELAYER 26 0
+EELAYER 29 0
 EELAYER END
 $Descr A4 11693 8268
@@
 Populate resistors to select I2C address\n
 $Comp
-L conn:Micro_SD_Card J8
+L Connector:Micro_SD_Card J8
 U 1 1 59517B7C
 P 8300 1900

Commit message: Updated Footprints
Updated the footprints to 5.1, added 3D models to all components.
Parts:
- R28, R29, R30, R31, R32, R33, R34: footprint Resistors_SMD:R_0603_HandSoldering -> Resistor_SMD:R_0603_1608Metric_Pad1.05x0.95mm_HandSolder
- U11: footprint Housings_SSOP:TSSOP-8_4.4x3mm_Pitch0.65mm -> Package_SO:TSSOP-8_4.4x3mm_P0.65mm
Changed lines of the file:
@@
 EESchema Schematic File Version 4
+LIBS:ZeroPilot-cache
 EELAYER 29 0
 EELAYER END
@@
 F 0 "R29" V 1730 5650 50  0000 C CNN
 F 1 "10K" V 1650 5650 50  0000 C CNN
-F 2 "Resistors_SMD:R_0603_HandSoldering" V 1580 5650 50  0001 C CNN
+F 2 "Resistor_SMD:R_0603_1608Metric_Pad1.05x0.95mm_HandSolder" V 1580 5650 50  0001 C CNN
 F 3 "http://industrial.panasonic.com/www-cgi/jvcr13pz.cgi?E+PZ+3+AOA0001+ERJ3GEYJ103V+7+WW" H 1650 5650 50  0001 C CNN
 F 4 "RESS-005" V 1650 5650 60  0001 C CNN "part_num"
@@
 F 0 "R28" V 1730 5100 50  0000 C CNN
 F 1 "0" V 1650 5100 50  0000 C CNN
-F 2 "Resistors_SMD:R_0603_HandSoldering" V 1580 5100 50  0001 C CNN
+F 2 "Resistor_SMD:R_0603_1608Metric_Pad1.05x0.95mm_HandSolder" V 1580 5100 50  0001 C CNN
 F 3 "http://www.yageo.com/documents/recent/PYu-RC_Group_51_RoHS_L_10.pdf" H 1650 5100 50  0001 C CNN
 F 4 "RESS-001" V 1650 5100 60  0001 C CNN "part_num"
@@
 F 0 "R31" V 1980 5650 50  0000 C CNN
 F 1 "10K" V 1900 5650 50  0000 C CNN
-F 2 "Resistors_SMD:R_0603_HandSoldering" V 1830 5650 50  0001 C CNN
+F 2 "Resistor_SMD:R_0603_1608Metric_Pad1.05x0.95mm_HandSolder" V 1830 5650 50  0001 C CNN
 F 3 "http://industrial.panasonic.com/www-cgi/jvcr13pz.cgi?E+PZ+3+AOA0001+ERJ3GEYJ103V+7+WW" H 1900 5650 50  0001 C CNN
 F 4 "RESS-005" V 1900 5650 60  0001 C CNN "part_num"
@@
 F 0 "R33" V 2230 5650 50  0000 C CNN
 F 1 "10K" V 2150 5650 50  0000 C CNN
-F 2 "Resistors_SMD:R_0603_HandSoldering" V 2080 5650 50  0001 C CNN
+F 2 "Resistor_SMD:R_0603_1608Metric_Pad1.05x0.95mm_HandSolder" V 2080 5650 50  0001 C CNN
 F 3 "http://industrial.panasonic.com/www-cgi/jvcr13pz.cgi?E+PZ+3+AOA0001+ERJ3GEYJ103V+7+WW" H 2150 5650 50  0001 C CNN
 F 4 "RESS-005" V 2150 5650 60  0001 C CNN "part_num"
@@
 F 0 "R30" V 1980 5100 50  0000 C CNN
 F 1 "0" V 1900 5100 50  0000 C CNN
-F 2 "Resistors_SMD:R_0603_HandSoldering" V 1830 5100 50  0001 C CNN
+F 2 "Resistor_SMD:R_0603_1608Metric_Pad1.05x0.95mm_HandSolder" V 1830 5100 50  0001 C CNN
 F 3 "http://www.yageo.com/documents/recent/PYu-RC_Group_51_RoHS_L_10.pdf" H 1900 5100 50  0001 C CNN
 F 4 "RESS-001" V 1900 5100 60  0001 C CNN "part_num"
@@
 F 0 "R32" V 2230 5100 50  0000 C CNN
 F 1 "0" V 2150 5100 50  0000 C CNN
-F 2 "Resistors_SMD:R_0603_HandSoldering" V 2080 5100 50  0001 C CNN
+F 2 "Resistor_SMD:R_0603_1608Metric_Pad1.05x0.95mm_HandSolder" V 2080 5100 50  0001 C CNN
 F 3 "http://www.yageo.com/documents/recent/PYu-RC_Group_51_RoHS_L_10.pdf" H 2150 5100 50  0001 C CNN
 F 4 "RESS-001" V 2150 5100 60  0001 C CNN "part_num"
@@
 F 0 "R34" V 4030 5300 50  0000 C CNN
 F 1 "10K" V 3950 5300 50  0000 C CNN
-F 2 "Resistors_SMD:R_0603_HandSoldering" V 3880 5300 50  0001 C CNN
+F 2 "Resistor_SMD:R_0603_1608Metric_Pad1.05x0.95mm_HandSolder" V 3880 5300 50  0001 C CNN
 F 3 "http://industrial.panasonic.com/www-cgi/jvcr13pz.cgi?E+PZ+3+AOA0001+ERJ3GEYJ103V+7+WW" H 3950 5300 50  0001 C CNN
 F 4 "RESS-005" V 3950 5300 60  0001 C CNN "part_num"
@@
 F 0 "U11" H 5300 5450 60  0000 C CNN
 F 1 "M24C64-WDW6TP" H 5250 4100 60  0000 C CNN
-F 2 "Housings_SSOP:TSSOP-8_4.4x3mm_Pitch0.65mm" H 5200 5350 60  0001 C CNN
+F 2 "Package_SO:TSSOP-8_4.4x3mm_P0.65mm" H 5200 5350 60  0001 C CNN
 F 3 "http://www.st.com/content/ccc/resource/technical/document/datasheet/5c/df/52/a5/15/f2/48/bd/CD00259166.pdf/files/CD00259166.pdf/jcr:content/translations/en.CD00259166.pdf" H 5300 5450 60  0001 C CNN
 F 4 "MEMM-001" H 5400 5550 60  0001 C CNN "part_num"

Commit message: HW Bootcamp for Zeropilot R1
Changed the board to R1.
Parts:
- renumbered R28 to R26, R29 to R27, R30 to R28, R31 to R29, R32 to R30, R33 to R31, R34 to R32, U11 to U6
Changed lines of the file:
@@
 EESchema Schematic File Version 4
-LIBS:ZeroPilot-cache
 EELAYER 29 0
 EELAYER END
@@
 $EndDescr
 $Comp
-L power:GND #PWR040
+L power:GND #PWR035
 U 1 1 5920672F
 P 9150 2600
-F 0 "#PWR040" H 9150 2350 50  0001 C CNN
+F 0 "#PWR035" H 9150 2350 50  0001 C CNN
 F 1 "GND" H 9150 2450 50  0000 C CNN
 F 2 "" H 9150 2600 50  0001 C CNN
@@
 SD_DAT3
 $Comp
-L power:GND #PWR039
+L power:GND #PWR034
 U 1 1 592067B5
 P 7300 2400
-F 0 "#PWR039" H 7300 2150 50  0001 C CNN
+F 0 "#PWR034" H 7300 2150 50  0001 C CNN
 F 1 "GND" H 7300 2250 50  0000 C CNN
 F 2 "" H 7300 2400 50  0001 C CNN
@@
 $EndComp
 $Comp
-L power:GND #PWR038
+L power:GND #PWR033
 U 1 1 592069E4
 P 5150 5850
-F 0 "#PWR038" H 5150 5600 50  0001 C CNN
+F 0 "#PWR033" H 5150 5600 50  0001 C CNN
 F 1 "GND" H 5150 5700 50  0000 C CNN
 F 2 "" H 5150 5850 50  0001 C CNN
@@
 E3
 $Comp
-L Device:R R29
+L Device:R R27
 U 1 1 59206C6F
 P 1650 5650
-F 0 "R29" V 1730 5650 50  0000 C CNN
+F 0 "R27" V 1730 5650 50  0000 C CNN
 F 1 "10K" V 1650 5650 50  0000 C CNN
 F 2 "Resistor_SMD:R_0603_1608Metric_Pad1.05x0.95mm_HandSolder" V 1580 5650 50  0001 C CNN
@@
 $EndComp
 $Comp
-L Device:R R28
+L Device:R R26
 U 1 1 59206D63
 P 1650 5100
-F 0 "R28" V 1730 5100 50  0000 C CNN
+F 0 "R26" V 1730 5100 50  0000 C CNN
 F 1 "0" V 1650 5100 50  0000 C CNN
 F 2 "Resistor_SMD:R_0603_1608Metric_Pad1.05x0.95mm_HandSolder" V 1580 5100 50  0001 C CNN
@@
 $EndComp
 $Comp
-L power:GND #PWR037
+L power:GND #PWR032
 U 1 1 59206DDE
 P 1900 5950
-F 0 "#PWR037" H 1900 5700 50  0001 C CNN
+F 0 "#PWR032" H 1900 5700 50  0001 C CNN
 F 1 "GND" H 1900 5800 50  0000 C CNN
 F 2 "" H 1900 5950 50  0001 C CNN
@@
 $EndComp
 $Comp
-L Device:R R31
+L Device:R R29
 U 1 1 59596B34
 P 1900 5650
-F 0 "R31" V 1980 5650 50  0000 C CNN
+F 0 "R29" V 1980 5650 50  0000 C CNN
 F 1 "10K" V 1900 5650 50  0000 C CNN
 F 2 "Resistor_SMD:R_0603_1608Metric_Pad1.05x0.95mm_HandSolder" V 1830 5650 50  0001 C CNN
@@
 $EndComp
 $Comp
-L Device:R R33
+L Device:R R31
 U 1 1 59596B68
 P 2150 5650
-F 0 "R33" V 2230 5650 50  0000 C CNN
+F 0 "R31" V 2230 5650 50  0000 C CNN
 F 1 "10K" V 2150 5650 50  0000 C CNN
 F 2 "Resistor_SMD:R_0603_1608Metric_Pad1.05x0.95mm_HandSolder" V 2080 5650 50  0001 C CNN
@@
 $EndComp
 $Comp
-L Device:R R30
+L Device:R R28
 U 1 1 59596BE6
 P 1900 5100
-F 0 "R30" V 1980 5100 50  0000 C CNN
+F 0 "R28" V 1980 5100 50  0000 C CNN
 F 1 "0" V 1900 5100 50  0000 C CNN
 F 2 "Resistor_SMD:R_0603_1608Metric_Pad1.05x0.95mm_HandSolder" V 1830 5100 50  0001 C CNN
@@
 $EndComp
 $Comp
-L Device:R R32
+L Device:R R30
 U 1 1 59596C1A
 P 2150 5100
-F 0 "R32" V 2230 5100 50  0000 C CNN
+F 0 "R30" V 2230 5100 50  0000 C CNN
 F 1 "0" V 2150 5100 50  0000 C CNN
 F 2 "Resistor_SMD:R_0603_1608Metric_Pad1.05x0.95mm_HandSolder" V 2080 5100 50  0001 C CNN
@@
 $EndComp
 $Comp
-L Device:R R34
+L Device:R R32
 U 1 1 59596D32
 P 3950 5300
-F 0 "R34" V 4030 5300 50  0000 C CNN
+F 0 "R32" V 4030 5300 50  0000 C CNN
 F 1 "10K" V 3950 5300 50  0000 C CNN
 F 2 "Resistor_SMD:R_0603_1608Metric_Pad1.05x0.95mm_HandSolder" V 3880 5300 50  0001 C CNN
@@
 $EndComp
 $Comp
-L WARG:M24C64-WDW6TP U11
+L WARG:M24C64-WDW6TP U6
 U 1 1 595FB585
 P 5300 5000
-F 0 "U11" H 5300 5450 60  0000 C CNN
+F 0 "U6" H 5300 5450 60  0000 C CNN
 F 1 "M24C64-WDW6TP" H 5250 4100 60  0000 C CNN
 F 2 "Package_SO:TSSOP-8_4.4x3mm_P0.65mm" H 5200 5350 60  0001 C CNN
